Commit message: Change on namespaces

File: rbsherpa_description/urdf/bases/base.gazebo.xacro (robot description, xacro)
@@ -16,5 +16,5 @@
 		<gazebo>
 		<plugin name="omni_drive_ackermann" filename="libomnidrive_ackermann_plugin.so">
-			<!--<robotNamespace>/sherpa</robotNamespace>-->
+			<!--<robotNamespace>/rbsherpa</robotNamespace>-->
 			<!--<robotParam>robot_description</robotParam>-->
 			<broadcastTF>1</broadcastTF>

File: rbsherpa_description/urdf/bases/base.urdf.xacro (robot description, xacro)
@@ -33,10 +33,10 @@
         <xacro:if value="${hq}">
           <geometry>
-            <mesh filename="package://rbsherpa_description/meshes/bases/sherpa_chassis.dae"/>
+            <mesh filename="package://rbsherpa_description/meshes/bases/rbsherpa_chassis.dae"/>
           </geometry>
         </xacro:if>
         <xacro:unless value="${hq}">
           <geometry>
-            <mesh filename="package://rbsherpa_description/meshes/bases/sherpa_chassis.dae"/>
+            <mesh filename="package://rbsherpa_description/meshes/bases/rbsherpa_chassis.dae"/>
           </geometry>
         </xacro:unless>
@@ -48,5 +48,5 @@
         <origin xyz="0.429 0 0" rpy="0 0 0 " />
         <geometry>
-          <mesh filename="package://rbsherpa_description/meshes/bases/sherpa_chassis.dae"/>
+          <mesh filename="package://rbsherpa_description/meshes/bases/rbsherpa_chassis.dae"/>
         </geometry>
       </collision>

Commit message: Minor fixes on params and add maps to localization folder

File: rbsherpa_description/urdf/bases/base.gazebo.xacro (robot description, xacro)
@@ -1,4 +1,4 @@
 <?xml version="1.0"?>
-<robot xmlns:xacro="http://ros.org/wiki/xacro">
+<robot xmlns:xacro="http://www.ros.org/wiki/xacro">
   <xacro:macro name="omni_steering">
 		<gazebo>

File: rbsherpa_description/urdf/common.gazebo.xacro (robot description, xacro)
@@ -1,4 +1,4 @@
 <?xml version="1.0"?>
-<robot xmlns:xacro="http://ros.org/wiki/xacro">
+<robot xmlns:xacro="http://www.ros.org/wiki/xacro">
   <!-- ros control plugin -->
   <xacro:macro name="ros_control" > <!--  params="ns"  -->

File: rbsherpa_description/urdf/wheels/motor_wheel.urdf.xacro (robot description, xacro)
@@ -3,7 +3,7 @@
   <xacro:property name="M_PI" value="3.1415926535897931" />
   <!-- Wheels -->
-  <property name="wheel_radius" value="0.110" />
-  <property name="wheel_height" value="0.110" />
-  <property name="wheel_mass" value="5.0" />
+  <xacro:property name="wheel_radius" value="0.110" />
+  <xacro:property name="wheel_height" value="0.110" />
+  <xacro:property name="wheel_mass" value="5.0" />
   <!-- in kg-->
   <xacro:property name="steer_joint_damping" value="2.0" />
@@ -26,5 +26,5 @@
       <parent link="${parent}"/>
       <child link="${prefix}motor_wheel"/>
-      <insert_block name="origin" />
+      <xacro:insert_block name="origin" />
       <axis xyz="0 0 1" rpy="0 0 0" />
       <!-- limit effort="${steer_joint_effort_limit}" velocity="${steer_joint_velocity_limit}" lower="-1.5708" upper="1.5708" / -->

File: rbsherpa_description/urdf/wheels/wheel.urdf.xacro (robot description, xacro)
@@ -3,7 +3,7 @@
   <xacro:property name="M_PI" value="3.1415926535897931" />
   <!-- Wheels -->
-  <property name="wheel_radius" value="0.110" />
-  <property name="wheel_height" value="0.110" />
-  <property name="wheel_mass" value="5.0" />
+  <xacro:property name="wheel_radius" value="0.110" />
+  <xacro:property name="wheel_height" value="0.110" />
+  <xacro:property name="wheel_mass" value="5.0" />
   <!-- in kg-->
   <xacro:property name="steer_joint_damping" value="2.0" />
@@ -26,5 +26,5 @@
       <parent link="${parent}"/>
       <child link="${prefix}wheel"/>
-      <insert_block name="origin" />
+      <xacro:insert_block name="origin" />
       <axis xyz="0 1 0" rpy="0 0 0" />
       <limit effort="${wheel_joint_effort_limit}" velocity="${wheel_joint_velocity_limit}"/>
