Commit message: Fix on URDF. Change controller. Minor fixes.

File: rbsherpa_description/urdf/bases/base.urdf.xacro (robot description, xacro)
@@ -26,9 +26,9 @@
       <inertial>
         <mass value="25.0" />
-        <origin xyz="0.429 0 0" />
+        <origin xyz="0 0 0" />
         <inertia ixx="1.0" ixy="0.0" ixz="0.0" iyy="1.0" iyz="0.0" izz="1.0" />
       </inertial>
       <visual>
-        <origin xyz="0.429 0 0" rpy="0 0 0" />
+        <origin xyz="0 0 0" rpy="0 0 0" />
         <xacro:if value="${hq}">
           <geometry>
@@ -46,5 +46,5 @@
       </visual>
       <collision>
-        <origin xyz="0.429 0 0" rpy="0 0 0 " />
+        <origin xyz="0 0 0" rpy="0 0 0 " />
         <geometry>
           <mesh filename="package://rbsherpa_description/meshes/bases/rbsherpa_chassis.dae"/>

File: rbsherpa_description/urdf/rbsherpa_base.urdf.xacro (robot description, xacro)
@@ -6,5 +6,5 @@
   <!-- First we import all posible elements defined in the urdf.xacro files. All these elements are defined as macro:xacros -->
   <xacro:include filename="$(find rbsherpa_description)/urdf/bases/base.urdf.xacro" />
-  <xacro:include filename="$(find rbsherpa_description)/urdf/bases/base.gazebo.xacro" />
+  <!--xacro:include filename="$(find rbsherpa_description)/urdf/bases/base.gazebo.xacro" /-->
   <xacro:include filename="$(find rbsherpa_description)/urdf/wheels/motor_wheel.urdf.xacro" />
   <xacro:include filename="$(find rbsherpa_description)/urdf/wheels/wheel.urdf.xacro" />
@@ -33,10 +33,10 @@
       <origin xyz="${wheel_offset_x} ${wheel_offset_y} ${wheel_offset_z}" rpy="0 0 ${180.0*deg2rad}"/>
     </xacro:motor_wheel>
-    <xacro:wheel prefix="${prefix}back_left_" parent="${prefix}base_link" reflect="false" hq="true">
+    <xacro:motor_wheel prefix="${prefix}back_left_" parent="${prefix}base_link" reflect="false" hq="true">
       <origin xyz="-${wheel_offset_x} ${wheel_offset_y} ${wheel_offset_z}" rpy="0 0 ${180.0*deg2rad}"/>
-    </xacro:wheel>
-    <xacro:wheel prefix="${prefix}back_right_" parent="${prefix}base_link" reflect="false" hq="true">
+    </xacro:motor_wheel>
+    <xacro:motor_wheel prefix="${prefix}back_right_" parent="${prefix}base_link" reflect="false" hq="true">
       <origin xyz="-${wheel_offset_x} -${wheel_offset_y} ${wheel_offset_z}" rpy="0 0 0"/>
-    </xacro:wheel>
+    </xacro:motor_wheel>
     <!-- SENSORS see robotnik_sensors for the specific configuration -->
     <xacro:sensor_imu_hector prefix="$(arg prefix)imu" parent="$(arg prefix)base_link">
@@ -48,10 +48,10 @@
       <origin xyz="-0.22 0 0.275" rpy="0 0 0"/>
     </xacro:sensor_gps>
-    <!--xacro:sensor_sick_s300 name="front_left" parent="${prefix}base_link">
+    <xacro:sensor_sick_s300 prefix="front_left" parent="${prefix}base_link">
       <origin xyz="0.606321 0.345821 0.3095" rpy="${180*deg2rad} 0 ${45*deg2rad}"/>
     </xacro:sensor_sick_s300>
-    <xacro:sensor_sick_s300 name="back_right" parent="${prefix}base_link">
+    <xacro:sensor_sick_s300 prefix="back_right" parent="${prefix}base_link">
         <origin xyz="-0.606321 -0.345821 0.3095" rpy="${180*deg2rad} 0 ${235*deg2rad}"/>
-    </xacro:sensor_sick_s300 -->
+    </xacro:sensor_sick_s300>
   </xacro:macro>
 </robot>

File: rbsherpa_description/urdf/wheels/motor_wheel.urdf.xacro (robot description, xacro)
@@ -27,5 +27,5 @@
       <child link="${prefix}motor_wheel"/>
       <xacro:insert_block name="origin" />
-      <axis xyz="0 0 1" rpy="0 0 0" />
+      <axis xyz="0 0 -1" rpy="0 0 0" />
       <!-- limit effort="${steer_joint_effort_limit}" velocity="${steer_joint_velocity_limit}" lower="-1.5708" upper="1.5708" / -->
       <limit effort="${steer_joint_effort_limit}" velocity="${steer_joint_velocity_limit}" lower="-3.00" upper="3.00"/>
