Commit message: bi_arm_support.urdf.xacro: added load_kinematics_file ur parameter

File: rbsherpa_description/urdf/bases/bi_arm_support.urdf.xacro (robot description, xacro)
@@ -41,47 +41,51 @@
     </gazebo>
     <!-- Left UR10 -->
-    <joint name="$(arg prefix)left_arm_base_joint" type="fixed">
-      <origin xyz="0 0.13861 0.10943" rpy="0.902 0 3.14"/>
-      <parent link="${prefix}G2_link" />
-      <child link="${prefix}left_arm_base_link" />
-    </joint>
-    <xacro:ur10_robot prefix="$(arg prefix)left_arm_" joint_limited="true"
-    shoulder_pan_lower_limit="${-pi}" shoulder_pan_upper_limit="${pi}"
-    wrist_3_lower_limit="${-pi}" wrist_3_upper_limit="${pi}">
-    </xacro:ur10_robot>
-    <!-- Right UR10 -->
-    <joint name="$(arg prefix)right_arm_base_joint" type="fixed">
-      <origin xyz="0 -0.13861 0.10943" rpy="0.902 0 0"/>
-      <parent link="${prefix}G2_link" />
-      <child link="${prefix}right_arm_base_link" />
-    </joint>
-    <xacro:ur10_robot prefix="$(arg prefix)right_arm_" joint_limited="true"
-    shoulder_pan_lower_limit="${-pi}" shoulder_pan_upper_limit="${pi}"
-    wrist_3_lower_limit="${-pi}" wrist_3_upper_limit="${pi}">
-    </xacro:ur10_robot>
-    <!--xacro:if value="$(arg load_kinematics_file)">
-      <xacro:ur10_robot prefix="$(arg prefix)right_arm_" joint_limited="true"
+    <xacro:if value="${load_kinematics_file}">
+      <joint name="${prefix}left_arm_base_joint" type="fixed">
+        <origin xyz="0 0.13861 0.10943" rpy="0.902 0 3.1416"/>
+        <parent link="${prefix}G2_link" />
+        <child link="${prefix}left_arm_base_link" />
+      </joint>
+      <xacro:ur10_robot prefix="${prefix}left_arm_" joint_limited="true"
         shoulder_pan_lower_limit="${-pi}" shoulder_pan_upper_limit="${pi}"
         wrist_3_lower_limit="${-pi}" wrist_3_upper_limit="${pi}"
-        kinematics_file="${load_yaml('$(find rbsherpa_control)/config/ur10_calibration.yaml')}">
+        kinematics_file="${load_yaml('$(find rbsherpa_control)/config/calibration/ur10_calibration.yaml')}">
       </xacro:ur10_robot>
-      <joint name="$(arg prefix)right_arm_base_joint" type="fixed">
-        <origin xyz="0 0.13861 0.10943" rpy="0.902 0 3.14"/>
+    </xacro:if>
+    <xacro:unless value="${load_kinematics_file}">
+      <joint name="${prefix}left_arm_base_joint" type="fixed">
+        <origin xyz="0 0.13861 0.10943" rpy="0.902 0 3.1416"/>
         <parent link="${prefix}G2_link" />
         <child link="${prefix}right_arm_base_link" />
       </joint>
-    </xacro:if-->
-    <!--xacro:if value="$(arg load_kinematics_file)">
-      <xacro:ur10_robot prefix="$(arg prefix)left_arm_" joint_limited="true"
+      <xacro:ur10_robot prefix="${prefix}left_arm_" joint_limited="true"
+        shoulder_pan_lower_limit="${-pi}" shoulder_pan_upper_limit="${pi}"
+        wrist_3_lower_limit="${-pi}" wrist_3_upper_limit="${pi}">
+      </xacro:ur10_robot>
+    </xacro:unless>
+    <!-- Right UR10 -->
+    <xacro:if value="${load_kinematics_file}">
+      <joint name="${prefix}right_arm_base_joint" type="fixed">
+        <origin xyz="0 -0.13861 0.10943" rpy="0.902 0 0"/>
+        <parent link="${prefix}G2_link" />
+        <child link="${prefix}right_arm_base_link" />
+      </joint>
+      <xacro:ur10_robot prefix="${prefix}right_arm_" joint_limited="true"
         shoulder_pan_lower_limit="${-pi}" shoulder_pan_upper_limit="${pi}"
         wrist_3_lower_limit="${-pi}" wrist_3_upper_limit="${pi}"
-        kinematics_file="${load_yaml('$(find rbsherpa_control)/config/ur10_calibration.yaml')}">
+        kinematics_file="${load_yaml('$(find rbsherpa_control)/config/calibration/ur10_calibration.yaml')}">
       </xacro:ur10_robot>
-      <joint name="$(arg prefix)left_arm_base_joint" type="fixed">
-        <origin xyz="0 0.13861 0.10943" rpy="0.902 0 3.14"/>
+    </xacro:if>
+    <xacro:unless value="${load_kinematics_file}">
+      <joint name="${prefix}right_arm_base_joint" type="fixed">
+        <origin xyz="0 -0.13861 0.10943" rpy="0.902 0 0"/>
         <parent link="${prefix}G2_link" />
-        <child link="${prefix}left_arm_base_link" />
+        <child link="${prefix}right_arm_base_link" />
       </joint>
-    </xacro:if-->
+      <xacro:ur10_robot prefix="${prefix}right_arm_" joint_limited="true"
+        shoulder_pan_lower_limit="${-pi}" shoulder_pan_upper_limit="${pi}"
+        wrist_3_lower_limit="${-pi}" wrist_3_upper_limit="${pi}">
+      </xacro:ur10_robot>
+    </xacro:unless>
   </xacro:macro>
 </robot>

Commit message: colors for gazebo&rviz visualization added

File: rbsherpa_description/urdf/bases/bi_arm_support.urdf.xacro (robot description, xacro)
@@ -17,4 +17,7 @@
           <mesh filename="package://rbsherpa_description/meshes/bases/bi_arm_support.stl" />
         </geometry>
+        <material name="lightblack">
+          <color rgba="0.1 0.1 0.1 1"/>
+        </material>
       </visual>
       <collision>

File: rbsherpa_description/urdf/bases/rbsherpa_xl_base.urdf.xacro (robot description, xacro)
@@ -75,6 +75,6 @@
           </geometry>
         </xacro:unless>
-        <material name="lightgrey">
-          <color rgba="0.9 0.9 0.9 1"/>
+        <material name="lightred">
+          <color rgba="0.9 0.2 0.2 1"/>
         </material>
       </visual>

File: rbsherpa_description/urdf/wheels/motor_wheel_xl.urdf.xacro (robot description, xacro)
@@ -69,4 +69,7 @@
           </geometry>
         </xacro:unless>
+        <material name="red">
+             <color rgba="0.9 0.1 0.1 1"/>
+        </material>
       </visual>
       <collision>
@@ -133,4 +136,7 @@
           </geometry>
         </xacro:unless>
+        <material name="black_wheel">
+          <color rgba="0.1 0.1 0.1 1"/>
+        </material>
       </visual>
       <collision>

File: rbsherpa_description/urdf/wheels/wheel.gazebo.xacro (robot description, xacro)
@@ -9,7 +9,7 @@
       <visual>
         <material>
-          <ambient>0.19225 0.19225 0.19225 1.0</ambient>
-          <diffuse>0.50754 0.50754 0.50754 1.0</diffuse>
-          <specular>0.508273 0.508273 0.508273 1.0</specular>
+          <ambient>0.1 0.1 0.1 1.0</ambient>
+          <diffuse>0.250754 0.250754 0.250754 1.0</diffuse>
+          <specular>0.2508273 0.2508273 0.2508273 1.0</specular>
           <emissive>0.0 0.0 0.0 0.0</emissive>
         </material>
