Commit message: Minor fixes

File: rbsherpa_description/urdf/wheels/motor_wheel.urdf.xacro (robot description, xacro)
@@ -27,5 +27,5 @@
       <child link="${prefix}motor_wheel"/>
       <xacro:insert_block name="origin" />
-      <axis xyz="0 0 -1" rpy="0 0 0" />
+      <axis xyz="0 0 1" rpy="0 0 0" />
       <!-- limit effort="${steer_joint_effort_limit}" velocity="${steer_joint_velocity_limit}" lower="-1.5708" upper="1.5708" / -->
       <limit effort="${steer_joint_effort_limit}" velocity="${steer_joint_velocity_limit}" lower="-3.00" upper="3.00"/>
