Commit message: Add load_kinematics_file param

File: rbsherpa_description/robots/rbsherpa_xl_std.urdf.xacro (robot description, xacro)
@@ -28,5 +28,7 @@
     <xacro:property name="publish_bf" value="true" />
     <xacro:arg name="prefix" default="robot_" />
-    <xacro:macro name="rbsherpa" params="prefix publish_bf hq">
+    <xacro:arg name="launch_arm" default="false" />
+    <xacro:arg name="load_kinematics_file" default="false" />
+    <xacro:macro name="rbsherpa" params="prefix launch_arm load_kinematics_file publish_bf hq">
         <!-- *************** -->
         <!-- Robots Elements -->
@@ -47,7 +49,9 @@
         </xacro:motor_wheel>
         <!-- ARM  -->
-        <xacro:bi_arm_support prefix="${prefix}" parent="${prefix}base_link" hq="true">
-            <origin xyz="${G2_offset_x} ${G2_offset_y} ${G2_offset_z}" rpy="0 0 0"/>
-        </xacro:bi_arm_support>
+        <xacro:if value="$(arg launch_arm)">
+          <xacro:bi_arm_support prefix="${prefix}" parent="${prefix}base_link" hq="true" load_kinematics_file="${load_kinematics_file}">
+              <origin xyz="${G2_offset_x} ${G2_offset_y} ${G2_offset_z}" rpy="0 0 0"/>
+          </xacro:bi_arm_support>
+        </xacro:if>
         <!-- SENSORS see robotnik_sensors for the specific configuration -->
         <!-- IMU -->
@@ -70,4 +74,4 @@
     <!-- Gazebo ros control pluggins -->
     <xacro:ros_control/>
-    <xacro:rbsherpa prefix="$(arg prefix)" publish_bf="${publish_bf}" hq="${hq}"/>
+    <xacro:rbsherpa prefix="$(arg prefix)" publish_bf="${publish_bf}" hq="${hq}" launch_arm="$(arg launch_arm)" load_kinematics_file="$(arg load_kinematics_file)"/>
 </robot>

File: rbsherpa_description/urdf/bases/bi_arm_support.urdf.xacro (robot description, xacro)
@@ -4,5 +4,5 @@
   <xacro:include filename="$(find rbsherpa_description)/urdf/inertia.urdf.xacro" />
   <xacro:property name="M_PI" value="3.1415926535897931" />
-  <xacro:macro name="bi_arm_support" params="prefix parent *origin hq">
+  <xacro:macro name="bi_arm_support" params="prefix parent load_kinematics_file *origin hq">
     <!-- G2 -->
     <joint name="${prefix}G2_joint" type="fixed">
@@ -60,4 +60,28 @@
     wrist_3_lower_limit="${-pi}" wrist_3_upper_limit="${pi}">
     </xacro:ur10_robot>
+    <!--xacro:if value="$(arg load_kinematics_file)">
+      <xacro:ur10_robot prefix="$(arg prefix)right_arm_" joint_limited="true"
+        shoulder_pan_lower_limit="${-pi}" shoulder_pan_upper_limit="${pi}"
+        wrist_3_lower_limit="${-pi}" wrist_3_upper_limit="${pi}"
+        kinematics_file="${load_yaml('$(find rbsherpa_control)/config/ur10_calibration.yaml')}">
+      </xacro:ur10_robot>
+      <joint name="$(arg prefix)right_arm_base_joint" type="fixed">
+        <origin xyz="0 0.13861 0.10943" rpy="0.902 0 3.14"/>
+        <parent link="${prefix}G2_link" />
+        <child link="${prefix}right_arm_base_link" />
+      </joint>
+    </xacro:if-->
+    <!--xacro:if value="$(arg load_kinematics_file)">
+      <xacro:ur10_robot prefix="$(arg prefix)left_arm_" joint_limited="true"
+        shoulder_pan_lower_limit="${-pi}" shoulder_pan_upper_limit="${pi}"
+        wrist_3_lower_limit="${-pi}" wrist_3_upper_limit="${pi}"
+        kinematics_file="${load_yaml('$(find rbsherpa_control)/config/ur10_calibration.yaml')}">
+      </xacro:ur10_robot>
+      <joint name="$(arg prefix)left_arm_base_joint" type="fixed">
+        <origin xyz="0 0.13861 0.10943" rpy="0.902 0 3.14"/>
+        <parent link="${prefix}G2_link" />
+        <child link="${prefix}left_arm_base_link" />
+      </joint>
+    </xacro:if-->
   </xacro:macro>
 </robot>
