Commit message: Minor corrections. Controllers not working

File: rbsherpa_description/robots/rbsherpa_std.urdf.xacro (robot description, xacro)
@@ -10,5 +10,5 @@
 	<!-- Import all available sensors -->
 	<xacro:include filename="$(find robotnik_sensors)/urdf/all_sensors.urdf.xacro" />
-	<xacro:property name="prefix" value="" />
+	<xacro:property name="prefix" value="rbsherpa_" />
 	<xacro:property name="publish_bf" value="true" />
 	<xacro:property name="hq" value="true" />

Commit message: Change on robot_id and remove unused files

File: rbsherpa_description/robots/rbsherpa_std.urdf.xacro (robot description, xacro)
@@ -10,5 +10,5 @@
 	<!-- Import all available sensors -->
 	<xacro:include filename="$(find robotnik_sensors)/urdf/all_sensors.urdf.xacro" />
-	<xacro:property name="prefix" value="rbsherpa_" />
+	<xacro:property name="prefix" value="robot_" />
 	<xacro:property name="publish_bf" value="true" />
 	<xacro:property name="hq" value="true" />

Commit message: Update to standard format

File: rbsherpa_description/robots/rbsherpa_std.urdf.xacro (robot description, xacro)
@@ -1,17 +1,64 @@
 <?xml version="1.0"?>
-<robot name="rbsherpa"
-	xmlns:xacro="http://www.ros.org/wiki/xacro">
-	<!-- ***************** -->
-	<!-- Imported elements -->
-	<!-- ***************** -->
-	<!-- First we import all posible elements defined in the urdf.xacro files. All these elements are defined as macro:xacros -->
-	<xacro:include filename="$(find rbsherpa_description)/urdf/rbsherpa_base.urdf.xacro" />
-	<xacro:include filename="$(find rbsherpa_description)/urdf/common.gazebo.xacro" />
-	<!-- Import all available sensors -->
-	<xacro:include filename="$(find robotnik_sensors)/urdf/all_sensors.urdf.xacro" />
-	<xacro:property name="prefix" value="robot_" />
-	<xacro:property name="publish_bf" value="true" />
-	<xacro:property name="hq" value="true" />
-	<xacro:rbsherpa_base prefix="${prefix}" publish_bf="${publish_bf}" hq="${hq}"/>
-	<xacro:ros_control />
+<!-- RBSherpa v2.0 -->
+<robot name="rbsherpa" xmlns:xacro="http://www.ros.org/wiki/xacro">
+    <!-- ***************** -->
+    <!-- Imported elements -->
+    <!-- ***************** -->
+    <!-- First we import all posible elements defined in the urdf.xacro files. All these elements are defined as macro:xacros -->
+    <!-- Import rbsherpa base elements-->
+    <xacro:include filename="$(find rbsherpa_description)/urdf/bases/rbsherpa_base_v2.urdf.xacro" />
+    <!-- Import rbsherpa wheels -->
+    <xacro:include filename="$(find rbsherpa_description)/urdf/wheels/motor_wheel.urdf.xacro" />
+    <xacro:include filename="$(find rbsherpa_description)/urdf/wheels/wheel.urdf.xacro" />
+    <!-- Import all available sensors -->
+    <xacro:include filename="$(find robotnik_sensors)/urdf/all_sensors.urdf.xacro" />
+    <xacro:property name="PI" value="3.1415926535897931"/>
+    <xacro:property name="deg2rad" value="0.01745329251"/>
+    <!-- Wheel parameters -->
+    <xacro:property name="wheel_offset_x" value="0.429" />    <!-- x,y,z in translation from base_link to the center of the wheel -->
+    <xacro:property name="wheel_offset_y" value="0.227" />
+    <xacro:property name="wheel_offset_z" value="0.0" />
+    <!-- Flag to select the high or low quality model -->
+    <xacro:property name="hq" value="true" />
+    <xacro:property name="publish_bf" value="true" />
+    <xacro:arg name="prefix" default="robot_" />
+    <xacro:macro name="rbsherpa" params="prefix publish_bf hq">
+        <!-- *************** -->
+        <!-- Robots Elements -->
+        <!-- *************** -->
+        <!-- Here we create the robot elements using the xacro:macros imported at the beggining of this file -->
+        <xacro:rbsherpa_base prefix="${prefix}" publish_bf="${publish_bf}" hq="${hq}"/>
+        <xacro:motor_wheel prefix="${prefix}front_right_" parent="${prefix}base_link" reflect="false" hq="true">
+            <origin xyz="${wheel_offset_x} -${wheel_offset_y} ${wheel_offset_z}" rpy="0 0 0"/>
+        </xacro:motor_wheel>
+        <xacro:motor_wheel prefix="${prefix}front_left_" parent="${prefix}base_link" reflect="false" hq="true">
+            <origin xyz="${wheel_offset_x} ${wheel_offset_y} ${wheel_offset_z}" rpy="0 0 ${180.0*deg2rad}"/>
+        </xacro:motor_wheel>
+        <xacro:motor_wheel prefix="${prefix}back_left_" parent="${prefix}base_link" reflect="false" hq="true">
+            <origin xyz="-${wheel_offset_x} ${wheel_offset_y} ${wheel_offset_z}" rpy="0 0 ${180.0*deg2rad}"/>
+        </xacro:motor_wheel>
+        <xacro:motor_wheel prefix="${prefix}back_right_" parent="${prefix}base_link" reflect="false" hq="true">
+            <origin xyz="-${wheel_offset_x} -${wheel_offset_y} ${wheel_offset_z}" rpy="0 0 0"/>
+        </xacro:motor_wheel>
+        <!-- SENSORS see robotnik_sensors for the specific configuration -->
+        <!-- IMU -->
+        <xacro:sensor_imu_hector prefix="$(arg prefix)imu" parent="$(arg prefix)base_link">
+            <origin xyz="0.3 0.3 0.250" rpy="0 0 0"/>
+        </xacro:sensor_imu_hector>
+        <!-- GPS -->
+        <xacro:sensor_gps prefix="$(arg prefix)gps" parent="$(arg prefix)base_link">
+        <origin xyz="-0.22 0 0.275" rpy="0 0 0"/>
+        </xacro:sensor_gps>
+        <!-- 2d laser -->
+        <xacro:sensor_sick_s300 prefix="$(arg prefix)front_laser" parent="${prefix}base_link" prefix_topic="front_laser">
+        <origin xyz="0.53 0.325821 0.3095" rpy="${180*deg2rad} 0 ${45*deg2rad}"/>
+        </xacro:sensor_sick_s300>
+        <!-- 2d laser -->
+        <xacro:sensor_sick_s300 prefix="$(arg prefix)rear_laser" parent="${prefix}base_link" prefix_topic="rear_laser">
+            <origin xyz="-0.532 -0.323821 0.3095" rpy="${180*deg2rad} 0 ${225*deg2rad}"/>
+        </xacro:sensor_sick_s300>
+    </xacro:macro>
+    <!-- Gazebo ros control pluggins -->
+    <xacro:ros_control/>
+    <xacro:rbsherpa prefix="$(arg prefix)" publish_bf="${publish_bf}" hq="${hq}"/>
 </robot>

File: rbsherpa_description/urdf/bases/rbsherpa_base_v2.urdf.xacro (robot description, xacro)
@@ -1,5 +1,6 @@
 <?xml version="1.0"?>
 <robot xmlns:xacro="http://www.ros.org/wiki/xacro">
-  <xacro:macro name="base" params="prefix publish_bf hq">
+  <xacro:include filename="$(find rbsherpa_description)/urdf/bases/rbsherpa_base.gazebo.xacro" />
+  <xacro:macro name="rbsherpa_base" params="prefix publish_bf hq">
     <!-- Robot mechanical and motor parameters -->
     <xacro:property name="PI" value="3.1415926535897931"/>

Commit message: Add stl v3 to description

File: rbsherpa_description/robots/rbsherpa_std.urdf.xacro (robot description, xacro)
@@ -10,5 +10,5 @@
     <!-- Import rbsherpa wheels -->
     <xacro:include filename="$(find rbsherpa_description)/urdf/wheels/motor_wheel.urdf.xacro" />
-    <xacro:include filename="$(find rbsherpa_description)/urdf/wheels/wheel.urdf.xacro" />
+    <xacro:include filename="$(find rbsherpa_description)/urdf/wheels/wheel_v3.urdf.xacro" />
     <!-- Import all available sensors -->
     <xacro:include filename="$(find robotnik_sensors)/urdf/all_sensors.urdf.xacro" />
@@ -48,13 +48,13 @@
         <!-- GPS -->
         <xacro:sensor_gps prefix="$(arg prefix)gps" parent="$(arg prefix)base_link">
-            <origin xyz="0.33375 0.0 1.115" rpy="0 0 0"/>
+            <origin xyz="-0.04625 0.0 1.115" rpy="0 0 0"/>
         </xacro:sensor_gps>
         <!-- Solid-State laser -->
-        <xacro:sensor_benewake_ce30 prefix="$(arg prefix)front_ss_laser" parent="${prefix}base_link" range_min="35" range_max="305" hfov="120" vfov="9" fps="20" gpu="false">
-            <origin xyz="0.5642 0.0 0.1857" rpy="${180*deg2rad} 0 0"/>
-        </xacro:sensor_benewake_ce30>
+        <xacro:sensor_benewake_ce30c prefix="$(arg prefix)front_ss_laser" parent="${prefix}base_link" gpu="false">
+            <origin xyz="0.5657 0.0 0.1622" rpy="0 0 0"/>
+        </xacro:sensor_benewake_ce30c>
         <!-- 2d laser -->
         <xacro:sensor_sick_tim551 prefix="$(arg prefix)front_laser" parent="${prefix}base_link" prefix_topic="front_laser">
-            <origin xyz="0.5307 0.0 0.157" rpy="${180*deg2rad} 0 0"/>
+            <origin xyz="0.5307 0.0 0.15389" rpy="${180*deg2rad} 0 0"/>
         </xacro:sensor_sick_tim551>
     </xacro:macro>

File: rbsherpa_description/robots/rbsherpa_std_v2.urdf.xacro (robot description, xacro)
@@ -10,5 +10,5 @@
     <!-- Import rbsherpa wheels -->
     <xacro:include filename="$(find rbsherpa_description)/urdf/wheels/motor_wheel.urdf.xacro" />
-    <xacro:include filename="$(find rbsherpa_description)/urdf/wheels/wheel.urdf.xacro" />
+    <xacro:include filename="$(find rbsherpa_description)/urdf/wheels/wheel_v2.urdf.xacro" />
     <!-- Import all available sensors -->
     <xacro:include filename="$(find robotnik_sensors)/urdf/all_sensors.urdf.xacro" />

File: rbsherpa_description/urdf/bases/rbsherpa_base_v2.urdf.xacro (robot description, xacro)
@@ -34,10 +34,10 @@
         <xacro:if value="${hq}">
           <geometry>
-            <mesh filename="package://rbsherpa_description/meshes/bases/rbsherpa_chassis.dae"/>
+            <mesh filename="package://rbsherpa_description/meshes/bases/rbsherpa_chassis_v2.stl"/>
           </geometry>
         </xacro:if>
         <xacro:unless value="${hq}">
           <geometry>
-            <mesh filename="package://rbsherpa_description/meshes/bases/rbsherpa_chassis.dae"/>
+            <mesh filename="package://rbsherpa_description/meshes/bases/rbsherpa_chassis_v2.dae"/>
           </geometry>
         </xacro:unless>
@@ -49,5 +49,5 @@
         <origin xyz="0 0 0" rpy="0 0 0 " />
         <geometry>
-          <mesh filename="package://rbsherpa_description/meshes/bases/rbsherpa_chassis.dae"/>
+          <mesh filename="package://rbsherpa_description/meshes/bases/rbsherpa_chassis_v2.dae"/>
         </geometry>
       </collision>

File: rbsherpa_description/urdf/bases/rbsherpa_base_v3.urdf.xacro (robot description, xacro)
@@ -34,10 +34,10 @@
         <xacro:if value="${hq}">
           <geometry>
-            <mesh filename="package://rbsherpa_description/meshes/bases/rbsherpa_chassis.dae"/>
+            <mesh filename="package://rbsherpa_description/meshes/bases/rbsherpa_chassis_v3.stl"/>
           </geometry>
         </xacro:if>
         <xacro:unless value="${hq}">
           <geometry>
-            <mesh filename="package://rbsherpa_description/meshes/bases/rbsherpa_chassis.dae"/>
+            <mesh filename="package://rbsherpa_description/meshes/bases/rbsherpa_chassis_v3.dae"/>
           </geometry>
         </xacro:unless>
@@ -49,5 +49,36 @@
         <origin xyz="0 0 0" rpy="0 0 0 " />
         <geometry>
-          <mesh filename="package://rbsherpa_description/meshes/bases/rbsherpa_chassis.dae"/>
+          <mesh filename="package://rbsherpa_description/meshes/bases/rbsherpa_chassis_v3.dae"/>
+        </geometry>
+      </collision>
+    </link>
+    <!-- Logos -->
+		<joint name="${prefix}base_logos_joint" type="fixed">
+			<origin xyz="0 0 0" rpy="0 0 0 " />
+			<parent link="${prefix}base_link"/>
+			<child link="${prefix}base_logos_link" />
+		</joint>
+		<!-- Logos -->
+		<link name="${prefix}base_logos_link" >
+      <visual>
+        <origin xyz="0 0 0" rpy="0 0 0" />
+        <xacro:if value="${hq}">
+          <geometry>
+            <mesh filename="package://rbsherpa_description/meshes/bases/rbsherpa_logos_v3.stl" scale="1.001 1.001 1.001"/>
+          </geometry>
+        </xacro:if>
+        <xacro:unless value="${hq}">
+          <geometry>
+            <mesh filename="package://rbsherpa_description/meshes/bases/rbsherpa_logos_v3.dae" scale="1.001 1.001 1.001"/>
+          </geometry>
+        </xacro:unless>
+        <material name="lightgrey">
+          <color rgba="0.9 0.9 0.9 1"/>
+        </material>
+      </visual>
+      <collision>
+        <origin xyz="0 0 0" rpy="0 0 0 " />
+        <geometry>
+          <mesh filename="package://rbsherpa_description/meshes/bases/rbsherpa_chassis_v3.dae" scale="1.001 1.001 1.001"/>
         </geometry>
       </collision>

Commit message: robot.urdf.xacro: corrected prefix issue
+ the prefix was sometimes added as an argument within the macro

File: rbsherpa_description/robots/rbsherpa_std.urdf.xacro (robot description, xacro)
@@ -43,17 +43,17 @@
         <!-- SENSORS see robotnik_sensors for the specific configuration -->
         <!-- IMU -->
-        <xacro:sensor_imu_hector prefix="$(arg prefix)imu" parent="$(arg prefix)base_link">
+        <xacro:sensor_imu_hector prefix="${prefix}imu" parent="${prefix}base_link">
             <origin xyz="0.3 0.3 0.250" rpy="0 0 0"/>
         </xacro:sensor_imu_hector>
         <!-- GPS -->
-        <xacro:sensor_gps prefix="$(arg prefix)gps" parent="$(arg prefix)base_link">
+        <xacro:sensor_gps prefix="${prefix}gps" parent="${prefix}base_link">
             <origin xyz="-0.04625 0.0 1.115" rpy="0 0 0"/>
         </xacro:sensor_gps>
         <!-- Solid-State laser -->
-        <xacro:sensor_benewake_ce30c prefix="$(arg prefix)front_ss_laser" parent="${prefix}base_link" gpu="false">
+        <xacro:sensor_benewake_ce30c prefix="${prefix}front_ss_laser" parent="${prefix}base_link" gpu="false">
             <origin xyz="0.5657 0.0 0.1622" rpy="0 0 0"/>
         </xacro:sensor_benewake_ce30c>
         <!-- 2d laser -->
-        <xacro:sensor_sick_tim551 prefix="$(arg prefix)front_laser" parent="${prefix}base_link" prefix_topic="front_laser">
+        <xacro:sensor_sick_tim551 prefix="${prefix}front_laser" parent="${prefix}base_link" prefix_topic="front_laser">
             <origin xyz="0.5307 0.0 0.15389" rpy="${180*deg2rad} 0 0"/>
         </xacro:sensor_sick_tim551>

File: rbsherpa_description/robots/rbsherpa_std_ur10.urdf.xacro (robot description, xacro)
@@ -35,5 +35,5 @@
     <xacro:property name="publish_bf" value="true" />
     <xacro:arg name="prefix" default="robot_" />
-    <xacro:macro name="rbsherpa" params="prefix publish_bf hq">
+    <xacro:macro name="rbsherpa" params="prefix publish_bf load_kinematics_file hq">
         <!-- *************** -->
         <!-- Robots Elements -->
@@ -55,36 +55,36 @@
         <!-- SENSORS see robotnik_sensors for the specific configuration -->
         <!-- IMU -->
-        <xacro:sensor_imu_hector prefix="$(arg prefix)imu" parent="$(arg prefix)base_link">
+        <xacro:sensor_imu_hector prefix="${prefix}imu" parent="${prefix}base_link">
             <origin xyz="0.3 0.3 0.250" rpy="0 0 0"/>
         </xacro:sensor_imu_hector>
         <!-- GPS -->
-        <!--xacro:sensor_gps prefix="$(arg prefix)gps" parent="$(arg prefix)base_link">
+        <!--xacro:sensor_gps prefix="${prefix}gps" parent="${prefix}base_link">
             <origin xyz="-0.04625 0.0 1.115" rpy="0 0 0"/>
         </xacro:sensor_gps-->
         <!-- Solid-State laser -->
-        <xacro:sensor_benewake_ce30c prefix="$(arg prefix)front_ss_laser" parent="${prefix}base_link" gpu="false">
+        <xacro:sensor_benewake_ce30c prefix="${prefix}front_ss_laser" parent="${prefix}base_link" gpu="false">
             <origin xyz="0.5657 0.0 0.1622" rpy="0 0 0"/>
         </xacro:sensor_benewake_ce30c>
         <!-- 2d laser -->
-        <xacro:sensor_sick_tim551 prefix="$(arg prefix)front_laser" parent="${prefix}base_link" prefix_topic="front_laser">
+        <xacro:sensor_sick_tim551 prefix="${prefix}front_laser" parent="${prefix}base_link" prefix_topic="front_laser">
             <origin xyz="0.5307 0.0 0.15389" rpy="${180*deg2rad} 0 0"/>
         </xacro:sensor_sick_tim551>
         <!-- UR-10 ARM -->
-        <xacro:if value="$(arg load_kinematics_file)">
-            <xacro:ur10_robot prefix="$(arg prefix)arm_" joint_limited="true" shoulder_pan_lower_limit="${-pi}" shoulder_pan_upper_limit="${pi}" wrist_3_lower_limit="${-pi}" wrist_3_upper_limit="${pi}" kinematics_file="${load_yaml('$(find rbkairos_control)/config/ur10_calibration.yaml')}">
+        <xacro:if value="${load_kinematics_file}">
+            <xacro:ur10_robot prefix="${prefix}arm_" joint_limited="true" shoulder_pan_lower_limit="${-pi}" shoulder_pan_upper_limit="${pi}" wrist_3_lower_limit="${-pi}" wrist_3_upper_limit="${pi}" kinematics_file="${load_yaml('$(find rbsherpa_control)/config/calibration/ur10_calibration.yaml')}">
             </xacro:ur10_robot>
-            <joint name="$(arg prefix)arm_base_joint" type="fixed">
+            <joint name="${prefix}arm_base_joint" type="fixed">
                 <origin xyz="${arm_position_x} ${arm_position_y} ${arm_position_z}" rpy="${arm_orientation_r} ${arm_orientation_p} ${arm_orientation_y}"/>
-                <parent link="$(arg prefix)base_link" />
-                <child link="$(arg prefix)arm_base_link" />
+                <parent link="${prefix}base_link" />
+                <child link="${prefix}arm_base_link" />
             </joint>
         </xacro:if>
-        <xacro:unless value="$(arg load_kinematics_file)">
-            <xacro:ur10_robot prefix="$(arg prefix)arm_" joint_limited="true" shoulder_pan_lower_limit="${-pi}" shoulder_pan_upper_limit="${pi}" wrist_3_lower_limit="${-pi}" wrist_3_upper_limit="${pi}">
+        <xacro:unless value="${load_kinematics_file}">
+            <xacro:ur10_robot prefix="${prefix}arm_" joint_limited="true" shoulder_pan_lower_limit="${-pi}" shoulder_pan_upper_limit="${pi}" wrist_3_lower_limit="${-pi}" wrist_3_upper_limit="${pi}">
             </xacro:ur10_robot>
-            <joint name="$(arg prefix)arm_base_joint" type="fixed">
+            <joint name="${prefix}arm_base_joint" type="fixed">
                 <origin xyz="${arm_position_x} ${arm_position_y} ${arm_position_z}" rpy="${arm_orientation_r} ${arm_orientation_p} ${arm_orientation_y}"/>
-                <parent link="$(arg prefix)base_link" />
-                <child link="$(arg prefix)arm_base_link" />
+                <parent link="${prefix}base_link" />
+                <child link="${prefix}arm_base_link" />
             </joint>
         </xacro:unless>
@@ -92,4 +92,4 @@
     <!-- Gazebo ros control pluggins -->
     <xacro:ros_control/>
-    <xacro:rbsherpa prefix="$(arg prefix)" publish_bf="${publish_bf}" hq="${hq}"/>
+    <xacro:rbsherpa prefix="$(arg prefix)" load_kinematics_file="$(arg load_kinematics_file)" publish_bf="${publish_bf}" hq="${hq}"/>
 </robot>
