Commit message: rbsherpa_description: added color, corrected missmatched meshes, updated rbsherpa_xl version

File: rbsherpa_description/robots/rbsherpa_std_ur10.urdf.xacro (robot description, xacro)
@@ -41,14 +41,14 @@
         <!-- Here we create the robot elements using the xacro:macros imported at the beggining of this file -->
         <xacro:rbsherpa_base prefix="${prefix}" publish_bf="${publish_bf}" hq="${hq}"/>
-        <xacro:motor_wheel prefix="${prefix}front_right_" parent="${prefix}base_link" reflect="false" hq="true">
+        <xacro:motor_wheel prefix="${prefix}front_right_" parent="${prefix}base_link" reflect="false" hq="${hq}">
             <origin xyz="${wheel_offset_x} -${wheel_offset_y} ${wheel_offset_z}" rpy="0 0 0"/>
         </xacro:motor_wheel>
-        <xacro:motor_wheel prefix="${prefix}front_left_" parent="${prefix}base_link" reflect="false" hq="true">
+        <xacro:motor_wheel prefix="${prefix}front_left_" parent="${prefix}base_link" reflect="false" hq="${hq}">
             <origin xyz="${wheel_offset_x} ${wheel_offset_y} ${wheel_offset_z}" rpy="0 0 ${180.0*deg2rad}"/>
         </xacro:motor_wheel>
-        <xacro:motor_wheel prefix="${prefix}back_left_" parent="${prefix}base_link" reflect="false" hq="true">
+        <xacro:motor_wheel prefix="${prefix}back_left_" parent="${prefix}base_link" reflect="false" hq="${hq}">
             <origin xyz="-${wheel_offset_x} ${wheel_offset_y} ${wheel_offset_z}" rpy="0 0 ${180.0*deg2rad}"/>
         </xacro:motor_wheel>
-        <xacro:motor_wheel prefix="${prefix}back_right_" parent="${prefix}base_link" reflect="false" hq="true">
+        <xacro:motor_wheel prefix="${prefix}back_right_" parent="${prefix}base_link" reflect="false" hq="${hq}">
             <origin xyz="-${wheel_offset_x} -${wheel_offset_y} ${wheel_offset_z}" rpy="0 0 0"/>
         </xacro:motor_wheel>
@@ -81,5 +81,5 @@
         </xacro:if>
         <xacro:unless value="${load_kinematics_file}">
-            <xacro:ur10_robot prefix="${prefix}arm_" joint_limited="true" shoulder_pan_lower_limit="${-pi}" shoulder_pan_upper_limit="${pi}" wrist_3_lower_limit="${-pi}" wrist_3_upper_limit="${pi}">
+            <xacro:ur10_robot prefix="${prefix}arm_" joint_limited="true" shoulder_pan_lower_limit="${-pi}" shoulder_pan_upper_limit="${pi}" wrist_3_lower_limit="${-pi}" wrist_3_upper_limit="${pi}" >
             </xacro:ur10_robot>
             <joint name="${prefix}arm_base_joint" type="fixed">

File: rbsherpa_description/robots/rbsherpa_std_v2.urdf.xacro (robot description, xacro)
@@ -29,14 +29,14 @@
         <!-- Here we create the robot elements using the xacro:macros imported at the beggining of this file -->
         <xacro:rbsherpa_base prefix="${prefix}" publish_bf="${publish_bf}" hq="${hq}"/>
-        <xacro:motor_wheel prefix="${prefix}front_right_" parent="${prefix}base_link" reflect="false" hq="true">
+        <xacro:motor_wheel prefix="${prefix}front_right_" parent="${prefix}base_link" reflect="false" hq="${hq}">
             <origin xyz="${wheel_offset_x} -${wheel_offset_y} ${wheel_offset_z}" rpy="0 0 0"/>
         </xacro:motor_wheel>
-        <xacro:motor_wheel prefix="${prefix}front_left_" parent="${prefix}base_link" reflect="false" hq="true">
+        <xacro:motor_wheel prefix="${prefix}front_left_" parent="${prefix}base_link" reflect="false" hq="${hq}">
             <origin xyz="${wheel_offset_x} ${wheel_offset_y} ${wheel_offset_z}" rpy="0 0 ${180.0*deg2rad}"/>
         </xacro:motor_wheel>
-        <xacro:motor_wheel prefix="${prefix}back_left_" parent="${prefix}base_link" reflect="false" hq="true">
+        <xacro:motor_wheel prefix="${prefix}back_left_" parent="${prefix}base_link" reflect="false" hq="${hq}">
             <origin xyz="-${wheel_offset_x} ${wheel_offset_y} ${wheel_offset_z}" rpy="0 0 ${180.0*deg2rad}"/>
         </xacro:motor_wheel>
-        <xacro:motor_wheel prefix="${prefix}back_right_" parent="${prefix}base_link" reflect="false" hq="true">
+        <xacro:motor_wheel prefix="${prefix}back_right_" parent="${prefix}base_link" reflect="false" hq="${hq}">
             <origin xyz="-${wheel_offset_x} -${wheel_offset_y} ${wheel_offset_z}" rpy="0 0 0"/>
         </xacro:motor_wheel>

File: rbsherpa_description/robots/rbsherpa_std_v3.urdf.xacro (robot description, xacro)
@@ -29,14 +29,14 @@
         <!-- Here we create the robot elements using the xacro:macros imported at the beggining of this file -->
         <xacro:rbsherpa_base prefix="${prefix}" publish_bf="${publish_bf}" hq="${hq}"/>
-        <xacro:motor_wheel prefix="${prefix}front_right_" parent="${prefix}base_link" reflect="false" hq="true">
+        <xacro:motor_wheel prefix="${prefix}front_right_" parent="${prefix}base_link" reflect="false" hq="${hq}">
             <origin xyz="${wheel_offset_x} -${wheel_offset_y} ${wheel_offset_z}" rpy="0 0 0"/>
         </xacro:motor_wheel>
-        <xacro:motor_wheel prefix="${prefix}front_left_" parent="${prefix}base_link" reflect="false" hq="true">
+        <xacro:motor_wheel prefix="${prefix}front_left_" parent="${prefix}base_link" reflect="false" hq="${hq}">
             <origin xyz="${wheel_offset_x} ${wheel_offset_y} ${wheel_offset_z}" rpy="0 0 ${180.0*deg2rad}"/>
         </xacro:motor_wheel>
-        <xacro:motor_wheel prefix="${prefix}back_left_" parent="${prefix}base_link" reflect="false" hq="true">
+        <xacro:motor_wheel prefix="${prefix}back_left_" parent="${prefix}base_link" reflect="false" hq="${hq}">
             <origin xyz="-${wheel_offset_x} ${wheel_offset_y} ${wheel_offset_z}" rpy="0 0 ${180.0*deg2rad}"/>
         </xacro:motor_wheel>
-        <xacro:motor_wheel prefix="${prefix}back_right_" parent="${prefix}base_link" reflect="false" hq="true">
+        <xacro:motor_wheel prefix="${prefix}back_right_" parent="${prefix}base_link" reflect="false" hq="${hq}">
             <origin xyz="-${wheel_offset_x} -${wheel_offset_y} ${wheel_offset_z}" rpy="0 0 0"/>
         </xacro:motor_wheel>

File: rbsherpa_description/robots/rbsherpa_xl.urdf.xacro (robot description, xacro)
@@ -17,11 +17,11 @@
     <xacro:property name="deg2rad" value="0.01745329251"/>
     <!-- Wheel parameters -->
-    <xacro:property name="wheel_offset_x" value="0.4655" />    <!-- x,y,z in translation from base_link to the center of the wheel -->
-    <xacro:property name="wheel_offset_y" value="0.294" />
+    <xacro:property name="wheel_offset_x" value="0.4795" />    <!-- x,y,z in translation from base_link to the center of the wheel -->
+    <xacro:property name="wheel_offset_y" value="0.2925" />
     <xacro:property name="wheel_offset_z" value="0.0" />
-    <!-- Wheel parameters -->
-    <xacro:property name="G2_offset_x" value="0.17286" />
+    <!-- Bi-arm support parameters -->
+    <xacro:property name="G2_offset_x" value="0.207" />
     <xacro:property name="G2_offset_y" value="0.0" />
-    <xacro:property name="G2_offset_z" value="0.50288" />
+    <xacro:property name="G2_offset_z" value="0.57188" />
     <!-- Flag to select the high or low quality model -->
     <xacro:property name="hq" value="true" />
@@ -36,14 +36,14 @@
         <!-- Here we create the robot elements using the xacro:macros imported at the beggining of this file -->
         <xacro:rbsherpa_base prefix="${prefix}" publish_bf="${publish_bf}" hq="${hq}"/>
-        <xacro:motor_wheel prefix="${prefix}front_right_" parent="${prefix}base_link" reflect="false" hq="true">
+        <xacro:motor_wheel prefix="${prefix}front_right_" parent="${prefix}base_link" reflect="false" hq="${hq}">
             <origin xyz="${wheel_offset_x} -${wheel_offset_y} ${wheel_offset_z}" rpy="0 0 0"/>
         </xacro:motor_wheel>
-        <xacro:motor_wheel prefix="${prefix}front_left_" parent="${prefix}base_link" reflect="false" hq="true">
+        <xacro:motor_wheel prefix="${prefix}front_left_" parent="${prefix}base_link" reflect="false" hq="${hq}">
             <origin xyz="${wheel_offset_x} ${wheel_offset_y} ${wheel_offset_z}" rpy="0 0 ${180.0*deg2rad}"/>
         </xacro:motor_wheel>
-        <xacro:motor_wheel prefix="${prefix}back_left_" parent="${prefix}base_link" reflect="false" hq="true">
+        <xacro:motor_wheel prefix="${prefix}back_left_" parent="${prefix}base_link" reflect="false" hq="${hq}">
             <origin xyz="-${wheel_offset_x} ${wheel_offset_y} ${wheel_offset_z}" rpy="0 0 ${180.0*deg2rad}"/>
         </xacro:motor_wheel>
-        <xacro:motor_wheel prefix="${prefix}back_right_" parent="${prefix}base_link" reflect="false" hq="true">
+        <xacro:motor_wheel prefix="${prefix}back_right_" parent="${prefix}base_link" reflect="false" hq="${hq}">
             <origin xyz="-${wheel_offset_x} -${wheel_offset_y} ${wheel_offset_z}" rpy="0 0 0"/>
         </xacro:motor_wheel>
@@ -56,11 +56,15 @@
         <!-- SENSORS see robotnik_sensors for the specific configuration -->
         <!-- IMU -->
-        <!--xacro:sensor_imu_hector prefix="${prefix}imu" parent="${prefix}base_link">
-            <origin xyz="0.3 0.3 0.250" rpy="0 0 0"/>
-        </xacro:sensor_imu_hector-->
+        <xacro:sensor_imu_hector prefix="${prefix}imu" parent="${prefix}base_link">
+            <origin xyz="0.3 0.0 0.3" rpy="0 0 0"/>
+        </xacro:sensor_imu_hector>
         <!-- GPS -->
         <!--xacro:sensor_gps prefix="${prefix}gps" parent="${prefix}base_link">
-            <origin xyz="-0.04625 0.0 1.115" rpy="0 0 0"/>
+            <origin xyz="-0.04625 0.0 0.59188" rpy="0 0 0"/>
         </xacro:sensor_gps-->
+        <!-- Lidar -->
+        <!--xacro:sensor_rslidar_16 prefix="${prefix}front_ss_laser" parent="${prefix}base_link" gpu="true">
+            <origin xyz="0.511 0 0.21" rpy="0 0 0"/>
+        </xacro:sensor_rslidar_16-->
         <!-- Solid-State laser -->
         <!--xacro:sensor_benewake_ce30c prefix="${prefix}front_ss_laser" parent="${prefix}base_link" gpu="false">

File: rbsherpa_description/urdf/bases/bi_arm_support.urdf.xacro (robot description, xacro)
@@ -1,5 +1,5 @@
 <?xml version="1.0"?>
 <robot xmlns:xacro="http://wiki.ros.org/xacro">
-	<xacro:include filename="$(find ur_description)/urdf/ur10.urdf.xacro" />
+	<xacro:include filename="$(find ur_e_description)/urdf/ur10e.urdf.xacro" />
   <xacro:include filename="$(find rbsherpa_description)/urdf/inertia.urdf.xacro" />
   <xacro:property name="M_PI" value="3.1415926535897931" />
@@ -13,5 +13,5 @@
     <link name="${prefix}G2_link">
       <visual>
-        <origin xyz="0 0 0" rpy="0 0 ${M_PI/2.0}" />
+        <origin xyz="0.0 0.0 0.0" rpy="0 0 ${M_PI/2.0}" />
         <geometry>
           <mesh filename="package://rbsherpa_description/meshes/bases/bi_arm_support.stl" />
@@ -25,6 +25,6 @@
       </collision>
       <inertial>
-        <mass value="10" />
-        <origin xyz="0 0 0" rpy="${M_PI/2.0} 0 0"/>
+        <mass value="5" />
+        <origin xyz="0 0 0" rpy="0 0 ${M_PI/2.0}"/>
         <solid_cuboid_inertia  w="0.4" h="0.4" d="0.2" m="5"/>
       </inertial>
@@ -43,48 +43,48 @@
     <xacro:if value="${load_kinematics_file}">
       <joint name="${prefix}left_arm_base_joint" type="fixed">
-        <origin xyz="0 0.13861 0.10943" rpy="0.902 0 3.1416"/>
+        <origin xyz="0 0.0915 0.15044" rpy="0.9 0 3.1416"/>
         <parent link="${prefix}G2_link" />
         <child link="${prefix}left_arm_base_link" />
       </joint>
-      <xacro:ur10_robot prefix="${prefix}left_arm_" joint_limited="true"
+      <xacro:ur10e_robot prefix="${prefix}left_arm_" joint_limited="true"
         shoulder_pan_lower_limit="${-pi}" shoulder_pan_upper_limit="${pi}"
         wrist_3_lower_limit="${-pi}" wrist_3_upper_limit="${pi}"
-        kinematics_file="${load_yaml('$(find rbsherpa_control)/config/calibration/ur10_calibration.yaml')}">
-      </xacro:ur10_robot>
+        kinematics_file="${load_yaml('$(find rbsherpa_control)/config/calibration/ur10e_default.yaml')}">
+      </xacro:ur10e_robot>
     </xacro:if>
     <xacro:unless value="${load_kinematics_file}">
       <joint name="${prefix}left_arm_base_joint" type="fixed">
-        <origin xyz="0 0.13861 0.10943" rpy="0.902 0 3.1416"/>
+        <origin xyz="0 -0.0915 0.15044" rpy="0.9 0 3.1416"/>
         <parent link="${prefix}G2_link" />
         <child link="${prefix}right_arm_base_link" />
       </joint>
-      <xacro:ur10_robot prefix="${prefix}left_arm_" joint_limited="true"
+      <xacro:ur10e_robot prefix="${prefix}left_arm_" joint_limited="true"
         shoulder_pan_lower_limit="${-pi}" shoulder_pan_upper_limit="${pi}"
         wrist_3_lower_limit="${-pi}" wrist_3_upper_limit="${pi}">
-      </xacro:ur10_robot>
+      </xacro:ur10e_robot>
     </xacro:unless>
     <!-- Right UR10 -->
     <xacro:if value="${load_kinematics_file}">
       <joint name="${prefix}right_arm_base_joint" type="fixed">
-        <origin xyz="0 -0.13861 0.10943" rpy="0.902 0 0"/>
+        <origin xyz="0 -0.0915 0.15044" rpy="0.9 0 0"/>
         <parent link="${prefix}G2_link" />
         <child link="${prefix}right_arm_base_link" />
       </joint>
-      <xacro:ur10_robot prefix="${prefix}right_arm_" joint_limited="true"
+      <xacro:ur10e_robot prefix="${prefix}right_arm_" joint_limited="true"
         shoulder_pan_lower_limit="${-pi}" shoulder_pan_upper_limit="${pi}"
         wrist_3_lower_limit="${-pi}" wrist_3_upper_limit="${pi}"
-        kinematics_file="${load_yaml('$(find rbsherpa_control)/config/calibration/ur10_calibration.yaml')}">
-      </xacro:ur10_robot>
+        kinematics_file="${load_yaml('$(find rbsherpa_control)/config/calibration/ur10e_default.yaml')}">
+      </xacro:ur10e_robot>
     </xacro:if>
     <xacro:unless value="${load_kinematics_file}">
       <joint name="${prefix}right_arm_base_joint" type="fixed">
-        <origin xyz="0 -0.13861 0.10943" rpy="0.902 0 0"/>
+        <origin xyz="0 -0.0915 0.15044" rpy="0.9 0 0"/>
         <parent link="${prefix}G2_link" />
         <child link="${prefix}right_arm_base_link" />
       </joint>
-      <xacro:ur10_robot prefix="${prefix}right_arm_" joint_limited="true"
+      <xacro:ur10e_robot prefix="${prefix}right_arm_" joint_limited="true"
         shoulder_pan_lower_limit="${-pi}" shoulder_pan_upper_limit="${pi}"
         wrist_3_lower_limit="${-pi}" wrist_3_upper_limit="${pi}">
-      </xacro:ur10_robot>
+      </xacro:ur10e_robot>
     </xacro:unless>
   </xacro:macro>

File: rbsherpa_description/urdf/bases/rbsherpa_base.gazebo.xacro (robot description, xacro)
@@ -45,6 +45,27 @@
         </gazebo>
     </xacro:macro>
-    <gazebo reference="base_footprint">
-        <material>Gazebo/Green</material>
-    </gazebo>
+    <xacro:macro name="gazebo_color_base_link" params="prefix">
+      <gazebo reference="${prefix}base_link">
+        <visual>
+          <material>
+            <ambient>0.0 0.0 0.0 1.0</ambient>
+            <diffuse>0.2 0.2 0.2 1.0</diffuse>
+            <specular>0.508273 0.508273 0.508273 1.0</specular>
+            <emissive>0.0 0.0 0.0 0.0</emissive>
+          </material>
+        </visual>
+      </gazebo>
+    </xacro:macro>
+    <xacro:macro name="gazebo_color_logo_link" params="prefix">
+      <gazebo reference="${prefix}base_logos_link">
+        <visual>
+          <material>
+            <ambient>1.0 0.0 0.0 1.0</ambient>
+            <diffuse>0.50754 0.50754 0.50754 1.0</diffuse>
+            <specular>0.508273 0.508273 0.508273 1.0</specular>
+            <emissive>0.0 0.0 0.0 0.0</emissive>
+          </material>
+        </visual>
+      </gazebo>
+    </xacro:macro>
 </robot>

File: rbsherpa_description/urdf/bases/rbsherpa_base_v2.urdf.xacro (robot description, xacro)
@@ -53,4 +53,5 @@
       </collision>
     </link>
+    <xacro:gazebo_color_base_link prefix="${prefix}"/>
   </xacro:macro>
 </robot>

File: rbsherpa_description/urdf/bases/rbsherpa_base_v3.urdf.xacro (robot description, xacro)
@@ -34,10 +34,10 @@
         <xacro:if value="${hq}">
           <geometry>
-            <mesh filename="package://rbsherpa_description/meshes/bases/rbsherpa_chassis_v3.stl"/>
+            <mesh filename="package://rbsherpa_description/meshes/bases/rbsherpa_chassis.dae"/>
           </geometry>
         </xacro:if>
         <xacro:unless value="${hq}">
           <geometry>
-            <mesh filename="package://rbsherpa_description/meshes/bases/rbsherpa_chassis_v3.dae"/>
+            <mesh filename="package://rbsherpa_description/meshes/bases/rbsherpa_chassis.dae"/>
           </geometry>
         </xacro:unless>
@@ -49,26 +49,26 @@
         <origin xyz="0 0 0" rpy="0 0 0 " />
         <geometry>
-          <mesh filename="package://rbsherpa_description/meshes/bases/rbsherpa_chassis_v3.dae"/>
+          <mesh filename="package://rbsherpa_description/meshes/bases/rbsherpa_chassis.dae"/>
         </geometry>
       </collision>
     </link>
     <!-- Logos -->
-		<joint name="${prefix}base_logos_joint" type="fixed">
-			<origin xyz="0 0 0" rpy="0 0 0 " />
-			<parent link="${prefix}base_link"/>
-			<child link="${prefix}base_logos_link" />
-		</joint>
-		<!-- Logos -->
-		<link name="${prefix}base_logos_link" >
+    <joint name="${prefix}base_logos_joint" type="fixed">
+      <origin xyz="0 0 0" rpy="0 0 0 " />
+      <parent link="${prefix}base_link"/>
+      <child link="${prefix}base_logos_link" />
+    </joint>
+    <!-- Logos -->
+    <link name="${prefix}base_logos_link">
       <visual>
         <origin xyz="0 0 0" rpy="0 0 0" />
         <xacro:if value="${hq}">
           <geometry>
-            <mesh filename="package://rbsherpa_description/meshes/bases/rbsherpa_logos_v3.stl" scale="1.001 1.001 1.001"/>
+            <mesh filename="package://rbsherpa_description/meshes/bases/rbsherpa_logos_v3.stl" scale="1.001 1.07 1.001"/>
           </geometry>
         </xacro:if>
         <xacro:unless value="${hq}">
           <geometry>
-            <mesh filename="package://rbsherpa_description/meshes/bases/rbsherpa_logos_v3.dae" scale="1.001 1.001 1.001"/>
+            <mesh filename="package://rbsherpa_description/meshes/bases/rbsherpa_logos_v3.dae" scale="1.001 1.07 1.001"/>
           </geometry>
         </xacro:unless>
@@ -77,11 +77,7 @@
         </material>
       </visual>
-      <collision>
-        <origin xyz="0 0 0" rpy="0 0 0 " />
-        <geometry>
-          <mesh filename="package://rbsherpa_description/meshes/bases/rbsherpa_chassis_v3.dae" scale="1.001 1.001 1.001"/>
-        </geometry>
-      </collision>
     </link>
+    <xacro:gazebo_color_base_link prefix="${prefix}"/>
+    <xacro:gazebo_color_logo_link prefix="${prefix}"/>
   </xacro:macro>
 </robot>

File: rbsherpa_description/urdf/bases/rbsherpa_xl_base.urdf.xacro (robot description, xacro)
@@ -25,10 +25,10 @@
     </xacro:if>
     <!-- BASE_LINK -->
-    <link name="${prefix}base_link">   x:1.025 y:0.75 z:0.3
+    <link name="${prefix}base_link">
       <inertial>
         <mass value="25.0" />
-        <origin xyz="0 0 0.35" />
+        <origin xyz="0 0 0.376" />
         <!--inertia ixx="1.0" ixy="0.0" ixz="0.0" iyy="1.0" iyz="0.0" izz="1.0" /-->
-        <solid_cuboid_inertia  w="1.025" h="0.75" d="0.3" m="25"/>
+        <solid_cuboid_inertia  w="1.265" h="0.812" d="0.465" m="25"/>
       </inertial>
       <visual>
@@ -36,10 +36,10 @@
         <xacro:if value="${hq}">
           <geometry>
-            <mesh filename="package://rbsherpa_description/meshes/bases/rbsherpa_xl_chassis.stl"/>
+            <mesh filename="package://rbsherpa_description/meshes/bases/rbsherpa_xl_base.stl"/>
           </geometry>
         </xacro:if>
         <xacro:unless value="${hq}">
           <geometry>
-            <mesh filename="package://rbsherpa_description/meshes/bases/rbsherpa_xl_chassis.stl"/>
+            <mesh filename="package://rbsherpa_description/meshes/bases/rbsherpa_xl_base.stl"/>
           </geometry>
         </xacro:unless>
@@ -51,18 +51,35 @@
         <origin xyz="0 0 0" rpy="0 0 0 " />
         <geometry>
-          <mesh filename="package://rbsherpa_description/meshes/bases/rbsherpa_xl_chassis.stl"/>
+          <mesh filename="package://rbsherpa_description/meshes/bases/rbsherpa_xl_base.stl"/>
         </geometry>
       </collision>
     </link>
-    <gazebo reference="${prefix}base_link">
+    <!-- Logos -->
+    <joint name="${prefix}base_logos_joint" type="fixed">
+      <origin xyz="0 0 0.15" rpy="0 0 0 " />
+      <parent link="${prefix}base_link"/>
+      <child link="${prefix}base_logos_link" />
+    </joint>
+    <!-- Logos -->
+    <link name="${prefix}base_logos_link">
       <visual>
-        <material>
-          <ambient>0.0 0.0 0.0 1.0</ambient>
-          <diffuse>0.2 0.2 0.2 1.0</diffuse>
-          <specular>0.508273 0.508273 0.508273 1.0</specular>
-          <emissive>0.0 0.0 0.0 0.0</emissive>
+        <origin xyz="0 0 0" rpy="0 0 0" />
+        <xacro:if value="${hq}">
+          <geometry>
+            <mesh filename="package://rbsherpa_description/meshes/bases/rbsherpa_logos_v3.stl" scale="1.23 1.23 1"/>
+          </geometry>
+        </xacro:if>
+        <xacro:unless value="${hq}">
+          <geometry>
+            <mesh filename="package://rbsherpa_description/meshes/bases/rbsherpa_logos_v3.dae" scale="1.3 1.3 1"/>
+          </geometry>
+        </xacro:unless>
+        <material name="lightgrey">
+          <color rgba="0.9 0.9 0.9 1"/>
         </material>
       </visual>
-    </gazebo>
+    </link>
+    <xacro:gazebo_color_base_link prefix="${prefix}"/>
+    <xacro:gazebo_color_logo_link prefix="${prefix}"/>
   </xacro:macro>
 </robot>

File: rbsherpa_description/urdf/wheels/motor_wheel.urdf.xacro (robot description, xacro)
@@ -1,4 +1,5 @@
 <?xml version="1.0"?>
 <robot xmlns:xacro="http://www.ros.org/wiki/xacro">
+  <xacro:include filename="$(find rbsherpa_description)/urdf/wheels/wheel.gazebo.xacro" />
   <xacro:property name="M_PI" value="3.1415926535897931" />
   <!-- Wheels -->
@@ -135,16 +136,10 @@
       <inertial>
         <mass value="${wheel_mass}" />
-        <origin xyz="0 0 0" />
+        <origin xyz="0 0 0" rpy="${M_PI/2} 0 0" />
         <cylinder_inertia m="${wheel_mass}" r="${wheel_radius}" h="${wheel_height}" />
       </inertial>
     </link>
-    <!-- gazebo reference="${prefix}wheel">
-        <mu1 value="1.0"/>
-        <mu2 value="1.0"/>
-        <kp value="10000000.0" />
-        <kd value="1.0" />
-        <fdir1 value="1 0 0"/>
-        <turnGravityOff>false</turnGravityOff>
-   </gazebo -->
+    <xacro:gazebo_color_wheel prefix="${prefix}"/>
+    <xacro:gazebo_color_steer_wheel prefix="${prefix}"/>
   </xacro:macro>
 </robot>
