Commit message: rbsherpa_description: added color, corrected missmatched meshes, updated rbsherpa_xl version

File: rbsherpa_description/urdf/wheels/motor_wheel_hard.urdf.xacro (robot description, xacro)
@@ -1,10 +1,10 @@
 <?xml version="1.0"?>
-<robot xmlns:xacro="http://wiki.ros.org/xacro">
+<robot xmlns:xacro="http://www.ros.org/wiki/xacro">
   <xacro:include filename="$(find rbsherpa_description)/urdf/wheels/wheel.gazebo.xacro" />
   <xacro:property name="M_PI" value="3.1415926535897931" />
   <!-- Wheels -->
-  <xacro:property name="wheel_radius" value="0.17" />
-  <xacro:property name="wheel_width" value="0.14" />
-  <xacro:property name="wheel_mass" value="4.0" />
+  <xacro:property name="wheel_radius" value="0.110" />
+  <xacro:property name="wheel_height" value="0.110" />
+  <xacro:property name="wheel_mass" value="5.0" />
   <!-- in kg-->
   <xacro:property name="steer_joint_damping" value="2.0" />
@@ -21,5 +21,5 @@
     <inertia ixx="${m*(3*r*r+h*h)/12}" ixy = "0" ixz = "0" iyy="${m*(3*r*r+h*h)/12}" iyz = "0" izz="${m*r*r/2}" />
   </xacro:macro>
-  <xacro:macro name="motor_wheel" params="prefix parent *origin reflect hq">
+  <xacro:macro name="motor_wheel_hard" params="prefix parent *origin reflect hq">
     <!-- TODO: check reflect parameter -->
     <!--MOTOR WHEEL -->
@@ -47,11 +47,11 @@
         <!-- HIGH RESOLUTION WHEELS -->
         <xacro:if value="${hq}">
-          <origin xyz="0 0 0.27952" rpy="0 0 0" />
+          <origin xyz="0 0 0" rpy="0 0 3.1416" />
           <geometry>
             <xacro:if value="${reflect}">
-              <mesh filename="package://rbsherpa_description/meshes/wheels/hub_rbsherpa_xl.stl" />
+              <mesh filename="package://rbsherpa_description/meshes/wheels/mw_frame.dae" />
             </xacro:if>
             <xacro:unless value="${reflect}">
-              <mesh filename="package://rbsherpa_description/meshes/wheels/hub_rbsherpa_xl.stl" />
+              <mesh filename="package://rbsherpa_description/meshes/wheels/mw_frame.dae" />
             </xacro:unless>
           </geometry>
@@ -59,11 +59,11 @@
         <!-- LOW RESOLUTION WHEELS -->
         <xacro:unless value="${hq}">
-          <origin xyz="0 0 0.27952" rpy="0 0 0" />
+          <origin xyz="0 0 0" rpy="0 0 3.1416" />
           <geometry>
             <xacro:if value="${reflect}">
-              <mesh filename="package://rbsherpa_description/meshes/wheels/hub_rbsherpa_xl.dae" />
+              <mesh filename="package://rbsherpa_description/meshes/wheels/mw_frame.stl" />
             </xacro:if>
             <xacro:unless value="${reflect}">
-              <mesh filename="package://rbsherpa_description/meshes/wheels/hub_rbsherpa_xl.dae" />
+              <mesh filename="package://rbsherpa_description/meshes/wheels/mw_frame.stl" />
             </xacro:unless>
           </geometry>
@@ -71,19 +71,18 @@
       </visual>
       <collision>
-        <origin xyz="0 0 0.27952" rpy="0 0 0" />
+        <origin xyz="0 0 0" rpy="0 0 3.1416" />
         <geometry>
           <xacro:if value="${reflect}">
-            <mesh filename="package://rbsherpa_description/meshes/wheels/hub_rbsherpa_xl.dae" />
+            <mesh filename="package://rbsherpa_description/meshes/wheels/mw_frame.dae" />
           </xacro:if>
           <xacro:unless value="${reflect}">
-            <mesh filename="package://rbsherpa_description/meshes/wheels/hub_rbsherpa_xl.dae" />
+            <mesh filename="package://rbsherpa_description/meshes/wheels/mw_frame.dae" />
           </xacro:unless>
         </geometry>
       </collision>
       <inertial>
-        <mass value="4" />
-        <origin xyz="0 0 0.12" rpy="0 0 0"/>
-        <!--inertia ixx="0.01" ixy="0.0" ixz="0.0" iyy="0.01" iyz="0.0" izz="0.01" /-->
-        <cylinder_inertia m="${wheel_mass}" r="${wheel_radius}" h="${wheel_width}" />
+        <mass value="10" />
+        <origin xyz="0 0 0" />
+        <inertia ixx="0.01" ixy="0.0" ixz="0.0" iyy="0.01" iyz="0.0" izz="0.01" />
       </inertial>
     </link>
@@ -114,8 +113,8 @@
           <geometry>
             <xacro:if value="${reflect}">
-              <mesh filename="package://rbsherpa_description/meshes/wheels/wheel_rbsherpa_xl.stl" />
+              <mesh filename="package://rbsherpa_description/meshes/wheels/hard_wheel.dae" />
             </xacro:if>
             <xacro:unless value="${reflect}">
-              <mesh filename="package://rbsherpa_description/meshes/wheels/wheel_rbsherpa_xl.stl" />
+              <mesh filename="package://rbsherpa_description/meshes/wheels/hard_wheel.dae" />
             </xacro:unless>
           </geometry>
@@ -123,11 +122,11 @@
         <!-- LOW RESOLUTION WHEELS -->
         <xacro:unless value="${hq}">
-          <origin xyz="0 0 0" rpy="0 0 0" />
+          <origin xyz="0 0 0" rpy="${M_PI/2} 0 0" />
           <geometry>
             <xacro:if value="${reflect}">
-              <mesh filename="package://rbsherpa_description/meshes/wheels/wheel_rbsherpa_xl.dae" />
+              <mesh filename="package://rbsherpa_description/meshes/wheels/hard_wheel.dae" />
             </xacro:if>
             <xacro:unless value="${reflect}">
-              <mesh filename="package://rbsherpa_description/meshes/wheels/wheel_rbsherpa_xl.dae" />
+              <mesh filename="package://rbsherpa_description/meshes/wheels/hard_wheel.dae" />
             </xacro:unless>
           </geometry>
@@ -135,18 +134,13 @@
       </visual>
       <collision>
-        <origin xyz="0 0 0" rpy="0 0 0" />
+        <origin xyz="0 0 0" rpy="${M_PI/2} 0 0" />
         <geometry>
-          <xacro:if value="${reflect}">
-              <mesh filename="package://rbsherpa_description/meshes/wheels/wheel_rbsherpa_xl.dae" />
-          </xacro:if>
-          <xacro:unless value="${reflect}">
-              <mesh filename="package://rbsherpa_description/meshes/wheels/wheel_rbsherpa_xl.dae" />
-          </xacro:unless>
+          <sphere radius="${wheel_radius}" />
         </geometry>
       </collision>
       <inertial>
         <mass value="${wheel_mass}" />
-        <origin xyz="0 0 0" rpy="${M_PI/2} 0 0"/>
-        <cylinder_inertia m="${wheel_mass}" r="${wheel_radius}" h="${wheel_width}" />
+        <origin xyz="0 0 0" />
+        <cylinder_inertia m="${wheel_mass}" r="${wheel_radius}" h="${wheel_height}" />
       </inertial>
     </link>

File: rbsherpa_description/urdf/wheels/wheel_v2.urdf.xacro (robot description, xacro)
@@ -1,4 +1,5 @@
 <?xml version="1.0"?>
 <robot xmlns:xacro="http://www.ros.org/wiki/xacro">
+  <xacro:include filename="$(find rbsherpa_description)/urdf/wheels/wheel.gazebo.xacro" />
   <xacro:property name="M_PI" value="3.1415926535897931" />
   <!-- Wheels -->
@@ -75,4 +76,6 @@
       </inertial>
     </link>
+    <xacro:gazebo_color_wheel prefix="${prefix}"/>
+    <xacro:gazebo_color_steer_wheel prefix="${prefix}"/>
   </xacro:macro>
 </robot>

File: rbsherpa_description/urdf/wheels/wheel_v3.urdf.xacro (robot description, xacro)
@@ -1,4 +1,5 @@
 <?xml version="1.0"?>
 <robot xmlns:xacro="http://www.ros.org/wiki/xacro">
+  <xacro:include filename="$(find rbsherpa_description)/urdf/wheels/wheel.gazebo.xacro" />
   <xacro:property name="M_PI" value="3.1415926535897931" />
   <!-- Wheels -->
@@ -75,4 +76,6 @@
       </inertial>
     </link>
+    <xacro:gazebo_color_wheel prefix="${prefix}"/>
+    <xacro:gazebo_color_steer_wheel prefix="${prefix}"/>
   </xacro:macro>
 </robot>
