Commit message: rbsherpa_description: added lasers to the rbsherpa_xl

File: rbsherpa_description/robots/rbsherpa_xl.urdf.xacro (robot description, xacro)
@@ -67,12 +67,11 @@
             <origin xyz="0.511 0 0.21" rpy="0 0 0"/>
         </xacro:sensor_rslidar_16-->
-        <!-- Solid-State laser -->
-        <!--xacro:sensor_benewake_ce30c prefix="${prefix}front_ss_laser" parent="${prefix}base_link" gpu="false">
-            <origin xyz="0.5657 0.0 0.1622" rpy="0 0 0"/>
-        </xacro:sensor_benewake_ce30c-->
-        <!-- 2d laser -->
-        <!--xacro:sensor_sick_tim551 prefix="${prefix}front_laser" parent="${prefix}base_link" prefix_topic="front_laser">
-            <origin xyz="0.5307 0.0 0.15389" rpy="${180*deg2rad} 0 0"/>
-        </xacro:sensor_sick_tim551-->
+        <!-- Laser -->
+        <xacro:sensor_sick_microscan3 prefix="${prefix}front_laser" parent="${prefix}base_link" prefix_topic="front_laser">
+            <origin xyz="0.647 -0.38975 0.40646" rpy="${PI} 0 0"/>
+        </xacro:sensor_sick_microscan3>
+        <xacro:sensor_sick_microscan3 prefix="${prefix}rear_laser" parent="${prefix}base_link" prefix_topic="rear_laser">
+            <origin xyz="-0.647 0.38975 0.40646" rpy="${PI} 0 ${PI}"/>
+        </xacro:sensor_sick_microscan3>
     </xacro:macro>
     <!-- Gazebo ros control pluggins -->

Commit message: updated moveit package and added new sensors to rbsherpa_xl

File: rbsherpa_description/robots/rbsherpa_xl.urdf.xacro (robot description, xacro)
@@ -51,5 +51,5 @@
         <xacro:if value="$(arg launch_arm)">
           <xacro:bi_arm_support prefix="${prefix}" parent="${prefix}base_link" hq="true" load_kinematics_file="${load_kinematics_file}">
-              <origin xyz="${G2_offset_x} ${G2_offset_y} ${G2_offset_z}" rpy="0 0 0"/>
+              <origin xyz="${G2_offset_x} ${G2_offset_y} ${G2_offset_z}" rpy="0 0 ${90*PI/180}"/>
           </xacro:bi_arm_support>
         </xacro:if>
@@ -63,14 +63,18 @@
             <origin xyz="-0.04625 0.0 0.59188" rpy="0 0 0"/>
         </xacro:sensor_gps-->
+        <!-- Camera Zed -->
+        <xacro:sensor_zed prefix="${prefix}zed" parent="${prefix}base_link" prefix_topic="zed">
+            <origin xyz="0.66135 0 0.31585" rpy="0 0 0"/>
+        </xacro:sensor_zed>
         <!-- Lidar -->
-        <!--xacro:sensor_rslidar_16 prefix="${prefix}front_ss_laser" parent="${prefix}base_link" gpu="true">
-            <origin xyz="0.511 0 0.21" rpy="0 0 0"/>
-        </xacro:sensor_rslidar_16-->
+        <xacro:sensor_rs_bpearl prefix="${prefix}front_3d_laser" parent="${prefix}base_link" prefix_topic="front_3d_laser" range_min="0.1" range_max="90" hfov="360" samples="1200" vfov="90.0" lasers="32" fps="15" gpu="true">
+            <origin xyz="0.645 0 0.52032" rpy="0 ${90*PI/180} 0"/>
+        </xacro:sensor_rs_bpearl>
         <!-- Laser -->
         <xacro:sensor_sick_microscan3 prefix="${prefix}front_laser" parent="${prefix}base_link" prefix_topic="front_laser">
-            <origin xyz="0.647 -0.38975 0.40646" rpy="${PI} 0 0"/>
+            <origin xyz="0.645 -0.396 0.44559" rpy="${PI} 0 -${45*PI/180}"/>
         </xacro:sensor_sick_microscan3>
         <xacro:sensor_sick_microscan3 prefix="${prefix}rear_laser" parent="${prefix}base_link" prefix_topic="rear_laser">
-            <origin xyz="-0.647 0.38975 0.40646" rpy="${PI} 0 ${PI}"/>
+            <origin xyz="-0.645 0.396 0.44559" rpy="${PI} 0 -${225*PI/180}"/>
         </xacro:sensor_sick_microscan3>
     </xacro:macro>

Commit message: added sick support and protector

File: rbsherpa_description/robots/rbsherpa_xl.urdf.xacro (robot description, xacro)
@@ -12,4 +12,8 @@
     <!-- Import arm structure -->
     <xacro:include filename="$(find rbsherpa_description)/urdf/bases/bi_arm_support.urdf.xacro" />
+    <!-- Import sick support -->
+    <xacro:include filename="$(find rbsherpa_description)/urdf/bases/sick_support.urdf.xacro" />
+    <!-- Import sick protector -->
+    <xacro:include filename="$(find rbsherpa_description)/urdf/bases/sick_protector.urdf.xacro" />
     <!-- Import all available sensors -->
     <xacro:include filename="$(find robotnik_sensors)/urdf/all_sensors.urdf.xacro" />
@@ -64,5 +68,5 @@
         </xacro:sensor_gps>
         <!-- Camera Zed -->
-        <xacro:sensor_zed prefix="${prefix}zed" parent="${prefix}base_link">
+        <xacro:sensor_zed prefix="${prefix}zed" parent="${prefix}base_link" model="zed2">
             <origin xyz="0.66135 0 0.31585" rpy="0 0 0"/>
         </xacro:sensor_zed>
@@ -71,10 +75,24 @@
             <origin xyz="0.645 0 0.52032" rpy="0 ${90*PI/180} 0"/>
         </xacro:sensor_rs_bpearl>
+        <!-- laser sick support-->
+        <xacro:sick_support prefix="${prefix}sick_front_support" parent="${prefix}base_link">
+            <origin xyz="0.472 0.3795 0.3774" rpy="0 ${90*PI/180} ${90*PI/180}"/>
+        </xacro:sick_support>
+        <xacro:sick_support prefix="${prefix}sick_rear_support" parent="${prefix}base_link">
+            <origin xyz="-0.472 -0.3795 0.3774" rpy="0 ${90*PI/180} -${90*PI/180}"/>
+        </xacro:sick_support>
+        <!-- laser sick protector-->
+        <xacro:sick_protector prefix="${prefix}sick_front_protector" parent="${prefix}base_link">
+            <origin xyz="0.645 0.396 0.3905" rpy="0 0 -${45*PI/180}"/>
+        </xacro:sick_protector>
+        <xacro:sick_protector prefix="${prefix}sick_rear_protector" parent="${prefix}base_link">
+            <origin xyz="-0.645 -0.396 0.3905" rpy="0 0 ${135*PI/180}"/>
+        </xacro:sick_protector>
         <!-- Laser -->
         <xacro:sensor_sick_microscan3 prefix="${prefix}front_laser" parent="${prefix}base_link" prefix_topic="front_laser">
-            <origin xyz="0.645 -0.396 0.44559" rpy="${PI} 0 -${45*PI/180}"/>
+            <origin xyz="0.645 0.396 0.4455" rpy="${PI} 0 ${45*PI/180}"/>
         </xacro:sensor_sick_microscan3>
         <xacro:sensor_sick_microscan3 prefix="${prefix}rear_laser" parent="${prefix}base_link" prefix_topic="rear_laser">
-            <origin xyz="-0.645 0.396 0.44559" rpy="${PI} 0 -${225*PI/180}"/>
+            <origin xyz="-0.645 -0.396 0.4455" rpy="${PI} 0 -${135*PI/180}"/>
         </xacro:sensor_sick_microscan3>
     </xacro:macro>

Commit message: laser and protector coordinates updated

File: rbsherpa_description/robots/rbsherpa_xl.urdf.xacro (robot description, xacro)
@@ -84,15 +84,15 @@
         <!-- laser sick protector-->
         <xacro:sick_protector prefix="${prefix}sick_front_protector" parent="${prefix}base_link">
-            <origin xyz="0.645 0.396 0.3905" rpy="0 0 -${45*PI/180}"/>
+            <origin xyz="0.645 0.396 0.39025" rpy="0 0 -${45*PI/180}"/>
         </xacro:sick_protector>
         <xacro:sick_protector prefix="${prefix}sick_rear_protector" parent="${prefix}base_link">
-            <origin xyz="-0.645 -0.396 0.3905" rpy="0 0 ${135*PI/180}"/>
+            <origin xyz="-0.645 -0.396 0.39025" rpy="0 0 ${135*PI/180}"/>
         </xacro:sick_protector>
         <!-- Laser -->
         <xacro:sensor_sick_microscan3 prefix="${prefix}front_laser" parent="${prefix}base_link" prefix_topic="front_laser">
-            <origin xyz="0.645 0.396 0.4455" rpy="${PI} 0 ${45*PI/180}"/>
+            <origin xyz="0.645 0.396 0.44559" rpy="${PI} 0 ${45*PI/180}"/>
         </xacro:sensor_sick_microscan3>
         <xacro:sensor_sick_microscan3 prefix="${prefix}rear_laser" parent="${prefix}base_link" prefix_topic="rear_laser">
-            <origin xyz="-0.645 -0.396 0.4455" rpy="${PI} 0 -${135*PI/180}"/>
+            <origin xyz="-0.645 -0.396 0.44559" rpy="${PI} 0 -${135*PI/180}"/>
         </xacro:sensor_sick_microscan3>
     </xacro:macro>

File: rbsherpa_description/urdf/bases/sick_support.urdf.xacro (robot description, xacro)
@@ -35,9 +35,9 @@
     </link>
     <gazebo reference="${prefix}sick_support_link">
-      <material>Gazebo/Green</material>
+      <material>Gazebo/Red</material>
       <visual>
         <material>
-          <ambient>0.0 0.0 0.0 1.0</ambient>
-          <diffuse>0.2 0.2 0.2 1.0</diffuse>
+          <ambient>1.0 0.0 0.0 1.0</ambient>
+          <diffuse>0.52 0.2 0.2 1.0</diffuse>
           <specular>0.508273 0.508273 0.508273 1.0</specular>
           <emissive>0.0 0.0 0.0 0.0</emissive>

Commit message: use of gpu parametrized, set to false by default

File: rbsherpa_description/robots/rbsherpa_xl.urdf.xacro (robot description, xacro)
@@ -34,5 +34,6 @@
     <xacro:arg name="launch_arm" default="false" />
     <xacro:arg name="load_kinematics_file" default="false" />
-    <xacro:macro name="rbsherpa" params="prefix launch_arm load_kinematics_file publish_bf hq">
+    <xacro:arg name="use_gpu" default="false" />
+    <xacro:macro name="rbsherpa" params="prefix launch_arm load_kinematics_file publish_bf hq use_gpu">
         <!-- *************** -->
         <!-- Robots Elements -->
@@ -72,5 +73,5 @@
         </xacro:sensor_zed>
         <!-- Lidar -->
-        <xacro:sensor_rs_bpearl prefix="${prefix}front_3d_laser" parent="${prefix}base_link" prefix_topic="front_3d_laser" range_min="0.1" range_max="90" hfov="360" samples="1200" vfov="90.0" lasers="32" fps="15" gpu="true">
+        <xacro:sensor_rs_bpearl prefix="${prefix}front_3d_laser" parent="${prefix}base_link" prefix_topic="front_3d_laser" range_min="0.1" range_max="90" hfov="360" samples="1200" vfov="90.0" lasers="32" fps="15" gpu="${use_gpu}">
             <origin xyz="0.645 0 0.52032" rpy="0 ${90*PI/180} 0"/>
         </xacro:sensor_rs_bpearl>
@@ -90,8 +91,8 @@
         </xacro:sick_protector>
         <!-- Laser -->
-        <xacro:sensor_sick_microscan3 prefix="${prefix}front_laser" parent="${prefix}base_link" prefix_topic="front_laser">
+        <xacro:sensor_sick_microscan3 prefix="${prefix}front_laser" parent="${prefix}base_link" prefix_topic="front_laser" gpu="${use_gpu}">
             <origin xyz="0.645 0.396 0.44559" rpy="${PI} 0 ${45*PI/180}"/>
         </xacro:sensor_sick_microscan3>
-        <xacro:sensor_sick_microscan3 prefix="${prefix}rear_laser" parent="${prefix}base_link" prefix_topic="rear_laser">
+        <xacro:sensor_sick_microscan3 prefix="${prefix}rear_laser" parent="${prefix}base_link" prefix_topic="rear_laser" gpu="${use_gpu}">
             <origin xyz="-0.645 -0.396 0.44559" rpy="${PI} 0 -${135*PI/180}"/>
         </xacro:sensor_sick_microscan3>
@@ -99,4 +100,4 @@
     <!-- Gazebo ros control pluggins -->
     <xacro:ros_control/>
-    <xacro:rbsherpa prefix="$(arg prefix)" publish_bf="${publish_bf}" hq="${hq}" launch_arm="$(arg launch_arm)" load_kinematics_file="$(arg load_kinematics_file)"/>
+    <xacro:rbsherpa prefix="$(arg prefix)" publish_bf="${publish_bf}" hq="${hq}" launch_arm="$(arg launch_arm)" load_kinematics_file="$(arg load_kinematics_file)" use_gpu="$(arg use_gpu)"/>
 </robot>

Commit message: parameter use_gpu renamed to gpu

File: rbsherpa_description/robots/rbsherpa_xl.urdf.xacro (robot description, xacro)
@@ -34,6 +34,6 @@
     <xacro:arg name="launch_arm" default="false" />
     <xacro:arg name="load_kinematics_file" default="false" />
-    <xacro:arg name="use_gpu" default="false" />
-    <xacro:macro name="rbsherpa" params="prefix launch_arm load_kinematics_file publish_bf hq use_gpu">
+    <xacro:arg name="gpu" default="false" />
+    <xacro:macro name="rbsherpa" params="prefix launch_arm load_kinematics_file publish_bf hq gpu">
         <!-- *************** -->
         <!-- Robots Elements -->
@@ -91,8 +91,8 @@
         </xacro:sick_protector>
         <!-- Laser -->
-        <xacro:sensor_sick_microscan3 prefix="${prefix}front_laser" parent="${prefix}base_link" prefix_topic="front_laser" gpu="${use_gpu}">
+        <xacro:sensor_sick_microscan3 prefix="${prefix}front_laser" parent="${prefix}base_link" prefix_topic="front_laser" gpu="${gpu}">
             <origin xyz="0.645 0.396 0.44559" rpy="${PI} 0 ${45*PI/180}"/>
         </xacro:sensor_sick_microscan3>
-        <xacro:sensor_sick_microscan3 prefix="${prefix}rear_laser" parent="${prefix}base_link" prefix_topic="rear_laser" gpu="${use_gpu}">
+        <xacro:sensor_sick_microscan3 prefix="${prefix}rear_laser" parent="${prefix}base_link" prefix_topic="rear_laser" gpu="${gpu}">
             <origin xyz="-0.645 -0.396 0.44559" rpy="${PI} 0 -${135*PI/180}"/>
         </xacro:sensor_sick_microscan3>
@@ -100,4 +100,4 @@
     <!-- Gazebo ros control pluggins -->
     <xacro:ros_control/>
-    <xacro:rbsherpa prefix="$(arg prefix)" publish_bf="${publish_bf}" hq="${hq}" launch_arm="$(arg launch_arm)" load_kinematics_file="$(arg load_kinematics_file)" use_gpu="$(arg use_gpu)"/>
+    <xacro:rbsherpa prefix="$(arg prefix)" publish_bf="${publish_bf}" hq="${hq}" launch_arm="$(arg launch_arm)" load_kinematics_file="$(arg load_kinematics_file)" gpu="$(arg gpu)"/>
 </robot>
