Commit message: arms and moveit: Working with the last version of univeral_robot package         - fmauch/universal_robot: 1ffdd69 Replace __ prefixes         - Update urdfs with the new ur description paths         - Update moveit collisions         - Fix deprecated ee_link

File: rbvogui_description/robots/rbvogui_std_ur10.urdf.xacro (robot description, xacro)
@@ -15,5 +15,5 @@
     <xacro:include filename="$(find robotnik_sensors)/urdf/all_sensors.urdf.xacro" />
     <!-- Include UR-10 ARM -->
-    <xacro:include filename="$(find ur_description)/urdf/ur10.urdf.xacro" />
+    <xacro:include filename="$(find ur_description)/urdf/inc/ur10_macro.xacro" />
     <xacro:property name="arm_position_x" value="0.0"/>
     <xacro:property name="arm_position_y" value="0"/>
@@ -72,5 +72,7 @@
         <!-- UR-10 ARM -->
         <xacro:if value="${load_kinematics_file}">
-            <xacro:ur10_robot prefix="${prefix}arm_" joint_limited="true" shoulder_pan_lower_limit="${-pi}" shoulder_pan_upper_limit="${pi}" wrist_3_lower_limit="${-pi}" wrist_3_upper_limit="${pi}" kinematics_file="${load_yaml('$(find rbvogui_control)/config/calibration/ur10_calibration.yaml')}">
+            <xacro:ur10_robot prefix="${prefix}arm_"
+                    kinematics_parameters_file="$(find rbvogui_control)/config/calibration/ur10_calibration.yaml"
+                    joint_limits_parameters_file="$(find rbvogui_control)/config/calibration/ur10_joint_limits.yaml">
             </xacro:ur10_robot>
             <joint name="${prefix}arm_base_joint" type="fixed">
@@ -81,5 +83,5 @@
         </xacro:if>
         <xacro:unless value="${load_kinematics_file}">
-            <xacro:ur10_robot prefix="${prefix}arm_" joint_limited="true" shoulder_pan_lower_limit="${-pi}" shoulder_pan_upper_limit="${pi}" wrist_3_lower_limit="${-pi}" wrist_3_upper_limit="${pi}" >
+            <xacro:ur10_robot prefix="${prefix}arm_">
             </xacro:ur10_robot>
             <joint name="${prefix}arm_base_joint" type="fixed">

File: rbvogui_description/robots/rbvogui_ur5e.urdf.xacro (robot description, xacro)
@@ -19,5 +19,5 @@
     <xacro:include filename="$(find rbvogui_description)/urdf/structures/gps.urdf.xacro" />
     <!-- Import ur arm -->
-    <xacro:include filename="$(find ur_e_description)/urdf/ur5e.urdf.xacro" />
+    <xacro:include filename="$(find ur_description)/urdf/inc/ur10_macro.xacro" />
     <!-- Import robotiq gripper -->
     <xacro:include filename="$(find robotiq_2f_85_gripper_visualization)/urdf/robotiq_arg2f_85_model_macro.xacro" />
@@ -41,15 +41,10 @@
     <xacro:if value="${load_kinematics_file}">
 		<!-- Ur5 Arm -->
-		<xacro:ur5e_robot prefix="$(arg prefix)arm_" joint_limited="false"
-			shoulder_pan_lower_limit="${-pi}" shoulder_pan_upper_limit="${pi}"
-			wrist_3_lower_limit="${-pi}" wrist_3_upper_limit="${pi}"
-			kinematics_file="${load_yaml('$(find rbvogui_control)/config/calibration/ur10_calibration.yaml')}">
+        <xacro:ur5e_robot prefix="${prefix}arm_" kinematics_parameters_file="$(find rbvogui_control)/config/calibration/ur10_calibration.yaml">
 		</xacro:ur5e_robot>
 	</xacro:if>
     <xacro:unless value="${load_kinematics_file}">
 		<!-- Ur5 Arm -->
-		<xacro:ur5e_robot prefix="$(arg prefix)arm_" joint_limited="false"
-			shoulder_pan_lower_limit="${-pi}" shoulder_pan_upper_limit="${pi}"
-			wrist_3_lower_limit="${-pi}" wrist_3_upper_limit="${pi}">
+		<xacro:ur5e_robot prefix="$(arg prefix)arm_">
 		</xacro:ur5e_robot>
 	</xacro:unless>

File: rbvogui_description/robots/rbvogui_xl_lift_ur10e.urdf.xacro (robot description, xacro)
@@ -11,5 +11,5 @@
     <xacro:include filename="$(find rbvogui_description)/urdf/wheels/motor_wheel_xl.urdf.xacro" />
     <!-- Import ur arm -->
-    <xacro:include filename="$(find ur_e_description)/urdf/ur10e.urdf.xacro" />
+    <xacro:include filename="$(find ur_description)/urdf/inc/ur10e_macro.xacro" />
     <!-- Import ewellix lift -->
     <xacro:include filename="$(find ewellix_description)/urdf/ewellix_lift_900mm.urdf.xacro" />
@@ -61,12 +61,11 @@
         <!-- UR-10e ARM -->
         <xacro:if value="${load_kinematics_file}">
-			<xacro:ur10e_robot prefix="${prefix}arm_" joint_limited="true" shoulder_pan_lower_limit="${-pi}"
-							shoulder_pan_upper_limit="${pi}" wrist_3_lower_limit="${-pi}" wrist_3_upper_limit="${pi}"
-							kinematics_file="${load_yaml('$(arg kinematics_config)')}">
+            <xacro:ur10e_robot prefix="${prefix}arm_"
+                        kinematics_parameters_file="$(find rbvogui_control)/config/calibration/ur10_calibration.yaml"
+                        joint_limits_parameters_file="$(find rbvogui_control)/config/calibration/ur10_joint_limits.yaml">
 			</xacro:ur10e_robot>
 		</xacro:if>
         <xacro:unless value="${load_kinematics_file}">
-			<xacro:ur10e_robot prefix="${prefix}arm_" joint_limited="true" shoulder_pan_lower_limit="${-pi}"
-							shoulder_pan_upper_limit="${pi}" wrist_3_lower_limit="${-pi}" wrist_3_upper_limit="${pi}">
+			<xacro:ur10e_robot prefix="${prefix}arm_">
 			</xacro:ur10e_robot>
 		</xacro:unless>

File: rbvogui_description/urdf/bases/bi_arm_support.urdf.xacro (robot description, xacro)
@@ -1,5 +1,5 @@
 <?xml version="1.0"?>
 <robot xmlns:xacro="http://wiki.ros.org/xacro">
-	<xacro:include filename="$(find ur_e_description)/urdf/ur10e.urdf.xacro" />
+	<xacro:include filename="$(find ur_description)/urdf/inc/ur10e_macro.xacro" />
   <xacro:include filename="$(find rbvogui_description)/urdf/inertia.urdf.xacro" />
   <xacro:property name="M_PI" value="3.1415926535897931" />
@@ -50,8 +50,7 @@
         <child link="${prefix}left_arm_base_link" />
       </joint>
-      <xacro:ur10e_robot prefix="${prefix}left_arm_" joint_limited="true"
-        shoulder_pan_lower_limit="${-pi}" shoulder_pan_upper_limit="${pi}"
-        wrist_3_lower_limit="${-pi}" wrist_3_upper_limit="${pi}"
-        kinematics_file="${load_yaml('$(find rbvogui_control)/config/calibration/ur10e_default.yaml')}">
+      <xacro:ur10e_robot prefix="${prefix}left_arm_"
+                kinematics_parameters_file="$(find rbvogui_control)/config/calibration/ur10_calibration.yaml"
+                joint_limits_parameters_file="$(find rbvogui_control)/config/calibration/ur10_joint_limits.yaml">
       </xacro:ur10e_robot>
     </xacro:if>
@@ -60,9 +59,7 @@
         <origin xyz="0 -0.0915 0.15044" rpy="0.9 0 3.1416"/>
         <parent link="${prefix}G2_link" />
-        <child link="${prefix}right_arm_base_link" />
+        <child link="${prefix}left_arm_base_link" />
       </joint>
-      <xacro:ur10e_robot prefix="${prefix}left_arm_" joint_limited="true"
-        shoulder_pan_lower_limit="${-pi}" shoulder_pan_upper_limit="${pi}"
-        wrist_3_lower_limit="${-pi}" wrist_3_upper_limit="${pi}">
+      <xacro:ur10e_robot prefix="${prefix}left_arm_" >
       </xacro:ur10e_robot>
     </xacro:unless>
@@ -74,8 +71,7 @@
         <child link="${prefix}right_arm_base_link" />
       </joint>
-      <xacro:ur10e_robot prefix="${prefix}right_arm_" joint_limited="true"
-        shoulder_pan_lower_limit="${-pi}" shoulder_pan_upper_limit="${pi}"
-        wrist_3_lower_limit="${-pi}" wrist_3_upper_limit="${pi}"
-        kinematics_file="${load_yaml('$(find rbvogui_control)/config/calibration/ur10e_default.yaml')}">
+      <xacro:ur10e_robot prefix="${prefix}right_arm_"
+                kinematics_parameters_file="$(find rbvogui_control)/config/calibration/ur10_calibration.yaml"
+                joint_limits_parameters_file="$(find rbvogui_control)/config/calibration/ur10_joint_limits.yaml">
       </xacro:ur10e_robot>
     </xacro:if>
@@ -86,7 +82,5 @@
         <child link="${prefix}right_arm_base_link" />
       </joint>
-      <xacro:ur10e_robot prefix="${prefix}right_arm_" joint_limited="true"
-        shoulder_pan_lower_limit="${-pi}" shoulder_pan_upper_limit="${pi}"
-        wrist_3_lower_limit="${-pi}" wrist_3_upper_limit="${pi}">
+      <xacro:ur10e_robot prefix="${prefix}right_arm_">
       </xacro:ur10e_robot>
     </xacro:unless>
