Commit message: description: Add vectornav for all rbvogui models

File: rbvogui_description/robots/rbvogui_6w_std.urdf.xacro (robot description, xacro)
@@ -67,7 +67,7 @@
         <!-- SENSORS see robotnik_sensors for the specific configuration -->
         <!-- IMU -->
-        <xacro:sensor_imu_hector prefix="${prefix}imu" parent="${prefix}chassis_link">
+        <xacro:sensor_vectornav prefix="${prefix}imu" parent="${prefix}chassis_link">
             <origin xyz="0.3 -0.3 0.0725" rpy="0 0 0"/>
-        </xacro:sensor_imu_hector>
+        </xacro:sensor_vectornav>
         <!-- Front Camera -->
         <xacro:sensor_orbbec_astra prefix="${prefix}front_rgbd_camera" parent="${prefix}chassis_link">

File: rbvogui_description/robots/rbvogui_6w_std_basket.urdf.xacro (robot description, xacro)
@@ -74,7 +74,7 @@
         <!-- SENSORS see robotnik_sensors for the specific configuration -->
         <!-- IMU -->
-        <xacro:sensor_imu_hector prefix="${prefix}imu" parent="${prefix}chassis_link">
+        <xacro:sensor_vectornav prefix="${prefix}imu" parent="${prefix}chassis_link">
             <origin xyz="0.3 -0.3 0.0725" rpy="0 0 0"/>
-        </xacro:sensor_imu_hector>
+        </xacro:sensor_vectornav>
         <!-- Front Camera -->
         <xacro:sensor_orbbec_astra prefix="${prefix}front_rgbd_camera" parent="${prefix}chassis_link">

File: rbvogui_description/robots/rbvogui_std_ur10.urdf.xacro (robot description, xacro)
@@ -54,7 +54,7 @@
         <!-- SENSORS see robotnik_sensors for the specific configuration -->
         <!-- IMU -->
-        <xacro:sensor_imu_hector prefix="${prefix}imu" parent="${prefix}chassis_link">
+        <xacro:sensor_vectornav prefix="${prefix}imu" parent="${prefix}chassis_link">
             <origin xyz="0.3 -0.3 0.0725" rpy="0 0 0"/>
-        </xacro:sensor_imu_hector>
+        </xacro:sensor_vectornav>
         <!-- Solid state laser -->
         <xacro:sensor_benewake_ce30c prefix="${prefix}front_ss_laser" parent="${prefix}chassis_link" gpu="false">

File: rbvogui_description/robots/rbvogui_std_ur10_egh.urdf.xacro (robot description, xacro)
@@ -56,7 +56,7 @@
         <!-- SENSORS see robotnik_sensors for the specific configuration -->
         <!-- IMU -->
-        <xacro:sensor_imu_hector prefix="${prefix}imu" parent="${prefix}chassis_link">
+        <xacro:sensor_vectornav prefix="${prefix}imu" parent="${prefix}chassis_link">
             <origin xyz="0.3 -0.3 0.0725" rpy="0 0 0"/>
-        </xacro:sensor_imu_hector>
+        </xacro:sensor_vectornav>
         <!-- Solid state laser -->
         <xacro:sensor_benewake_ce30c prefix="${prefix}front_ss_laser" parent="${prefix}chassis_link" gpu="false">

File: rbvogui_description/robots/rbvogui_std_ur10_rg2.urdf.xacro (robot description, xacro)
@@ -56,7 +56,7 @@
         <!-- SENSORS see robotnik_sensors for the specific configuration -->
         <!-- IMU -->
-        <xacro:sensor_imu_hector prefix="${prefix}imu" parent="${prefix}chassis_link">
+        <xacro:sensor_vectornav prefix="${prefix}imu" parent="${prefix}chassis_link">
             <origin xyz="0.3 -0.3 0.0725" rpy="0 0 0"/>
-        </xacro:sensor_imu_hector>
+        </xacro:sensor_vectornav>
         <!-- Solid state laser -->
         <xacro:sensor_benewake_ce30c prefix="${prefix}front_ss_laser" parent="${prefix}chassis_link" gpu="false">

File: rbvogui_description/robots/rbvogui_std_ur5.urdf.xacro (robot description, xacro)
@@ -54,7 +54,7 @@
         <!-- SENSORS see robotnik_sensors for the specific configuration -->
         <!-- IMU -->
-        <xacro:sensor_imu_hector prefix="${prefix}imu" parent="${prefix}chassis_link">
+        <xacro:sensor_vectornav prefix="${prefix}imu" parent="${prefix}chassis_link">
             <origin xyz="0.3 -0.3 0.0725" rpy="0 0 0"/>
-        </xacro:sensor_imu_hector>
+        </xacro:sensor_vectornav>
         <!-- Solid State laser -->
         <xacro:sensor_benewake_ce30c prefix="${prefix}front_ss_laser" parent="${prefix}chassis_link" gpu="false">

File: rbvogui_description/robots/rbvogui_std_ur5_rg2.urdf.xacro (robot description, xacro)
@@ -56,7 +56,7 @@
         <!-- SENSORS see robotnik_sensors for the specific configuration -->
         <!-- IMU -->
-        <xacro:sensor_imu_hector prefix="${prefix}imu" parent="${prefix}chassis_link">
+        <xacro:sensor_vectornav prefix="${prefix}imu" parent="${prefix}chassis_link">
             <origin xyz="0.3 -0.3 0.0725" rpy="0 0 0"/>
-        </xacro:sensor_imu_hector>
+        </xacro:sensor_vectornav>
         <!-- Solid State laser -->
         <xacro:sensor_benewake_ce30c prefix="${prefix}front_ss_laser" parent="${prefix}chassis_link" gpu="false">

File: rbvogui_description/robots/rbvogui_ur5e.urdf.xacro (robot description, xacro)
@@ -72,7 +72,7 @@
     <!-- SENSORS see robotnik_sensors for the specific configuration -->
     <!-- IMU -->
-    <xacro:sensor_imu_hector prefix="${prefix}imu" parent="${prefix}base_link">
-        <origin xyz="0.3 0.3 0.250" rpy="0 0 0"/>
-    </xacro:sensor_imu_hector>
+    <xacro:sensor_vectornav prefix="${prefix}imu" parent="${prefix}chassis_link">
+        <origin xyz="0.3 -0.3 0.0725" rpy="0 0 0"/>
+    </xacro:sensor_vectornav>
     <!-- GPS -->
     <xacro:sensor_gps_mast prefix="${prefix}gps" parent="${prefix}base_link">

File: rbvogui_description/robots/rbvogui_xl_biarm.urdf.xacro (robot description, xacro)
@@ -65,7 +65,7 @@
         <!-- SENSORS see robotnik_sensors for the specific configuration -->
         <!-- IMU -->
-        <xacro:sensor_imu_hector prefix="${prefix}imu" parent="${prefix}chassis_link">
-            <origin xyz="0.3 0.0 0.06624" rpy="0 0 0"/>
-        </xacro:sensor_imu_hector>
+        <xacro:sensor_vectornav prefix="${prefix}imu" parent="${prefix}chassis_link">
+            <origin xyz="0.3 -0.3 0.0725" rpy="0 0 0"/>
+        </xacro:sensor_vectornav>
         <!-- Orbbec camera -->
         <xacro:sensor_orbbec_astra prefix="${prefix}front_rgbd_camera" parent="${prefix}chassis_link">

File: rbvogui_description/robots/rbvogui_xl_lift_ur10e.urdf.xacro (robot description, xacro)
@@ -84,7 +84,7 @@
         <!-- SENSORS see robotnik_sensors for the specific configuration -->
         <!-- IMU -->
-        <xacro:sensor_imu_hector prefix="${prefix}imu" parent="${prefix}chassis_link">
-            <origin xyz="0.3 0.0 0.06624" rpy="0 0 0"/>
-        </xacro:sensor_imu_hector>
+        <xacro:sensor_vectornav prefix="${prefix}imu" parent="${prefix}chassis_link">
+            <origin xyz="0.3 -0.3 0.0725" rpy="0 0 0"/>
+        </xacro:sensor_vectornav>
         <!-- Orbbec camera -->
         <xacro:sensor_orbbec_astra prefix="${prefix}front_rgbd_camera" parent="${prefix}chassis_link">

File: rbvogui_description/robots/rbvogui_xl_lift_ur10e_hand_e.urdf.xacro (robot description, xacro)
@@ -86,7 +86,7 @@
         <!-- SENSORS see robotnik_sensors for the specific configuration -->
         <!-- IMU -->
-        <xacro:sensor_imu_hector prefix="${prefix}imu" parent="${prefix}chassis_link">
-            <origin xyz="0.3 0.0 0.06624" rpy="0 0 0"/>
-        </xacro:sensor_imu_hector>
+        <xacro:sensor_vectornav prefix="${prefix}imu" parent="${prefix}chassis_link">
+            <origin xyz="0.3 -0.3 0.0725" rpy="0 0 0"/>
+        </xacro:sensor_vectornav>
         <!-- Orbbec camera -->
         <xacro:sensor_orbbec_astra prefix="${prefix}front_rgbd_camera" parent="${prefix}chassis_link">

File: rbvogui_description/robots/rbvogui_xl_std.urdf.xacro (robot description, xacro)
@@ -67,7 +67,7 @@
         <!-- SENSORS see robotnik_sensors for the specific configuration -->
         <!-- IMU -->
-        <xacro:sensor_imu_hector prefix="${prefix}imu" parent="${prefix}chassis_link">
-            <origin xyz="0.3 0.0 0.06624" rpy="0 0 0"/>
-        </xacro:sensor_imu_hector>
+        <xacro:sensor_vectornav prefix="${prefix}imu" parent="${prefix}chassis_link">
+            <origin xyz="0.3 -0.3 0.0725" rpy="0 0 0"/>
+        </xacro:sensor_vectornav>
         <!-- GPS -->
         <xacro:sensor_gps_mast prefix="${prefix}gps" parent="${prefix}chassis_link">
