Commit message: Fixed xacro errors, rbvogui xl

File: rbvogui_description/robots/rbvogui_xl_std.urdf.xacro (robot description, xacro)
@@ -13,5 +13,5 @@
     <xacro:include filename="$(find rbvogui_description)/urdf/wheels/fixed_wheel_xl.urdf.xacro" />
     <!-- Import arm structure -->
-    <xacro:include filename="$(find rbvogui_description)/urdf/structures/bi_arm_support.urdf.xacro" />
+    <!--xacro:include filename="$(find rbvogui_description)/urdf/structures/bi_arm_support.urdf.xacro" /-->
     <!-- Structures -->
     <xacro:include filename="$(find rbvogui_description)/urdf/structures/top_cover.urdf.xacro" />
@@ -58,5 +58,5 @@
         </xacro:if>
         <xacro:if value="${kinematics == 'ackermann'}">
-            <xacro:fixed_wheel prefix="${prefix}rear_left_" parent="${prefix}base_link4" reflect="false" hq="${hq}">
+            <xacro:fixed_wheel prefix="${prefix}rear_left_" parent="${prefix}base_link" reflect="false" hq="${hq}">
                 <origin xyz="-${wheel_offset_x} ${wheel_offset_y} ${wheel_offset_z}" rpy="0 0 0"/>
             </xacro:fixed_wheel>
@@ -104,4 +104,28 @@
             <origin xyz="-0.64555 -0.39985 0.16608" rpy="${PI} 0 -${135*PI/180}"/>
         </xacro:sensor_sick_microscan3>
+        <xacro:macro name="ros2_joint" params="interface jmin jmax prefix name">
+          <joint name="${prefix}${name}">
+            <command_interface name="${interface}">
+              <param name="min">${jmin}</param>
+              <param name="max">${jmax}</param>
+            </command_interface>
+            <state_interface name="position"/>
+            <state_interface name="velocity"/>
+            <state_interface name="effort"/>
+          </joint>
+        </xacro:macro>
+        <ros2_control name="GazeboSystem" type="system">
+          <hardware>
+              <plugin>gazebo_ros2_control/GazeboSystem</plugin>
+          </hardware>
+          <xacro:ros2_joint interface="position" jmin="-2" jmax="2" prefix="${prefix}" name="front_left_motor_wheel_joint"/>
+          <xacro:ros2_joint interface="position" jmin="-2" jmax="2" prefix="${prefix}" name="front_right_motor_wheel_joint"/>
+          <xacro:ros2_joint interface="position" jmin="-2" jmax="2" prefix="${prefix}" name="rear_left_motor_wheel_joint"/>
+          <xacro:ros2_joint interface="position" jmin="-2" jmax="2" prefix="${prefix}" name="rear_right_motor_wheel_joint"/>
+          <xacro:ros2_joint interface="velocity" jmin="-10" jmax="10" prefix="${prefix}" name="front_left_wheel_joint"/>
+          <xacro:ros2_joint interface="velocity" jmin="-10" jmax="10" prefix="${prefix}" name="front_right_wheel_joint"/>
+          <xacro:ros2_joint interface="velocity" jmin="-20" jmax="20" prefix="${prefix}" name="rear_left_wheel_joint"/>
+          <xacro:ros2_joint interface="velocity" jmin="-20" jmax="20" prefix="${prefix}" name="rear_right_wheel_joint"/>
+        </ros2_control>
     </xacro:macro>
     <!-- Gazebo ros control pluggins -->

File: rbvogui_description/urdf/bases/rbvogui_xl_base.urdf.xacro (robot description, xacro)
@@ -37,5 +37,5 @@
         <origin xyz="0 0 0.376" />
         <!--inertia ixx="1.0" ixy="0.0" ixz="0.0" iyy="1.0" iyz="0.0" izz="1.0" /-->
-        <solid_cuboid_inertia  w="1.265" h="0.812" d="0.465" m="25"/>
+        <xacro:solid_cuboid_inertia w="1.265" h="0.812" d="0.465" m="25"/>
       </inertial>
       <visual>

File: rbvogui_description/urdf/structures/bi_arm_support.urdf.xacro (robot description, xacro)
@@ -30,5 +30,5 @@
         <mass value="5" />
         <origin xyz="0 0 0" rpy="0 0 ${M_PI/2.0}"/>
-        <solid_cuboid_inertia  w="0.4" h="0.4" d="0.2" m="5"/>
+        <xacro:solid_cuboid_inertia  w="0.4" h="0.4" d="0.2" m="5"/>
       </inertial>
     </link>

File: rbvogui_description/urdf/structures/sick_protector.urdf.xacro (robot description, xacro)
@@ -31,5 +31,5 @@
         <mass value="5" />
         <origin xyz="0 0 0" rpy="0 0 ${M_PI/2.0}"/>
-        <solid_cuboid_inertia  w="0.4" h="0.4" d="0.2" m="5"/>
+        <xacro:solid_cuboid_inertia  w="0.4" h="0.4" d="0.2" m="5"/>
       </inertial>
     </link>

File: rbvogui_description/urdf/structures/sick_support.urdf.xacro (robot description, xacro)
@@ -31,5 +31,5 @@
         <mass value="5" />
         <origin xyz="0 0 0" rpy="0 0 ${M_PI/2.0}"/>
-        <solid_cuboid_inertia  w="0.4" h="0.4" d="0.2" m="5"/>
+        <xacro:solid_cuboid_inertia  w="0.4" h="0.4" d="0.2" m="5"/>
       </inertial>
     </link>

File: rbvogui_description/urdf/wheels/rubber_wheel_285mm.urdf.xacro (robot description, xacro)
@@ -5,4 +5,5 @@
   <!-- Wheels -->
   <xacro:property name="wheel_radius" value="0.1425" />
+  <xacro:property name="wheel_width" value="0.1275" />
   <xacro:property name="wheel_height" value="0.14" />
   <xacro:property name="wheel_mass" value="4.0" />
@@ -79,5 +80,5 @@
         <mass value="${wheel_mass}" />
         <origin xyz="0 0 0" />
-        <cylinder_inertia m="${wheel_mass}" r="${wheel_radius}" h="${wheel_height}" />
+        <xacro:cylinder_inertia m="${wheel_mass}" r="${wheel_radius}" h="${wheel_height}" />
       </inertial>
     </link>

File: rbvogui_description/urdf/wheels/rubber_wheel_350mm.urdf.xacro (robot description, xacro)
@@ -5,4 +5,5 @@
   <!-- Wheels -->
   <xacro:property name="wheel_radius" value="0.1745" />
+  <xacro:property name="wheel_width" value="0.1275" />
   <xacro:property name="wheel_height" value="0.1165" /> <!--Check -->
   <xacro:property name="wheel_mass" value="5.0" />
@@ -79,5 +80,5 @@
         <mass value="${wheel_mass}" />
         <origin xyz="0 0 0" />
-        <cylinder_inertia m="${wheel_mass}" r="${wheel_radius}" h="${wheel_height}" />
+        <xacro:cylinder_inertia m="${wheel_mass}" r="${wheel_radius}" h="${wheel_height}" />
       </inertial>
     </link>

File: rbvogui_description/urdf/wheels/steering_wheel_xl.urdf.xacro (robot description, xacro)
@@ -88,5 +88,5 @@
 		</xacro:unless>
         <!-- To do: add real intertia-->
-        <cylinder_inertia m="5" r="0.1425" h="0.14"/>
+        <xacro:cylinder_inertia m="5" r="0.1425" h="0.14"/>
       </inertial>
     </link>

File: rbvogui_description/urdf/wheels/steering_wheel_xl_offroad.urdf.xacro (robot description, xacro)
@@ -88,5 +88,5 @@
 		</xacro:unless>
         <!-- To do: add real intertia-->
-        <cylinder_inertia m="5" r="0.1425" h="0.14"/>
+        <xacro:cylinder_inertia m="5" r="0.1425" h="0.14"/>
       </inertial>
     </link>
