Commit message: FIx rbvogui xl inertias and ros2_control

File: rbvogui_description/robots/rbvogui_xl_std.urdf.xacro (robot description, xacro)
@@ -9,5 +9,5 @@
     <xacro:include filename="$(find rbvogui_description)/urdf/bases/rbvogui_xl_base.urdf.xacro" />
     <!-- Import rbvogui wheels -->
-    <xacro:include filename="$(find rbvogui_description)/urdf/wheels/motor_wheel_xl.urdf.xacro" />
+    <xacro:include filename="$(find rbvogui_description)/urdf/wheels/steering_wheel_xl.urdf.xacro" />
     <!-- Import rbvogui fix wheels -->
     <xacro:include filename="$(find rbvogui_description)/urdf/wheels/fixed_wheel_xl.urdf.xacro" />
@@ -43,23 +43,23 @@
         <!-- Here we create the robot elements using the xacro:macros imported at the beggining of this file -->
         <xacro:rbvogui_base prefix="${prefix}" publish_bf="${publish_bf}" base_height="${wheel_radius}" hq="${hq}"/>
-        <xacro:motor_wheel prefix="${prefix}front_right_" parent="${prefix}base_link" reflect="true" hq="${hq}">
+        <xacro:steering_wheel prefix="${prefix}front_right_" parent="${prefix}base_link" reflect="true" hq="${hq}">
             <origin xyz="${wheel_offset_x} -${wheel_offset_y} ${wheel_offset_z}" rpy="0 0 0"/>
-        </xacro:motor_wheel>
-        <xacro:motor_wheel prefix="${prefix}front_left_" parent="${prefix}base_link" reflect="false" hq="${hq}">
+        </xacro:steering_wheel>
+        <xacro:steering_wheel prefix="${prefix}front_left_" parent="${prefix}base_link" reflect="false" hq="${hq}">
             <origin xyz="${wheel_offset_x} ${wheel_offset_y} ${wheel_offset_z}" rpy="0 0 0"/>
-        </xacro:motor_wheel>
+        </xacro:steering_wheel>
         <xacro:if value="${kinematics == 'omni'}">
-            <xacro:motor_wheel prefix="${prefix}rear_left_" parent="${prefix}base_link" reflect="false" hq="${hq}">
+            <xacro:steering_wheel prefix="${prefix}back_left_" parent="${prefix}base_link" reflect="false" hq="${hq}">
                 <origin xyz="-${wheel_offset_x} ${wheel_offset_y} ${wheel_offset_z}" rpy="0 0 0"/>
-            </xacro:motor_wheel>
-            <xacro:motor_wheel prefix="${prefix}rear_right_" parent="${prefix}base_link" reflect="true" hq="${hq}">
+            </xacro:steering_wheel>
+            <xacro:steering_wheel prefix="${prefix}back_right_" parent="${prefix}base_link" reflect="true" hq="${hq}">
                 <origin xyz="-${wheel_offset_x} -${wheel_offset_y} ${wheel_offset_z}" rpy="0 0 0"/>
-            </xacro:motor_wheel>
+            </xacro:steering_wheel>
         </xacro:if>
         <xacro:if value="${kinematics == 'ackermann'}">
-            <xacro:fixed_wheel prefix="${prefix}rear_left_" parent="${prefix}base_link" reflect="false" hq="${hq}">
+            <xacro:fixed_wheel prefix="${prefix}back_left_" parent="${prefix}base_link" reflect="false" hq="${hq}">
                 <origin xyz="-${wheel_offset_x} ${wheel_offset_y} ${wheel_offset_z}" rpy="0 0 0"/>
             </xacro:fixed_wheel>
-            <xacro:fixed_wheel prefix="${prefix}rear_right_" parent="${prefix}base_link" reflect="true" hq="${hq}">
+            <xacro:fixed_wheel prefix="${prefix}back_right_" parent="${prefix}base_link" reflect="true" hq="${hq}">
                 <origin xyz="-${wheel_offset_x} -${wheel_offset_y} ${wheel_offset_z}" rpy="0 0 0"/>
             </xacro:fixed_wheel>
@@ -104,34 +104,11 @@
             <origin xyz="-0.64555 -0.39985 0.16608" rpy="${PI} 0 -${135*PI/180}"/>
         </xacro:sensor_sick_microscan3>
-        <xacro:macro name="ros2_joint" params="interface jmin jmax prefix name">
-          <joint name="${prefix}${name}">
-            <command_interface name="${interface}">
-              <param name="min">${jmin}</param>
-              <param name="max">${jmax}</param>
-            </command_interface>
-            <state_interface name="position"/>
-            <state_interface name="velocity"/>
-            <state_interface name="effort"/>
-          </joint>
-        </xacro:macro>
-        <ros2_control name="GazeboSystem" type="system">
-          <hardware>
-              <plugin>gazebo_ros2_control/GazeboSystem</plugin>
-          </hardware>
-          <xacro:ros2_joint interface="position" jmin="-2" jmax="2" prefix="${prefix}" name="front_left_motor_wheel_joint"/>
-          <xacro:ros2_joint interface="position" jmin="-2" jmax="2" prefix="${prefix}" name="front_right_motor_wheel_joint"/>
-          <xacro:ros2_joint interface="position" jmin="-2" jmax="2" prefix="${prefix}" name="rear_left_motor_wheel_joint"/>
-          <xacro:ros2_joint interface="position" jmin="-2" jmax="2" prefix="${prefix}" name="rear_right_motor_wheel_joint"/>
-          <xacro:ros2_joint interface="velocity" jmin="-10" jmax="10" prefix="${prefix}" name="front_left_wheel_joint"/>
-          <xacro:ros2_joint interface="velocity" jmin="-10" jmax="10" prefix="${prefix}" name="front_right_wheel_joint"/>
-          <xacro:ros2_joint interface="velocity" jmin="-20" jmax="20" prefix="${prefix}" name="rear_left_wheel_joint"/>
-          <xacro:ros2_joint interface="velocity" jmin="-20" jmax="20" prefix="${prefix}" name="rear_right_wheel_joint"/>
-        </ros2_control>
     </xacro:macro>
-    <!-- Gazebo ros control pluggins -->
-    <xacro:ros_control/>
     <xacro:rbvogui prefix="$(arg prefix)" kinematics="$(arg kinematics)" load_kinematics_file="$(arg load_kinematics_file)" gpu="$(arg gpu)" publish_bf="${publish_bf}" hq="${hq}"
                    launch_arm="$(arg launch_arm)" arm_manufacturer="$(arg arm_manufacturer)" arm_model="$(arg arm_model)"
                    launch_gripper="$(arg launch_gripper)" gripper_manufacturer="$(arg gripper_manufacturer)" gripper_model="$(arg gripper_model)"
                    launch_lift="$(arg launch_lift)" lift_manufacturer="$(arg lift_manufacturer)" lift_model="$(arg lift_model)" />
+    <!-- Gazebo ros control pluggins -->
+    <xacro:include filename="$(find rbvogui_description)/urdf/ros2_control.urdf.xacro"/>
+    <xacro:ros2_control prefix="$(arg prefix)"/>
 </robot>

File: rbvogui_description/urdf/bases/rbvogui_xl_base.urdf.xacro (robot description, xacro)
@@ -2,6 +2,11 @@
 <robot xmlns:xacro="http://wiki.ros.org/xacro">
   <xacro:include filename="$(find rbvogui_description)/urdf/bases/rbvogui_base.gazebo.xacro" />
-  <xacro:include filename="$(find rbvogui_description)/urdf/inertia.urdf.xacro" />
   <xacro:macro name="rbvogui_base" params="prefix publish_bf base_height:=0.1425 hq">
+    <xacro:macro name="solid_cuboid_inertia" params="w h d m">
+      <inertia  ixx="${(m*(h*h+d*d))/12}" ixy = "0" ixz = "0"
+                iyy="${(m*(w*w+d*d))/12}" iyz = "0"
+                izz="${(m*(w*w+h*h))/12}"
+      />
+    </xacro:macro>
     <!-- Robot mechanical and motor parameters -->
     <xacro:property name="PI" value="3.1415926535897931"/>
@@ -34,8 +39,8 @@
     <link name="${prefix}chassis_link">
       <inertial>
-        <mass value="25.0" />
-        <origin xyz="0 0 0.376" />
+        <mass value="65.0" />
+        <origin xyz="0 0 -0.12" />
         <!--inertia ixx="1.0" ixy="0.0" ixz="0.0" iyy="1.0" iyz="0.0" izz="1.0" /-->
-        <xacro:solid_cuboid_inertia w="1.265" h="0.812" d="0.465" m="25"/>
+        <xacro:solid_cuboid_inertia w="1.265" h="0.812" d="0.465" m="65.0"/>
       </inertial>
       <visual>
@@ -71,7 +76,7 @@
     <link name="${prefix}battery_link">
       <inertial>
-        <mass value="20.0" />
-        <origin xyz="0 0 0" />
-        <inertia ixx="1.0" ixy="0.0" ixz="0.0" iyy="1.0" iyz="0.0" izz="1.0" />
+        <mass value="40.0" />
+        <origin xyz="0 0 -0.25" />
+        <xacro:solid_cuboid_inertia w="0.265" h="0.212" d="0.165" m="40.0"/>
       </inertial>
       <visual>

File: rbvogui_description/urdf/wheels/rubber_wheel_285mm.urdf.xacro (robot description, xacro)
@@ -2,26 +2,16 @@
 <robot xmlns:xacro="http://www.ros.org/wiki/xacro">
   <xacro:include filename="$(find rbvogui_description)/urdf/wheels/wheel.gazebo.xacro" />
-  <xacro:property name="M_PI" value="3.1415926535897931" />
-  <!-- Wheels -->
   <xacro:property name="wheel_radius" value="0.1425" />
-  <xacro:property name="wheel_width" value="0.1275" />
-  <xacro:property name="wheel_height" value="0.14" />
-  <xacro:property name="wheel_mass" value="4.0" />
-  <!-- in kg-->
-  <xacro:property name="steer_joint_damping" value="2.0" />
-  <xacro:property name="steer_joint_friction" value="1.0" />
-  <xacro:property name="steer_joint_effort_limit" value="100.0" />
-  <xacro:property name="steer_joint_velocity_limit" value="2.83" />
-  <xacro:property name="motor_wheel_mechanical_reduction" value="1.0" />
-  <xacro:property name="wheel_joint_damping" value="0.1" />
-  <xacro:property name="wheel_joint_friction" value="0.1" />
-  <xacro:property name="wheel_joint_effort_limit" value="1000.0" />
-  <xacro:property name="wheel_joint_velocity_limit" value="2000.0" />
-  <xacro:property name="wheel_mechanical_reduction" value="1.0" />
-  <xacro:macro name="cylinder_inertia" params="m r h">
-    <inertia ixx="${m*(3*r*r+h*h)/12}" ixy = "0" ixz = "0" iyy="${m*(3*r*r+h*h)/12}" iyz = "0" izz="${m*r*r/2}" />
-  </xacro:macro>
   <xacro:macro name="wheel_285mm" params="prefix parent *origin reflect hq">
-    <!-- TODO: check reflect parameter -->
+    <xacro:macro name="cylinder_inertia" params="m r h">
+      <inertia ixx="${m*(3*r*r+h*h)/12}" ixy = "0" ixz = "0" iyy="${m*(3*r*r+h*h)/12}" iyz = "0" izz="${m*r*r/2}" />
+    </xacro:macro>
+    <xacro:property name="M_PI" value="3.1415926535897931" />
+    <xacro:property name="wheel_width" value="0.14" />
+    <xacro:property name="wheel_mass" value="4.0" />
+    <xacro:property name="wheel_joint_damping" value="0.1" />
+    <xacro:property name="wheel_joint_friction" value="0.1" />
+    <xacro:property name="wheel_joint_effort_limit" value="1000.0" />
+    <xacro:property name="wheel_joint_velocity_limit" value="2000.0" />
     <!--WHEEL TIRE -->
     <joint name="${prefix}wheel_joint" type="continuous">
@@ -31,16 +21,6 @@
       <axis xyz="0 1 0" rpy="0 0 0" />
       <limit effort="${wheel_joint_effort_limit}" velocity="${wheel_joint_velocity_limit}"/>
-      <joint_properties damping="${wheel_joint_damping}" friction="{wheel_joint_friction}"/>
+      <dynamics damping="${wheel_joint_damping}" friction="${wheel_joint_friction}"/>
     </joint>
-    <transmission name="${prefix}wheel_trans">
-      <type>transmission_interface/SimpleTransmission</type>
-      <joint name="${prefix}wheel_joint">
-        <hardwareInterface>hardware_interface/VelocityJointInterface</hardwareInterface>
-      </joint>
-      <actuator name="${prefix}wheel_motor">
-        <hardwareInterface>hardware_interface/VelocityActuatorInterface</hardwareInterface>
-        <mechanicalReduction>${wheel_mechanical_reduction}</mechanicalReduction>
-      </actuator>
-    </transmission>
     <link name="${prefix}wheel">
       <visual>
@@ -64,5 +44,5 @@
           <origin xyz="0 0 0" rpy="${M_PI/2} 0 0" />
           <geometry>
-            <cylinder length="${wheel_height}" radius="${wheel_radius}" />
+            <cylinder length="${wheel_width}" radius="${wheel_radius}" />
           </geometry>
         </xacro:unless>
@@ -74,15 +54,16 @@
         <origin xyz="0 0 0" rpy="${M_PI/2} 0 0" />
         <geometry>
-          <sphere radius="${wheel_radius}" />
+          <cylinder length="${wheel_radius}" radius="${wheel_radius}" />
         </geometry>
       </collision>
       <inertial>
         <mass value="${wheel_mass}" />
-        <origin xyz="0 0 0" />
-        <xacro:cylinder_inertia m="${wheel_mass}" r="${wheel_radius}" h="${wheel_height}" />
+        <origin xyz="0 0 0" rpy="${M_PI/2} 0 0"/>
+        <xacro:cylinder_inertia m="${wheel_mass}" r="${wheel_radius}" h="${wheel_width}" />
       </inertial>
     </link>
-    <xacro:gazebo_color_wheel prefix="${prefix}"/>
-    <xacro:gazebo_color_steer_wheel prefix="${prefix}"/>
+    <!-- GAZEBO PARAMETERS -->
+    <xacro:gazebo_rubber_tire_physics name="${prefix}wheel" />
+    <xacro:gazebo_rubber_tire_material name="${prefix}wheel" />
   </xacro:macro>
 </robot>

File: rbvogui_description/urdf/wheels/steering_wheel_xl.urdf.xacro (robot description, xacro)
@@ -3,49 +3,32 @@
   <xacro:include filename="$(find rbvogui_description)/urdf/wheels/wheel.gazebo.xacro" />
   <xacro:include filename="$(find rbvogui_description)/urdf/wheels/rubber_wheel_285mm.urdf.xacro" />
-  <xacro:property name="M_PI" value="3.1415926535897931" />
-  <xacro:property name="steer_joint_damping" value="2.0" />
-  <xacro:property name="steer_joint_friction" value="1.0" />
-  <xacro:property name="steer_joint_effort_limit" value="100.0" />
-  <xacro:property name="steer_joint_velocity_limit" value="2.83" />
-  <xacro:property name="motor_wheel_mechanical_reduction" value="1.0" />
-  <xacro:property name="wheel_joint_damping" value="0.1" />
-  <xacro:property name="wheel_joint_friction" value="0.1" />
-  <xacro:property name="wheel_joint_effort_limit" value="1000.0" />
-  <xacro:property name="wheel_joint_velocity_limit" value="2000.0" />
-  <xacro:property name="wheel_mechanical_reduction" value="1.0" />
-  <xacro:macro name="cylinder_inertia" params="m r h">
-    <inertia ixx="${m*(3*r*r+h*h)/12}" ixy = "0" ixz = "0" iyy="${m*(3*r*r+h*h)/12}" iyz = "0" izz="${m*r*r/2}" />
-  </xacro:macro>
-  <xacro:macro name="motor_wheel" params="prefix parent *origin reflect hq">
+  <xacro:macro name="steering_wheel" params="prefix parent *origin reflect hq">
+    <xacro:macro name="cylinder_inertia" params="m r h">
+      <inertia ixx="${m*(3*r*r+h*h)/12}" ixy = "0" ixz = "0" iyy="${m*(3*r*r+h*h)/12}" iyz = "0" izz="${m*r*r/2}" />
+    </xacro:macro>
+    <xacro:property name="M_PI" value="3.1415926535897931" />
+    <xacro:property name="steer_joint_damping" value="2.0" />
+    <xacro:property name="steer_joint_friction" value="1.0" />
+    <xacro:property name="steer_joint_effort_limit" value="2000.0" />
+    <xacro:property name="steer_joint_velocity_limit" value="1000.0" />
     <!--MOTOR WHEEL -->
-    <joint name="${prefix}motor_wheel_joint" type="revolute">
+    <joint name="${prefix}steering_joint" type="revolute">
       <parent link="${parent}"/>
-      <child link="${prefix}motor_wheel"/>
+      <child link="${prefix}base_wheel"/>
       <xacro:insert_block name="origin" />
       <axis xyz="0 0 1" rpy="0 0 0" />
-      <!-- limit effort="${steer_joint_effort_limit}" velocity="${steer_joint_velocity_limit}" lower="-1.5708" upper="1.5708" / -->
       <limit effort="${steer_joint_effort_limit}" velocity="${steer_joint_velocity_limit}" lower="-3.00" upper="3.00"/>
-      <joint_properties damping="${steer_joint_damping}" friction="${steer_joint_friction}"/>
+      <dynamics damping="${steer_joint_damping}" friction="${steer_joint_friction}"/>
     </joint>
-    <transmission name="${prefix}motor_wheel_trans">
-      <type>transmission_interface/SimpleTransmission</type>
-      <joint name="${prefix}motor_wheel_joint">
-        <hardwareInterface>hardware_interface/PositionJointInterface</hardwareInterface>
-      </joint>
-      <actuator name="${prefix}motor_wheel_motor">
-        <hardwareInterface>hardware_interface/PositionActuatorInterface</hardwareInterface>
-        <mechanicalReduction>${motor_wheel_mechanical_reduction}</mechanicalReduction>
-      </actuator>
-    </transmission>
-    <link name="${prefix}motor_wheel">
+    <link name="${prefix}base_wheel">
       <visual>
         <!-- HIGH RESOLUTION WHEELS -->
         <xacro:if value="${hq}">
-		  <xacro:if value="${reflect}">
-			<origin xyz="0 0 0" rpy="0 0 ${M_PI}" />
-		  </xacro:if>
-		  <xacro:unless value="${reflect}">
-			<origin xyz="0 0 0.0" rpy="0 0 0" />
-		  </xacro:unless>
+          <xacro:if value="${reflect}">
+            <origin xyz="0 0 0" rpy="0 0 ${M_PI}" />
+          </xacro:if>
+          <xacro:unless value="${reflect}">
+            <origin xyz="0 0 0.0" rpy="0 0 0" />
+          </xacro:unless>
           <geometry>
             <mesh filename="package://rbvogui_description/meshes/wheels/hub_rbvogui_xl.stl" />
@@ -55,26 +38,26 @@
         <xacro:unless value="${hq}">
           <xacro:if value="${reflect}">
-			<origin xyz="0 0 0" rpy="0 0 ${M_PI}" />
-		  </xacro:if>
-		  <xacro:unless value="${reflect}">
-			<origin xyz="0 0 0" rpy="0 0 0" />
-		  </xacro:unless>
+			      <origin xyz="0 0 0" rpy="0 0 ${M_PI}" />
+          </xacro:if>
+          <xacro:unless value="${reflect}">
+            <origin xyz="0 0 0" rpy="0 0 0" />
+          </xacro:unless>
           <geometry>
-              <mesh filename="package://rbvogui_description/meshes/wheels/hub_rbvogui_xl.stl" />
+            <mesh filename="package://rbvogui_description/meshes/wheels/hub_rbvogui_xl.stl" />
           </geometry>
         </xacro:unless>
         <material name="red">
-             <color rgba="0.9 0.1 0.1 1"/>
+          <color rgba="0.9 0.1 0.1 1"/>
         </material>
       </visual>
       <collision>
-		<xacro:if value="${reflect}">
-			<origin xyz="0 0 0" rpy="0 0 ${M_PI}" />
-		</xacro:if>
-		<xacro:unless value="${reflect}">
-			<origin xyz="0 0 0.0" rpy="0 0 0" />
-		</xacro:unless>
+        <xacro:if value="${reflect}">
+          <origin xyz="0 0 0" rpy="0 0 ${M_PI}" />
+        </xacro:if>
+        <xacro:unless value="${reflect}">
+          <origin xyz="0 0 0.0" rpy="0 0 0" />
+        </xacro:unless>
         <geometry>
-            <mesh filename="package://rbvogui_description/meshes/wheels/hub_rbvogui_xl.stl" />
+          <mesh filename="package://rbvogui_description/meshes/wheels/hub_rbvogui_xl.stl" />
         </geometry>
       </collision>
@@ -82,15 +65,15 @@
         <mass value="4" />
         <xacro:if value="${reflect}">
-			<origin xyz="0 0 0.12" rpy="0 0 ${M_PI}"/>
-		</xacro:if>
-		<xacro:unless value="${reflect}">
-			<origin xyz="0 0 0.12" rpy="0 0 0"/>
-		</xacro:unless>
-        <!-- To do: add real intertia-->
+          <origin xyz="0 0 ${wheel_radius/1.5}" rpy="${M_PI/2.0} ${M_PI/2.0} 0"/>
+        </xacro:if>
+        <xacro:unless value="${reflect}">
+          <origin xyz="0 0 ${wheel_radius/1.5}" rpy="${M_PI/2.0} ${M_PI/2.0} ${M_PI/2.0}"/>
+        </xacro:unless>
         <xacro:cylinder_inertia m="5" r="0.1425" h="0.14"/>
       </inertial>
     </link>
-    <xacro:gazebo_color_wheel_frame prefix="${prefix}"/>
-    <xacro:wheel_285mm prefix="${prefix}" parent="${prefix}motor_wheel" reflect="${reflect}" hq="${hq}">
+    <xacro:gazebo_steering_frame_physics name="${prefix}base_wheel"/>
+    <xacro:gazebo_steering_frame_material name="${prefix}base_wheel"/>
+    <xacro:wheel_285mm prefix="${prefix}" parent="${prefix}base_wheel" reflect="${reflect}" hq="${hq}">
         <origin xyz="0 0 0" rpy="0 0 0"/>
     </xacro:wheel_285mm>
