Commit message: description: Update rbvogui xl urdf for all configurations

File: rbvogui_description/robots/rbvogui_xl_biarm.urdf.xacro (robot description, xacro)
@@ -46,8 +46,8 @@
             <origin xyz="${wheel_offset_x} -${wheel_offset_y} ${wheel_offset_z}" rpy="0 0 0"/>
         </xacro:motor_wheel>
-        <xacro:motor_wheel prefix="${prefix}front_left_" parent="${prefix}base_link" reflect="false" hq="${hq}"> <!-- good -->
+        <xacro:motor_wheel prefix="${prefix}front_left_" parent="${prefix}base_link" reflect="false" hq="${hq}">
             <origin xyz="${wheel_offset_x} ${wheel_offset_y} ${wheel_offset_z}" rpy="0 0 0"/>
         </xacro:motor_wheel>
-        <xacro:motor_wheel prefix="${prefix}back_left_" parent="${prefix}base_link" reflect="false" hq="${hq}"> <!-- good -->
+        <xacro:motor_wheel prefix="${prefix}back_left_" parent="${prefix}base_link" reflect="false" hq="${hq}">
             <origin xyz="-${wheel_offset_x} ${wheel_offset_y} ${wheel_offset_z}" rpy="0 0 0"/>
         </xacro:motor_wheel>
@@ -70,5 +70,5 @@
         <!-- Orbbec camera -->
         <xacro:sensor_orbbec_astra prefix="${prefix}front_rgbd_camera" parent="${prefix}chassis_link">
-            <origin xyz="0.63658 0.0 -0.03643" rpy="0 0 0"/>
+            <origin xyz="0.637 0.0 -0.036" rpy="0 0 0"/>
         </xacro:sensor_orbbec_astra>
         <!-- Zed camera
@@ -102,4 +102,8 @@
             <origin xyz="-0.64555 -0.39985 0.16608" rpy="${PI} 0 -${135*PI/180}"/>
         </xacro:sensor_sick_microscan3>
+        <!-- GPS -->
+        <xacro:sensor_ublox prefix="${prefix}gps" parent="${prefix}chassis_link">
+            <origin xyz="-0.472 0.4 0.456" rpy="0 0 0"/>
+        </xacro:sensor_ublox>
     </xacro:macro>
     <!-- Gazebo ros control pluggins -->

File: rbvogui_description/robots/rbvogui_xl_lift_ur10e.urdf.xacro (robot description, xacro)
@@ -30,7 +30,7 @@
     <xacro:property name="wheel_offset_z" value="0.0" />
     <!-- Arm with lift parameters -->
-    <xacro:property name="lift_arm_offset_x" value="0.207" />
+    <xacro:property name="lift_arm_offset_x" value="0.275" />
     <xacro:property name="lift_arm_offset_y" value="0.0" />
-    <xacro:property name="lift_arm_offset_z" value="0.235" />
+    <xacro:property name="lift_arm_offset_z" value="0.01" />
     <!-- Flag to select the high or low quality model -->
     <xacro:property name="hq" value="true" />
@@ -74,5 +74,5 @@
 		</xacro:unless>
         <joint name="${prefix}arm_base_joint" type="fixed">
-            <origin xyz="0 0 0.015" rpy="0 0 0"/>
+            <origin xyz="0 0 0.015" rpy="0 0 ${PI/4}"/>
             <parent link="${prefix}ewellix_lift_top_link" />
             <child link="${prefix}arm_base_link" />
@@ -89,5 +89,5 @@
         <!-- Orbbec camera -->
         <xacro:sensor_orbbec_astra prefix="${prefix}front_rgbd_camera" parent="${prefix}chassis_link">
-            <origin xyz="0.63658 0.0 -0.03643" rpy="0 0 0"/>
+            <origin xyz="0.637 0.0 -0.036" rpy="0 0 0"/>
         </xacro:sensor_orbbec_astra>
         <!-- Zed camera
@@ -98,5 +98,5 @@
         <!-- 3D lidar -->
         <xacro:sensor_rs_bpearl prefix="${prefix}front_3d_laser" parent="${prefix}chassis_link" prefix_topic="front_3d_laser" range_min="0.1" range_max="90" hfov="360" samples="1200" vfov="90.0" lasers="32" fps="15" gpu="${gpu}">
-            <origin xyz="0.57918 0 0.24072" rpy="0 ${90*PI/180} 0"/>
+            <origin xyz="0.579 0 0.241" rpy="0 ${90*PI/180} 0"/>
         </xacro:sensor_rs_bpearl>
         <!-- Laser sick support -->
@@ -121,4 +121,8 @@
             <origin xyz="-0.64555 -0.39985 0.16608" rpy="${PI} 0 -${135*PI/180}"/>
         </xacro:sensor_sick_microscan3>
+        <!-- GPS -->
+        <xacro:sensor_ublox prefix="${prefix}gps" parent="${prefix}chassis_link">
+            <origin xyz="-0.472 0.4 0.456" rpy="0 0 0"/>
+        </xacro:sensor_ublox>
     </xacro:macro>
     <!-- Gazebo ros control pluggins -->

File: rbvogui_description/robots/rbvogui_xl_lift_ur10e_hand_e.urdf.xacro (robot description, xacro)
@@ -32,7 +32,7 @@
     <xacro:property name="wheel_offset_z" value="0.0" />
     <!-- Arm with lift parameters -->
-    <xacro:property name="lift_arm_offset_x" value="0.207" />
+    <xacro:property name="lift_arm_offset_x" value="0.275" />
     <xacro:property name="lift_arm_offset_y" value="0.0" />
-    <xacro:property name="lift_arm_offset_z" value="0.235" />
+    <xacro:property name="lift_arm_offset_z" value="0.01" />
     <!-- Flag to select the high or low quality model -->
     <xacro:property name="hq" value="true" />
@@ -76,5 +76,5 @@
 		</xacro:unless>
         <joint name="${prefix}arm_base_joint" type="fixed">
-            <origin xyz="0 0 0.015" rpy="0 0 0"/>
+            <origin xyz="0 0 0.015" rpy="0 0 ${PI/4}"/>
             <parent link="${prefix}ewellix_lift_top_link" />
             <child link="${prefix}arm_base_link" />
@@ -91,5 +91,5 @@
         <!-- Orbbec camera -->
         <xacro:sensor_orbbec_astra prefix="${prefix}front_rgbd_camera" parent="${prefix}chassis_link">
-            <origin xyz="0.63658 0.0 -0.03643" rpy="0 0 0"/>
+            <origin xyz="0.637 0.0 -0.036" rpy="0 0 0"/>
         </xacro:sensor_orbbec_astra>
         <!-- Zed camera
@@ -100,5 +100,5 @@
         <!-- 3D lidar -->
         <xacro:sensor_rs_bpearl prefix="${prefix}front_3d_laser" parent="${prefix}chassis_link" prefix_topic="front_3d_laser" range_min="0.1" range_max="90" hfov="360" samples="1200" vfov="90.0" lasers="32" fps="15" gpu="${gpu}">
-            <origin xyz="0.57918 0 0.24072" rpy="0 ${90*PI/180} 0"/>
+            <origin xyz="0.579 0 0.241" rpy="0 ${90*PI/180} 0"/>
         </xacro:sensor_rs_bpearl>
         <!-- Laser sick support -->
@@ -123,4 +123,8 @@
             <origin xyz="-0.64555 -0.39985 0.16608" rpy="${PI} 0 -${135*PI/180}"/>
         </xacro:sensor_sick_microscan3>
+        <!-- GPS -->
+        <xacro:sensor_ublox prefix="${prefix}gps" parent="${prefix}chassis_link">
+            <origin xyz="-0.472 0.4 0.456" rpy="0 0 0"/>
+        </xacro:sensor_ublox>
         <!-- Robotiq hand_e -->
         <xacro:hand_e_gripper prefix="$(arg prefix)gripper" parent="$(arg prefix)arm_tool0">

File: rbvogui_description/robots/rbvogui_xl_std.urdf.xacro (robot description, xacro)
@@ -76,5 +76,5 @@
         <!-- Orbbec camera -->
         <xacro:sensor_orbbec_astra prefix="${prefix}front_rgbd_camera" parent="${prefix}chassis_link">
-            <origin xyz="0.63658 0.0 -0.03643" rpy="0 0 0"/>
+            <origin xyz="0.637 0.0 -0.036" rpy="0 0 0"/>
         </xacro:sensor_orbbec_astra>
         <!-- Zed camera

File: rbvogui_description/urdf/wheels/motor_wheel_xl.urdf.xacro (robot description, xacro)
@@ -21,5 +21,5 @@
     <inertia ixx="${m*(3*r*r+h*h)/12}" ixy = "0" ixz = "0" iyy="${m*(3*r*r+h*h)/12}" iyz = "0" izz="${m*r*r/2}" />
   </xacro:macro>
-  <xacro:macro name="motor_wheel" params="prefix parent *origin reflect hq">
+  <xacro:macro name="motor_wheel" params="prefix parent *origin reflect hq offroad:=false">
     <!--MOTOR WHEEL -->
     <joint name="${prefix}motor_wheel_joint" type="revolute">
@@ -130,7 +130,14 @@
             <origin xyz="0 0 0" rpy="0 0 0" />
           </xacro:unless>
-          <geometry>
-              <mesh filename="package://rbvogui_description/meshes/wheels/wheel_rbvogui_xl.stl" />
-          </geometry>
+          <xacro:if value="${offroad}">
+              <geometry>
+                <mesh filename="package://rbvogui_description/meshes/wheels/wheel_rbvogui_xl_offroad.stl" />
+              </geometry>
+          </xacro:if>
+          <xacro:unless value="${offroad}">
+              <geometry>
+                <mesh filename="package://rbvogui_description/meshes/wheels/wheel_rbvogui_xl.stl" />
+              </geometry>
+          </xacro:unless>
         </xacro:if>
         <!-- LOW RESOLUTION WHEELS -->
@@ -142,7 +149,14 @@
 			    <origin xyz="0 0 0" rpy="0 0 0" />
 		    </xacro:unless>
-          <geometry>
-             <mesh filename="package://rbvogui_description/meshes/wheels/wheel_rbvogui_xl.dae" />
-          </geometry>
+          <xacro:if value="${offroad}">
+              <geometry>
+                <mesh filename="package://rbvogui_description/meshes/wheels/wheel_rbvogui_xl_offroad.stl" />
+              </geometry>
+          </xacro:if>
+          <xacro:unless value="${offroad}">
+              <geometry>
+                <mesh filename="package://rbvogui_description/meshes/wheels/wheel_rbvogui_xl.stl" />
+              </geometry>
+          </xacro:unless>
         </xacro:unless>
         <material name="black_wheel">

Commit message: description/rbvogui_xl: Refector wheel selection and add offroad wheel

File: rbvogui_description/robots/rbvogui_xl_biarm.urdf.xacro (robot description, xacro)
@@ -9,5 +9,5 @@
     <xacro:include filename="$(find rbvogui_description)/urdf/bases/rbvogui_xl_base.urdf.xacro" />
     <!-- Import rbvogui wheels -->
-    <xacro:include filename="$(find rbvogui_description)/urdf/wheels/motor_wheel_xl.urdf.xacro" />
+    <xacro:include filename="$(find rbvogui_description)/urdf/wheels/motor_wheel_xl_offroad.urdf.xacro" />
     <!-- Import arm structure -->
     <xacro:include filename="$(find rbvogui_description)/urdf/structures/bi_arm_support.urdf.xacro" />
@@ -42,5 +42,5 @@
         <!-- *************** -->
         <!-- Here we create the robot elements using the xacro:macros imported at the beggining of this file -->
-        <xacro:rbvogui_base prefix="${prefix}" publish_bf="${publish_bf}" hq="${hq}"/>
+        <xacro:rbvogui_base prefix="${prefix}" publish_bf="${publish_bf}" base_height="${wheel_radius}" hq="${hq}"/>
         <xacro:motor_wheel prefix="${prefix}front_right_" parent="${prefix}base_link" reflect="true" hq="${hq}">
             <origin xyz="${wheel_offset_x} -${wheel_offset_y} ${wheel_offset_z}" rpy="0 0 0"/>

File: rbvogui_description/robots/rbvogui_xl_lift_ur10e.urdf.xacro (robot description, xacro)
@@ -45,5 +45,5 @@
         <!-- *************** -->
         <!-- Here we create the robot elements using the xacro:macros imported at the beggining of this file -->
-        <xacro:rbvogui_base prefix="${prefix}" publish_bf="${publish_bf}" hq="${hq}"/>
+        <xacro:rbvogui_base prefix="${prefix}" publish_bf="${publish_bf}" base_height="${wheel_radius}" hq="${hq}"/>
         <xacro:motor_wheel prefix="${prefix}front_right_" parent="${prefix}base_link" reflect="true" hq="${hq}">
             <origin xyz="${wheel_offset_x} -${wheel_offset_y} ${wheel_offset_z}" rpy="0 0 0"/>

File: rbvogui_description/robots/rbvogui_xl_lift_ur10e_hand_e.urdf.xacro (robot description, xacro)
@@ -47,5 +47,5 @@
         <!-- *************** -->
         <!-- Here we create the robot elements using the xacro:macros imported at the beggining of this file -->
-        <xacro:rbvogui_base prefix="${prefix}" publish_bf="${publish_bf}" hq="${hq}"/>
+        <xacro:rbvogui_base prefix="${prefix}" publish_bf="${publish_bf}" base_height="${wheel_radius}" hq="${hq}"/>
         <xacro:motor_wheel prefix="${prefix}front_right_" parent="${prefix}base_link" reflect="true" hq="${hq}">
             <origin xyz="${wheel_offset_x} -${wheel_offset_y} ${wheel_offset_z}" rpy="0 0 0"/>

File: rbvogui_description/robots/rbvogui_xl_std.urdf.xacro (robot description, xacro)
@@ -42,5 +42,5 @@
         <!-- *************** -->
         <!-- Here we create the robot elements using the xacro:macros imported at the beggining of this file -->
-        <xacro:rbvogui_base prefix="${prefix}" publish_bf="${publish_bf}" hq="${hq}"/>
+        <xacro:rbvogui_base prefix="${prefix}" publish_bf="${publish_bf}" base_height="${wheel_radius}" hq="${hq}"/>
         <xacro:motor_wheel prefix="${prefix}front_right_" parent="${prefix}base_link" reflect="true" hq="${hq}">
             <origin xyz="${wheel_offset_x} -${wheel_offset_y} ${wheel_offset_z}" rpy="0 0 0"/>
@@ -58,5 +58,5 @@
         </xacro:if>
         <xacro:if value="${kinematics == 'ackermann'}">
-            <xacro:fixed_wheel prefix="${prefix}back_left_" parent="${prefix}base_link" reflect="false" hq="${hq}"> <!-- good -->
+            <xacro:fixed_wheel prefix="${prefix}back_left_" parent="${prefix}base_link" reflect="false" hq="${hq}">
                 <origin xyz="-${wheel_offset_x} ${wheel_offset_y} ${wheel_offset_z}" rpy="0 0 0"/>
             </xacro:fixed_wheel>

File: rbvogui_description/urdf/bases/rbvogui_xl_base.urdf.xacro (robot description, xacro)
@@ -3,8 +3,7 @@
   <xacro:include filename="$(find rbvogui_description)/urdf/bases/rbvogui_base.gazebo.xacro" />
   <xacro:include filename="$(find rbvogui_description)/urdf/inertia.urdf.xacro" />
-  <xacro:macro name="rbvogui_base" params="prefix publish_bf hq">
+  <xacro:macro name="rbvogui_base" params="prefix publish_bf base_height:=0.1425 hq">
     <!-- Robot mechanical and motor parameters -->
     <xacro:property name="PI" value="3.1415926535897931"/>
-    <xacro:property name="wheel_width" value="0.146" />
     <!-- BASE FOOTPRINT -->
     <xacro:if value="${publish_bf}">
@@ -18,5 +17,5 @@
       </link>
       <joint name="${prefix}base_footprint_joint" type="fixed">
-        <origin xyz="0 0 ${wheel_radius}" rpy="0 0 0" />
+        <origin xyz="0 0 ${base_height}" rpy="0 0 0" />
         <!-- ${wheel_radius} property must be defined inside wheel description -->
         <parent link="${prefix}base_footprint"/>

File: rbvogui_description/urdf/wheels/fixed_wheel_xl.urdf.xacro (robot description, xacro)
@@ -3,9 +3,4 @@
   <xacro:include filename="$(find rbvogui_description)/urdf/wheels/wheel.gazebo.xacro" />
   <xacro:property name="M_PI" value="3.1415926535897931" />
-  <!-- Wheels -->
-  <xacro:property name="wheel_radius" value="0.1425" />
-  <xacro:property name="wheel_width" value="0.14" />
-  <xacro:property name="wheel_mass" value="4.0" />
-  <!-- in kg-->
   <xacro:property name="steer_joint_damping" value="2.0" />
   <xacro:property name="steer_joint_friction" value="1.0" />
@@ -79,93 +74,12 @@
 			<origin xyz="0 0 0.12" rpy="0 0 0"/>
 		</xacro:unless>
-     <!--inertia ixx="0.01" ixy="0.0" ixz="0.0" iyy="0.01" iyz="0.0" izz="0.01" /-->
-        <cylinder_inertia m="${wheel_mass}" r="${wheel_radius}" h="${wheel_width}" />
+        <!-- To do: add real intertia-->
+        <cylinder_inertia m="5" r="0.1425" h="0.14"/>
       </inertial>
     </link>
-    <!--WHEEL TIRE -->
-    <joint name="${prefix}wheel_joint" type="continuous">
-      <parent link="${prefix}fixed_wheel"/>
-      <child link="${prefix}wheel"/>
-      <xacro:if value="${reflect}">
-      <origin xyz="0 0 0" rpy="0 0 0" />
-		<axis xyz="0 1 0" rpy="0 0 0" />
-	  </xacro:if>
-      <xacro:unless value="${reflect}">
-       <origin xyz="0 0 0" rpy="0 0 0" />
-		<axis xyz="0 1 0" rpy="0 0 0" />
-	  </xacro:unless>
-      <limit effort="${wheel_joint_effort_limit}" velocity="${wheel_joint_velocity_limit}"/>
-      <joint_properties damping="${wheel_joint_damping}" friction="{wheel_joint_friction}"/>
-    </joint>
-    <transmission name="${prefix}wheel_trans">
-      <type>transmission_interface/SimpleTransmission</type>
-      <joint name="${prefix}wheel_joint">
-        <hardwareInterface>hardware_interface/VelocityJointInterface</hardwareInterface>
-      </joint>
-      <actuator name="${prefix}wheel_motor">
-        <hardwareInterface>hardware_interface/VelocityActuatorInterface</hardwareInterface>
-        <mechanicalReduction>${wheel_mechanical_reduction}</mechanicalReduction>
-      </actuator>
-    </transmission>
-    <link name="${prefix}wheel">
-      <visual>
-        <!-- HIGH RESOLUTION WHEELS -->
-        <xacro:if value="${hq}">
-		  <xacro:if value="${reflect}">
-			<origin xyz="0 0 0" rpy="0 0 ${M_PI}" />
-		  </xacro:if>
-		  <xacro:unless value="${reflect}">
-			<origin xyz="0 0 0" rpy="0 0 0" />
-		  </xacro:unless>
-          <geometry>
-             <mesh filename="package://rbvogui_description/meshes/wheels/wheel_rbvogui_xl.stl" />
-          </geometry>
-        </xacro:if>
-        <!-- LOW RESOLUTION WHEELS -->
-        <xacro:unless value="${hq}">
-          <xacro:if value="${reflect}">
-			<origin xyz="0 0 0" rpy="0 0 ${M_PI}" />
-		  </xacro:if>
-		  <xacro:unless value="${reflect}">
-			<origin xyz="0 0 0" rpy="0 0 0" />
-		  </xacro:unless>
-          <geometry>
-             <mesh filename="package://rbvogui_description/meshes/wheels/wheel_rbvogui_xl.stl" />
-          </geometry>
-        </xacro:unless>
-        <material name="black_wheel">
-          <color rgba="0.1 0.1 0.1 1"/>
-        </material>
-      </visual>
-      <collision>
-      <!--
-        <xacro:if value="${reflect}">
-			<origin xyz="0 0 0" rpy="${M_PI} 0 0" />
-		  </xacro:if>
-		  <xacro:unless value="${reflect}">
-			<origin xyz="0 0 0" rpy="0 0 0" />
-		  </xacro:unless>
-          <geometry>
-             <mesh filename="package://rbvogui_description/meshes/wheels/wheel_rbvogui_xl.stl" />
-        </geometry>
-        -->
-        <origin xyz="0 0 0" rpy="${M_PI/2} 0 0" />
-        <geometry>
-          <cylinder radius="${wheel_radius}" length="${wheel_width}"/>
-          </geometry>
-      </collision>
-      <inertial>
-        <mass value="${wheel_mass}" />
-        <xacro:if value="${reflect}">
-			<origin xyz="0 0 0" rpy="${M_PI/2 + M_PI} 0 0" />
-		  </xacro:if>
-		  <xacro:unless value="${reflect}">
-			<origin xyz="0 0 0" rpy="${M_PI/2} 0 0" />
-		  </xacro:unless>
-        <cylinder_inertia m="${wheel_mass}" r="${wheel_radius}" h="${wheel_width}" />
-      </inertial>
-    </link>
-    <xacro:gazebo_color_wheel prefix="${prefix}"/>
-    <xacro:gazebo_color_steer_wheel prefix="${prefix}"/>
+    <xacro:gazebo_color_fixed_wheel_frame prefix="${prefix}"/>
+    <xacro:wheel_285mm prefix="${prefix}" parent="${prefix}fixed_wheel" reflect="${reflect}" hq="${hq}">
+        <origin xyz="0 0 0" rpy="0 0 0"/>
+    </xacro:wheel_285mm>
   </xacro:macro>
 </robot>

File: rbvogui_description/urdf/wheels/fixed_wheel_xl_offroad.urdf.xacro (robot description, xacro)
@@ -1,6 +1,5 @@
 <?xml version="1.0"?>
-<robot xmlns:xacro="http://www.ros.org/wiki/xacro">
+<robot xmlns:xacro="http://wiki.ros.org/xacro">
   <xacro:include filename="$(find rbvogui_description)/urdf/wheels/wheel.gazebo.xacro" />
-  <xacro:include filename="$(find rbvogui_description)/urdf/wheels/rubber_wheel_285mm.urdf.xacro" />
   <xacro:property name="M_PI" value="3.1415926535897931" />
   <xacro:property name="steer_joint_damping" value="2.0" />
@@ -17,26 +16,14 @@
     <inertia ixx="${m*(3*r*r+h*h)/12}" ixy = "0" ixz = "0" iyy="${m*(3*r*r+h*h)/12}" iyz = "0" izz="${m*r*r/2}" />
   </xacro:macro>
-  <xacro:macro name="motor_wheel" params="prefix parent *origin reflect hq">
+  <xacro:macro name="fixed_wheel" params="prefix parent *origin reflect hq">
+    <!-- TODO: check reflect parameter -->
     <!--MOTOR WHEEL -->
-    <joint name="${prefix}motor_wheel_joint" type="revolute">
+    <joint name="${prefix}fixed_wheel_joint" type="fixed">
       <parent link="${parent}"/>
-      <child link="${prefix}motor_wheel"/>
+      <child link="${prefix}fixed_wheel"/>
       <xacro:insert_block name="origin" />
       <axis xyz="0 0 1" rpy="0 0 0" />
-      <!-- limit effort="${steer_joint_effort_limit}" velocity="${steer_joint_velocity_limit}" lower="-1.5708" upper="1.5708" / -->
-      <limit effort="${steer_joint_effort_limit}" velocity="${steer_joint_velocity_limit}" lower="-3.00" upper="3.00"/>
-      <joint_properties damping="${steer_joint_damping}" friction="${steer_joint_friction}"/>
     </joint>
-    <transmission name="${prefix}motor_wheel_trans">
-      <type>transmission_interface/SimpleTransmission</type>
-      <joint name="${prefix}motor_wheel_joint">
-        <hardwareInterface>hardware_interface/PositionJointInterface</hardwareInterface>
-      </joint>
-      <actuator name="${prefix}motor_wheel_motor">
-        <hardwareInterface>hardware_interface/PositionActuatorInterface</hardwareInterface>
-        <mechanicalReduction>${motor_wheel_mechanical_reduction}</mechanicalReduction>
-      </actuator>
-    </transmission>
-    <link name="${prefix}motor_wheel">
+    <link name="${prefix}fixed_wheel">
       <visual>
         <!-- HIGH RESOLUTION WHEELS -->
@@ -91,8 +78,8 @@
       </inertial>
     </link>
-    <xacro:gazebo_color_wheel_frame prefix="${prefix}"/>
-    <xacro:wheel_285mm prefix="${prefix}" parent="${prefix}motor_wheel" reflect="${reflect}" hq="${hq}">
+    <xacro:gazebo_color_fixed_wheel_frame prefix="${prefix}"/>
+    <xacro:wheel_350mm prefix="${prefix}" parent="${prefix}fixed_wheel" reflect="${reflect}" hq="${hq}">
         <origin xyz="0 0 0" rpy="0 0 0"/>
-    </xacro:wheel_285mm>
+    </xacro:wheel_350mm>
   </xacro:macro>
 </robot>

File: rbvogui_description/urdf/wheels/motor_wheel_xl_offroad.urdf.xacro (robot description, xacro)
@@ -2,5 +2,5 @@
 <robot xmlns:xacro="http://www.ros.org/wiki/xacro">
   <xacro:include filename="$(find rbvogui_description)/urdf/wheels/wheel.gazebo.xacro" />
-  <xacro:include filename="$(find rbvogui_description)/urdf/wheels/rubber_wheel_285mm.urdf.xacro" />
+  <xacro:include filename="$(find rbvogui_description)/urdf/wheels/rubber_wheel_350mm.urdf.xacro" />
   <xacro:property name="M_PI" value="3.1415926535897931" />
   <xacro:property name="steer_joint_damping" value="2.0" />
@@ -92,7 +92,7 @@
     </link>
     <xacro:gazebo_color_wheel_frame prefix="${prefix}"/>
-    <xacro:wheel_285mm prefix="${prefix}" parent="${prefix}motor_wheel" reflect="${reflect}" hq="${hq}">
+    <xacro:wheel_350mm prefix="${prefix}" parent="${prefix}motor_wheel" reflect="${reflect}" hq="${hq}">
         <origin xyz="0 0 0" rpy="0 0 0"/>
-    </xacro:wheel_285mm>
+    </xacro:wheel_350mm>
   </xacro:macro>
 </robot>
