Commit message: Revert "Fix noetic devel"

File: rbvogui_description/robots/rbvogui_xl_biarm.urdf.xacro (robot description, xacro)
@@ -78,5 +78,5 @@
         -->
         <!-- 3D lidar -->
-        <xacro:sensor_rs_bpearl prefix="${prefix}front_3d_laser" parent="${prefix}chassis_link" prefix_topic="front_3d_laser" suffix_topic="pcl" range_min="0.1" range_max="90" hfov="360" samples="1200" vfov="90.0" lasers="32" fps="15" gpu="${gpu}">
+        <xacro:sensor_rs_bpearl prefix="${prefix}front_3d_laser" parent="${prefix}chassis_link" prefix_topic="front_3d_laser" range_min="0.1" range_max="90" hfov="360" samples="1200" vfov="90.0" lasers="32" fps="15" gpu="${gpu}">
             <origin xyz="0.57918 0 0.24072" rpy="0 ${90*PI/180} 0"/>
         </xacro:sensor_rs_bpearl>

File: rbvogui_description/robots/rbvogui_xl_lift_ur10e.urdf.xacro (robot description, xacro)
@@ -97,5 +97,5 @@
         -->
         <!-- 3D lidar -->
-        <xacro:sensor_rs_bpearl prefix="${prefix}front_3d_laser" parent="${prefix}chassis_link" prefix_topic="front_3d_laser" suffix_topic="pcl" range_min="0.1" range_max="90" hfov="360" samples="1200" vfov="90.0" lasers="32" fps="15" gpu="${gpu}">
+        <xacro:sensor_rs_bpearl prefix="${prefix}front_3d_laser" parent="${prefix}chassis_link" prefix_topic="front_3d_laser" range_min="0.1" range_max="90" hfov="360" samples="1200" vfov="90.0" lasers="32" fps="15" gpu="${gpu}">
             <origin xyz="0.579 0 0.241" rpy="0 ${90*PI/180} 0"/>
         </xacro:sensor_rs_bpearl>

File: rbvogui_description/urdf/bases/rbvogui_xl_base.urdf.xacro (robot description, xacro)
@@ -37,5 +37,5 @@
         <origin xyz="0 0 0.376" />
         <!--inertia ixx="1.0" ixy="0.0" ixz="0.0" iyy="1.0" iyz="0.0" izz="1.0" /-->
-        <xacro:solid_cuboid_inertia  w="1.265" h="0.812" d="0.465" m="25"/>
+        <solid_cuboid_inertia  w="1.265" h="0.812" d="0.465" m="25"/>
       </inertial>
       <visual>

File: rbvogui_description/urdf/structures/bi_arm_support.urdf.xacro (robot description, xacro)
@@ -30,5 +30,5 @@
         <mass value="5" />
         <origin xyz="0 0 0" rpy="0 0 ${M_PI/2.0}"/>
-        <xacro:solid_cuboid_inertia  w="0.4" h="0.4" d="0.2" m="5"/>
+        <solid_cuboid_inertia  w="0.4" h="0.4" d="0.2" m="5"/>
       </inertial>
     </link>

File: rbvogui_description/urdf/structures/sick_protector.urdf.xacro (robot description, xacro)
@@ -31,5 +31,5 @@
         <mass value="5" />
         <origin xyz="0 0 0" rpy="0 0 ${M_PI/2.0}"/>
-        <xacro:solid_cuboid_inertia  w="0.4" h="0.4" d="0.2" m="5"/>
+        <solid_cuboid_inertia  w="0.4" h="0.4" d="0.2" m="5"/>
       </inertial>
     </link>

File: rbvogui_description/urdf/structures/sick_support.urdf.xacro (robot description, xacro)
@@ -31,5 +31,5 @@
         <mass value="5" />
         <origin xyz="0 0 0" rpy="0 0 ${M_PI/2.0}"/>
-        <xacro:solid_cuboid_inertia  w="0.4" h="0.4" d="0.2" m="5"/>
+        <solid_cuboid_inertia  w="0.4" h="0.4" d="0.2" m="5"/>
       </inertial>
     </link>

File: rbvogui_description/urdf/wheels/fixed_wheel.urdf.xacro (robot description, xacro)
@@ -140,5 +140,5 @@
         <mass value="${wheel_mass}" />
         <origin xyz="0 0 0" rpy="${M_PI/2} 0 0" />
-        <xacro:cylinder_inertia m="${wheel_mass}" r="${wheel_radius}" h="${wheel_height}" />
+        <cylinder_inertia m="${wheel_mass}" r="${wheel_radius}" h="${wheel_height}" />
       </inertial>
     </link>

File: rbvogui_description/urdf/wheels/fixed_wheel_xl.urdf.xacro (robot description, xacro)
@@ -69,11 +69,11 @@
         <mass value="4" />
         <xacro:if value="${reflect}">
-			    <origin xyz="0 0 0.12" rpy="0 0 ${M_PI}"/>
-		    </xacro:if>
-		    <xacro:unless value="${reflect}">
-			    <origin xyz="0 0 0.12" rpy="0 0 0"/>
-		    </xacro:unless>
+			<origin xyz="0 0 0.12" rpy="0 0 ${M_PI}"/>
+		</xacro:if>
+		<xacro:unless value="${reflect}">
+			<origin xyz="0 0 0.12" rpy="0 0 0"/>
+		</xacro:unless>
         <!-- To do: add real intertia-->
-        <xacro:cylinder_inertia m="5" r="0.1425" h="0.14"/>
+        <cylinder_inertia m="5" r="0.1425" h="0.14"/>
       </inertial>
     </link>

File: rbvogui_description/urdf/wheels/fixed_wheel_xl_offroad.urdf.xacro (robot description, xacro)
@@ -69,11 +69,11 @@
         <mass value="4" />
         <xacro:if value="${reflect}">
-			    <origin xyz="0 0 0.12" rpy="0 0 ${M_PI}"/>
-		    </xacro:if>
-		    <xacro:unless value="${reflect}">
-			    <origin xyz="0 0 0.12" rpy="0 0 0"/>
-		    </xacro:unless>
+			<origin xyz="0 0 0.12" rpy="0 0 ${M_PI}"/>
+		</xacro:if>
+		<xacro:unless value="${reflect}">
+			<origin xyz="0 0 0.12" rpy="0 0 0"/>
+		</xacro:unless>
         <!-- To do: add real intertia-->
-        <xacro:cylinder_inertia m="5" r="0.1425" h="0.14"/>
+        <cylinder_inertia m="5" r="0.1425" h="0.14"/>
       </inertial>
     </link>

File: rbvogui_description/urdf/wheels/motor_wheel.urdf.xacro (robot description, xacro)
@@ -93,5 +93,5 @@
           <origin xyz="0 0 0.0" rpy="0 0 ${M_PI}"/>
         </xacro:unless>
-        <xacro:cylinder_inertia m="${wheel_mass}" r="${wheel_radius}" h="${wheel_width}" />
+        <cylinder_inertia m="${wheel_mass}" r="${wheel_radius}" h="${wheel_width}" />
       </inertial>
     </link>
@@ -171,5 +171,5 @@
 			<origin xyz="0 0 0" rpy="${M_PI/2} 0 0" />
 		</xacro:unless>
-        <xacro:cylinder_inertia m="${wheel_mass}" r="${wheel_radius}" h="${wheel_width}" />
+        <cylinder_inertia m="${wheel_mass}" r="${wheel_radius}" h="${wheel_width}" />
       </inertial>
     </link>

File: rbvogui_description/urdf/wheels/motor_wheel_xl.urdf.xacro (robot description, xacro)
@@ -82,11 +82,11 @@
         <mass value="4" />
         <xacro:if value="${reflect}">
-			    <origin xyz="0 0 0.12" rpy="0 0 ${M_PI}"/>
-		    </xacro:if>
-		    <xacro:unless value="${reflect}">
-		    	<origin xyz="0 0 0.12" rpy="0 0 0"/>
-		    </xacro:unless>
+			<origin xyz="0 0 0.12" rpy="0 0 ${M_PI}"/>
+		</xacro:if>
+		<xacro:unless value="${reflect}">
+			<origin xyz="0 0 0.12" rpy="0 0 0"/>
+		</xacro:unless>
         <!-- To do: add real intertia-->
-        <xacro:cylinder_inertia m="5" r="0.1425" h="0.14"/>
+        <cylinder_inertia m="5" r="0.1425" h="0.14"/>
       </inertial>
     </link>

File: rbvogui_description/urdf/wheels/motor_wheel_xl_offroad.urdf.xacro (robot description, xacro)
@@ -82,11 +82,11 @@
         <mass value="4" />
         <xacro:if value="${reflect}">
-			    <origin xyz="0 0 0.12" rpy="0 0 ${M_PI}"/>
-		    </xacro:if>
-		    <xacro:unless value="${reflect}">
-			    <origin xyz="0 0 0.12" rpy="0 0 0"/>
-		    </xacro:unless>
+			<origin xyz="0 0 0.12" rpy="0 0 ${M_PI}"/>
+		</xacro:if>
+		<xacro:unless value="${reflect}">
+			<origin xyz="0 0 0.12" rpy="0 0 0"/>
+		</xacro:unless>
         <!-- To do: add real intertia-->
-        <xacro:cylinder_inertia m="5" r="0.1425" h="0.14"/>
+        <cylinder_inertia m="5" r="0.1425" h="0.14"/>
       </inertial>
     </link>

File: rbvogui_description/urdf/wheels/rubber_wheel.urdf.xacro (robot description, xacro)
@@ -76,5 +76,5 @@
         <mass value="${wheel_mass}" />
         <origin xyz="0 0 0" />
-        <xacro:cylinder_inertia m="${wheel_mass}" r="${wheel_radius}" h="${wheel_height}" />
+        <cylinder_inertia m="${wheel_mass}" r="${wheel_radius}" h="${wheel_height}" />
       </inertial>
     </link>

File: rbvogui_description/urdf/wheels/rubber_wheel_285mm.urdf.xacro (robot description, xacro)
@@ -79,5 +79,5 @@
         <mass value="${wheel_mass}" />
         <origin xyz="0 0 0" />
-        <xacro:cylinder_inertia m="${wheel_mass}" r="${wheel_radius}" h="${wheel_height}" />
+        <cylinder_inertia m="${wheel_mass}" r="${wheel_radius}" h="${wheel_height}" />
       </inertial>
     </link>

File: rbvogui_description/urdf/wheels/rubber_wheel_350mm.urdf.xacro (robot description, xacro)
@@ -79,5 +79,5 @@
         <mass value="${wheel_mass}" />
         <origin xyz="0 0 0" />
-        <xacro:cylinder_inertia m="${wheel_mass}" r="${wheel_radius}" h="${wheel_height}" />
+        <cylinder_inertia m="${wheel_mass}" r="${wheel_radius}" h="${wheel_height}" />
       </inertial>
     </link>
