Commit message: Change default orientation of the steering motor on std rbvogui

File: rbvogui_description/robots/rbvogui_std.urdf.xacro (robot description, xacro)
@@ -32,9 +32,9 @@
             <origin xyz="${wheel_offset_x} -${wheel_offset_y} ${wheel_offset_z}" rpy="0 0 0"/>
         </xacro:motor_wheel>
-        <xacro:motor_wheel prefix="${prefix}front_left_" parent="${prefix}base_link" reflect="false" hq="true">
-            <origin xyz="${wheel_offset_x} ${wheel_offset_y} ${wheel_offset_z}" rpy="0 0 ${180.0*deg2rad}"/>
+        <xacro:motor_wheel prefix="${prefix}front_left_" parent="${prefix}base_link" reflect="true" hq="true">
+            <origin xyz="${wheel_offset_x} ${wheel_offset_y} ${wheel_offset_z}" rpy="0 0 0"/>
         </xacro:motor_wheel>
-        <xacro:motor_wheel prefix="${prefix}back_left_" parent="${prefix}base_link" reflect="false" hq="true">
-            <origin xyz="-${wheel_offset_x} ${wheel_offset_y} ${wheel_offset_z}" rpy="0 0 ${180.0*deg2rad}"/>
+        <xacro:motor_wheel prefix="${prefix}back_left_" parent="${prefix}base_link" reflect="true" hq="true">
+            <origin xyz="-${wheel_offset_x} ${wheel_offset_y} ${wheel_offset_z}" rpy="0 0 0"/>
         </xacro:motor_wheel>
         <xacro:motor_wheel prefix="${prefix}back_right_" parent="${prefix}base_link" reflect="false" hq="true">

File: rbvogui_description/urdf/wheels/motor_wheel.urdf.xacro (robot description, xacro)
@@ -5,5 +5,5 @@
   <!-- Wheels -->
   <xacro:property name="wheel_radius" value="0.110" />
-  <xacro:property name="wheel_height" value="0.110" />
+  <xacro:property name="wheel_width" value="0.110" />
   <xacro:property name="wheel_mass" value="5.0" />
   <!-- in kg-->
@@ -47,42 +47,47 @@
         <!-- HIGH RESOLUTION WHEELS -->
         <xacro:if value="${hq}">
-          <origin xyz="0 0 0" rpy="0 0 3.1416" />
+		  <xacro:if value="${reflect}">
+			<origin xyz="0 0 0.0" rpy="0 0 0" />
+		  </xacro:if>
+		  <xacro:unless value="${reflect}">
+			<origin xyz="0 0 0.0" rpy="0 0 ${M_PI}" />
+		  </xacro:unless>
           <geometry>
-            <xacro:if value="${reflect}">
-              <mesh filename="package://rbvogui_description/meshes/wheels/mw_frame.dae" />
-            </xacro:if>
-            <xacro:unless value="${reflect}">
-              <mesh filename="package://rbvogui_description/meshes/wheels/mw_frame.dae" />
-            </xacro:unless>
+            <mesh filename="package://rbvogui_description/meshes/wheels/mw_frame.dae" />
           </geometry>
         </xacro:if>
         <!-- LOW RESOLUTION WHEELS -->
         <xacro:unless value="${hq}">
-          <origin xyz="0 0 0" rpy="0 0 3.1416" />
+          <xacro:if value="${reflect}">
+			<origin xyz="0 0 0.0" rpy="0 0 0" />
+		  </xacro:if>
+		  <xacro:unless value="${reflect}">
+			<origin xyz="0 0 0.0" rpy="0 0 ${M_PI}" />
+		  </xacro:unless>
           <geometry>
-            <xacro:if value="${reflect}">
-              <mesh filename="package://rbvogui_description/meshes/wheels/mw_frame.stl" />
-            </xacro:if>
-            <xacro:unless value="${reflect}">
-              <mesh filename="package://rbvogui_description/meshes/wheels/mw_frame.stl" />
-            </xacro:unless>
+            <mesh filename="package://rbvogui_description/meshes/wheels/mw_frame.stl" />
           </geometry>
         </xacro:unless>
       </visual>
       <collision>
-        <origin xyz="0 0 0" rpy="0 0 3.1416" />
-        <geometry>
-          <xacro:if value="${reflect}">
-            <mesh filename="package://rbvogui_description/meshes/wheels/mw_frame.dae" />
-          </xacro:if>
-          <xacro:unless value="${reflect}">
-            <mesh filename="package://rbvogui_description/meshes/wheels/mw_frame.dae" />
-          </xacro:unless>
-        </geometry>
+		  <xacro:if value="${reflect}">
+			<origin xyz="0 0 0.0" rpy="0 0 0" />
+		  </xacro:if>
+		  <xacro:unless value="${reflect}">
+			<origin xyz="0 0 0.0" rpy="0 0 ${M_PI}" />
+		  </xacro:unless>
+		  <geometry>
+			<mesh filename="package://rbvogui_description/meshes/wheels/mw_frame.dae" />
+		  </geometry>
       </collision>
       <inertial>
-        <mass value="10" />
-        <origin xyz="0 0 0" />
-        <inertia ixx="0.01" ixy="0.0" ixz="0.0" iyy="0.01" iyz="0.0" izz="0.01" />
+        <mass value="4" />
+        <xacro:if value="${reflect}">
+			<origin xyz="0 0 0.0" rpy="0 0 0"/>
+		</xacro:if>
+		<xacro:unless value="${reflect}">
+			<origin xyz="0 0 0.0" rpy="0 0 ${M_PI}"/>
+		</xacro:unless>
+        <cylinder_inertia m="${wheel_mass}" r="${wheel_radius}" h="${wheel_width}" />
       </inertial>
     </link>
@@ -91,6 +96,11 @@
       <parent link="${prefix}motor_wheel"/>
       <child link="${prefix}wheel"/>
-      <origin xyz="0 0 0" rpy="0 0 ${M_PI}" />
-      <axis xyz="0 1 0" rpy="0 0 0" />
+      <origin xyz="0 0 0" rpy="0 0 0" />
+      <xacro:if value="${reflect}">
+		<axis xyz="0 1 0" rpy="0 0 0" />
+	  </xacro:if>
+      <xacro:unless value="${reflect}">
+		<axis xyz="0 1 0" rpy="0 0 0" />
+	  </xacro:unless>
       <limit effort="${wheel_joint_effort_limit}" velocity="${wheel_joint_velocity_limit}"/>
       <joint_properties damping="${wheel_joint_damping}" friction="{wheel_joint_friction}"/>
@@ -110,24 +120,34 @@
         <!-- HIGH RESOLUTION WHEELS -->
         <xacro:if value="${hq}">
-          <origin xyz="0 0 0" rpy="0 0 0" />
+		  <xacro:if value="${reflect}">
+			<origin xyz="0 0 0" rpy="0 0 0" />
+		  </xacro:if>
+		  <xacro:unless value="${reflect}">
+			<origin xyz="0 0 0" rpy="0 0 0" />
+		  </xacro:unless>
           <geometry>
-            <xacro:if value="${reflect}">
               <mesh filename="package://rbvogui_description/meshes/wheels/wheel_sxl.dae" />
-            </xacro:if>
-            <xacro:unless value="${reflect}">
-              <mesh filename="package://rbvogui_description/meshes/wheels/wheel_sxl.dae" />
-            </xacro:unless>
           </geometry>
         </xacro:if>
         <!-- LOW RESOLUTION WHEELS -->
         <xacro:unless value="${hq}">
-          <origin xyz="0 0 0" rpy="${M_PI/2} 0 0" />
+           <xacro:if value="${reflect}">
+			<origin xyz="0 0 0" rpy="0 0 0" />
+		  </xacro:if>
+		  <xacro:unless value="${reflect}">
+			<origin xyz="0 0 0" rpy="0 0 0" />
+		  </xacro:unless>
           <geometry>
-            <cylinder length="${wheel_height}" radius="${wheel_radius}" />
+            <cylinder length="${wheel_width}" radius="${wheel_radius}" />
           </geometry>
         </xacro:unless>
       </visual>
       <collision>
-        <origin xyz="0 0 0" rpy="${M_PI/2} 0 0" />
+        <xacro:if value="${reflect}">
+		  <origin xyz="0 0 0" rpy="0 0 0" />
+		</xacro:if>
+		<xacro:unless value="${reflect}">
+			<origin xyz="0 0 0" rpy="0 0 0" />
+		</xacro:unless>
         <geometry>
           <sphere radius="${wheel_radius}" />
@@ -136,6 +156,11 @@
       <inertial>
         <mass value="${wheel_mass}" />
-        <origin xyz="0 0 0" rpy="${M_PI/2} 0 0" />
-        <cylinder_inertia m="${wheel_mass}" r="${wheel_radius}" h="${wheel_height}" />
+        <xacro:if value="${reflect}">
+			<origin xyz="0 0 0" rpy="${M_PI/2} 0 0" />
+		</xacro:if>
+		<xacro:unless value="${reflect}">
+			<origin xyz="0 0 0" rpy="${M_PI/2} 0 0" />
+		</xacro:unless>
+        <cylinder_inertia m="${wheel_mass}" r="${wheel_radius}" h="${wheel_width}" />
       </inertial>
     </link>

File: rbvogui_description/urdf/wheels/motor_wheel_xl.urdf.xacro (robot description, xacro)
@@ -22,5 +22,4 @@
   </xacro:macro>
   <xacro:macro name="motor_wheel" params="prefix parent *origin reflect hq">
-    <!-- TODO: check reflect parameter -->
     <!--MOTOR WHEEL -->
     <joint name="${prefix}motor_wheel_joint" type="revolute">

Commit message: Add load_kinematics_file argument in all versions - Compatibility with UR arms option

File: rbvogui_description/robots/rbvogui_std.urdf.xacro (robot description, xacro)
@@ -23,5 +23,6 @@
     <xacro:property name="publish_bf" value="true" />
     <xacro:arg name="prefix" default="robot_" />
-    <xacro:macro name="rbvogui" params="prefix publish_bf hq">
+    <xacro:arg name="load_kinematics_file" default="false"/>
+    <xacro:macro name="rbvogui" params="prefix publish_bf hq load_kinematics_file">
         <!-- *************** -->
         <!-- Robots Elements -->
@@ -50,15 +51,11 @@
             <origin xyz="-0.04625 0.0 1.115" rpy="0 0 0"/>
         </xacro:sensor_gps>
-        <!-- Solid-State laser -->
-        <xacro:sensor_benewake_ce30c prefix="${prefix}front_ss_laser" parent="${prefix}base_link" gpu="false">
-            <origin xyz="0.5657 0.0 0.1622" rpy="0 0 0"/>
-        </xacro:sensor_benewake_ce30c>
         <!-- 2d laser -->
-        <xacro:sensor_sick_tim551 prefix="${prefix}front_laser" parent="${prefix}base_link" prefix_topic="front_laser">
+        <xacro:sensor_sick_outdoorscan3 prefix="${prefix}front_laser" parent="${prefix}base_link" prefix_topic="front_laser">
             <origin xyz="0.5307 0.0 0.15389" rpy="${180*deg2rad} 0 0"/>
-        </xacro:sensor_sick_tim551>
+        </xacro:sensor_sick_outdoorscan3>
     </xacro:macro>
     <!-- Gazebo ros control pluggins -->
     <xacro:ros_control/>
-    <xacro:rbvogui prefix="$(arg prefix)" publish_bf="${publish_bf}" hq="${hq}"/>
+    <xacro:rbvogui prefix="$(arg prefix)" load_kinematics_file="$(arg load_kinematics_file)" publish_bf="${publish_bf}" hq="${hq}"/>
 </robot>

File: rbvogui_description/robots/rbvogui_std_ur10.urdf.xacro (robot description, xacro)
@@ -44,9 +44,9 @@
             <origin xyz="${wheel_offset_x} -${wheel_offset_y} ${wheel_offset_z}" rpy="0 0 0"/>
         </xacro:motor_wheel>
-        <xacro:motor_wheel prefix="${prefix}front_left_" parent="${prefix}base_link" reflect="false" hq="${hq}">
-            <origin xyz="${wheel_offset_x} ${wheel_offset_y} ${wheel_offset_z}" rpy="0 0 ${180.0*deg2rad}"/>
+        <xacro:motor_wheel prefix="${prefix}front_left_" parent="${prefix}base_link" reflect="true" hq="${hq}">
+            <origin xyz="${wheel_offset_x} ${wheel_offset_y} ${wheel_offset_z}" rpy="0 0 0"/>
         </xacro:motor_wheel>
-        <xacro:motor_wheel prefix="${prefix}back_left_" parent="${prefix}base_link" reflect="false" hq="${hq}">
-            <origin xyz="-${wheel_offset_x} ${wheel_offset_y} ${wheel_offset_z}" rpy="0 0 ${180.0*deg2rad}"/>
+        <xacro:motor_wheel prefix="${prefix}back_left_" parent="${prefix}base_link" reflect="true" hq="${hq}">
+            <origin xyz="-${wheel_offset_x} ${wheel_offset_y} ${wheel_offset_z}" rpy="0 0 0"/>
         </xacro:motor_wheel>
         <xacro:motor_wheel prefix="${prefix}back_right_" parent="${prefix}base_link" reflect="false" hq="${hq}">

File: rbvogui_description/robots/rbvogui_std_v2.urdf.xacro (robot description, xacro)
@@ -23,4 +23,5 @@
     <xacro:property name="publish_bf" value="true" />
     <xacro:arg name="prefix" default="robot_" />
+    <xacro:arg name="load_kinematics_file" default="false"/>
     <xacro:macro name="rbvogui" params="prefix publish_bf hq">
         <!-- *************** -->
@@ -32,9 +33,9 @@
             <origin xyz="${wheel_offset_x} -${wheel_offset_y} ${wheel_offset_z}" rpy="0 0 0"/>
         </xacro:motor_wheel>
-        <xacro:motor_wheel prefix="${prefix}front_left_" parent="${prefix}base_link" reflect="false" hq="${hq}">
-            <origin xyz="${wheel_offset_x} ${wheel_offset_y} ${wheel_offset_z}" rpy="0 0 ${180.0*deg2rad}"/>
+        <xacro:motor_wheel prefix="${prefix}front_left_" parent="${prefix}base_link" reflect="true" hq="${hq}">
+            <origin xyz="${wheel_offset_x} ${wheel_offset_y} ${wheel_offset_z}" rpy="0 0 0"/>
         </xacro:motor_wheel>
-        <xacro:motor_wheel prefix="${prefix}back_left_" parent="${prefix}base_link" reflect="false" hq="${hq}">
-            <origin xyz="-${wheel_offset_x} ${wheel_offset_y} ${wheel_offset_z}" rpy="0 0 ${180.0*deg2rad}"/>
+        <xacro:motor_wheel prefix="${prefix}back_left_" parent="${prefix}base_link" reflect="true" hq="${hq}">
+            <origin xyz="-${wheel_offset_x} ${wheel_offset_y} ${wheel_offset_z}" rpy="0 0 0"/>
         </xacro:motor_wheel>
         <xacro:motor_wheel prefix="${prefix}back_right_" parent="${prefix}base_link" reflect="false" hq="${hq}">
@@ -61,4 +62,4 @@
     <!-- Gazebo ros control pluggins -->
     <xacro:ros_control/>
-    <xacro:rbvogui prefix="$(arg prefix)" publish_bf="${publish_bf}" hq="${hq}"/>
+    <xacro:rbvogui prefix="$(arg prefix)" load_kinematics_file="$(arg load_kinematics_file)" publish_bf="${publish_bf}" hq="${hq}"/>
 </robot>

File: rbvogui_description/robots/rbvogui_std_v3.urdf.xacro (robot description, xacro)
@@ -23,4 +23,5 @@
     <xacro:property name="publish_bf" value="true" />
     <xacro:arg name="prefix" default="robot_" />
+    <xacro:arg name="load_kinematics_file" default="false"/>
     <xacro:macro name="rbvogui" params="prefix publish_bf hq">
         <!-- *************** -->
@@ -32,9 +33,9 @@
             <origin xyz="${wheel_offset_x} -${wheel_offset_y} ${wheel_offset_z}" rpy="0 0 0"/>
         </xacro:motor_wheel>
-        <xacro:motor_wheel prefix="${prefix}front_left_" parent="${prefix}base_link" reflect="false" hq="${hq}">
-            <origin xyz="${wheel_offset_x} ${wheel_offset_y} ${wheel_offset_z}" rpy="0 0 ${180.0*deg2rad}"/>
+        <xacro:motor_wheel prefix="${prefix}front_left_" parent="${prefix}base_link" reflect="true" hq="${hq}">
+            <origin xyz="${wheel_offset_x} ${wheel_offset_y} ${wheel_offset_z}" rpy="0 0 0"/>
         </xacro:motor_wheel>
-        <xacro:motor_wheel prefix="${prefix}back_left_" parent="${prefix}base_link" reflect="false" hq="${hq}">
-            <origin xyz="-${wheel_offset_x} ${wheel_offset_y} ${wheel_offset_z}" rpy="0 0 ${180.0*deg2rad}"/>
+        <xacro:motor_wheel prefix="${prefix}back_left_" parent="${prefix}base_link" reflect="true" hq="${hq}">
+            <origin xyz="-${wheel_offset_x} ${wheel_offset_y} ${wheel_offset_z}" rpy="0 0 0"/>
         </xacro:motor_wheel>
         <xacro:motor_wheel prefix="${prefix}back_right_" parent="${prefix}base_link" reflect="false" hq="${hq}">
@@ -61,4 +62,4 @@
     <!-- Gazebo ros control pluggins -->
     <xacro:ros_control/>
-    <xacro:rbvogui prefix="$(arg prefix)" publish_bf="${publish_bf}" hq="${hq}"/>
+    <xacro:rbvogui prefix="$(arg prefix)" load_kinematics_file="$(arg load_kinematics_file)" publish_bf="${publish_bf}" hq="${hq}"/>
 </robot>

File: rbvogui_description/robots/rbvogui_ur5e.urdf.xacro (robot description, xacro)
@@ -32,6 +32,6 @@
     <xacro:property name="publish_bf" value="true" />
     <xacro:arg name="prefix" default="robot_" />
-    <xacro:arg name="kinematics_config" default="$(find ur_e_description)/config/ur5e_default.yaml"/>
-    <xacro:macro name="rbvogui" params="prefix publish_bf hq">
+    <xacro:arg name="load_kinematics_file" default="false"/>
+    <xacro:macro name="rbvogui" params="prefix publish_bf hq load_kinematics_file">
         <!-- *************** -->
         <!-- Robots Elements -->
@@ -39,10 +39,19 @@
         <!-- Here we create the robot elements using the xacro:macros imported at the beggining of this file -->
     <xacro:rbvogui_base prefix="${prefix}" publish_bf="${publish_bf}" hq="${hq}"/>
-    <!-- Ur5 Arm -->
-    <xacro:ur5e_robot prefix="$(arg prefix)arm_" joint_limited="false"
-        shoulder_pan_lower_limit="${-pi}" shoulder_pan_upper_limit="${pi}"
-        wrist_3_lower_limit="${-pi}" wrist_3_upper_limit="${pi}"
-        kinematics_file="${load_yaml('$(arg kinematics_config)')}">
-    </xacro:ur5e_robot>
+    <xacro:if value="${load_kinematics_file}">
+		<!-- Ur5 Arm -->
+		<xacro:ur5e_robot prefix="$(arg prefix)arm_" joint_limited="false"
+			shoulder_pan_lower_limit="${-pi}" shoulder_pan_upper_limit="${pi}"
+			wrist_3_lower_limit="${-pi}" wrist_3_upper_limit="${pi}"
+			kinematics_file="${load_yaml('$(find rbvogui_control)/config/calibration/ur10_calibration.yaml')}">
+		</xacro:ur5e_robot>
+	</xacro:if>
+    <xacro:unless value="${load_kinematics_file}">
+		<!-- Ur5 Arm -->
+		<xacro:ur5e_robot prefix="$(arg prefix)arm_" joint_limited="false"
+			shoulder_pan_lower_limit="${-pi}" shoulder_pan_upper_limit="${pi}"
+			wrist_3_lower_limit="${-pi}" wrist_3_upper_limit="${pi}">
+		</xacro:ur5e_robot>
+	</xacro:unless>
     <joint name="$(arg prefix)arm_base_joint" type="fixed">
         <origin xyz="0.1815 0.0 0.4405" rpy="0 0 -1.57"/>
@@ -62,9 +71,9 @@
         <origin xyz="${wheel_offset_x} -${wheel_offset_y} ${wheel_offset_z}" rpy="0 0 0"/>
     </xacro:motor_wheel>
-    <xacro:motor_wheel prefix="${prefix}front_left_" parent="${prefix}base_link" reflect="false" hq="true">
-        <origin xyz="${wheel_offset_x} ${wheel_offset_y} ${wheel_offset_z}" rpy="0 0 ${180.0*deg2rad}"/>
+    <xacro:motor_wheel prefix="${prefix}front_left_" parent="${prefix}base_link" reflect="true" hq="true">
+        <origin xyz="${wheel_offset_x} ${wheel_offset_y} ${wheel_offset_z}" rpy="0 0 0"/>
     </xacro:motor_wheel>
-    <xacro:motor_wheel prefix="${prefix}back_left_" parent="${prefix}base_link" reflect="false" hq="true">
-        <origin xyz="-${wheel_offset_x} ${wheel_offset_y} ${wheel_offset_z}" rpy="0 0 ${180.0*deg2rad}"/>
+    <xacro:motor_wheel prefix="${prefix}back_left_" parent="${prefix}base_link" reflect="true" hq="true">
+        <origin xyz="-${wheel_offset_x} ${wheel_offset_y} ${wheel_offset_z}" rpy="0 0 0"/>
     </xacro:motor_wheel>
     <xacro:motor_wheel prefix="${prefix}back_right_" parent="${prefix}base_link" reflect="false" hq="true">
@@ -101,4 +110,4 @@
     <!-- Gazebo ros control pluggins -->
     <xacro:ros_control/>
-    <xacro:rbvogui prefix="$(arg prefix)" publish_bf="${publish_bf}" hq="${hq}"/>
+    <xacro:rbvogui prefix="$(arg prefix)" load_kinematics_file="$(arg load_kinematics_file)" publish_bf="${publish_bf}" hq="${hq}"/>
 </robot>

File: rbvogui_description/robots/rbvogui_xl_lift_ur10e.urdf.xacro (robot description, xacro)
@@ -36,5 +36,6 @@
     <xacro:arg name="kinematics_config" default="$(find rbvogui_control)/config/calibration/ur10e_default.yaml"/>
     <xacro:arg name="gpu" default="false" />
-    <xacro:macro name="rbvogui" params="prefix publish_bf hq gpu">
+    <xacro:arg name="load_kinematics_file" default="false" />
+    <xacro:macro name="rbvogui" params="prefix publish_bf hq gpu load_kinematics_file">
         <!-- *************** -->
         <!-- Robots Elements -->
@@ -59,8 +60,15 @@
         </xacro:ewellix_lift_900mm>
         <!-- UR-10e ARM -->
-        <xacro:ur10e_robot prefix="${prefix}arm_" joint_limited="true" shoulder_pan_lower_limit="${-pi}"
-                        shoulder_pan_upper_limit="${pi}" wrist_3_lower_limit="${-pi}" wrist_3_upper_limit="${pi}"
-                        kinematics_file="${load_yaml('$(arg kinematics_config)')}">>
-        </xacro:ur10e_robot>
+        <xacro:if value="${load_kinematics_file}">
+			<xacro:ur10e_robot prefix="${prefix}arm_" joint_limited="true" shoulder_pan_lower_limit="${-pi}"
+							shoulder_pan_upper_limit="${pi}" wrist_3_lower_limit="${-pi}" wrist_3_upper_limit="${pi}"
+							kinematics_file="${load_yaml('$(arg kinematics_config)')}">
+			</xacro:ur10e_robot>
+		</xacro:if>
+        <xacro:unless value="${load_kinematics_file}">
+			<xacro:ur10e_robot prefix="${prefix}arm_" joint_limited="true" shoulder_pan_lower_limit="${-pi}"
+							shoulder_pan_upper_limit="${pi}" wrist_3_lower_limit="${-pi}" wrist_3_upper_limit="${pi}">
+			</xacro:ur10e_robot>
+		</xacro:unless>
         <joint name="${prefix}arm_base_joint" type="fixed">
             <origin xyz="0 0 0.015" rpy="0 0 0"/>
@@ -109,4 +117,4 @@
     <!-- Gazebo ros control pluggins -->
     <xacro:ros_control/>
-    <xacro:rbvogui prefix="$(arg prefix)" publish_bf="${publish_bf}" hq="${hq}" gpu="$(arg gpu)"/>
+    <xacro:rbvogui prefix="$(arg prefix)" load_kinematics_file="$(arg load_kinematics_file)" publish_bf="${publish_bf}" hq="${hq}" gpu="$(arg gpu)"/>
 </robot>

Commit message: description: Update urdf for the standard rbvogui:      - Set tim551 as default laser      - Add benewake sensor      - Add gpu param

File: rbvogui_description/robots/rbvogui_std.urdf.xacro (robot description, xacro)
@@ -23,6 +23,7 @@
     <xacro:property name="publish_bf" value="true" />
     <xacro:arg name="prefix" default="robot_" />
+    <xacro:arg name="gpu" default="true" />
     <xacro:arg name="load_kinematics_file" default="false"/>
-    <xacro:macro name="rbvogui" params="prefix publish_bf hq load_kinematics_file">
+    <xacro:macro name="rbvogui" params="prefix publish_bf hq load_kinematics_file gpu">
         <!-- *************** -->
         <!-- Robots Elements -->
@@ -49,13 +50,17 @@
         <!-- GPS -->
         <xacro:sensor_gps prefix="${prefix}gps" parent="${prefix}base_link">
-            <origin xyz="-0.04625 0.0 1.115" rpy="0 0 0"/>
+            <origin xyz="-0.04625 0.0 0.4" rpy="0 0 0"/>
         </xacro:sensor_gps>
         <!-- 2d laser -->
-        <xacro:sensor_sick_outdoorscan3 prefix="${prefix}front_laser" parent="${prefix}base_link" prefix_topic="front_laser">
-            <origin xyz="0.5307 0.0 0.15389" rpy="${180*deg2rad} 0 0"/>
-        </xacro:sensor_sick_outdoorscan3>
+        <xacro:sensor_sick_tim551 prefix="$(arg prefix)front_laser" parent="${prefix}base_link" gpu="${gpu}" min_angle="${-PI/2}" max_angle="${PI/2}" prefix_topic="front_laser">
+            <origin xyz="0.53 0.0 0.153" rpy="${PI} 0 0"/>
+        </xacro:sensor_sick_tim551>
+        <!-- Front 3d laser -->
+        <xacro:sensor_benewake_ce30c prefix="$(arg prefix)front_3d_laser" parent="${prefix}base_link"  gpu="${gpu}" prefix_topic="front_3d_laser">
+            <origin xyz="0.59 0 0.189" rpy="0 0 0"/>
+        </xacro:sensor_benewake_ce30c>
     </xacro:macro>
     <!-- Gazebo ros control pluggins -->
     <xacro:ros_control/>
-    <xacro:rbvogui prefix="$(arg prefix)" load_kinematics_file="$(arg load_kinematics_file)" publish_bf="${publish_bf}" hq="${hq}"/>
+    <xacro:rbvogui prefix="$(arg prefix)" load_kinematics_file="$(arg load_kinematics_file)" gpu="$(arg gpu)" publish_bf="${publish_bf}" hq="${hq}"/>
 </robot>

Commit message: rbvogui_description: Remove benewake for standard rbvogui

File: rbvogui_description/robots/rbvogui_std.urdf.xacro (robot description, xacro)
@@ -53,11 +53,7 @@
         </xacro:sensor_gps>
         <!-- 2d laser -->
-        <xacro:sensor_sick_tim551 prefix="$(arg prefix)front_laser" parent="${prefix}base_link" gpu="${gpu}" min_angle="${-PI/2}" max_angle="${PI/2}" prefix_topic="front_laser">
+        <xacro:sensor_sick_tim551 prefix="${prefix}front_laser" parent="${prefix}base_link" gpu="${gpu}" min_angle="${-PI/2}" max_angle="${PI/2}" prefix_topic="front_laser">
             <origin xyz="0.53 0.0 0.153" rpy="${PI} 0 0"/>
         </xacro:sensor_sick_tim551>
-        <!-- Front 3d laser -->
-        <xacro:sensor_benewake_ce30c prefix="$(arg prefix)front_3d_laser" parent="${prefix}base_link"  gpu="${gpu}" prefix_topic="front_3d_laser">
-            <origin xyz="0.59 0 0.189" rpy="0 0 0"/>
-        </xacro:sensor_benewake_ce30c>
     </xacro:macro>
     <!-- Gazebo ros control pluggins -->
