Commit message: Fix some issues

File: rbvogui_description/robots/rbvogui_std.urdf.xacro (robot description, xacro)
@@ -78,4 +78,28 @@
         </xacro:sensor_rslidar_16>
         -->
+        <xacro:macro name="ros2_joint" params="interface jmin jmax prefix name">
+          <joint name="${prefix}${name}">
+            <command_interface name="${interface}">
+              <param name="min">${jmin}</param>
+              <param name="max">${jmax}</param>
+            </command_interface>
+            <state_interface name="position"/>
+            <state_interface name="velocity"/>
+            <state_interface name="effort"/>
+          </joint>
+        </xacro:macro>
+        <ros2_control name="GazeboSystem" type="system">
+          <hardware>
+              <plugin>gazebo_ros2_control/GazeboSystem</plugin>
+          </hardware>
+          <xacro:ros2_joint interface="position" jmin="-2" jmax="2" prefix="${prefix}" name="front_left_motor_wheel_joint"/>
+          <xacro:ros2_joint interface="position" jmin="-2" jmax="2" prefix="${prefix}" name="front_right_motor_wheel_joint"/>
+          <xacro:ros2_joint interface="position" jmin="-2" jmax="2" prefix="${prefix}" name="back_left_motor_wheel_joint"/>
+          <xacro:ros2_joint interface="position" jmin="-2" jmax="2" prefix="${prefix}" name="back_right_motor_wheel_joint"/>
+          <xacro:ros2_joint interface="velocity" jmin="-10" jmax="10" prefix="${prefix}" name="front_left_wheel_joint"/>
+          <xacro:ros2_joint interface="velocity" jmin="-10" jmax="10" prefix="${prefix}" name="front_right_wheel_joint"/>
+          <xacro:ros2_joint interface="velocity" jmin="-20" jmax="20" prefix="${prefix}" name="back_left_wheel_joint"/>
+          <xacro:ros2_joint interface="velocity" jmin="-20" jmax="20" prefix="${prefix}" name="back_right_wheel_joint"/>
+        </ros2_control>
     </xacro:macro>
     <!-- Gazebo ros control pluggins -->

File: rbvogui_description/urdf/bases/rbvogui_base.gazebo.xacro (robot description, xacro)
@@ -4,11 +4,11 @@
     <xacro:macro name="ros_control">
         <gazebo>
-            <plugin name="ros_control" filename="libgazebo_ros_control.so">
-                <!--<robotNamespace>/summit_xl</robotNamespace>-->
-                <robotParam>robot_description</robotParam>
-                <controlPeriod>0.001</controlPeriod>
-                <robotSimType>gazebo_ros_control/DefaultRobotHWSim</robotSimType>
-                <legacyModeNS>true</legacyModeNS>
-            </plugin>
+          <plugin name="ros_control" filename="libgazebo_ros2_control.so">
+            <namespace>$(arg robot_id)</namespace>
+            <parameters>$(arg config_controllers)</parameters>
+            <!--robot_param>robot_description</robot_param-->
+            <!--robot_param_node>robot_state_publisher</robot_param_node-->
+            <!--remaping>$(find rbvogui_description)/config/remapping.yaml</remaping-->
+          </plugin>
         </gazebo>
     </xacro:macro>

File: rbvogui_description/urdf/wheels/motor_wheel.urdf.xacro (robot description, xacro)
@@ -93,5 +93,5 @@
           <origin xyz="0 0 0.0" rpy="0 0 ${M_PI}"/>
         </xacro:unless>
-        <cylinder_inertia m="${wheel_mass}" r="${wheel_radius}" h="${wheel_width}" />
+        <xacro:cylinder_inertia m="${wheel_mass}" r="${wheel_radius}" h="${wheel_width}" />
       </inertial>
     </link>

File: rbvogui_description/urdf/wheels/rubber_wheel.urdf.xacro (robot description, xacro)
@@ -30,16 +30,6 @@
       <axis xyz="0 1 0" rpy="0 0 0" />
       <limit effort="${wheel_joint_effort_limit}" velocity="${wheel_joint_velocity_limit}"/>
-      <joint_properties damping="${wheel_joint_damping}" friction="{wheel_joint_friction}"/>
+      <dynamics damping="${wheel_joint_damping}" friction="${wheel_joint_friction}"/>
     </joint>
-    <transmission name="${prefix}wheel_trans">
-      <type>transmission_interface/SimpleTransmission</type>
-      <joint name="${prefix}wheel_joint">
-        <hardwareInterface>hardware_interface/VelocityJointInterface</hardwareInterface>
-      </joint>
-      <actuator name="${prefix}wheel_motor">
-        <hardwareInterface>hardware_interface/VelocityActuatorInterface</hardwareInterface>
-        <mechanicalReduction>${wheel_mechanical_reduction}</mechanicalReduction>
-      </actuator>
-    </transmission>
     <link name="${prefix}wheel">
       <visual>
@@ -70,5 +60,5 @@
         <origin xyz="0 0 0" rpy="${M_PI/2} 0 0" />
         <geometry>
-          <sphere radius="${wheel_radius}" />
+          <cylinder length="${wheel_radius}" radius="${wheel_radius}" />
         </geometry>
       </collision>
@@ -76,5 +66,5 @@
         <mass value="${wheel_mass}" />
         <origin xyz="0 0 0" />
-        <cylinder_inertia m="${wheel_mass}" r="${wheel_radius}" h="${wheel_height}" />
+        <xacro:cylinder_inertia m="${wheel_mass}" r="${wheel_radius}" h="${wheel_height}" />
       </inertial>
     </link>

File: rbvogui_description/urdf/wheels/wheel.gazebo.xacro (robot description, xacro)
@@ -4,8 +4,9 @@
   <xacro:macro name="gazebo_color_wheel" params="prefix">
     <gazebo reference="${prefix}wheel">
-      <mu1 value="1.0"/>
-      <mu2 value="1.0"/>
+      <mu1 value="0.85"/>
+      <mu2 value="0.68"/>
       <kp value="10000000.0" />
       <kd value="1.0" />
+      <fdir1>1 0 0</fdir1>
       <visual>
         <material>

Commit message: Fixed inertias and other stuff in rbvogui_std

File: rbvogui_description/robots/rbvogui_std.urdf.xacro (robot description, xacro)
@@ -9,5 +9,5 @@
     <xacro:include filename="$(find rbvogui_description)/urdf/bases/rbvogui_base.urdf.xacro" />
     <!-- Import rbvogui wheels -->
-    <xacro:include filename="$(find rbvogui_description)/urdf/wheels/motor_wheel.urdf.xacro" />
+    <xacro:include filename="$(find rbvogui_description)/urdf/wheels/steering_wheel.urdf.xacro" />
     <!-- Import rbvogui fix wheels -->
     <xacro:include filename="$(find rbvogui_description)/urdf/wheels/fixed_wheel.urdf.xacro" />
@@ -24,5 +24,6 @@
     <xacro:property name="hq" value="true" />
     <xacro:property name="publish_bf" value="true" />
-    <xacro:arg name="prefix" default="robot_" />
+    <xacro:arg name="robot_id" default="robot" />
+    <xacro:arg name="prefix" default="$(arg robot)_" />
     <xacro:arg name="gpu" default="true" />
     <xacro:arg name="kinematics" default="omni" />
@@ -34,23 +35,23 @@
         <!-- Here we create the robot elements using the xacro:macros imported at the beggining of this file -->
         <xacro:rbvogui_base prefix="${prefix}" publish_bf="${publish_bf}" hq="${hq}"/>
-        <xacro:motor_wheel prefix="${prefix}front_right_" parent="${prefix}base_link" reflect="false" hq="true">
+        <xacro:steering_wheel prefix="${prefix}front_right_" parent="${prefix}base_link" reflect="false" hq="true">
             <origin xyz="${wheel_offset_x} -${wheel_offset_y} ${wheel_offset_z}" rpy="0 0 0"/>
-        </xacro:motor_wheel>
-        <xacro:motor_wheel prefix="${prefix}front_left_" parent="${prefix}base_link" reflect="true" hq="true">
+        </xacro:steering_wheel>
+        <xacro:steering_wheel prefix="${prefix}front_left_" parent="${prefix}base_link" reflect="true" hq="true">
             <origin xyz="${wheel_offset_x} ${wheel_offset_y} ${wheel_offset_z}" rpy="0 0 0"/>
-        </xacro:motor_wheel>
+        </xacro:steering_wheel>
         <xacro:if value="${kinematics == 'omni'}">
-            <xacro:motor_wheel prefix="${prefix}rear_left_" parent="${prefix}base_link" reflect="true" hq="true">
+            <xacro:steering_wheel prefix="${prefix}back_left_" parent="${prefix}base_link" reflect="true" hq="true">
                 <origin xyz="-${wheel_offset_x} ${wheel_offset_y} ${wheel_offset_z}" rpy="0 0 0"/>
-            </xacro:motor_wheel>
-            <xacro:motor_wheel prefix="${prefix}rear_right_" parent="${prefix}base_link" reflect="false" hq="true">
+            </xacro:steering_wheel>
+            <xacro:steering_wheel prefix="${prefix}back_right_" parent="${prefix}base_link" reflect="false" hq="true">
                 <origin xyz="-${wheel_offset_x} -${wheel_offset_y} ${wheel_offset_z}" rpy="0 0 0"/>
-            </xacro:motor_wheel>
+            </xacro:steering_wheel>
         </xacro:if>
         <xacro:if value="${kinematics == 'ackermann'}">
-            <xacro:fixed_wheel prefix="${prefix}rear_left_" parent="${prefix}base_link" reflect="true" hq="true">
+            <xacro:fixed_wheel prefix="${prefix}back_left_" parent="${prefix}base_link" reflect="true" hq="true">
                 <origin xyz="-${wheel_offset_x} ${wheel_offset_y} ${wheel_offset_z}" rpy="0 0 0"/>
             </xacro:fixed_wheel>
-            <xacro:fixed_wheel prefix="${prefix}rear_right_" parent="${prefix}base_link" reflect="false" hq="true">
+            <xacro:fixed_wheel prefix="${prefix}back_right_" parent="${prefix}base_link" reflect="false" hq="true">
                 <origin xyz="-${wheel_offset_x} -${wheel_offset_y} ${wheel_offset_z}" rpy="0 0 0"/>
             </xacro:fixed_wheel>
@@ -58,17 +59,19 @@
         <!-- SENSORS see robotnik_sensors for the specific configuration -->
         <!-- IMU -->
-        <xacro:sensor_vectornav prefix="${prefix}imu" parent="${prefix}chassis_link">
+        <xacro:sensor_vectornav prefix="${prefix}imu" parent="${prefix}chassis_link" topic="/$(arg robot_id)/imu/data">
             <origin xyz="0.3 -0.3 0.0725" rpy="0 0 0"/>
         </xacro:sensor_vectornav>
-        <!-- Front Camera -->
+        <!-- Front Camera
         <xacro:sensor_orbbec_astra prefix="${prefix}front_rgbd_camera" parent="${prefix}chassis_link">
             <origin xyz="0.46462 0.0 0.18258" rpy="0 0 0"/>
         </xacro:sensor_orbbec_astra>
-        <!-- GPS -->
+        -->
+        <!-- GPS
         <xacro:sensor_ublox prefix="${prefix}gps" parent="${prefix}chassis_link">
             <origin xyz="-0.3875 0.34553 0.3965" rpy="0 0 0"/>
         </xacro:sensor_ublox>
+        -->
         <!-- 2d laser -->
-        <xacro:sensor_sick_tim551 prefix="${prefix}front_laser" parent="${prefix}chassis_link" gpu="${gpu}" min_angle="${-PI/2}" max_angle="${PI/2}" prefix_topic="front_laser">
+        <xacro:sensor_sick_tim551 prefix="${prefix}front_laser" parent="${prefix}chassis_link" gpu="${gpu}" min_angle="${-PI/2}" max_angle="${PI/2}" prefix_topic="/$(arg robot_id)/front_laser">
             <origin xyz="0.53 0.0 -0.0245" rpy="${PI} 0 0"/> <!-- Verificar X -->
         </xacro:sensor_sick_tim551>
@@ -93,12 +96,12 @@
               <plugin>gazebo_ros2_control/GazeboSystem</plugin>
           </hardware>
-          <xacro:ros2_joint interface="position" jmin="-2" jmax="2" prefix="${prefix}" name="front_left_motor_wheel_joint"/>
-          <xacro:ros2_joint interface="position" jmin="-2" jmax="2" prefix="${prefix}" name="front_right_motor_wheel_joint"/>
-          <xacro:ros2_joint interface="position" jmin="-2" jmax="2" prefix="${prefix}" name="rear_left_motor_wheel_joint"/>
-          <xacro:ros2_joint interface="position" jmin="-2" jmax="2" prefix="${prefix}" name="rear_right_motor_wheel_joint"/>
+          <xacro:ros2_joint interface="position" jmin="-2" jmax="2" prefix="${prefix}" name="front_left_steering_joint"/>
+          <xacro:ros2_joint interface="position" jmin="-2" jmax="2" prefix="${prefix}" name="front_right_steering_joint"/>
+          <xacro:ros2_joint interface="position" jmin="-2" jmax="2" prefix="${prefix}" name="back_left_steering_joint"/>
+          <xacro:ros2_joint interface="position" jmin="-2" jmax="2" prefix="${prefix}" name="back_right_steering_joint"/>
           <xacro:ros2_joint interface="velocity" jmin="-10" jmax="10" prefix="${prefix}" name="front_left_wheel_joint"/>
           <xacro:ros2_joint interface="velocity" jmin="-10" jmax="10" prefix="${prefix}" name="front_right_wheel_joint"/>
-          <xacro:ros2_joint interface="velocity" jmin="-20" jmax="20" prefix="${prefix}" name="rear_left_wheel_joint"/>
-          <xacro:ros2_joint interface="velocity" jmin="-20" jmax="20" prefix="${prefix}" name="rear_right_wheel_joint"/>
+          <xacro:ros2_joint interface="velocity" jmin="-20" jmax="20" prefix="${prefix}" name="back_left_wheel_joint"/>
+          <xacro:ros2_joint interface="velocity" jmin="-20" jmax="20" prefix="${prefix}" name="back_right_wheel_joint"/>
         </ros2_control>
     </xacro:macro>

File: rbvogui_description/urdf/bases/rbvogui_base.urdf.xacro (robot description, xacro)
@@ -5,15 +5,7 @@
     <!-- Robot mechanical and motor parameters -->
     <xacro:property name="PI" value="3.1415926535897931"/>
-    <xacro:property name="wheel_width" value="0.146" />
     <!-- BASE FOOTPRINT -->
     <xacro:if value="${publish_bf}">
-      <link name="${prefix}base_footprint">
-        <visual>
-          <origin xyz="0 0 0" rpy="0 0 0" />
-          <geometry>
-            <box size="0.001 0.001 0.001" />
-          </geometry>
-        </visual>
-      </link>
+      <link name="${prefix}base_footprint" />
       <joint name="${prefix}base_footprint_joint" type="fixed">
         <origin xyz="0 0 ${wheel_radius}" rpy="0 0 0" />
@@ -35,6 +27,6 @@
       <inertial>
         <mass value="25.0" />
-        <origin xyz="0 0 0" />
-        <inertia ixx="1.0" ixy="0.0" ixz="0.0" iyy="1.0" iyz="0.0" izz="1.0" />
+        <origin xyz="0 0 0.10" />
+        <xacro:solid_cuboid_inertia w="1.265" h="0.812" d="0.22" m="25.0"/>
       </inertial>
       <visual>
@@ -70,7 +62,7 @@
     <link name="${prefix}battery_link">
       <inertial>
-        <mass value="20.0" />
-        <origin xyz="0 0 0" />
-        <inertia ixx="1.0" ixy="0.0" ixz="0.0" iyy="1.0" iyz="0.0" izz="1.0" />
+        <mass value="45.0" />
+        <origin xyz="0 0 -0.05" />
+        <xacro:solid_cuboid_inertia w="0.265" h="0.112" d="0.06" m="45.0"/>
       </inertial>
       <visual>

File: rbvogui_description/urdf/wheels/rubber_wheel.urdf.xacro (robot description, xacro)
@@ -3,24 +3,17 @@
   <xacro:include filename="$(find rbvogui_description)/urdf/wheels/wheel.gazebo.xacro" />
   <xacro:property name="M_PI" value="3.1415926535897931" />
-  <!-- Wheels -->
-  <xacro:property name="wheel_radius" value="0.1165" /> <!-- rbvogui uses wheels with 0.233 m of diameter-->
-  <xacro:property name="wheel_height" value="0.1165" />
-  <xacro:property name="wheel_mass" value="5.0" />
   <!-- in kg-->
-  <xacro:property name="steer_joint_damping" value="2.0" />
-  <xacro:property name="steer_joint_friction" value="1.0" />
-  <xacro:property name="steer_joint_effort_limit" value="100.0" />
-  <xacro:property name="steer_joint_velocity_limit" value="2.83" />
-  <xacro:property name="motor_wheel_mechanical_reduction" value="1.0" />
-  <xacro:property name="wheel_joint_damping" value="0.1" />
-  <xacro:property name="wheel_joint_friction" value="0.1" />
-  <xacro:property name="wheel_joint_effort_limit" value="1000.0" />
-  <xacro:property name="wheel_joint_velocity_limit" value="2000.0" />
-  <xacro:property name="wheel_mechanical_reduction" value="1.0" />
   <xacro:macro name="cylinder_inertia" params="m r h">
     <inertia ixx="${m*(3*r*r+h*h)/12}" ixy = "0" ixz = "0" iyy="${m*(3*r*r+h*h)/12}" iyz = "0" izz="${m*r*r/2}" />
   </xacro:macro>
   <xacro:macro name="wheel" params="prefix parent *origin reflect hq">
-    <!-- TODO: check reflect parameter -->
+    <!-- Wheels -->
+    <xacro:property name="wheel_radius" value="0.1165" /> <!-- rbvogui uses wheels with 0.233 m of diameter-->
+    <xacro:property name="wheel_width" value="0.1375" />
+    <xacro:property name="wheel_mass" value="5.0" />
+    <xacro:property name="wheel_joint_damping" value="0.5" />
+    <xacro:property name="wheel_joint_friction" value="2.0" />
+    <xacro:property name="wheel_joint_effort_limit" value="200.0" />
+    <xacro:property name="wheel_joint_velocity_limit" value="100.0" />
     <!--WHEEL TIRE -->
     <joint name="${prefix}wheel_joint" type="continuous">
@@ -53,5 +46,5 @@
           <origin xyz="0 0 0" rpy="${M_PI/2} 0 0" />
           <geometry>
-            <cylinder length="${wheel_height}" radius="${wheel_radius}" />
+            <cylinder length="${wheel_width}" radius="${wheel_radius}" />
           </geometry>
         </xacro:unless>
@@ -65,10 +58,11 @@
       <inertial>
         <mass value="${wheel_mass}" />
-        <origin xyz="0 0 0" />
-        <xacro:cylinder_inertia m="${wheel_mass}" r="${wheel_radius}" h="${wheel_height}" />
+        <origin xyz="0 0 0" rpy="${M_PI/2} 0 0"/>
+        <xacro:cylinder_inertia m="${wheel_mass}" r="${wheel_radius}" h="${wheel_width}" />
       </inertial>
     </link>
-    <xacro:gazebo_color_wheel prefix="${prefix}"/>
-    <xacro:gazebo_color_steer_wheel prefix="${prefix}"/>
+    <!-- GAZEBO PARAMETERS -->
+    <xacro:gazebo_rubber_tire_physics name="${prefix}wheel" />
+    <xacro:gazebo_rubber_tire_material name="${prefix}wheel" />
   </xacro:macro>
 </robot>

File: rbvogui_description/urdf/wheels/wheel.gazebo.xacro (robot description, xacro)
@@ -2,11 +2,55 @@
 <robot xmlns:xacro="http://wiki.ros.org/xacro">
   <!-- Rubber wheel color -->
+  <xacro:macro name="gazebo_rubber_tire_physics" params="name">
+    <gazebo reference="${name}">
+      <mu1>0.90</mu1>
+      <mu2>0.85</mu2>
+      <kp>8.75e5</kp>
+      <kd>8.25e1</kd>
+      <fdir1>0 0 0</fdir1>
+      <maxContacts>4</maxContacts>
+    </gazebo>
+  </xacro:macro>
+  <xacro:macro name="gazebo_rubber_tire_material" params="name">
+    <gazebo reference="${name}">
+      <visual>
+        <material>
+          <ambient>0.1 0.1 0.1 1.0</ambient>
+          <diffuse>0.250754 0.250754 0.250754 1.0</diffuse>
+          <specular>0.2508273 0.2508273 0.2508273 1.0</specular>
+          <emissive>0.0 0.0 0.0 0.0</emissive>
+        </material>
+      </visual>
+    </gazebo>
+  </xacro:macro>
+  <xacro:macro name="gazebo_steering_frame_physics" params="name">
+    <gazebo reference="${name}">
+      <mu1>0.40</mu1>
+      <mu2>0.35</mu2>
+      <kp>8.75e9</kp>
+      <kd>8.25e0</kd>
+      <fdir1>0 0 0</fdir1>
+    </gazebo>
+  </xacro:macro>
+  <xacro:macro name="gazebo_steering_frame_material" params="name">
+    <gazebo reference="${name}">
+      <visual>
+        <material>
+          <ambient>1.0 0.0 0.0 1.0</ambient>
+          <diffuse>0.50754 0.50754 0.50754 1.0</diffuse>
+          <specular>0.508273 0.508273 0.508273 1.0</specular>
+          <emissive>0.0 0.0 0.0 0.0</emissive>
+        </material>
+      </visual>
+    </gazebo>
+  </xacro:macro>
   <xacro:macro name="gazebo_color_wheel" params="prefix">
     <gazebo reference="${prefix}wheel">
-      <mu1 value="0.85"/>
-      <mu2 value="0.68"/>
-      <kp value="10000000.0" />
-      <kd value="1.0" />
-      <fdir1>1 0 0</fdir1>
+      <mu1>0.90</mu1>
+      <mu2>0.85</mu2>
+      <kp>8.75e5</kp>
+      <kd>8.25e1</kd>
+      <fdir1>0 1 0</fdir1>
+      <maxContacts>4</maxContacts>
       <visual>
         <material>
@@ -21,5 +65,5 @@
   <!-- Steer wheel color -->
   <xacro:macro name="gazebo_color_steer_wheel" params="prefix">
-    <gazebo reference="${prefix}motor_wheel">
+    <gazebo reference="${prefix}base_wheel">
       <visual>
         <material>

Commit message: Moved ros2_control tag to external file

File: rbvogui_description/robots/rbvogui_std.urdf.xacro (robot description, xacro)
@@ -81,34 +81,11 @@
         </xacro:sensor_rslidar_16>
         -->
-        <xacro:macro name="ros2_joint" params="interface jmin jmax prefix name">
-          <joint name="${prefix}${name}">
-            <command_interface name="${interface}">
-              <param name="min">${jmin}</param>
-              <param name="max">${jmax}</param>
-            </command_interface>
-            <state_interface name="position"/>
-            <state_interface name="velocity"/>
-            <state_interface name="effort"/>
-          </joint>
-        </xacro:macro>
-        <ros2_control name="GazeboSystem" type="system">
-          <hardware>
-              <plugin>gazebo_ros2_control/GazeboSystem</plugin>
-          </hardware>
-          <xacro:ros2_joint interface="position" jmin="-2" jmax="2" prefix="${prefix}" name="front_left_steering_joint"/>
-          <xacro:ros2_joint interface="position" jmin="-2" jmax="2" prefix="${prefix}" name="front_right_steering_joint"/>
-          <xacro:ros2_joint interface="position" jmin="-2" jmax="2" prefix="${prefix}" name="back_left_steering_joint"/>
-          <xacro:ros2_joint interface="position" jmin="-2" jmax="2" prefix="${prefix}" name="back_right_steering_joint"/>
-          <xacro:ros2_joint interface="velocity" jmin="-10" jmax="10" prefix="${prefix}" name="front_left_wheel_joint"/>
-          <xacro:ros2_joint interface="velocity" jmin="-10" jmax="10" prefix="${prefix}" name="front_right_wheel_joint"/>
-          <xacro:ros2_joint interface="velocity" jmin="-20" jmax="20" prefix="${prefix}" name="back_left_wheel_joint"/>
-          <xacro:ros2_joint interface="velocity" jmin="-20" jmax="20" prefix="${prefix}" name="back_right_wheel_joint"/>
-        </ros2_control>
     </xacro:macro>
-    <!-- Gazebo ros control pluggins -->
-    <xacro:ros_control/>
     <xacro:rbvogui prefix="$(arg prefix)" kinematics="$(arg kinematics)" load_kinematics_file="$(arg load_kinematics_file)" gpu="$(arg gpu)" publish_bf="${publish_bf}" hq="${hq}"
                    launch_arm="$(arg launch_arm)" arm_manufacturer="$(arg arm_manufacturer)" arm_model="$(arg arm_model)"
                    launch_gripper="$(arg launch_gripper)" gripper_manufacturer="$(arg gripper_manufacturer)" gripper_model="$(arg gripper_model)"
                    launch_lift="$(arg launch_lift)" lift_manufacturer="$(arg lift_manufacturer)" lift_model="$(arg lift_model)" />
+    <!-- Gazebo ros control pluggins -->
+    <xacro:include filename="$(find rbvogui_description)/urdf/ros2_control.urdf.xacro"/>
+    <xacro:ros2_control prefix="$(arg prefix)"/>
 </robot>

File: rbvogui_description/urdf/wheels/rubber_wheel.urdf.xacro (robot description, xacro)
@@ -2,10 +2,10 @@
 <robot xmlns:xacro="http://www.ros.org/wiki/xacro">
   <xacro:include filename="$(find rbvogui_description)/urdf/wheels/wheel.gazebo.xacro" />
-  <xacro:property name="M_PI" value="3.1415926535897931" />
-  <!-- in kg-->
-  <xacro:macro name="cylinder_inertia" params="m r h">
-    <inertia ixx="${m*(3*r*r+h*h)/12}" ixy = "0" ixz = "0" iyy="${m*(3*r*r+h*h)/12}" iyz = "0" izz="${m*r*r/2}" />
-  </xacro:macro>
+  <xacro:property name="wheel_radius" value="0.1165" />
   <xacro:macro name="wheel" params="prefix parent *origin reflect hq">
+    <xacro:macro name="cylinder_inertia" params="m r h">
+      <inertia ixx="${m*(3*r*r+h*h)/12}" ixy = "0" ixz = "0" iyy="${m*(3*r*r+h*h)/12}" iyz = "0" izz="${m*r*r/2}" />
+    </xacro:macro>
+    <xacro:property name="M_PI" value="3.1415926535897931" />
     <!-- Wheels -->
     <xacro:property name="wheel_radius" value="0.1165" /> <!-- rbvogui uses wheels with 0.233 m of diameter-->

File: rbvogui_description/urdf/wheels/wheel.gazebo.xacro (robot description, xacro)
@@ -6,5 +6,5 @@
       <mu1>0.90</mu1>
       <mu2>0.85</mu2>
-      <kp>8.75e5</kp>
+      <kp>2.75e6</kp>
       <kd>8.25e1</kd>
       <fdir1>0 0 0</fdir1>
