Commit message: Added two sick_s300 front and back lidar

File: rbvogui_description/robots/rbvogui_std.urdf.xacro (robot description, xacro)
@@ -73,7 +73,10 @@
         -->
         <!-- 2d laser -->
-        <xacro:sensor_sick_tim551 prefix="${prefix}front_laser" parent="${prefix}chassis_link" gpu="${gpu}" min_angle="${-PI/2}" max_angle="${PI/2}" prefix_topic="/$(arg robot_id)/front_laser">
-            <origin xyz="0.53 0.0 -0.0245" rpy="${PI} 0 0"/> <!-- Verificar X -->
-        </xacro:sensor_sick_tim551>
+        <xacro:sensor_sick_s300 prefix="${prefix}front_laser" parent="${prefix}chassis_link" gpu="${gpu}" prefix_topic="/$(arg robot_id)/front_laser">
+          <origin xyz="0.53 0.33 0.1245" rpy="${PI} 0 ${PI/4}"/>
+        </xacro:sensor_sick_s300>
+        <xacro:sensor_sick_s300 prefix="${prefix}rear_laser" parent="${prefix}chassis_link" gpu="${gpu}" prefix_topic="/$(arg robot_id)/rear_laser">
+          <origin xyz="-0.53 -0.33 0.1245" rpy="${PI} 0 ${-PI*3/4}"/>
+        </xacro:sensor_sick_s300>
         <!-- 3D Laser
         <xacro:sensor_rslidar_16 prefix="${prefix}top_3d_laser" parent="${prefix}chassis_link" prefix_topic="top_3d_laser" gpu="${gpu}">

Commit message: Added some features
- Added Intel realsense 435d
- Update sick painted, realsense, wheels and chassis

File: rbvogui_description/robots/rbvogui_std.urdf.xacro (robot description, xacro)
@@ -62,9 +62,8 @@
             <origin xyz="0.3 -0.3 0.0725" rpy="0 0 0"/>
         </xacro:sensor_vectornav>
-        <!-- Front Camera
-        <xacro:sensor_orbbec_astra prefix="${prefix}front_rgbd_camera" parent="${prefix}chassis_link">
+        <!-- Front Camera -->
+        <xacro:sensor_intel_d435 prefix="${prefix}front_rgbd_camera" parent="${prefix}chassis_link" prefix_topic="/$(arg robot_id)/front_rgbd_camera" use_nominal_extrinsics="true">
             <origin xyz="0.46462 0.0 0.18258" rpy="0 0 0"/>
-        </xacro:sensor_orbbec_astra>
-        -->
+        </xacro:sensor_intel_d435>
         <!-- GPS
         <xacro:sensor_ublox prefix="${prefix}gps" parent="${prefix}chassis_link">
@@ -74,8 +73,8 @@
         <!-- 2d laser -->
         <xacro:sensor_sick_s300 prefix="${prefix}front_laser" parent="${prefix}chassis_link" gpu="${gpu}" prefix_topic="/$(arg robot_id)/front_laser">
-          <origin xyz="0.53 0.33 0.1245" rpy="${PI} 0 ${PI/4}"/>
+          <origin xyz="0.53 0.33 0.1145" rpy="${PI} 0 ${PI/4}"/>
         </xacro:sensor_sick_s300>
         <xacro:sensor_sick_s300 prefix="${prefix}rear_laser" parent="${prefix}chassis_link" gpu="${gpu}" prefix_topic="/$(arg robot_id)/rear_laser">
-          <origin xyz="-0.53 -0.33 0.1245" rpy="${PI} 0 ${-PI*3/4}"/>
+          <origin xyz="-0.53 -0.33 0.1145" rpy="${PI} 0 ${-PI*3/4}"/>
         </xacro:sensor_sick_s300>
         <!-- 3D Laser

File: rbvogui_description/urdf/bases/rbvogui_base.urdf.xacro (robot description, xacro)
@@ -34,20 +34,17 @@
         <xacro:if value="${hq}">
           <geometry>
-            <mesh filename="package://rbvogui_description/meshes/bases/rbvogui_chassis.stl"/>
+            <mesh filename="package://rbvogui_description/meshes/bases/rbvogui_chassis_color.dae"/>
           </geometry>
         </xacro:if>
         <xacro:unless value="${hq}">
           <geometry>
-            <mesh filename="package://rbvogui_description/meshes/bases/rbvogui_chassis.stl"/>
+            <mesh filename="package://rbvogui_description/meshes/bases/rbvogui_chassis_color.dae"/>
           </geometry>
         </xacro:unless>
-        <material name="darkgrey">
-          <color rgba="0.1 0.1 0.1 1"/>
-        </material>
       </visual>
       <collision>
         <origin xyz="0 0 0" rpy="0 0 0 " />
         <geometry>
-          <mesh filename="package://rbvogui_description/meshes/bases/rbvogui_chassis.stl"/>
+          <mesh filename="package://rbvogui_description/meshes/bases/rbvogui_chassis_color.dae"/>
         </geometry>
       </collision>
@@ -157,5 +154,5 @@
     </link>
     <xacro:gazebo_color_base_link prefix="${prefix}"/>
-    <xacro:gazebo_color_chassis_link prefix="${prefix}"/>
+    <!--xacro:gazebo_color_chassis_link prefix="${prefix}"/-->
     <xacro:gazebo_color_battery_link prefix="${prefix}"/>
     <xacro:gazebo_color_contactors_link prefix="${prefix}"/>

File: rbvogui_description/urdf/wheels/steering_wheel.urdf.xacro (robot description, xacro)
@@ -36,5 +36,5 @@
           </xacro:unless>
           <geometry>
-            <mesh filename="package://rbvogui_description/meshes/wheels/mw_frame.stl" />
+            <mesh filename="package://rbvogui_description/meshes/wheels/mw_frame_stl_color.dae" />
           </geometry>
         </xacro:if>
@@ -48,5 +48,5 @@
           </xacro:unless>
           <geometry>
-            <mesh filename="package://rbvogui_description/meshes/wheels/mw_frame.stl" />
+            <mesh filename="package://rbvogui_description/meshes/wheels/mw_frame_stl_color.dae" />
           </geometry>
         </xacro:unless>
@@ -63,5 +63,5 @@
         </xacro:unless>
         <geometry>
-          <mesh filename="package://rbvogui_description/meshes/wheels/mw_frame.stl" />
+          <mesh filename="package://rbvogui_description/meshes/wheels/mw_frame_stl_color.dae" />
         </geometry>
       </collision>
@@ -78,5 +78,5 @@
     </link>
     <xacro:gazebo_steering_frame_physics name="${prefix}base_wheel"/>
-    <xacro:gazebo_steering_frame_material name="${prefix}base_wheel"/>
+    <!--xacro:gazebo_steering_frame_material name="${prefix}base_wheel"/-->
     <xacro:wheel prefix="${prefix}" parent="${prefix}base_wheel" reflect="${reflect}" hq="${hq}">
         <origin xyz="0 0 0" rpy="0 0 0"/>

Commit message: Fix urdf parse ros2_control error

File: rbvogui_description/robots/rbvogui_std.urdf.xacro (robot description, xacro)
@@ -25,7 +25,17 @@
     <xacro:property name="publish_bf" value="true" />
     <xacro:arg name="robot_id" default="robot" />
-    <xacro:arg name="prefix" default="$(arg robot)_" />
+    <xacro:arg name="prefix" default="$(arg robot_id)_" />
     <xacro:arg name="gpu" default="true" />
     <xacro:arg name="kinematics" default="omni" />
+    <xacro:arg name="load_kinematics_file" default="false" />
+    <xacro:arg name="launch_gripper" default="false" />
+    <xacro:arg name="gripper_manufacturer" default="false" />
+    <xacro:arg name="gripper_model" default="false" />
+    <xacro:arg name="launch_lift" default="false" />
+    <xacro:arg name="lift_manufacturer" default="false" />
+    <xacro:arg name="lift_model" default="false" />
+    <xacro:arg name="launch_arm" default="false" />
+    <xacro:arg name="arm_manufacturer" default="false" />
+    <xacro:arg name="arm_model" default="false" />
     <xacro:macro name="rbvogui" params="prefix publish_bf hq kinematics launch_arm arm_manufacturer arm_model load_kinematics_file
                                         launch_gripper gripper_manufacturer gripper_model launch_lift lift_manufacturer lift_model gpu">

File: rbvogui_description/urdf/ros2_control.urdf.xacro (robot description, xacro)
@@ -1,13 +1,11 @@
 <?xml version="1.0"?>
 <robot xmlns:xacro="http://wiki.ros.org/xacro">
-    <!-- ros control plugin -->
     <xacro:macro name="ros2_control" params="prefix">
         <gazebo>
           <plugin name="ros_control" filename="libgazebo_ros2_control.so">
-            <namespace>$(arg robot_id)</namespace>
-            <parameters>$(arg config_controllers)</parameters>
-            <!--robot_param>robot_description</robot_param-->
-            <!--robot_param_node>robot_state_publisher</robot_param_node-->
-            <!--remaping>$(find rbvogui_description)/config/remapping.yaml</remaping-->
+            <namespace>robot</namespace>
+            <robot_param>robot_description</robot_param>
+            <robot_param_node>robot_state_publisher</robot_param_node>
+            <parameters>$(find rbvogui_gazebo)/config/base_controller.yaml</parameters>
           </plugin>
         </gazebo>
@@ -37,35 +35,3 @@
         </ros2_control>
     </xacro:macro>
-    <xacro:macro name="omni_steering">
-        <gazebo>
-            <plugin name="omni_steering" filename="libgazebo_ros_planar_move.so">
-                <robotNamespace>/robot</robotNamespace>
-                <commandTopic>robotnik_base_control/cmd_vel</commandTopic>
-                <odometryTopic>robotnik_base_control/odom</odometryTopic>
-                <odometryFrame>odom</odometryFrame>
-                <odometryRate>20.0</odometryRate>
-                <robotBaseFrame>base_footprint</robotBaseFrame>
-            </plugin>
-          </gazebo>
-    </xacro:macro>
-    <xacro:macro name="omni_drive_ackermann">
-        <gazebo>
-            <plugin name="omni_drive_ackermann" filename="libomnidrive_ackermann_plugin.so">
-                <!--<robotNamespace>/rbvogui</robotNamespace>-->
-                <!--<robotParam>robot_description</robotParam>-->
-                <broadcastTF>1</broadcastTF>
-                <wheelDiameter>0.220</wheelDiameter>
-                <wheelBase>0.858</wheelBase>
-                <trackWidth>0.454</trackWidth>
-                <wheelTorque>44.2</wheelTorque>
-                <motorWheelTorque>15.0</motorWheelTorque>
-                <commandTopic>cmd_vel</commandTopic>  <!-- TODO: review topics -->
-                <odometryTopic>odom</odometryTopic>
-                <odometryFrame>odom</odometryFrame>
-                <odometrySource>encoder</odometrySource>
-                <robotBaseFrame>base_footprint</robotBaseFrame>
-                <updateRate>100.0</updateRate>
-            </plugin>
-        </gazebo>
-    </xacro:macro>
 </robot>

File: rbvogui_description/urdf/wheels/steering_wheel.urdf.xacro (robot description, xacro)
@@ -3,5 +3,5 @@
   <xacro:include filename="$(find rbvogui_description)/urdf/wheels/wheel.gazebo.xacro" />
   <xacro:include filename="$(find rbvogui_description)/urdf/wheels/rubber_wheel.urdf.xacro" />
-  <xacro:property name="wheel_radius" value="0.1175" /> <!-- teorically D: 0.235-->
+  <xacro:property name="wheel_radius" value="0.1175" />
   <xacro:macro name="steering_wheel" params="prefix parent *origin reflect hq">
     <xacro:macro name="cylinder_inertia" params="m r h">
@@ -14,6 +14,4 @@
     <xacro:property name="steer_joint_effort_limit" value="200.0" />
     <xacro:property name="steer_joint_velocity_limit" value="100.0" />
-    <!-- TODO: check reflect parameter -->
-    <!--MOTOR WHEEL -->
     <joint name="${prefix}steering_joint" type="revolute">
       <parent link="${parent}"/>
@@ -21,5 +19,4 @@
       <xacro:insert_block name="origin" />
       <axis xyz="0 0 1" rpy="0 0 0" />
-      <!-- limit effort="${steer_joint_effort_limit}" velocity="${steer_joint_velocity_limit}" lower="-1.5708" upper="1.5708" / -->
       <limit effort="${steer_joint_effort_limit}" velocity="${steer_joint_velocity_limit}" lower="-3.00" upper="3.00"/>
       <dynamics damping="${steer_joint_damping}" friction="${steer_joint_friction}"/>
@@ -27,5 +24,4 @@
     <link name="${prefix}base_wheel">
       <visual>
-        <!-- HIGH RESOLUTION WHEEL -->
         <xacro:if value="${hq}">
           <xacro:if value="${reflect}">
@@ -39,5 +35,4 @@
           </geometry>
         </xacro:if>
-          <!-- LOW RESOLUTION WHEEL -->
         <xacro:unless value="${hq}">
           <xacro:if value="${reflect}">
@@ -78,5 +73,4 @@
     </link>
     <xacro:gazebo_steering_frame_physics name="${prefix}base_wheel"/>
-    <!--xacro:gazebo_steering_frame_material name="${prefix}base_wheel"/-->
     <xacro:wheel prefix="${prefix}" parent="${prefix}base_wheel" reflect="${reflect}" hq="${hq}">
         <origin xyz="0 0 0" rpy="0 0 0"/>

Commit message: Fixed errors and added ROBETARME cart

File: rbvogui_description/robots/rbvogui_std.urdf.xacro (robot description, xacro)
@@ -15,4 +15,6 @@
     <xacro:include filename="$(find robotnik_sensors)/urdf/all_sensors.urdf.xacro" />
     <xacro:include filename="$(find rbvogui_description)/urdf/structures/gps_mast.urdf.xacro" />
+    <!-- Import cart -->
+    <xacro:include filename="$(find rbvogui_description)/urdf/cart/cart.urdf.xacro" />
     <xacro:property name="PI" value="3.1415926535897931"/>
     <xacro:property name="deg2rad" value="0.01745329251"/>
@@ -38,6 +40,8 @@
     <xacro:arg name="arm_manufacturer" default="false" />
     <xacro:arg name="arm_model" default="false" />
+    <!-- Cart -->
+    <xacro:arg name="cart" default="false" />
     <xacro:macro name="rbvogui" params="prefix publish_bf hq kinematics launch_arm arm_manufacturer arm_model load_kinematics_file
-                                        launch_gripper gripper_manufacturer gripper_model launch_lift lift_manufacturer lift_model gpu">
+                                        launch_gripper gripper_manufacturer gripper_model launch_lift lift_manufacturer lift_model gpu cart">
         <!-- ***************   -->
         <!-- Robots Elements -->
@@ -93,11 +97,15 @@
         </xacro:sensor_rslidar_16>
         -->
+        <xacro:if value="${cart}">
+            <xacro:cart prefix="${prefix}cart_" parent="${prefix}base_footprint">
+            </xacro:cart>
+        </xacro:if>
     </xacro:macro>
     <xacro:rbvogui prefix="$(arg prefix)" kinematics="$(arg kinematics)" load_kinematics_file="$(arg load_kinematics_file)" gpu="$(arg gpu)" publish_bf="${publish_bf}" hq="${hq}"
                    launch_arm="$(arg launch_arm)" arm_manufacturer="$(arg arm_manufacturer)" arm_model="$(arg arm_model)"
                    launch_gripper="$(arg launch_gripper)" gripper_manufacturer="$(arg gripper_manufacturer)" gripper_model="$(arg gripper_model)"
-                   launch_lift="$(arg launch_lift)" lift_manufacturer="$(arg lift_manufacturer)" lift_model="$(arg lift_model)" />
+                   launch_lift="$(arg launch_lift)" lift_manufacturer="$(arg lift_manufacturer)" lift_model="$(arg lift_model)" cart="$(arg cart)"/>
     <!-- Gazebo ros control pluggins -->
     <xacro:include filename="$(find rbvogui_description)/urdf/ros2_control.urdf.xacro"/>
-    <xacro:ros2_control prefix="$(arg prefix)"/>
+    <xacro:ros2_control prefix="$(arg prefix)" cart="$(arg cart)"/>
 </robot>

File: rbvogui_description/urdf/inertia.urdf.xacro (robot description, xacro)
@@ -1,5 +1,4 @@
 <?xml version="1.0"?>
 <robot xmlns:xacro="http://wiki.ros.org/xacro">
-  <!-- Source: https://en.wikipedia.org/wiki/List_of_moments_of_inertia-->
   <!-- TODO Solid sphere of radius r and mass m-->
   <xacro:macro name="solid_sphere_inertia" params="m r">

File: rbvogui_description/urdf/ros2_control.urdf.xacro (robot description, xacro)
@@ -1,5 +1,5 @@
 <?xml version="1.0"?>
 <robot xmlns:xacro="http://wiki.ros.org/xacro">
-    <xacro:macro name="ros2_control" params="prefix">
+    <xacro:macro name="ros2_control" params="prefix cart">
         <gazebo>
           <plugin name="ros_control" filename="libgazebo_ros2_control.so">
@@ -9,4 +9,20 @@
             <parameters>$(find rbvogui_gazebo)/config/base_controller.yaml</parameters>
           </plugin>
+          <xacro:if value="${cart}">
+            <plugin name="cart_joint_state" filename="libgazebo_ros_joint_state_publisher.so">
+              <namespace>robot</namespace>
+              <update_rate>30</update_rate>
+              <joint_name>robot_cart_hitch_z_joint</joint_name>
+              <joint_name>robot_cart_hitch_y_joint</joint_name>
+              <joint_name>robot_cart_hitch_x_joint</joint_name>
+              <joint_name>robot_cart_body_joint</joint_name>
+              <joint_name>robot_cart_left_wheel_joint</joint_name>
+              <joint_name>robot_cart_right_wheel_joint</joint_name>
+              <joint_name>robot_cart_support_front_right_wheel_joint</joint_name>
+              <joint_name>robot_cart_support_front_left_wheel_joint</joint_name>
+              <joint_name>robot_cart_front_right_wheel_joint</joint_name>
+              <joint_name>robot_cart_front_left_wheel_joint</joint_name>
+            </plugin>
+          </xacro:if>
         </gazebo>
         <xacro:macro name="ros2_joint" params="interface jmin jmax prefix name">
