Commit message: Update meshes

File: rbvogui_description/robots/rbvogui_std.urdf.xacro (robot description, xacro)
@@ -80,4 +80,8 @@
             <origin xyz="0.46462 0.0 0.18258" rpy="0 0 0"/>
         </xacro:sensor_intel_d435>
+        <!-- Rear Camera -->
+        <xacro:sensor_intel_d435 prefix="${prefix}rear_rgbd_camera" parent="${prefix}base_link" prefix_topic="/$(arg robot_id)/rear_rgbd_camera" use_nominal_extrinsics="true">
+            <origin xyz="-0.503 0.0 0.29" rpy="0 0 -${PI}"/>
+        </xacro:sensor_intel_d435>
         <!-- GPS
         <xacro:sensor_ublox prefix="${prefix}gps" parent="${prefix}chassis_link">
@@ -98,5 +102,5 @@
         -->
         <xacro:if value="${cart}">
-            <xacro:cart prefix="${prefix}cart_" parent="${prefix}base_footprint">
+            <xacro:cart prefix="${prefix}cart_" parent="${prefix}base_link">
             </xacro:cart>
         </xacro:if>

File: rbvogui_description/urdf/cart/cart.urdf.xacro (robot description, xacro)
@@ -6,10 +6,10 @@
   <xacro:property name="PI" value="3.141592" />
   <!-- Size cart -->
-  <xacro:property name="cart_length" value="1.25" />
-  <xacro:property name="cart_width" value="1.098" />
+  <xacro:property name="cart_length" value="1.4" />
+  <xacro:property name="cart_width" value="1.4" />
   <xacro:property name="cart_height" value="0.25" />
   <xacro:property name="cart_mass" value="80" />
   <!-- Size wheels -->
-  <xacro:property name="wheels_radius" value="0.20" />
+  <xacro:property name="wheels_radius" value="0.225" />
   <xacro:property name="wheels_width" value="0.08" />
   <xacro:property name="wheels_center_dist_x" value="0.41" />
@@ -23,8 +23,46 @@
   <xacro:property name="support_width" value="0.03" />
   <!-- Hitch -->
-  <xacro:property name="hitch_length" value="0.4" />
-  <xacro:property name="hitch_width" value="0.05" />
+  <xacro:property name="hitch_length" value="0.215" />
+  <xacro:property name="hitch_width" value="0.160" />
+  <xacro:property name="hitch_height" value="0.064" />
+  <!-- NEW CART VALUES -->
+  <!-- Transform from robot_base_link to bulon -->
+  <xacro:property name="bulon_x" value="-0.669" />
+  <xacro:property name="bulon_z" value="0.391" />
+  <!-- Transform from hitch to chassis UNKOWN -->
+  <xacro:property name="hitch_x" value="-0.620" />
+  <xacro:property name="hitch_z" value="0.161" />
+  <!-- Transform from chassis to wheels -->
+  <xacro:property name="front_caster_wheel_x" value="0.620" />
+  <xacro:property name="front_caster_wheel_y" value="0.6045" />
+  <xacro:property name="front_caster_wheel_z" value="-0.11201" />
+  <xacro:property name="rear_wheel_x" value="-0.40883" />
+  <xacro:property name="rear_wheel_y" value="0.5895" />
+  <xacro:property name="rear_wheel_z" value="-0.075" />
+  <!-- Transform from front_caster_wheel to front_wheel -->
+  <xacro:property name="front_wheel_x" value="-0.04545" />
+  <xacro:property name="front_wheel_z" value="-0.115" />
   <xacro:macro name="cart" params="prefix parent">
-    <!-- Robot to Hitch -->
+    <!-- Robot to bulon NOMBRE PROVISIONAL SUPONGO??-->
+      <link name="${prefix}bulon">
+        <inertial>
+              <mass value="1" />
+              <origin xyz="0 0 0" rpy="0 0 0" />
+              <xacro:solid_cuboid_inertia w="${0.01}" d="${0.01}" h="${0.01}" m="10"/>
+        </inertial>
+        <visual>
+          <origin xyz="0.0 0.0 -0.0975" rpy="0.0 0.0 0.0"/>
+          <geometry>
+            <cylinder radius="0.015" length="0.195"/>
+          </geometry>
+        </visual>
+        <collision>
+          <origin xyz="0.0 0.0 -0.0975" rpy="0.0 0.0 0.0"/>
+          <geometry>
+            <cylinder radius="0.015" length="0.195"/>
+          </geometry>
+        </collision>
+      </link>
+    <!-- bulon to Hitch -->
     <link name="${prefix}hitch_z">
       <inertial>
@@ -44,11 +82,17 @@
       <inertial>
             <mass value="1" />
-            <origin xyz="-${hitch_length/2} 0 0" rpy="0 0 0" />
-            <xacro:solid_cuboid_inertia w="${hitch_length}" d="${hitch_width}" h="${hitch_width}" m="1"/>
-      </inertial>
-      <collision>
-        <origin xyz="-${hitch_length/2} 0.0 0.0" rpy="0.0 0.0 0.0"/>
-        <geometry>
-          <box size="${hitch_length} ${hitch_width} ${hitch_width}"/>
+            <origin xyz="0.0 0 0" rpy="0 0 0" />
+            <xacro:solid_cuboid_inertia w="${hitch_length}" d="${hitch_height}" h="${hitch_width}" m="1"/>
+      </inertial>
+      <visual>
+        <origin xyz="0.0 0.0 0.0" rpy="0.0 0.0 0.0"/>
+        <geometry>
+          <box size="0.215 0.160 0.064"/>
+        </geometry>
+      </visual>
+      <collision>
+        <origin xyz="0.0 0.0 0.0" rpy="0.0 0.0 0.0"/>
+        <geometry>
+          <box size="${hitch_length} ${hitch_width} ${hitch_height}"/>
         </geometry>
       </collision>
@@ -64,5 +108,5 @@
       </inertial>
       <visual>
-        <origin xyz="0.0 0.0 ${-cart_height/2}" rpy="${PI/2} 0.0 ${PI}"/>
+        <origin xyz="0.0 0.0 0" rpy="0 0.0 0"/>
         <geometry>
           <mesh filename="package://rbvogui_description/meshes/cart/cart.stl" scale="1.0 1.0 1.0"/>
@@ -82,6 +126,6 @@
       <material>Gazebo/Red</material>
     </gazebo>
-    <!-- Left wheel -->
-    <link name="${prefix}left_wheel">
+    <!-- Rear Left wheel -->
+    <link name="${prefix}rear_left_wheel">
       <inertial>
             <mass value="1" />
@@ -90,5 +134,5 @@
       </inertial>
       <visual>
-        <origin xyz="0.0 0.0 0.0" rpy="0 0.0 ${PI/2}"/>
+        <origin xyz="0.0 0.0 0.0" rpy="0 0.0 0"/>
         <geometry>
           <mesh filename="package://rbvogui_description/meshes/cart/back_wheel.stl" scale="1.0 1.0 1.0"/>
@@ -105,9 +149,9 @@
       </collision>
     </link>
-    <gazebo reference="${prefix}left_wheel">
+    <gazebo reference="${prefix}rear_left_wheel">
       <material>Gazebo/Grey</material>
     </gazebo>
-    <!-- Right wheel -->
-    <link name="${prefix}right_wheel">
+    <!-- Rear Right wheel -->
+    <link name="${prefix}rear_right_wheel">
       <inertial>
             <mass value="1" />
@@ -116,5 +160,5 @@
       </inertial>
       <visual>
-        <origin xyz="0.0 0.0 0.0" rpy="0 0.0 ${PI/2}"/>
+        <origin xyz="0.0 0.0 0.0" rpy="0 0.0 0"/>
         <geometry>
           <mesh filename="package://rbvogui_description/meshes/cart/back_wheel.stl" scale="1.0 1.0 1.0"/>
@@ -131,9 +175,33 @@
       </collision>
     </link>
-    <gazebo reference="${prefix}right_wheel">
+    <gazebo reference="${prefix}rear_right_wheel">
       <material>Gazebo/Grey</material>
     </gazebo>
+    <!-- Front Right Wheel base support -->
+    <link name="${prefix}front_right_wheel_base_support">
+      <visual>
+        <origin xyz="0.0 0.0 0.0" rpy="0 0 0"/>
+        <geometry>
+          <mesh filename="package://rbvogui_description/meshes/cart/base_support_wheel.stl" scale="1.0 1.0 1.0"/>
+        </geometry>
+      </visual>
+    </link>
+    <gazebo reference="${prefix}front_right_wheel_base_support">
+      <material>Gazebo/Red</material>
+    </gazebo>
+    <!-- Front Left Wheel base support -->
+    <link name="${prefix}front_left_wheel_base_support">
+      <visual>
+        <origin xyz="0.0 0.0 0.0" rpy="0 0 0"/>
+        <geometry>
+          <mesh filename="package://rbvogui_description/meshes/cart/base_support_wheel.stl" scale="1.0 1.0 1.0"/>
+        </geometry>
+      </visual>
+    </link>
+    <gazebo reference="${prefix}front_left_wheel_base_support">
+      <material>Gazebo/Red</material>
+    </gazebo>
     <!-- Front Right Wheel support -->
-    <link name="${prefix}support_front_right_wheel">
+    <link name="${prefix}front_right_wheel_support">
       <inertial>
             <mass value="1" />
@@ -142,5 +210,5 @@
       </inertial>
       <visual>
-        <origin xyz="0.0 0.0 0.06" rpy="${PI/2} 0 -${PI/4}"/>
+        <origin xyz="0.0 0.0 0.0" rpy="0 0 -${40*PI/180}"/>
         <geometry>
           <mesh filename="package://rbvogui_description/meshes/cart/support_wheel.stl" scale="1.0 1.0 1.0"/>
@@ -154,9 +222,9 @@
       </collision>
     </link>
-    <gazebo reference="${prefix}support_front_right_wheel">
+    <gazebo reference="${prefix}front_right_wheel_support">
       <material>Gazebo/Red</material>
     </gazebo>
     <!-- Front Left Wheel support -->
-    <link name="${prefix}support_front_left_wheel">
+    <link name="${prefix}front_left_wheel_support">
       <inertial>
             <mass value="1" />
@@ -165,5 +233,5 @@
       </inertial>
       <visual>
-        <origin xyz="0.0 0.0 0.06" rpy="${PI/2} 0 -${PI/4}"/>
+        <origin xyz="0.0 0.0 0.0" rpy="0 0 -${40*PI/180}"/>
         <geometry>
           <mesh filename="package://rbvogui_description/meshes/cart/support_wheel.stl" scale="1.0 1.0 1.0"/>
@@ -177,5 +245,5 @@
       </collision>
     </link>
-    <gazebo reference="${prefix}support_front_left_wheel">
+    <gazebo reference="${prefix}front_left_wheel_support">
       <material>Gazebo/Red</material>
     </gazebo>

File: rbvogui_description/urdf/cart/cart_joint.urdf.xacro (robot description, xacro)
@@ -2,7 +2,13 @@
 <robot xmlns:xacro="http://www.ros.org/wiki/xacro" name="robot_name">
     <xacro:macro name="cart_joints" params="prefix parent">
-    <!-- Robot to Hitch -->
+    <!-- Robot to BULON -->
+        <joint name="${prefix}bulon_joint" type="fixed">
+            <origin xyz="${bulon_x} 0 ${bulon_z}" rpy="0.0 0.0 0.0"/>
+            <parent link="${parent}"/>
+            <child link="${prefix}bulon"/>
+        </joint>
+    <!-- BULON to Hitch -->
         <joint name="${prefix}hitch_z_joint" type="revolute">
-            <origin xyz="-0.6 0 ${wheels_radius + cart_height/2}" rpy="0.0 0.0 0.0"/>
+            <origin xyz="${hitch_x} 0 ${hitch_z}" rpy="0.0 0.0 0.0"/>
             <parent link="${parent}"/>
             <child link="${prefix}hitch_z"/>
@@ -26,5 +32,5 @@
     <!-- Hitch to Body -->
         <joint name="${prefix}body_joint" type="revolute">
-            <origin xyz="${-cart_length/2 -hitch_length} 0 0" rpy="0.0 0.0 0.0"/>
+            <origin xyz="${-cart_length/2 -hitch_length/2} 0 0" rpy="0.0 0.0 0.0"/>
             <parent link="${prefix}hitch_x"/>
             <child link="${prefix}body"/>
@@ -32,33 +38,45 @@
             <limit effort="1000" velocity="2000" lower="-0.2" upper="0.2"/>
         </joint>
-    <!-- Left wheel -->
-        <joint name="${prefix}left_wheel_joint" type="continuous">
-            <origin xyz="${-wheels_center_dist_x} ${cart_width / 2 + wheels_width / 2} ${-cart_height/2}" rpy="0.0 0.0 0.0"/>
+    <!-- Rear Left wheel -->
+        <joint name="${prefix}rear_left_wheel_joint" type="continuous">
+            <origin xyz="${rear_wheel_x} ${rear_wheel_y} ${rear_wheel_z}" rpy="0.0 0.0 0.0"/>
             <parent link="${prefix}body"/>
-            <child link="${prefix}left_wheel"/>
+            <child link="${prefix}rear_left_wheel"/>
             <axis xyz="0.0 1.0 0.0"/>
             <limit effort="1000" velocity="2000"/>
         </joint>
-    <!-- Right wheel -->
-        <joint name="${prefix}right_wheel_joint" type="continuous">
-            <origin xyz="${-wheels_center_dist_x} ${-cart_width / 2 - wheels_width / 2} ${-cart_height/2}" rpy="0.0 0.0 0.0"/>
+    <!-- Rear Right wheel -->
+        <joint name="${prefix}rear_right_wheel_joint" type="continuous">
+            <origin xyz="${rear_wheel_x} -${rear_wheel_y} ${rear_wheel_z}" rpy="0.0 0.0 0.0"/>
             <parent link="${prefix}body"/>
-            <child link="${prefix}right_wheel"/>
+            <child link="${prefix}rear_right_wheel"/>
             <axis xyz="0.0 1.0 0.0"/>
             <limit effort="1000" velocity="2000"/>
         </joint>
+    <!-- Front Right Wheel support base-->
+        <joint name="${prefix}front_right_wheel_base_support_joint" type="fixed">
+            <origin xyz="${front_caster_wheel_x} ${-front_caster_wheel_y} ${front_caster_wheel_z}" rpy="0.0 0.0 0.0"/>
+            <parent link="${prefix}body"/>
+            <child link="${prefix}front_right_wheel_base_support"/>
+        </joint>
+    <!-- Front Left Wheel support base-->
+        <joint name="${prefix}front_left_wheel_base_support_joint" type="fixed">
+            <origin xyz="${front_caster_wheel_x} ${front_caster_wheel_y} ${front_caster_wheel_z}" rpy="0.0 0.0 0.0"/>
+            <parent link="${prefix}body"/>
+            <child link="${prefix}front_left_wheel_base_support"/>
+        </joint>
     <!-- Front Right Wheel support -->
-        <joint name="${prefix}support_front_right_wheel_joint" type="continuous">
-            <origin xyz="${front_wheel_center_dist_x} ${-front_wheel_center_dist_y} ${-cart_height/2-support_length/2}" rpy="0.0 0.0 0.0"/>
+        <joint name="${prefix}front_right_wheel_support_joint" type="continuous">
+            <origin xyz="${front_caster_wheel_x} ${-front_caster_wheel_y} ${front_caster_wheel_z}" rpy="0.0 0.0 0.0"/>
             <parent link="${prefix}body"/>
-            <child link="${prefix}support_front_right_wheel"/>
+            <child link="${prefix}front_right_wheel_support"/>
             <axis xyz="0.0 0.0 1.0"/>
             <limit effort="1000" velocity="2000"/>
         </joint>
     <!-- Front Left Wheel support -->
-        <joint name="${prefix}support_front_left_wheel_joint" type="continuous">
-            <origin xyz="${front_wheel_center_dist_x} ${front_wheel_center_dist_y} ${-cart_height/2-support_length/2}" rpy="0.0 0.0 0.0"/>
+        <joint name="${prefix}front_left_wheel_support_joint" type="continuous">
+            <origin xyz="${front_caster_wheel_x} ${front_caster_wheel_y} ${front_caster_wheel_z}" rpy="0.0 0.0 0.0"/>
             <parent link="${prefix}body"/>
-            <child link="${prefix}support_front_left_wheel"/>
+            <child link="${prefix}front_left_wheel_support"/>
             <axis xyz="0.0 0.0 1.0"/>
             <limit effort="1000" velocity="2000"/>
@@ -66,6 +84,6 @@
     <!-- Front Left wheel -->
         <joint name="${prefix}front_left_wheel_joint" type="continuous">
-            <origin xyz="-0.05 0 ${-support_length/2}" rpy="0.0 0.0 0.0"/>
-            <parent link="${prefix}support_front_left_wheel"/>
+            <origin xyz="${front_wheel_x} 0 ${front_wheel_z}" rpy="0.0 0.0 0.0"/>
+            <parent link="${prefix}front_left_wheel_support"/>
             <child link="${prefix}front_left_wheel"/>
             <axis xyz="0.0 1.0 0.0"/>
@@ -74,6 +92,6 @@
     <!-- Front Right wheel -->
         <joint name="${prefix}front_right_wheel_joint" type="continuous">
-            <origin xyz="-0.05 0 ${-support_length/2}" rpy="0.0 0.0 0.0"/>
-            <parent link="${prefix}support_front_right_wheel"/>
+            <origin xyz="${front_wheel_x} 0 ${front_wheel_z}" rpy="0.0 0.0 0.0"/>
+            <parent link="${prefix}front_right_wheel_support"/>
             <child link="${prefix}front_right_wheel"/>
             <axis xyz="0.0 1.0 0.0"/>

File: rbvogui_description/urdf/ros2_control.urdf.xacro (robot description, xacro)
@@ -19,8 +19,8 @@
               <joint_name>robot_cart_hitch_x_joint</joint_name>
               <joint_name>robot_cart_body_joint</joint_name>
-              <joint_name>robot_cart_left_wheel_joint</joint_name>
-              <joint_name>robot_cart_right_wheel_joint</joint_name>
-              <joint_name>robot_cart_support_front_right_wheel_joint</joint_name>
-              <joint_name>robot_cart_support_front_left_wheel_joint</joint_name>
+              <joint_name>robot_cart_rear_left_wheel_joint</joint_name>
+              <joint_name>robot_cart_rear_right_wheel_joint</joint_name>
+              <joint_name>robot_cart_front_right_wheel_support_joint</joint_name>
+              <joint_name>robot_cart_front_left_wheel_support_joint</joint_name>
               <joint_name>robot_cart_front_right_wheel_joint</joint_name>
               <joint_name>robot_cart_front_left_wheel_joint</joint_name>

Commit message: Fixed inertias and rotation movement

File: rbvogui_description/robots/rbvogui_std.urdf.xacro (robot description, xacro)
@@ -102,5 +102,5 @@
         -->
         <xacro:if value="${cart}">
-            <xacro:cart prefix="${prefix}cart_" parent="${prefix}base_link">
+            <xacro:cart prefix="${prefix}cart_" parent="${prefix}base_link" connection="true">
             </xacro:cart>
         </xacro:if>

File: rbvogui_description/urdf/cart/cart.urdf.xacro (robot description, xacro)
@@ -6,7 +6,7 @@
   <xacro:property name="PI" value="3.141592" />
   <!-- Size cart -->
-  <xacro:property name="cart_length" value="1.4" />
-  <xacro:property name="cart_width" value="1.4" />
-  <xacro:property name="cart_height" value="0.25" />
+  <xacro:property name="cart_length" value="1.3" />
+  <xacro:property name="cart_width" value="1.3" />
+  <xacro:property name="cart_height" value="0.23" />
   <xacro:property name="cart_mass" value="80" />
   <!-- Size wheels -->
@@ -43,5 +43,5 @@
   <xacro:property name="front_wheel_x" value="-0.04545" />
   <xacro:property name="front_wheel_z" value="-0.115" />
-  <xacro:macro name="cart" params="prefix parent">
+  <xacro:macro name="cart" params="prefix parent connection">
     <!-- Robot to bulon NOMBRE PROVISIONAL SUPONGO??-->
       <link name="${prefix}bulon">
@@ -67,21 +67,21 @@
     <link name="${prefix}hitch_z">
       <inertial>
-            <mass value="1" />
+            <mass value="3" />
             <origin xyz="0 0 0" rpy="0 0 0" />
-            <xacro:solid_cuboid_inertia w="${0.01}" d="${0.01}" h="${0.01}" m="10"/>
+            <xacro:solid_cuboid_inertia w="0.215" d="0.064" h="0.160" m="3"/>
       </inertial>
     </link>
     <link name="${prefix}hitch_y">
       <inertial>
-            <mass value="1" />
+            <mass value="3" />
             <origin xyz="0 0 0" rpy="0 0 0" />
-            <xacro:solid_cuboid_inertia w="${0.01}" d="${0.01}" h="${0.01}" m="10"/>
+            <xacro:solid_cuboid_inertia w="0.215" d="0.064" h="0.160" m="3"/>
       </inertial>
     </link>
     <link name="${prefix}hitch_x">
       <inertial>
-            <mass value="1" />
-            <origin xyz="0.0 0 0" rpy="0 0 0" />
-            <xacro:solid_cuboid_inertia w="${hitch_length}" d="${hitch_height}" h="${hitch_width}" m="1"/>
+            <mass value="3" />
+            <origin xyz="0 0 0" rpy="0 0 0" />
+            <xacro:solid_cuboid_inertia w="0.215" d="0.064" h="0.160" m="3"/>
       </inertial>
       <visual>
@@ -300,5 +300,23 @@
       <material>Gazebo/Grey</material>
     </gazebo>
-    <xacro:cart_joints prefix="${prefix}" parent="${parent}"/>
+    <!-- Marker0 -->
+    <link name="${prefix}marker0">
+      <visual>
+        <origin xyz="0.0 0.0 0.0" rpy="0.0 0 0"/>
+        <geometry>
+          <mesh filename="package://rbvogui_description/meshes/cart/Markers/meshes/Marker0.dae" scale="0.1 0.1 0.1"/>
+        </geometry>
+      </visual>
+    </link>
+    <!-- Marker1 -->
+    <link name="${prefix}marker1">
+      <visual>
+        <origin xyz="0.0 0.0 0.0" rpy="0.0 0 0"/>
+        <geometry>
+          <mesh filename="package://rbvogui_description/meshes/cart/Markers/meshes/Marker1.dae" scale="0.1 0.1 0.1"/>
+        </geometry>
+      </visual>
+    </link>
+    <xacro:cart_joints prefix="${prefix}" parent="${parent}" connection="${connection}"/>
   </xacro:macro>
 </robot>

File: rbvogui_description/urdf/cart/cart_joint.urdf.xacro (robot description, xacro)
@@ -1,5 +1,5 @@
 <?xml version="1.0"?>
 <robot xmlns:xacro="http://www.ros.org/wiki/xacro" name="robot_name">
-    <xacro:macro name="cart_joints" params="prefix parent">
+    <xacro:macro name="cart_joints" params="prefix parent connection">
     <!-- Robot to BULON -->
         <joint name="${prefix}bulon_joint" type="fixed">
@@ -14,5 +14,5 @@
             <child link="${prefix}hitch_z"/>
             <axis xyz="0.0 0.0 1.0"/>
-            <limit effort="1000" velocity="2000" lower="${-PI/6}" upper="${PI/6}"/>
+            <limit effort="1000" velocity="2000" lower="${-PI/7}" upper="${PI/7}"/>
         </joint>
         <joint name="${prefix}hitch_y_joint" type="revolute">
@@ -21,5 +21,5 @@
             <child link="${prefix}hitch_y"/>
             <axis xyz="0.0 1.0 0.0"/>
-            <limit effort="1000" velocity="2000" lower="${-PI/6}" upper="${PI/6}"/>
+            <limit effort="1000" velocity="2000" lower="${-PI/7}" upper="${PI/7}"/>
         </joint>
         <joint name="${prefix}hitch_x_joint" type="revolute">
@@ -28,5 +28,5 @@
             <child link="${prefix}hitch_x"/>
             <axis xyz="1.0 0.0 0.0"/>
-            <limit effort="1000" velocity="2000" lower="${-PI/6}" upper="${PI/6}"/>
+            <limit effort="1000" velocity="2000" lower="${-PI/7}" upper="${PI/7}"/>
         </joint>
     <!-- Hitch to Body -->
@@ -98,4 +98,16 @@
             <limit effort="1000" velocity="2000"/>
         </joint>
+    <!-- Marker0 -->
+        <joint name="${prefix}marker0_joint" type="fixed">
+            <origin xyz="0.66 -0.08 0.05" rpy="0.0 0.0 0.0"/>
+            <parent link="${prefix}body"/>
+            <child link="${prefix}marker0"/>
+        </joint>
+    <!-- Marker1 -->
+        <joint name="${prefix}marker1_joint" type="fixed">
+            <origin xyz="0.66 0.08 0.05" rpy="0.0 0.0 0.0"/>
+            <parent link="${prefix}body"/>
+            <child link="${prefix}marker1"/>
+        </joint>
     </xacro:macro>
 </robot>
