Commit message: Fixed URDF and updated navigation params

File: rbvogui_description/robots/rbvogui_std.urdf.xacro (robot description, xacro)
@@ -16,5 +16,5 @@
     <xacro:include filename="$(find rbvogui_description)/urdf/structures/gps_mast.urdf.xacro" />
     <!-- Import cart -->
-    <xacro:include filename="$(find rbvogui_description)/urdf/cart/cart.urdf.xacro" />
+    <!-- <xacro:include filename="$(find rbvogui_description)/urdf/cart/cart.urdf.xacro" /> -->
     <xacro:property name="PI" value="3.1415926535897931"/>
     <xacro:property name="deg2rad" value="0.01745329251"/>
@@ -42,6 +42,7 @@
     <!-- Cart -->
     <xacro:arg name="cart" default="false" />
+    <xacro:arg name="connected" default="false" />
     <xacro:macro name="rbvogui" params="prefix publish_bf hq kinematics launch_arm arm_manufacturer arm_model load_kinematics_file
-                                        launch_gripper gripper_manufacturer gripper_model launch_lift lift_manufacturer lift_model gpu cart">
+                                        launch_gripper gripper_manufacturer gripper_model launch_lift lift_manufacturer lift_model gpu cart connected">
         <!-- ***************   -->
         <!-- Robots Elements -->
@@ -102,6 +103,10 @@
         -->
         <xacro:if value="${cart}">
-            <xacro:cart prefix="${prefix}cart_" parent="${prefix}base_link" connection="true">
-            </xacro:cart>
+            <xacro:include filename="$(find rbvogui_description)/urdf/cart/cart_robot_connection.urdf.xacro" />
+            <xacro:cart_connection prefix="${prefix}" connected="${connected}"/>
+            <xacro:if value="${connected}">
+                <xacro:include filename="$(find rbvogui_description)/urdf/cart/cart.urdf.xacro" />
+                <xacro:cart prefix="${prefix}cart_" connected="${connected}"/>
+            </xacro:if>
         </xacro:if>
     </xacro:macro>
@@ -109,7 +114,7 @@
                    launch_arm="$(arg launch_arm)" arm_manufacturer="$(arg arm_manufacturer)" arm_model="$(arg arm_model)"
                    launch_gripper="$(arg launch_gripper)" gripper_manufacturer="$(arg gripper_manufacturer)" gripper_model="$(arg gripper_model)"
-                   launch_lift="$(arg launch_lift)" lift_manufacturer="$(arg lift_manufacturer)" lift_model="$(arg lift_model)" cart="$(arg cart)"/>
+                   launch_lift="$(arg launch_lift)" lift_manufacturer="$(arg lift_manufacturer)" lift_model="$(arg lift_model)" cart="$(arg cart)" connected="$(arg connected)"/>
     <!-- Gazebo ros control pluggins -->
     <xacro:include filename="$(find rbvogui_description)/urdf/ros2_control.urdf.xacro"/>
-    <xacro:ros2_control prefix="$(arg prefix)" cart="$(arg cart)"/>
+    <xacro:ros2_control prefix="$(arg prefix)"/>
 </robot>

File: rbvogui_description/urdf/cart/cart.urdf.xacro (robot description, xacro)
@@ -3,4 +3,7 @@
   <xacro:include filename="$(find rbvogui_description)/urdf/inertia.urdf.xacro" />
   <xacro:include filename="$(find rbvogui_description)/urdf/cart/cart_joint.urdf.xacro" />
+  <xacro:include filename="$(find rbvogui_description)/urdf/cart/cart_robot_connection.urdf.xacro" />
+  <xacro:arg name="prefix" default="robot_" />
+  <xacro:arg name="connected" default="false" />
   <!-- Math -->
   <xacro:property name="PI" value="3.141592" />
@@ -43,64 +46,13 @@
   <xacro:property name="front_wheel_x" value="-0.04545" />
   <xacro:property name="front_wheel_z" value="-0.115" />
-  <xacro:macro name="cart" params="prefix parent connection">
-    <!-- Robot to bulon NOMBRE PROVISIONAL SUPONGO??-->
-      <link name="${prefix}bulon">
-        <inertial>
-              <mass value="1" />
-              <origin xyz="0 0 0" rpy="0 0 0" />
-              <xacro:solid_cuboid_inertia w="${0.01}" d="${0.01}" h="${0.01}" m="10"/>
-        </inertial>
-        <visual>
-          <origin xyz="0.0 0.0 -0.0975" rpy="0.0 0.0 0.0"/>
-          <geometry>
-            <cylinder radius="0.015" length="0.195"/>
-          </geometry>
-        </visual>
-        <collision>
-          <origin xyz="0.0 0.0 -0.0975" rpy="0.0 0.0 0.0"/>
-          <geometry>
-            <cylinder radius="0.015" length="0.195"/>
-          </geometry>
-        </collision>
-      </link>
-    <!-- bulon to Hitch -->
-    <link name="${prefix}hitch_z">
-      <inertial>
-            <mass value="3" />
-            <origin xyz="0 0 0" rpy="0 0 0" />
-            <xacro:solid_cuboid_inertia w="0.215" d="0.064" h="0.160" m="3"/>
-      </inertial>
-    </link>
-    <link name="${prefix}hitch_y">
-      <inertial>
-            <mass value="3" />
-            <origin xyz="0 0 0" rpy="0 0 0" />
-            <xacro:solid_cuboid_inertia w="0.215" d="0.064" h="0.160" m="3"/>
-      </inertial>
-    </link>
-    <link name="${prefix}hitch_x">
-      <inertial>
-            <mass value="3" />
-            <origin xyz="0 0 0" rpy="0 0 0" />
-            <xacro:solid_cuboid_inertia w="0.215" d="0.064" h="0.160" m="3"/>
-      </inertial>
-      <visual>
-        <origin xyz="0.0 0.0 0.0" rpy="0.0 0.0 0.0"/>
-        <geometry>
-          <box size="0.215 0.160 0.064"/>
-        </geometry>
-      </visual>
-      <collision>
-        <origin xyz="0.0 0.0 0.0" rpy="0.0 0.0 0.0"/>
-        <geometry>
-          <box size="${hitch_length} ${hitch_width} ${hitch_height}"/>
-        </geometry>
-      </collision>
-    </link>
-    <!-- Hitch to Body -->
-    <link name="${prefix}body">
+  <xacro:macro name="cart" params="prefix connected">
+    <xacro:unless value="${connected}">
+      <link name="${prefix}base_footprint"/>
+    </xacro:unless>
+    <!-- Hitch to chassis -->
+    <link name="${prefix}chassis">
       <inertial>
         <mass value="${cart_mass}" />
-        <origin xyz="0 0 0" rpy="0 0 0" />
+        <origin xyz="-0.1 0 -0.1" rpy="0 0 0" />
         <inertia ixx="${(cart_mass*(cart_width*cart_width+cart_height*cart_height))/12}" ixy="0" ixz="0"
                   iyy="${(cart_mass*(cart_length*cart_length+cart_height*cart_height))/12}" iyz="0"
@@ -123,5 +75,5 @@
       </collision>
     </link>
-    <gazebo reference="${prefix}body">
+    <gazebo reference="${prefix}chassis">
       <material>Gazebo/Red</material>
     </gazebo>
@@ -129,7 +81,7 @@
     <link name="${prefix}rear_left_wheel">
       <inertial>
-            <mass value="1" />
+            <mass value="3" />
             <origin xyz="0 0 0" rpy="${PI/2} 0 0" />
-            <xacro:solid_cylinder_inertia m="1" r="${wheels_radius}" h="${wheels_width}"/>
+            <xacro:solid_cylinder_inertia m="3" r="${wheels_radius}" h="${wheels_width}"/>
       </inertial>
       <visual>
@@ -147,4 +99,5 @@
           <cylinder radius="${wheels_radius}" length="${wheels_width}"/>
         </geometry>
+        <contact_coefficients mu="1.0" kp="1.0" kd="1.0" />
       </collision>
     </link>
@@ -155,7 +108,7 @@
     <link name="${prefix}rear_right_wheel">
       <inertial>
-            <mass value="1" />
+            <mass value="3" />
             <origin xyz="0 0 0" rpy="${PI/2} 0 0" />
-            <xacro:solid_cylinder_inertia m="1" r="${wheels_radius}" h="${wheels_width}"/>
+            <xacro:solid_cylinder_inertia m="3" r="${wheels_radius}" h="${wheels_width}"/>
       </inertial>
       <visual>
@@ -173,4 +126,5 @@
           <cylinder radius="${wheels_radius}" length="${wheels_width}"/>
         </geometry>
+        <contact_coefficients mu="1.0" kp="1.0" kd="1.0" />
       </collision>
     </link>
@@ -269,4 +223,5 @@
           <cylinder radius="${front_wheel_radius}" length="${front_wheel_width}"/>
         </geometry>
+        <contact_coefficients mu="1.0" kp="1.0" kd="1.0" />
       </collision>
     </link>
@@ -295,4 +250,5 @@
           <cylinder radius="${front_wheel_radius}" length="${front_wheel_width}"/>
         </geometry>
+        <contact_coefficients mu="1.0" kp="1.0" kd="1.0" />
       </collision>
     </link>
@@ -305,5 +261,5 @@
         <origin xyz="0.0 0.0 0.0" rpy="0.0 0 0"/>
         <geometry>
-          <mesh filename="package://rbvogui_description/meshes/cart/Markers/meshes/Marker0.dae" scale="0.1 0.1 0.1"/>
+          <mesh filename="package://rbvogui_description/meshes/cart/Markers/meshes/Marker0.dae" scale="0.16 0.16 0.16"/>
         </geometry>
       </visual>
@@ -314,9 +270,37 @@
         <origin xyz="0.0 0.0 0.0" rpy="0.0 0 0"/>
         <geometry>
-          <mesh filename="package://rbvogui_description/meshes/cart/Markers/meshes/Marker1.dae" scale="0.1 0.1 0.1"/>
-        </geometry>
-      </visual>
-    </link>
-    <xacro:cart_joints prefix="${prefix}" parent="${parent}" connection="${connection}"/>
+          <mesh filename="package://rbvogui_description/meshes/cart/Markers/meshes/Marker1.dae" scale="0.16 0.16 0.16"/>
+        </geometry>
+      </visual>
+    </link>
+    <xacro:cart_joints prefix="${prefix}" connected="${connected}"/>
+    <gazebo>
+      <plugin name="cart_joint_state" filename="libgazebo_ros_joint_state_publisher.so">
+        <ros>
+          <xacro:if value="${connected}">
+            <namespace>robot</namespace>
+          </xacro:if>
+          <xacro:unless value="${connected}">
+            <namespace>robot/cart</namespace>
+          </xacro:unless>
+        </ros>
+        <update_rate>30</update_rate>
+        <xacro:if value="${connected}">
+          <joint_name>robot_hitch_x_joint</joint_name>
+          <joint_name>robot_hitch_y_joint</joint_name>
+          <joint_name>robot_hitch_z_joint</joint_name>
+          <joint_name>${prefix}chassis_joint</joint_name>
+        </xacro:if>
+        <joint_name>${prefix}rear_left_wheel_joint</joint_name>
+        <joint_name>${prefix}rear_right_wheel_joint</joint_name>
+        <joint_name>${prefix}front_right_wheel_support_joint</joint_name>
+        <joint_name>${prefix}front_left_wheel_support_joint</joint_name>
+        <joint_name>${prefix}front_right_wheel_joint</joint_name>
+        <joint_name>${prefix}front_left_wheel_joint</joint_name>
+      </plugin>
+    </gazebo>
   </xacro:macro>
+  <xacro:unless value="$(arg connected)">
+    <xacro:cart prefix="$(arg prefix)cart_" connected="$(arg connected)"/>
+  </xacro:unless>
 </robot>

File: rbvogui_description/urdf/cart/cart_joint.urdf.xacro (robot description, xacro)
@@ -1,61 +1,46 @@
 <?xml version="1.0"?>
 <robot xmlns:xacro="http://www.ros.org/wiki/xacro" name="robot_name">
-    <xacro:macro name="cart_joints" params="prefix parent connection">
-    <!-- Robot to BULON -->
-        <joint name="${prefix}bulon_joint" type="fixed">
-            <origin xyz="${bulon_x} 0 ${bulon_z}" rpy="0.0 0.0 0.0"/>
-            <parent link="${parent}"/>
-            <child link="${prefix}bulon"/>
-        </joint>
-    <!-- BULON to Hitch -->
-        <joint name="${prefix}hitch_z_joint" type="revolute">
-            <origin xyz="${hitch_x} 0 ${hitch_z}" rpy="0.0 0.0 0.0"/>
-            <parent link="${parent}"/>
-            <child link="${prefix}hitch_z"/>
-            <axis xyz="0.0 0.0 1.0"/>
-            <limit effort="1000" velocity="2000" lower="${-PI/7}" upper="${PI/7}"/>
-        </joint>
-        <joint name="${prefix}hitch_y_joint" type="revolute">
-            <origin xyz="0.0 0.0 0.0" rpy="0.0 0.0 0.0"/>
-            <parent link="${prefix}hitch_z"/>
-            <child link="${prefix}hitch_y"/>
-            <axis xyz="0.0 1.0 0.0"/>
-            <limit effort="1000" velocity="2000" lower="${-PI/7}" upper="${PI/7}"/>
-        </joint>
-        <joint name="${prefix}hitch_x_joint" type="revolute">
-            <origin xyz="0.0 0.0 0.0" rpy="0.0 0.0 0.0"/>
-            <parent link="${prefix}hitch_y"/>
-            <child link="${prefix}hitch_x"/>
-            <axis xyz="1.0 0.0 0.0"/>
-            <limit effort="1000" velocity="2000" lower="${-PI/7}" upper="${PI/7}"/>
-        </joint>
-    <!-- Hitch to Body -->
-        <joint name="${prefix}body_joint" type="revolute">
-            <origin xyz="${-cart_length/2 -hitch_length/2} 0 0" rpy="0.0 0.0 0.0"/>
-            <parent link="${prefix}hitch_x"/>
-            <child link="${prefix}body"/>
-            <axis xyz="0.0 1.0 0.0"/>
-            <limit effort="1000" velocity="2000" lower="-0.2" upper="0.2"/>
-        </joint>
+    <xacro:arg name="prefix" default="robot_cart_" />
+    <xacro:arg name="connected" default="true" />
+    <xacro:macro name="cart_joints" params="prefix connected">
+    <!-- Hitch to chassis -->
+        <xacro:if value="${connected}">
+            <joint name="${prefix}chassis_joint" type="revolute">
+                <origin xyz="${-cart_length/2 -hitch_length/2} 0 0" rpy="0.0 0.0 0.0"/>
+                <parent link="robot_hitch_x"/>
+                <child link="${prefix}chassis"/>
+                <axis xyz="0.0 1.0 0.0"/>
+                <limit effort="1000" velocity="2000" lower="-0.2" upper="0.2"/>
+            </joint>
+        </xacro:if>
+        <xacro:unless value="${connected}">
+            <joint name="${prefix}chassis_joint" type="fixed">
+                <origin xyz="0 0 0.3" rpy="0.0 0.0 0.0"/>
+                <parent link="${prefix}base_footprint"/>
+                <child link="${prefix}chassis"/>
+            </joint>
+        </xacro:unless>
     <!-- Rear Left wheel -->
         <joint name="${prefix}rear_left_wheel_joint" type="continuous">
             <origin xyz="${rear_wheel_x} ${rear_wheel_y} ${rear_wheel_z}" rpy="0.0 0.0 0.0"/>
-            <parent link="${prefix}body"/>
+            <parent link="${prefix}chassis"/>
             <child link="${prefix}rear_left_wheel"/>
             <axis xyz="0.0 1.0 0.0"/>
             <limit effort="1000" velocity="2000"/>
+            <dynamics damping="0.8" friction="2.0"/>
         </joint>
     <!-- Rear Right wheel -->
         <joint name="${prefix}rear_right_wheel_joint" type="continuous">
             <origin xyz="${rear_wheel_x} -${rear_wheel_y} ${rear_wheel_z}" rpy="0.0 0.0 0.0"/>
-            <parent link="${prefix}body"/>
+            <parent link="${prefix}chassis"/>
             <child link="${prefix}rear_right_wheel"/>
             <axis xyz="0.0 1.0 0.0"/>
             <limit effort="1000" velocity="2000"/>
+            <dynamics damping="0.8" friction="2.0"/>
         </joint>
     <!-- Front Right Wheel support base-->
         <joint name="${prefix}front_right_wheel_base_support_joint" type="fixed">
             <origin xyz="${front_caster_wheel_x} ${-front_caster_wheel_y} ${front_caster_wheel_z}" rpy="0.0 0.0 0.0"/>
-            <parent link="${prefix}body"/>
+            <parent link="${prefix}chassis"/>
             <child link="${prefix}front_right_wheel_base_support"/>
         </joint>
@@ -63,5 +48,5 @@
         <joint name="${prefix}front_left_wheel_base_support_joint" type="fixed">
             <origin xyz="${front_caster_wheel_x} ${front_caster_wheel_y} ${front_caster_wheel_z}" rpy="0.0 0.0 0.0"/>
-            <parent link="${prefix}body"/>
+            <parent link="${prefix}chassis"/>
             <child link="${prefix}front_left_wheel_base_support"/>
         </joint>
@@ -69,16 +54,18 @@
         <joint name="${prefix}front_right_wheel_support_joint" type="continuous">
             <origin xyz="${front_caster_wheel_x} ${-front_caster_wheel_y} ${front_caster_wheel_z}" rpy="0.0 0.0 0.0"/>
-            <parent link="${prefix}body"/>
+            <parent link="${prefix}chassis"/>
             <child link="${prefix}front_right_wheel_support"/>
             <axis xyz="0.0 0.0 1.0"/>
             <limit effort="1000" velocity="2000"/>
+            <dynamics damping="0.8" friction="2.0"/>
         </joint>
     <!-- Front Left Wheel support -->
         <joint name="${prefix}front_left_wheel_support_joint" type="continuous">
             <origin xyz="${front_caster_wheel_x} ${front_caster_wheel_y} ${front_caster_wheel_z}" rpy="0.0 0.0 0.0"/>
-            <parent link="${prefix}body"/>
+            <parent link="${prefix}chassis"/>
             <child link="${prefix}front_left_wheel_support"/>
             <axis xyz="0.0 0.0 1.0"/>
             <limit effort="1000" velocity="2000"/>
+            <dynamics damping="0.8" friction="2.0"/>
         </joint>
     <!-- Front Left wheel -->
@@ -89,4 +76,5 @@
             <axis xyz="0.0 1.0 0.0"/>
             <limit effort="1000" velocity="2000"/>
+            <dynamics damping="0.8" friction="2.0"/>
         </joint>
     <!-- Front Right wheel -->
@@ -97,15 +85,16 @@
             <axis xyz="0.0 1.0 0.0"/>
             <limit effort="1000" velocity="2000"/>
+            <dynamics damping="0.8" friction="2.0"/>
         </joint>
     <!-- Marker0 -->
         <joint name="${prefix}marker0_joint" type="fixed">
-            <origin xyz="0.66 -0.08 0.05" rpy="0.0 0.0 0.0"/>
-            <parent link="${prefix}body"/>
+            <origin xyz="0.67 -0.12 0.05" rpy="0.0 0.0 0.0"/>
+            <parent link="${prefix}chassis"/>
             <child link="${prefix}marker0"/>
         </joint>
     <!-- Marker1 -->
         <joint name="${prefix}marker1_joint" type="fixed">
-            <origin xyz="0.66 0.08 0.05" rpy="0.0 0.0 0.0"/>
-            <parent link="${prefix}body"/>
+            <origin xyz="0.67 0.12 0.05" rpy="0.0 0.0 0.0"/>
+            <parent link="${prefix}chassis"/>
             <child link="${prefix}marker1"/>
         </joint>

File: rbvogui_description/urdf/ros2_control.urdf.xacro (robot description, xacro)
@@ -1,5 +1,5 @@
 <?xml version="1.0"?>
 <robot xmlns:xacro="http://wiki.ros.org/xacro">
-    <xacro:macro name="ros2_control" params="prefix cart">
+    <xacro:macro name="ros2_control" params="prefix">
         <gazebo>
           <plugin name="ros_control" filename="libgazebo_ros2_control.so">
@@ -9,22 +9,4 @@
             <parameters>$(find rbvogui_gazebo)/config/base_controller.yaml</parameters>
           </plugin>
-          <xacro:if value="${cart}">
-            <plugin name="cart_joint_state" filename="libgazebo_ros_joint_state_publisher.so">
-              <ros>
-                <namespace>robot</namespace>
-              </ros>
-              <update_rate>30</update_rate>
-              <joint_name>robot_cart_hitch_z_joint</joint_name>
-              <joint_name>robot_cart_hitch_y_joint</joint_name>
-              <joint_name>robot_cart_hitch_x_joint</joint_name>
-              <joint_name>robot_cart_body_joint</joint_name>
-              <joint_name>robot_cart_rear_left_wheel_joint</joint_name>
-              <joint_name>robot_cart_rear_right_wheel_joint</joint_name>
-              <joint_name>robot_cart_front_right_wheel_support_joint</joint_name>
-              <joint_name>robot_cart_front_left_wheel_support_joint</joint_name>
-              <joint_name>robot_cart_front_right_wheel_joint</joint_name>
-              <joint_name>robot_cart_front_left_wheel_joint</joint_name>
-            </plugin>
-          </xacro:if>
         </gazebo>
         <xacro:macro name="ros2_joint" params="interface jmin jmax prefix name">

File: rbvogui_description/urdf/wheels/fixed_wheel.urdf.xacro (robot description, xacro)
@@ -23,6 +23,4 @@
   </xacro:macro>
   <xacro:macro name="fixed_wheel" params="prefix parent *origin reflect hq">
-    <!-- TODO: check reflect parameter -->
-    <!--MOTOR WHEEL -->
     <joint name="${prefix}fixed_wheel_joint" type="fixed">
       <parent link="${parent}"/>
@@ -30,5 +28,4 @@
       <xacro:insert_block name="origin" />
       <axis xyz="0 0 1" rpy="0 0 0" />
-      <!-- limit effort="${steer_joint_effort_limit}" velocity="${steer_joint_velocity_limit}" lower="-1.5708" upper="1.5708" / -->
       <limit effort="${steer_joint_effort_limit}" velocity="${steer_joint_velocity_limit}" lower="-3.00" upper="3.00"/>
       <joint_properties damping="${steer_joint_damping}" friction="${steer_joint_friction}"/>
@@ -90,60 +87,4 @@
         <origin xyz="0 0 0" rpy="0 0 0"/>
     </xacro:wheel>
-    <!--WHEEL TIRE
-    <joint name="${prefix}wheel_joint" type="continuous">
-      <parent link="${prefix}fixed_wheel"/>
-      <child link="${prefix}wheel"/>
-      <origin xyz="0 0 0" rpy="0 0 ${M_PI}" />
-      <axis xyz="0 1 0" rpy="0 0 0" />
-      <limit effort="${wheel_joint_effort_limit}" velocity="${wheel_joint_velocity_limit}"/>
-      <joint_properties damping="${wheel_joint_damping}" friction="{wheel_joint_friction}"/>
-    </joint>
-    <transmission name="${prefix}wheel_trans">
-      <type>transmission_interface/SimpleTransmission</type>
-      <joint name="${prefix}wheel_joint">
-        <hardwareInterface>hardware_interface/VelocityJointInterface</hardwareInterface>
-      </joint>
-      <actuator name="${prefix}wheel_motor">
-        <hardwareInterface>hardware_interface/VelocityActuatorInterface</hardwareInterface>
-        <mechanicalReduction>${wheel_mechanical_reduction}</mechanicalReduction>
-      </actuator>
-    </transmission>
-    <link name="${prefix}wheel">
-      <visual>
-         HIGH RESOLUTION WHEELS
-        <xacro:if value="${hq}">
-          <origin xyz="0 0 0" rpy="0 0 0" />
-          <geometry>
-            <xacro:if value="${reflect}">
-              <mesh filename="package://rbvogui_description/meshes/wheels/wheel_sxl.stl" />
-            </xacro:if>
-            <xacro:unless value="${reflect}">
-              <mesh filename="package://rbvogui_description/meshes/wheels/wheel_sxl.stl" />
-            </xacro:unless>
-          </geometry>
-        </xacro:if>
-         LOW RESOLUTION WHEELS
-        <xacro:unless value="${hq}">
-          <origin xyz="0 0 0" rpy="${M_PI/2} 0 0" />
-          <geometry>
-            <cylinder length="${wheel_height}" radius="${wheel_radius}" />
-          </geometry>
-        </xacro:unless>
-      </visual>
-      <collision>
-        <origin xyz="0 0 0" rpy="${M_PI/2} 0 0" />
-        <geometry>
-          <sphere radius="${wheel_radius}" />
-        </geometry>
-      </collision>
-      <inertial>
-        <mass value="${wheel_mass}" />
-        <origin xyz="0 0 0" rpy="${M_PI/2} 0 0" />
-        <cylinder_inertia m="${wheel_mass}" r="${wheel_radius}" h="${wheel_height}" />
-      </inertial>
-    </link>
-    <xacro:gazebo_color_wheel prefix="${prefix}"/>
-    <xacro:gazebo_color_steer_wheel prefix="${prefix}"/>
--->
   </xacro:macro>
 </robot>

File: rbvogui_description/urdf/wheels/fixed_wheel_xl.urdf.xacro (robot description, xacro)
@@ -17,5 +17,4 @@
   </xacro:macro>
   <xacro:macro name="fixed_wheel" params="prefix parent *origin reflect hq">
-    <!-- TODO: check reflect parameter -->
     <!--MOTOR WHEEL -->
     <joint name="${prefix}fixed_wheel_joint" type="fixed">

File: rbvogui_description/urdf/wheels/fixed_wheel_xl_offroad.urdf.xacro (robot description, xacro)
@@ -17,5 +17,4 @@
   </xacro:macro>
   <xacro:macro name="fixed_wheel" params="prefix parent *origin reflect hq">
-    <!-- TODO: check reflect parameter -->
     <!--MOTOR WHEEL -->
     <joint name="${prefix}fixed_wheel_joint" type="fixed">
