Commit message: Fixed URDF and updated navigation params

File: rbvogui_description/urdf/wheels/rubber_wheel_350mm.urdf.xacro (robot description, xacro)
@@ -23,5 +23,4 @@
   </xacro:macro>
   <xacro:macro name="wheel_350mm" params="prefix parent *origin reflect hq">
-    <!-- TODO: check reflect parameter -->
     <!--WHEEL TIRE -->
     <joint name="${prefix}wheel_joint" type="continuous">

Commit message: Nav config for ackermann

File: rbvogui_description/robots/rbvogui_std.urdf.xacro (robot description, xacro)
@@ -116,5 +116,5 @@
                    launch_lift="$(arg launch_lift)" lift_manufacturer="$(arg lift_manufacturer)" lift_model="$(arg lift_model)" cart="$(arg cart)" connected="$(arg connected)"/>
     <!-- Gazebo ros control pluggins -->
-    <xacro:include filename="$(find rbvogui_description)/urdf/ros2_control.urdf.xacro"/>
+    <xacro:include filename="$(find rbvogui_description)/urdf/ros2_control_ackermann.urdf.xacro"/>
     <xacro:ros2_control prefix="$(arg prefix)"/>
 </robot>

File: rbvogui_description/urdf/cart/cart_joint.urdf.xacro (robot description, xacro)
@@ -7,5 +7,5 @@
         <xacro:if value="${connected}">
             <joint name="${prefix}chassis_joint" type="revolute">
-                <origin xyz="${-cart_length/2 - 0.1} 0 0" rpy="0.0 0.0 0.0"/>
+                <origin xyz="${-cart_length/2 - 0.2} 0 0" rpy="0.0 0.0 0.0"/>
                 <parent link="robot_hitch_x"/>
                 <child link="${prefix}chassis"/>
@@ -101,5 +101,5 @@
     <!-- Marker10 -->
         <joint name="${prefix}marker10_joint" type="fixed">
-            <origin xyz="0.67 -0.08 0.05" rpy="0.0 0.0 0.0"/>
+            <origin xyz="0.67 -0.10 0.05" rpy="0.0 0.0 0.0"/>
             <parent link="${prefix}chassis"/>
             <child link="${prefix}marker10"/>
@@ -107,5 +107,5 @@
     <!-- Marker11 -->
         <joint name="${prefix}marker11_joint" type="fixed">
-            <origin xyz="0.67 0.08 0.05" rpy="0.0 0.0 0.0"/>
+            <origin xyz="0.67 0.10 0.05" rpy="0.0 0.0 0.0"/>
             <parent link="${prefix}chassis"/>
             <child link="${prefix}marker11"/>

Commit message: Add debs controller

File: rbvogui_description/robots/rbvogui_std.urdf.xacro (robot description, xacro)
@@ -57,4 +57,5 @@
         </xacro:steering_wheel>
         <xacro:if value="${kinematics == 'omni'}">
+            <xacro:include filename="$(find rbvogui_description)/urdf/ros2_control.urdf.xacro"/>
             <xacro:steering_wheel prefix="${prefix}back_left_" parent="${prefix}base_link" reflect="true" hq="true">
                 <origin xyz="-${wheel_offset_x} ${wheel_offset_y} ${wheel_offset_z}" rpy="0 0 0"/>
@@ -65,10 +66,18 @@
         </xacro:if>
         <xacro:if value="${kinematics == 'ackermann'}">
-            <xacro:fixed_wheel prefix="${prefix}back_left_" parent="${prefix}base_link" reflect="true" hq="true">
+            <xacro:include filename="$(find rbvogui_description)/urdf/ros2_control_ackermann.urdf.xacro"/>
+            <!-- TODO CHANGE WHEN CONTROLLER IS BETTER ADAPTED -->
+            <!-- <xacro:fixed_wheel prefix="${prefix}back_left_" parent="${prefix}base_link" reflect="true" hq="true">
                 <origin xyz="-${wheel_offset_x} ${wheel_offset_y} ${wheel_offset_z}" rpy="0 0 0"/>
             </xacro:fixed_wheel>
             <xacro:fixed_wheel prefix="${prefix}back_right_" parent="${prefix}base_link" reflect="false" hq="true">
                 <origin xyz="-${wheel_offset_x} -${wheel_offset_y} ${wheel_offset_z}" rpy="0 0 0"/>
-            </xacro:fixed_wheel>
+            </xacro:fixed_wheel> -->
+            <xacro:steering_wheel prefix="${prefix}back_left_" parent="${prefix}base_link" reflect="true" hq="true">
+                <origin xyz="-${wheel_offset_x} ${wheel_offset_y} ${wheel_offset_z}" rpy="0 0 0"/>
+            </xacro:steering_wheel>
+            <xacro:steering_wheel prefix="${prefix}back_right_" parent="${prefix}base_link" reflect="false" hq="true">
+                <origin xyz="-${wheel_offset_x} -${wheel_offset_y} ${wheel_offset_z}" rpy="0 0 0"/>
+            </xacro:steering_wheel>
         </xacro:if>
         <!-- SENSORS see robotnik_sensors for the specific configuration -->
@@ -110,4 +119,6 @@
             </xacro:if>
         </xacro:if>
+        <!-- Gazebo ros control pluggins -->
+        <xacro:ros2_control prefix="${prefix}"/>ç
     </xacro:macro>
     <xacro:rbvogui prefix="$(arg prefix)" kinematics="$(arg kinematics)" load_kinematics_file="$(arg load_kinematics_file)" gpu="$(arg gpu)" publish_bf="${publish_bf}" hq="${hq}"
@@ -115,6 +126,3 @@
                    launch_gripper="$(arg launch_gripper)" gripper_manufacturer="$(arg gripper_manufacturer)" gripper_model="$(arg gripper_model)"
                    launch_lift="$(arg launch_lift)" lift_manufacturer="$(arg lift_manufacturer)" lift_model="$(arg lift_model)" cart="$(arg cart)" connected="$(arg connected)"/>
-    <!-- Gazebo ros control pluggins -->
-    <xacro:include filename="$(find rbvogui_description)/urdf/ros2_control_ackermann.urdf.xacro"/>
-    <xacro:ros2_control prefix="$(arg prefix)"/>
 </robot>

Commit message: URDF updated

File: rbvogui_description/robots/rbvogui_std.urdf.xacro (robot description, xacro)
@@ -112,5 +112,5 @@
         -->
         <xacro:if value="${cart}">
-            <xacro:include filename="$(find rbvogui_description)/urdf/cart/cart_robot_connection.urdf.xacro" />
+            <xacro:include filename="$(find rbvogui_description)/urdf/cart/robot_cart_connection.urdf.xacro" />
             <xacro:cart_connection prefix="${prefix}" connected="${connected}"/>
             <xacro:if value="${connected}">
@@ -120,5 +120,5 @@
         </xacro:if>
         <!-- Gazebo ros control pluggins -->
-        <xacro:ros2_control prefix="${prefix}"/>ç
+        <xacro:ros2_control prefix="${prefix}"/>
     </xacro:macro>
     <xacro:rbvogui prefix="$(arg prefix)" kinematics="$(arg kinematics)" load_kinematics_file="$(arg load_kinematics_file)" gpu="$(arg gpu)" publish_bf="${publish_bf}" hq="${hq}"

File: rbvogui_description/urdf/cart/cart.urdf.xacro (robot description, xacro)
@@ -3,5 +3,6 @@
   <xacro:include filename="$(find rbvogui_description)/urdf/inertia.urdf.xacro" />
   <xacro:include filename="$(find rbvogui_description)/urdf/cart/cart_joint.urdf.xacro" />
-  <xacro:include filename="$(find rbvogui_description)/urdf/cart/cart_robot_connection.urdf.xacro" />
+  <xacro:include filename="$(find rbvogui_description)/urdf/cart/robot_cart_connection.urdf.xacro" />
+  <xacro:include filename="$(find rbvogui_description)/urdf/cart/markers.urdf.xacro" />
   <xacro:arg name="prefix" default="robot_" />
   <xacro:arg name="connected" default="false" />
@@ -50,5 +51,20 @@
       <link name="${prefix}base_footprint"/>
     </xacro:unless>
-    <!-- Hitch to chassis -->
+    <!-- Lanza -->
+    <link name="${prefix}lanza">
+      <visual>
+        <origin xyz="0.0 0.0 0.0" rpy="0.0 0 0"/>
+        <geometry>
+          <mesh filename="package://rbvogui_description/meshes/cart/lanza.stl" scale="1.0 1.0 1.0"/>
+        </geometry>
+      </visual>
+      <collision>
+        <origin xyz="0.0 0.0 0.0" rpy="0.0 0.0 0.0"/>
+        <geometry>
+          <mesh filename="package://rbvogui_description/meshes/cart/lanza.stl" scale="1.0 1.0 1.0"/>
+        </geometry>
+      </collision>
+    </link>
+    <!-- Chassis -->
     <link name="${prefix}chassis">
       <inertial>
@@ -256,41 +272,6 @@
       <material>Gazebo/Grey</material>
     </gazebo>
-    <!-- Marker00 -->
-    <link name="${prefix}marker00">
-      <visual>
-        <origin xyz="0.0 0.0 0.0" rpy="0.0 0 0"/>
-        <geometry>
-          <mesh filename="package://rbvogui_description/meshes/cart/Markers/meshes/Marker0.dae" scale="0.16 0.16 0.16"/>
-        </geometry>
-      </visual>
-    </link>
-    <!-- Marker01 -->
-    <link name="${prefix}marker01">
-      <visual>
-        <origin xyz="0.0 0.0 0.0" rpy="0.0 0 0"/>
-        <geometry>
-          <mesh filename="package://rbvogui_description/meshes/cart/Markers/meshes/Marker0.dae" scale="0.16 0.16 0.16"/>
-        </geometry>
-      </visual>
-    </link>
-    <!-- Marker10 -->
-    <link name="${prefix}marker10">
-      <visual>
-        <origin xyz="0.0 0.0 0.0" rpy="0.0 0 0"/>
-        <geometry>
-          <mesh filename="package://rbvogui_description/meshes/cart/Markers/meshes/Marker1.dae" scale="0.16 0.16 0.16"/>
-        </geometry>
-      </visual>
-    </link>
-    <!-- Marker11 -->
-    <link name="${prefix}marker11">
-      <visual>
-        <origin xyz="0.0 0.0 0.0" rpy="0.0 0 0"/>
-        <geometry>
-          <mesh filename="package://rbvogui_description/meshes/cart/Markers/meshes/Marker1.dae" scale="0.16 0.16 0.16"/>
-        </geometry>
-      </visual>
-    </link>
     <xacro:cart_joints prefix="${prefix}" connected="${connected}"/>
+    <xacro:markers prefix="${prefix}"/>
     <gazebo>
       <plugin name="cart_joint_state" filename="libgazebo_ros_joint_state_publisher.so">

File: rbvogui_description/urdf/cart/cart_joint.urdf.xacro (robot description, xacro)
@@ -4,8 +4,14 @@
     <xacro:arg name="connected" default="true" />
     <xacro:macro name="cart_joints" params="prefix connected">
+    <!-- Lanza -->
+        <joint name="${prefix}lanza_joint" type="fixed">
+            <origin xyz="0.0 0.0 0.0" rpy="3.141592 0.0 0.0"/>
+            <parent link="${prefix}chassis"/>
+            <child link="${prefix}lanza"/>
+        </joint>
     <!-- Hitch to chassis -->
         <xacro:if value="${connected}">
             <joint name="${prefix}chassis_joint" type="revolute">
-                <origin xyz="${-cart_length/2 - 0.2} 0 0" rpy="0.0 0.0 0.0"/>
+                <origin xyz="${-cart_length/2 - 0.285} 0 0" rpy="0.0 0.0 0.0"/>
                 <parent link="robot_hitch_x"/>
                 <child link="${prefix}chassis"/>
@@ -87,28 +93,4 @@
             <dynamics damping="0.8" friction="2.0"/>
         </joint>
-    <!-- Marker00 -->
-        <joint name="${prefix}marker00_joint" type="fixed">
-            <origin xyz="0.67 -0.3 0.05" rpy="0.0 0.0 0.0"/>
-            <parent link="${prefix}chassis"/>
-            <child link="${prefix}marker00"/>
-        </joint>
-    <!-- Marker01 -->
-        <joint name="${prefix}marker01_joint" type="fixed">
-            <origin xyz="0.67 0.3 0.05" rpy="0.0 0.0 0.0"/>
-            <parent link="${prefix}chassis"/>
-            <child link="${prefix}marker01"/>
-        </joint>
-    <!-- Marker10 -->
-        <joint name="${prefix}marker10_joint" type="fixed">
-            <origin xyz="0.67 -0.10 0.05" rpy="0.0 0.0 0.0"/>
-            <parent link="${prefix}chassis"/>
-            <child link="${prefix}marker10"/>
-        </joint>
-    <!-- Marker11 -->
-        <joint name="${prefix}marker11_joint" type="fixed">
-            <origin xyz="0.67 0.10 0.05" rpy="0.0 0.0 0.0"/>
-            <parent link="${prefix}chassis"/>
-            <child link="${prefix}marker11"/>
-        </joint>
     </xacro:macro>
 </robot>
