Commit message: description: Add color for rbvogui in rviz

File: rbvogui_description/urdf/bases/rbvogui_base_v3.urdf.xacro (robot description, xacro)
@@ -1,4 +1,4 @@
 <?xml version="1.0"?>
-<robot xmlns:xacro="http://www.ros.org/wiki/xacro">
+<robot xmlns:xacro="http://wiki.ros.org/xacro">
   <xacro:include filename="$(find rbvogui_description)/urdf/bases/rbvogui_base.gazebo.xacro" />
   <xacro:macro name="rbvogui_base" params="prefix publish_bf hq">
@@ -34,10 +34,10 @@
         <xacro:if value="${hq}">
           <geometry>
-            <mesh filename="package://rbvogui_description/meshes/bases/rbvogui_chassis.dae"/>
+            <mesh filename="package://rbvogui_description/meshes/bases/rbvogui_chassis_v3.stl"/>
           </geometry>
         </xacro:if>
         <xacro:unless value="${hq}">
           <geometry>
-            <mesh filename="package://rbvogui_description/meshes/bases/rbvogui_chassis.dae"/>
+            <mesh filename="package://rbvogui_description/meshes/bases/rbvogui_chassis_v3.dae"/>
           </geometry>
         </xacro:unless>
@@ -49,5 +49,5 @@
         <origin xyz="0 0 0" rpy="0 0 0 " />
         <geometry>
-          <mesh filename="package://rbvogui_description/meshes/bases/rbvogui_chassis.dae"/>
+          <mesh filename="package://rbvogui_description/meshes/bases/rbvogui_chassis_v3.stl"/>
         </geometry>
       </collision>
@@ -73,6 +73,6 @@
           </geometry>
         </xacro:unless>
-        <material name="lightgrey">
-          <color rgba="0.9 0.9 0.9 1"/>
+        <material name="lightred">
+          <color rgba="0.9 0.2 0.2 1"/>
         </material>
       </visual>

File: rbvogui_description/urdf/wheels/motor_wheel.urdf.xacro (robot description, xacro)
@@ -54,5 +54,5 @@
 		  </xacro:unless>
           <geometry>
-            <mesh filename="package://rbvogui_description/meshes/wheels/mw_frame.dae" />
+            <mesh filename="package://rbvogui_description/meshes/wheels/mw_frame.stl" />
           </geometry>
         </xacro:if>
@@ -66,7 +66,10 @@
 		  </xacro:unless>
           <geometry>
-            <mesh filename="package://rbvogui_description/meshes/wheels/mw_frame.stl" />
+            <mesh filename="package://rbvogui_description/meshes/wheels/mw_frame.dae" />
           </geometry>
         </xacro:unless>
+        <material name="red2">
+          <color rgba="0.9 0.1 0.1 1"/>
+        </material>
       </visual>
       <collision>
@@ -127,5 +130,5 @@
 		  </xacro:unless>
           <geometry>
-              <mesh filename="package://rbvogui_description/meshes/wheels/wheel_sxl.dae" />
+              <mesh filename="package://rbvogui_description/meshes/wheels/wheel_sxl.stl" />
           </geometry>
         </xacro:if>
@@ -142,4 +145,7 @@
           </geometry>
         </xacro:unless>
+        <material name="dark-gray">
+          <color rgba="0.25 0.25 0.25 1.0"/>
+        </material>
       </visual>
       <collision>
