Commit message: Update  physics, mass, frictions and deformations

File: rbvogui_description/urdf/bases/rbvogui_base.urdf.xacro (robot description, xacro)
@@ -9,7 +9,7 @@
     <link name="${prefix}case_link">
       <inertial>
-        <mass value="100.0" />
-        <origin xyz="0 0 0.128" />
-        <xacro:cuboid_inertia m="100.0" d="0.6" h="0.23" w="1.0" />
+        <mass value="150.0" />
+        <origin xyz="0 0 0.028" />
+        <xacro:cuboid_inertia m="150.0" d="0.6" h="0.23" w="1.0" />
       </inertial>
       <visual>

File: rbvogui_description/urdf/wheels/steering_wheel.urdf.xacro (robot description, xacro)
@@ -13,4 +13,5 @@
       <child link="${prefix}steer_link" />
       <axis xyz="0 0 1" />
+      <dynamics damping="1.0" friction="2.0"/>
       <limit effort="100" velocity="100" lower="-${2*M_PI/3}" upper="${2*M_PI/3}" />
     </joint>
@@ -44,5 +45,5 @@
       </inertial>
     </link>
-    <gazebo reference="${prefix}set_wheel_link">
+    <gazebo reference="${prefix}base_wheel_link">
       <material>Gazebo/Red</material>
     </gazebo>

File: rbvogui_description/urdf/wheels/wheel.urdf.xacro (robot description, xacro)
@@ -65,8 +65,8 @@
     <gazebo reference="${prefix}wheel_link">
       <material>Gazebo/DarkGrey</material>
-      <mu1>0.98</mu1>
-      <mu2>0.98</mu2>
-      <kp>2.75e5</kp>
-      <kd>5.25e2</kd>
+      <mu1>0.90</mu1>
+      <mu2>0.85</mu2>
+      <kp>4.75e5</kp>
+      <kd>8.25e2</kd>
     </gazebo>
   </xacro:macro>
