Commit message: Get urdf-devel branch changes

File: rbvogui_description/urdf/bases/rbvogui_6w_base.urdf.xacro (robot description, xacro)
@@ -27,5 +27,5 @@
     <!-- Chassis -->
     <joint name="${prefix}chassis_joint" type="fixed">
-      <origin xyz="-0.012 0 0.1775" rpy="0 0 0" /> <!-- Modificar para cada vogui -->
+      <origin xyz="0 0 0.24117" rpy="0 0 0 " /> <!-- Modificar para cada vogui -->
       <parent link="${prefix}base_link"/>
       <child link="${prefix}chassis_link" />
@@ -42,10 +42,10 @@
         <xacro:if value="${hq}">
           <geometry>
-            <mesh filename="package://rbvogui_description/meshes/bases/rbvogui_chassis.stl"/>
+            <mesh filename="package://rbvogui_description/meshes/bases/rbvogui_6w_chassis.stl"/>
           </geometry>
         </xacro:if>
         <xacro:unless value="${hq}">
           <geometry>
-            <mesh filename="package://rbvogui_description/meshes/bases/rbvogui_chassis.stl"/>
+            <mesh filename="package://rbvogui_description/meshes/bases/rbvogui_6w_chassis.stl"/>
           </geometry>
         </xacro:unless>
@@ -57,5 +57,5 @@
         <origin xyz="0 0 0" rpy="0 0 0 " />
         <geometry>
-          <mesh filename="package://rbvogui_description/meshes/bases/rbvogui_chassis.stl"/>
+          <mesh filename="package://rbvogui_description/meshes/bases/rbvogui_6w_chassis.stl"/>
         </geometry>
       </collision>
@@ -63,5 +63,5 @@
     <!-- Battery -->
     <joint name="${prefix}battery_joint" type="fixed">
-      <origin xyz="0.02952 0 0" rpy="0 0 0 " />
+      <origin xyz="0.02952 0 0" rpy="0 0 0 " /> <!-- To do: check and set new battery stl from origin -->
       <parent link="${prefix}chassis_link"/>
       <child link="${prefix}battery_link" />
@@ -99,5 +99,5 @@
     <!-- Contactors -->
     <joint name="${prefix}contactors_joint" type="fixed">
-      <origin xyz="0.5235 0 0.09265" rpy="0 0 0 " />
+      <origin xyz="0.5235 0 0.09265" rpy="0 0 0 " /> <!-- To do: check -->
       <parent link="${prefix}chassis_link"/>
       <child link="${prefix}contactors_link" />
@@ -124,5 +124,5 @@
     <!-- Logos -->
     <joint name="${prefix}base_logos_joint" type="fixed">
-      <origin xyz="0 0 -0.1775" rpy="0 0 0" />
+      <origin xyz="0 0 -0.1775" rpy="0 0 0 " />
       <parent link="${prefix}chassis_link"/>
       <child link="${prefix}base_logos_link" />
@@ -131,23 +131,29 @@
     <link name="${prefix}base_logos_link">
       <visual>
-        <origin xyz="-0.015 0 0" rpy="0 0 0 " />
+        <origin xyz="0 0 0" rpy="0 0 0" />
         <xacro:if value="${hq}">
           <geometry>
-            <mesh filename="package://rbvogui_description/meshes/bases/rbvogui_logos.stl" scale="1.001 1.076 1.001"/>
+            <mesh filename="package://rbvogui_description/meshes/bases/rbvogui_logos.stl" scale="1.001 1.001 1.001"/>
           </geometry>
         </xacro:if>
         <xacro:unless value="${hq}">
           <geometry>
-            <mesh filename="package://rbvogui_description/meshes/bases/rbvogui_logos.dae" scale="1.001 1.076 1.001"/>
+            <mesh filename="package://rbvogui_description/meshes/bases/rbvogui_logos.dae" scale="1.001 1.001 1.001"/>
           </geometry>
         </xacro:unless>
-        <material name="lightred">
-          <color rgba="0.9 0.2 0.2 1"/>
+        <material name="lightgrey">
+          <color rgba="0.9 0.9 0.9 1"/>
         </material>
       </visual>
+      <collision>
+        <origin xyz="0 0 0" rpy="0 0 0 " />
+        <geometry>
+          <mesh filename="package://rbvogui_description/meshes/bases/rbvogui_logos.stl" scale="1.001 1.001 1.001"/>
+        </geometry>
+      </collision>
     </link>
     <!-- Leds -->
     <joint name="${prefix}leds_joint" type="fixed">
-      <origin xyz="0 0 0.1025" rpy="0 0 0 " />
+      <origin xyz="0 0 0.1025" rpy="0 0 0 " /> <!-- To do: check -->
       <parent link="${prefix}chassis_link"/>
       <child link="${prefix}leds_link" />
@@ -165,6 +171,6 @@
     </link>
     <xacro:gazebo_color_base_link prefix="${prefix}"/>
+    <xacro:gazebo_color_battery_link prefix="${prefix}"/>
     <xacro:gazebo_color_chassis_link prefix="${prefix}"/>
-    <xacro:gazebo_color_battery_link prefix="${prefix}"/>
     <xacro:gazebo_color_contactors_link prefix="${prefix}"/>
     <xacro:gazebo_color_logo_link prefix="${prefix}"/>

File: rbvogui_description/urdf/bases/rbvogui_xl_base.urdf.xacro (robot description, xacro)
@@ -1,9 +1,9 @@
 <?xml version="1.0"?>
-<robot xmlns:xacro="http://www.ros.org/wiki/xacro">
+<robot xmlns:xacro="http://wiki.ros.org/xacro">
   <xacro:include filename="$(find rbvogui_description)/urdf/bases/rbvogui_base.gazebo.xacro" />
-  <xacro:macro name="rbvogui_base" params="prefix publish_bf hq">
+  <xacro:include filename="$(find rbvogui_description)/urdf/inertia.urdf.xacro" />
+  <xacro:macro name="rbvogui_base" params="prefix publish_bf base_height:=0.1425 hq">
     <!-- Robot mechanical and motor parameters -->
     <xacro:property name="PI" value="3.1415926535897931"/>
-    <xacro:property name="wheel_width" value="0.146" />
     <!-- BASE FOOTPRINT -->
     <xacro:if value="${publish_bf}">
@@ -17,5 +17,5 @@
       </link>
       <joint name="${prefix}base_footprint_joint" type="fixed">
-        <origin xyz="0 0 ${wheel_radius}" rpy="0 0 0" />
+        <origin xyz="0 0 ${base_height}" rpy="0 0 0" />
         <!-- ${wheel_radius} property must be defined inside wheel description -->
         <parent link="${prefix}base_footprint"/>
@@ -27,14 +27,15 @@
     <!-- Chassis -->
     <joint name="${prefix}chassis_joint" type="fixed">
-      <origin xyz="-0.012 0 0.1775" rpy="0 0 0" /> <!-- Modificar para cada vogui -->
+      <origin xyz="0 0 0.23376" rpy="0 0 0" />
       <parent link="${prefix}base_link"/>
       <child link="${prefix}chassis_link" />
     </joint>
-    <!-- Chassis -->
+   <!-- Chassis -->
     <link name="${prefix}chassis_link">
       <inertial>
         <mass value="25.0" />
-        <origin xyz="0 0 0" />
-        <inertia ixx="1.0" ixy="0.0" ixz="0.0" iyy="1.0" iyz="0.0" izz="1.0" />
+        <origin xyz="0 0 0.376" />
+        <!--inertia ixx="1.0" ixy="0.0" ixz="0.0" iyy="1.0" iyz="0.0" izz="1.0" /-->
+        <solid_cuboid_inertia  w="1.265" h="0.812" d="0.465" m="25"/>
       </inertial>
       <visual>
@@ -42,10 +43,10 @@
         <xacro:if value="${hq}">
           <geometry>
-            <mesh filename="package://rbvogui_description/meshes/bases/rbvogui_chassis.stl"/>
+            <mesh filename="package://rbvogui_description/meshes/bases/rbvogui_xl_chassis.stl"/>
           </geometry>
         </xacro:if>
         <xacro:unless value="${hq}">
           <geometry>
-            <mesh filename="package://rbvogui_description/meshes/bases/rbvogui_chassis.stl"/>
+            <mesh filename="package://rbvogui_description/meshes/bases/rbvogui_xl_chassis.stl"/>
           </geometry>
         </xacro:unless>
@@ -57,5 +58,5 @@
         <origin xyz="0 0 0" rpy="0 0 0 " />
         <geometry>
-          <mesh filename="package://rbvogui_description/meshes/bases/rbvogui_chassis.stl"/>
+          <mesh filename="package://rbvogui_description/meshes/bases/rbvogui_xl_chassis.stl"/>
         </geometry>
       </collision>
@@ -63,5 +64,5 @@
     <!-- Battery -->
     <joint name="${prefix}battery_joint" type="fixed">
-      <origin xyz="0.02952 0 0" rpy="0 0 0 " />
+      <origin xyz="0 0 0" rpy="0 0 0 " />
       <parent link="${prefix}chassis_link"/>
       <child link="${prefix}battery_link" />
@@ -78,10 +79,10 @@
         <xacro:if value="${hq}">
           <geometry>
-             <mesh filename="package://rbvogui_description/meshes/bases/rbvogui_battery.stl"/>
+             <mesh filename="package://rbvogui_description/meshes/bases/rbvogui_xl_battery.stl"/>
           </geometry>
         </xacro:if>
         <xacro:unless value="${hq}">
           <geometry>
-             <mesh filename="package://rbvogui_description/meshes/bases/rbvogui_battery.stl"/>
+             <mesh filename="package://rbvogui_description/meshes/bases/rbvogui_xl_battery.stl"/>
           </geometry>
         </xacro:unless>
@@ -93,5 +94,5 @@
         <origin xyz="0 0 0" rpy="0 0 0 " />
         <geometry>
-           <mesh filename="package://rbvogui_description/meshes/bases/rbvogui_battery.stl"/>
+           <mesh filename="package://rbvogui_description/meshes/bases/rbvogui_xl_battery.stl"/>
         </geometry>
       </collision>
@@ -99,5 +100,5 @@
     <!-- Contactors -->
     <joint name="${prefix}contactors_joint" type="fixed">
-      <origin xyz="0.5235 0 0.09265" rpy="0 0 0 " />
+      <origin xyz="0.6405 0 0.10264" rpy="0 0 0 " />
       <parent link="${prefix}chassis_link"/>
       <child link="${prefix}contactors_link" />
@@ -124,5 +125,5 @@
     <!-- Logos -->
     <joint name="${prefix}base_logos_joint" type="fixed">
-      <origin xyz="0 0 -0.1775" rpy="0 0 0" />
+      <origin xyz="0 0 -0.08376" rpy="0 0 0 " />
       <parent link="${prefix}chassis_link"/>
       <child link="${prefix}base_logos_link" />
@@ -131,13 +132,13 @@
     <link name="${prefix}base_logos_link">
       <visual>
-        <origin xyz="-0.015 0 0" rpy="0 0 0 " />
+        <origin xyz="0 0 -0.06" rpy="0 0 0" />
         <xacro:if value="${hq}">
           <geometry>
-            <mesh filename="package://rbvogui_description/meshes/bases/rbvogui_logos.stl" scale="1.001 1.076 1.001"/>
+            <mesh filename="package://rbvogui_description/meshes/bases/rbvogui_logos.stl" scale="1.24 1.24 1"/>
           </geometry>
         </xacro:if>
         <xacro:unless value="${hq}">
           <geometry>
-            <mesh filename="package://rbvogui_description/meshes/bases/rbvogui_logos.dae" scale="1.001 1.076 1.001"/>
+            <mesh filename="package://rbvogui_description/meshes/bases/rbvogui_logos.dae" scale="1.3 1.3 1"/>
           </geometry>
         </xacro:unless>
@@ -147,7 +148,6 @@
       </visual>
     </link>
-    <!-- Leds -->
     <joint name="${prefix}leds_joint" type="fixed">
-      <origin xyz="0 0 0.1025" rpy="0 0 0 " />
+      <origin xyz="0 0 0.12624" rpy="0 0 0 " />
       <parent link="${prefix}chassis_link"/>
       <child link="${prefix}leds_link" />
@@ -157,5 +157,5 @@
         <origin xyz="0 0 0" rpy="0 0 0.0" />
           <geometry>
-              <mesh filename="package://rbvogui_description/meshes/bases/rbvogui_leds.stl" />
+              <mesh filename="package://rbvogui_description/meshes/bases/rbvogui_xl_leds.stl" />
           </geometry>
         <material name="lightgreen">

Commit message: rbvogui_description: corrected inertias

File: rbvogui_description/urdf/bases/rbvogui_6w_base.urdf.xacro (robot description, xacro)
@@ -2,4 +2,5 @@
 <robot xmlns:xacro="http://www.ros.org/wiki/xacro">
   <xacro:include filename="$(find rbvogui_description)/urdf/bases/rbvogui_base.gazebo.xacro" />
+  <xacro:include filename="$(find rbvogui_description)/urdf/inertia.urdf.xacro" />
   <xacro:macro name="rbvogui_base" params="prefix publish_bf hq">
     <!-- Robot mechanical and motor parameters -->
@@ -36,5 +37,5 @@
         <mass value="25.0" />
         <origin xyz="0 0 0" />
-        <inertia ixx="1.0" ixy="0.0" ixz="0.0" iyy="1.0" iyz="0.0" izz="1.0" />
+        <xacro:solid_cuboid_inertia  w="1.04" h="0.65" d="0.352" m="25"/>
       </inertial>
       <visual>

File: rbvogui_description/urdf/bases/rbvogui_base.urdf.xacro (robot description, xacro)
@@ -2,4 +2,5 @@
 <robot xmlns:xacro="http://www.ros.org/wiki/xacro">
   <xacro:include filename="$(find rbvogui_description)/urdf/bases/rbvogui_base.gazebo.xacro" />
+  <xacro:include filename="$(find rbvogui_description)/urdf/inertia.urdf.xacro" />
   <xacro:macro name="rbvogui_base" params="prefix publish_bf hq">
     <!-- Robot mechanical and motor parameters -->
@@ -35,6 +36,6 @@
       <inertial>
         <mass value="25.0" />
-        <origin xyz="0 0 0" />
-        <inertia ixx="1.0" ixy="0.0" ixz="0.0" iyy="1.0" iyz="0.0" izz="1.0" />
+        <origin xyz="0 0 0" rpy="0.0 0.0 0.0"/>
+        <xacro:solid_cuboid_inertia  w="1.04" h="0.65" d="0.352" m="25"/>
       </inertial>
       <visual>

File: rbvogui_description/urdf/inertia.urdf.xacro (robot description, xacro)
@@ -10,5 +10,5 @@
   </xacro:macro>
   <!-- TODO Hollow sphere of radius r and mass m-->
-  <xacro:macro name="solid_sphere_inertia" params="m r">
+  <xacro:macro name="hollow_sphere_inertia" params="m r">
     <inertia  ixx="${(2*r*r*m)/3}" ixy = "0" ixz = "0"
               iyy="${(2*r*r*m)/3}" iyz = "0"

File: rbvogui_description/urdf/wheels/motor_wheel.urdf.xacro (robot description, xacro)
@@ -88,8 +88,8 @@
         <mass value="4" />
           <xacro:if value="${reflect}">
-            <origin xyz="0 0 0.0" rpy="0 0 0"/>
+            <origin xyz="0 0 0.12" rpy="0 ${M_PI/2} ${M_PI/2}"/>
           </xacro:if>
         <xacro:unless value="${reflect}">
-          <origin xyz="0 0 0.0" rpy="0 0 ${M_PI}"/>
+          <origin xyz="0 0 0.12" rpy="0 ${M_PI/2} ${3*M_PI/2}"/>
         </xacro:unless>
         <xacro:cylinder_inertia m="${wheel_mass}" r="${wheel_radius}" h="${wheel_width}" />

File: rbvogui_description/urdf/wheels/motor_wheel_xl.urdf.xacro (robot description, xacro)
@@ -82,11 +82,11 @@
         <mass value="4" />
         <xacro:if value="${reflect}">
-			    <origin xyz="0 0 0.12" rpy="0 0 ${M_PI}"/>
+			    <origin xyz="0 0.03 0.1" rpy="0 0 ${M_PI}"/>
 		    </xacro:if>
 		    <xacro:unless value="${reflect}">
-		    	<origin xyz="0 0 0.12" rpy="0 0 0"/>
+		    	<origin xyz="0 -0.03 0.1" rpy="0 0 0"/>
 		    </xacro:unless>
         <!-- To do: add real intertia-->
-        <xacro:cylinder_inertia m="5" r="0.1425" h="0.14"/>
+        <xacro:cylinder_inertia m="5" r="0.07" h="0.26"/>
       </inertial>
     </link>

File: rbvogui_description/urdf/wheels/rubber_wheel.urdf.xacro (robot description, xacro)
@@ -75,5 +75,5 @@
       <inertial>
         <mass value="${wheel_mass}" />
-        <origin xyz="0 0 0" />
+        <origin xyz="0 0 0" rpy="0 ${M_PI/2} ${M_PI/2}"/>
         <xacro:cylinder_inertia m="${wheel_mass}" r="${wheel_radius}" h="${wheel_height}" />
       </inertial>

File: rbvogui_description/urdf/wheels/rubber_wheel_285mm.urdf.xacro (robot description, xacro)
@@ -78,5 +78,5 @@
       <inertial>
         <mass value="${wheel_mass}" />
-        <origin xyz="0 0 0" />
+        <origin xyz="0 0 0" rpy="0 ${M_PI/2} ${M_PI/2}"/>
         <xacro:cylinder_inertia m="${wheel_mass}" r="${wheel_radius}" h="${wheel_height}" />
       </inertial>
