Commit message: common: Add six wheel rbvogui

File: rbvogui_description/urdf/structures/rocker.urdf.xacro (robot description, xacro)
@@ -1,12 +1,13 @@
 <?xml version="1.0"?>
 <robot name="structure" xmlns:xacro="http://wiki.ros.org/xacro">
-    <xacro:macro name="structure_drawer" params="prefix parent *origin">
-        <joint name="${prefix}_joint" type="fixed">
+    <xacro:macro name="structure_rocker" params="prefix parent *origin">
+        <!-- This joint should be flexible +-24deg in y -->
+        <joint name="${prefix}joint" type="fixed">
             <axis xyz="0 1 0"/>
             <xacro:insert_block name="origin"/>
             <parent link="${parent}"/>
-            <child link="${prefix}_link"/>
+            <child link="${prefix}link"/>
         </joint>
-        <link name="${prefix}_link">
+        <link name="${prefix}link">
             <!-- TODO: check inertia -->
             <inertial>
@@ -17,20 +18,20 @@
             <visual>
                 <origin rpy="0 0 0" xyz="0 0 0"/>
-                <material name="alu_color">
-                    <color rgba="0.1 0.1 0.1 1"/>
+                <material name="red_rocker">
+                    <color rgba="1.0 0.0 0.0 1"/>
                 </material>
                 <geometry>
-                    <mesh filename="package://rbvogui_description/meshes/structures/structure_drawer.stl"/>
+                    <mesh filename="package://rbvogui_description/meshes/structures/rocker_structure.stl"/>
                 </geometry>
             </visual>
             <collision>
-            <origin rpy="0 0 0" xyz="0 0 0"/>
-            <geometry>
-                <mesh filename="package://rbvogui_description/meshes/structures/structure_drawer.stl"/>
-            </geometry>
+                <origin rpy="0 0 0" xyz="0 0 0"/>
+                <geometry>
+                    <mesh filename="package://rbvogui_description/meshes/structures/rocker_structure.stl"/>
+                </geometry>
             </collision>
         </link>
-        <gazebo reference="${prefix}_link">
-            <material>Gazebo/Black</material>
+        <gazebo reference="${prefix}link">
+            <material>Gazebo/Red</material>
             <gravity>true</gravity>
         </gazebo>

File: rbvogui_description/urdf/wheels/wheel_v3.urdf.xacro (robot description, xacro)
@@ -44,4 +44,7 @@
     <link name="${prefix}wheel">
       <visual>
+        <material name="dark-gray">
+          <color rgba="0.25 0.25 0.25 1.0"/>
+        </material>
         <!-- HIGH RESOLUTION WHEELS -->
         <xacro:if value="${hq}">
@@ -49,8 +52,8 @@
           <geometry>
             <xacro:if value="${reflect}">
-              <mesh filename="package://rbvogui_description/meshes/wheels/wheel_sxl.dae" />
+              <mesh filename="package://rbvogui_description/meshes/wheels/wheel_sxl.stl" />
             </xacro:if>
             <xacro:unless value="${reflect}">
-              <mesh filename="package://rbvogui_description/meshes/wheels/wheel_sxl.dae" />
+              <mesh filename="package://rbvogui_description/meshes/wheels/wheel_sxl.stl" />
             </xacro:unless>
           </geometry>
