Commit message: description: Update bi arm support positions

File: rbvogui_description/urdf/structures/bi_arm_support.urdf.xacro (robot description, xacro)
@@ -46,5 +46,5 @@
     <xacro:if value="${load_kinematics_file}">
       <joint name="${prefix}left_arm_base_joint" type="fixed">
-        <origin xyz="0 0.0915 0.15044" rpy="0.9 0 3.1416"/>
+        <origin xyz="0 0.09549 0.14538" rpy="-0.9 0 0"/>
         <parent link="${prefix}G2_link" />
         <child link="${prefix}left_arm_base_link" />
@@ -57,5 +57,5 @@
     <xacro:unless value="${load_kinematics_file}">
       <joint name="${prefix}left_arm_base_joint" type="fixed">
-        <origin xyz="0 -0.0915 0.15044" rpy="0.9 0 3.1416"/>
+        <origin xyz="0 0.09549 0.14538" rpy="-0.9 0 0"/>
         <parent link="${prefix}G2_link" />
         <child link="${prefix}left_arm_base_link" />
@@ -67,5 +67,5 @@
     <xacro:if value="${load_kinematics_file}">
       <joint name="${prefix}right_arm_base_joint" type="fixed">
-        <origin xyz="0 -0.0915 0.15044" rpy="0.9 0 0"/>
+        <origin xyz="0 -0.09549 0.14538" rpy="-0.9 0 ${M_PI}"/>
         <parent link="${prefix}G2_link" />
         <child link="${prefix}right_arm_base_link" />
@@ -78,5 +78,5 @@
     <xacro:unless value="${load_kinematics_file}">
       <joint name="${prefix}right_arm_base_joint" type="fixed">
-        <origin xyz="0 -0.0915 0.15044" rpy="0.9 0 0"/>
+        <origin xyz="0 -0.09549 0.14538" rpy="-0.9 0 ${M_PI}"/>
         <parent link="${prefix}G2_link" />
         <child link="${prefix}right_arm_base_link" />
