Commit message: description: Update basket structure

File: rbvogui_description/urdf/structures/basket.urdf.xacro (robot description, xacro)
@@ -2,34 +2,5 @@
 <robot name="structure" xmlns:xacro="http://wiki.ros.org/xacro">
     <xacro:macro name="structure_basket" params="prefix parent *origin">
-        <joint name="${prefix}joint" type="fixed">
-            <axis xyz="0 1 0"/>
-            <xacro:insert_block name="origin"/>
-            <parent link="${parent}"/>
-            <child link="${prefix}basket_container_link"/>
-        </joint>
-        <link name="${prefix}basket_container_link">
-            <!-- TODO: check inertia -->
-            <inertial>
-                <mass value="0.001"/>
-                <origin rpy="0 0 0" xyz="0 0 0"/>
-                <inertia ixx="0.0001" ixy="0" ixz="0" iyy="0.000001" iyz="0" izz="0.0001"/>
-            </inertial>
-            <visual>
-                <origin rpy="0 0 0" xyz="0 0 0"/>
-                <material name="alu_color">
-                    <color rgba="0.1 0.1 0.1 1"/>
-                </material>
-                <geometry>
-                    <mesh filename="package://rbvogui_description/meshes/structures/basket_container.stl"/>
-                </geometry>
-            </visual>
-            <collision>
-            <origin rpy="0 0 0" xyz="0 0 0"/>
-            <geometry>
-                <mesh filename="package://rbvogui_description/meshes/structures/basket_container.stl"/>
-            </geometry>
-            </collision>
-        </link>
-        <joint name="${prefix}basket_container_joint" type="fixed">
+        <joint name="${prefix}basket_chassis_joint" type="fixed">
             <axis xyz="0 1 0"/>
             <xacro:insert_block name="origin"/>
@@ -60,6 +31,35 @@
             </collision>
         </link>
+        <joint name="${prefix}basket_container_joint" type="fixed">
+            <axis xyz="0 1 0"/>
+            <origin xyz="-0.068 0 0.013" rpy="0 0 0"/>
+            <parent link="${prefix}basket_chassis_link"/>
+            <child link="${prefix}basket_container_link"/>
+        </joint>
+        <link name="${prefix}basket_container_link">
+            <!-- TODO: check inertia -->
+            <inertial>
+                <mass value="0.001"/>
+                <origin rpy="0 0 0" xyz="0 0 0"/>
+                <inertia ixx="0.0001" ixy="0" ixz="0" iyy="0.000001" iyz="0" izz="0.0001"/>
+            </inertial>
+            <visual>
+                <origin rpy="0 0 0" xyz="0 0 0"/>
+                <material name="alu_color">
+                    <color rgba="0.1 0.1 0.1 1"/>
+                </material>
+                <geometry>
+                    <mesh filename="package://rbvogui_description/meshes/structures/basket_container.stl"/>
+                </geometry>
+            </visual>
+            <collision>
+            <origin rpy="0 0 0" xyz="0 0 0"/>
+            <geometry>
+                <mesh filename="package://rbvogui_description/meshes/structures/basket_container.stl"/>
+            </geometry>
+            </collision>
+        </link>
         <gazebo reference="${prefix}basket_container_link">
-            <material>Gazebo/Black</material>
+            <material>Gazebo/Red</material>
             <gravity>true</gravity>
         </gazebo>
