Commit message: Update gps_wifi_antenna.urdf.xacro collisions

File: rbvogui_description/urdf/structures/gps_wifi_antenna.urdf.xacro (robot description, xacro)
@@ -15,5 +15,5 @@
 			<mass value="0.2" />
 			<xacro:solid_cuboid_inertia m="0.2" w="0.081" h="0.081" d="0.03" />
-      </inertial>masl
+      </inertial>
 	    <visual>
 	      <origin rpy="0 0 0" xyz="0 0 0"/>
@@ -28,5 +28,5 @@
 	      <origin rpy="0 0 0" xyz="0 0 -0.15"/>
 	      <geometry>
-	        <cylinder radius="0.05" length="0.4"/>
+	        <cylinder radius="0.08" length="0.48"/>
 	      </geometry>
 	    </collision>
