Commit message: description: Reflect param for vogui xl wheels fixed

File: rbvogui_description/urdf/wheels/motor_wheel_xl.urdf.xacro (robot description, xacro)
@@ -47,8 +47,8 @@
         <xacro:if value="${hq}">
 		  <xacro:if value="${reflect}">
-			<origin xyz="0 0 0.27952" rpy="0 0 ${M_PI}" />
+			<origin xyz="0 0 0.27952" rpy="0 0 0" />
 		  </xacro:if>
 		  <xacro:unless value="${reflect}">
-			<origin xyz="0 0 0.27952" rpy="0 0 0.0" />
+			<origin xyz="0 0 0.27952" rpy="0 0 ${M_PI}" />
 		  </xacro:unless>
           <geometry>
@@ -59,8 +59,8 @@
         <xacro:unless value="${hq}">
           <xacro:if value="${reflect}">
-			<origin xyz="0 0 0.27952" rpy="0 0 ${M_PI}" />
+			<origin xyz="0 0 0.27952" rpy="0 0 0" />
 		  </xacro:if>
 		  <xacro:unless value="${reflect}">
-			<origin xyz="0 0 0.27952" rpy="0 0 0.0" />
+			<origin xyz="0 0 0.27952" rpy="0 0 ${M_PI}" />
 		  </xacro:unless>
           <geometry>
@@ -74,8 +74,8 @@
       <collision>
 		<xacro:if value="${reflect}">
-			<origin xyz="0 0 0.27952" rpy="0 0 ${M_PI}" />
+			<origin xyz="0 0 0.27952" rpy="0 0 0" />
 		</xacro:if>
 		<xacro:unless value="${reflect}">
-			<origin xyz="0 0 0.27952" rpy="0 0 0.0" />
+			<origin xyz="0 0 0.27952" rpy="0 0 ${M_PI}" />
 		</xacro:unless>
         <geometry>
@@ -99,11 +99,12 @@
       <parent link="${prefix}motor_wheel"/>
       <child link="${prefix}wheel"/>
-      <origin xyz="0 0 0" rpy="0 0 ${M_PI}" />
       <xacro:if value="${reflect}">
-		<axis xyz="0 -1 0" rpy="0 0 0" />
-	  </xacro:if>
+		     <origin xyz="0 0 0" rpy="0 0 0" />
+         <axis xyz="0 1 0" rpy="0 0 0" />
+	    </xacro:if>
       <xacro:unless value="${reflect}">
-		<axis xyz="0 1 0" rpy="0 0 0" />
-	  </xacro:unless>
+         <origin xyz="0 0 0" rpy="0 0 0" />
+		     <axis xyz="0 1 0" rpy="0 0 0" />
+	    </xacro:unless>
       <limit effort="${wheel_joint_effort_limit}" velocity="${wheel_joint_velocity_limit}"/>
       <joint_properties damping="${wheel_joint_damping}" friction="{wheel_joint_friction}"/>
@@ -124,5 +125,5 @@
         <xacro:if value="${hq}">
 		  <xacro:if value="${reflect}">
-			<origin xyz="0 0 0" rpy="${M_PI} 0 0" />
+			<origin xyz="0 0 0" rpy="0 0 ${M_PI}" />
 		  </xacro:if>
 		  <xacro:unless value="${reflect}">
@@ -136,5 +137,5 @@
         <xacro:unless value="${hq}">
           <xacro:if value="${reflect}">
-			<origin xyz="0 0 0" rpy="${M_PI} 0 0" />
+			<origin xyz="0 0 0" rpy="0 0 ${M_PI}" />
 		  </xacro:if>
 		  <xacro:unless value="${reflect}">

Commit message: rbvogui_description: rbvogui xl wheel collision replaced with a cylinder

File: rbvogui_description/urdf/wheels/motor_wheel_xl.urdf.xacro (robot description, xacro)
@@ -124,12 +124,12 @@
         <!-- HIGH RESOLUTION WHEELS -->
         <xacro:if value="${hq}">
-		  <xacro:if value="${reflect}">
-			<origin xyz="0 0 0" rpy="0 0 ${M_PI}" />
-		  </xacro:if>
-		  <xacro:unless value="${reflect}">
-			<origin xyz="0 0 0" rpy="0 0 0" />
-		  </xacro:unless>
+		      <xacro:if value="${reflect}">
+			      <origin xyz="0 0 0" rpy="0 0 ${M_PI}" />
+		      </xacro:if>
+          <xacro:unless value="${reflect}">
+            <origin xyz="0 0 0" rpy="0 0 0" />
+          </xacro:unless>
           <geometry>
-             <mesh filename="package://rbvogui_description/meshes/wheels/wheel_rbvogui_xl.stl" />
+              <mesh filename="package://rbvogui_description/meshes/wheels/wheel_rbvogui_xl.stl" />
           </geometry>
         </xacro:if>
@@ -137,9 +137,9 @@
         <xacro:unless value="${hq}">
           <xacro:if value="${reflect}">
-			<origin xyz="0 0 0" rpy="0 0 ${M_PI}" />
-		  </xacro:if>
-		  <xacro:unless value="${reflect}">
-			<origin xyz="0 0 0" rpy="0 0 0" />
-		  </xacro:unless>
+			      <origin xyz="0 0 0" rpy="0 0 ${M_PI}" />
+		      </xacro:if>
+		    <xacro:unless value="${reflect}">
+			    <origin xyz="0 0 0" rpy="0 0 0" />
+		    </xacro:unless>
           <geometry>
              <mesh filename="package://rbvogui_description/meshes/wheels/wheel_rbvogui_xl.dae" />
@@ -151,13 +151,19 @@
       </visual>
       <collision>
+        <!--
         <xacro:if value="${reflect}">
-			<origin xyz="0 0 0" rpy="${M_PI} 0 0" />
-		  </xacro:if>
-		  <xacro:unless value="${reflect}">
-			<origin xyz="0 0 0" rpy="0 0 0" />
-		  </xacro:unless>
-          <geometry>
-             <mesh filename="package://rbvogui_description/meshes/wheels/wheel_rbvogui_xl.dae" />
-          </geometry>
+			    <origin xyz="0 0 0" rpy="${M_PI} 0 0" />
+		    </xacro:if>
+		    <xacro:unless value="${reflect}">
+			    <origin xyz="0 0 0" rpy="0 0 0" />
+		    </xacro:unless>
+        <geometry>
+            <mesh filename="package://rbvogui_description/meshes/wheels/wheel_rbvogui_xl.dae" />
+        </geometry>
+        -->
+        <origin xyz="0 0 0" rpy="${M_PI/2} 0 0" />
+        <geometry>
+          <cylinder radius="${wheel_radius}" length="${wheel_width}"/>
+        </geometry>
       </collision>
       <inertial>
