Commit message: Update physics parameters

File: rbvogui_description/urdf/wheels/steering_wheel.urdf.xacro (robot description, xacro)
@@ -14,5 +14,5 @@
       <axis xyz="0 0 1" />
       <dynamics damping="1.0" friction="2.0"/>
-      <limit effort="100" velocity="100" lower="-${2*M_PI/3}" upper="${2*M_PI/3}" />
+      <limit effort="200" velocity="10" lower="-${2*M_PI/3}" upper="${2*M_PI/3}" />
     </joint>
     <link name="${prefix}steer_link" />

File: rbvogui_description/urdf/wheels/wheel.urdf.xacro (robot description, xacro)
@@ -17,7 +17,7 @@
       <child link="${prefix}wheel_link"/>
       <axis xyz="0 0 1"/>
-      <dynamics damping="0.1" friction="0.1"/>
-      <limit effort="1e9" velocity="1000.0"/>
-      <safety_controller k_velocity="0.1" k_position="0.1" soft_lower_limit="-${M_PI}" soft_upper_limit="${M_PI}"/>
+      <dynamics damping="0.1" friction="2"/>
+      <limit effort="100" velocity="100.0"/>
+      <!--safety_controller k_velocity="0.1" k_position="0.1" soft_lower_limit="-${M_PI}" soft_upper_limit="${M_PI}"/-->
     </joint>
     <link name="${prefix}wheel_link">
@@ -67,6 +67,6 @@
       <mu1>0.90</mu1>
       <mu2>0.85</mu2>
-      <kp>4.75e5</kp>
-      <kd>8.25e2</kd>
+      <kp>8.75e5</kp>
+      <kd>8.25e1</kd>
     </gazebo>
   </xacro:macro>

Commit message: Update physics

File: rbvogui_description/urdf/wheels/steering_wheel.urdf.xacro (robot description, xacro)
@@ -13,6 +13,7 @@
       <child link="${prefix}steer_link" />
       <axis xyz="0 0 1" />
-      <dynamics damping="1.0" friction="2.0"/>
-      <limit effort="200" velocity="10" lower="-${2*M_PI/3}" upper="${2*M_PI/3}" />
+      <dynamics damping="0.1" friction="2.0"/>
+      <limit effort="200.0" velocity="100.0" lower="-${2*M_PI/3}" upper="${2*M_PI/3}" />
+      <!--safety_limits lower="-${2*M_PI/3}" upper="${2*M_PI/3}" k_position="1" k_velocity="0.5" /-->
     </joint>
     <link name="${prefix}steer_link" />

File: rbvogui_description/urdf/wheels/wheel.urdf.xacro (robot description, xacro)
@@ -59,5 +59,5 @@
         </xacro:unless>
         <geometry>
-          <cylinder length="${tire_width}" radius="${tire_radius}" />
+          <cylinder length="${tire_width/2}" radius="${tire_radius}" />
         </geometry>
       </collision>
@@ -69,4 +69,6 @@
       <kp>8.75e5</kp>
       <kd>8.25e1</kd>
+      <fdir1>0 0 1</fdir1>
+      <maxContacts>4</maxContacts>
     </gazebo>
   </xacro:macro>

Commit message: Fix dynamics tag

File: rbvogui_description/urdf/wheels/steering_wheel.urdf.xacro (robot description, xacro)
@@ -12,5 +12,5 @@
     <xacro:property name="steer_joint_damping" value="1.0" />
     <xacro:property name="steer_joint_friction" value="1.0" />
-    <xacro:property name="steer_joint_effort_limit" value="100.0" />
+    <xacro:property name="steer_joint_effort_limit" value="200.0" />
     <xacro:property name="steer_joint_velocity_limit" value="100.0" />
     <!-- TODO: check reflect parameter -->
@@ -23,5 +23,5 @@
       <!-- limit effort="${steer_joint_effort_limit}" velocity="${steer_joint_velocity_limit}" lower="-1.5708" upper="1.5708" / -->
       <limit effort="${steer_joint_effort_limit}" velocity="${steer_joint_velocity_limit}" lower="-3.00" upper="3.00"/>
-      <joint_properties damping="${steer_joint_damping}" friction="${steer_joint_friction}"/>
+      <dynamics damping="${steer_joint_damping}" friction="${steer_joint_friction}"/>
     </joint>
     <link name="${prefix}base_wheel">
