Commit message: Wheels for xl version with reflect argument

File: rbvogui_description/urdf/wheels/fixed_wheel_xl.urdf.xacro (robot description, xacro)
@@ -21,26 +21,13 @@
     <inertia ixx="${m*(3*r*r+h*h)/12}" ixy = "0" ixz = "0" iyy="${m*(3*r*r+h*h)/12}" iyz = "0" izz="${m*r*r/2}" />
   </xacro:macro>
-  <xacro:macro name="motor_wheel" params="prefix parent *origin reflect hq">
+  <xacro:macro name="fixed_wheel" params="prefix parent *origin reflect hq">
     <!-- TODO: check reflect parameter -->
     <!--MOTOR WHEEL -->
-    <joint name="${prefix}motor_wheel_joint" type="revolute">
+    <joint name="${prefix}motor_wheel_joint" type="fixed">
       <parent link="${parent}"/>
       <child link="${prefix}motor_wheel"/>
       <xacro:insert_block name="origin" />
       <axis xyz="0 0 1" rpy="0 0 0" />
-      <!-- limit effort="${steer_joint_effort_limit}" velocity="${steer_joint_velocity_limit}" lower="-1.5708" upper="1.5708" / -->
-      <limit effort="${steer_joint_effort_limit}" velocity="${steer_joint_velocity_limit}" lower="-3.00" upper="3.00"/>
-      <joint_properties damping="${steer_joint_damping}" friction="${steer_joint_friction}"/>
     </joint>
-    <transmission name="${prefix}motor_wheel_trans">
-      <type>transmission_interface/SimpleTransmission</type>
-      <joint name="${prefix}motor_wheel_joint">
-        <hardwareInterface>hardware_interface/PositionJointInterface</hardwareInterface>
-      </joint>
-      <actuator name="${prefix}motor_wheel_motor">
-        <hardwareInterface>hardware_interface/PositionActuatorInterface</hardwareInterface>
-        <mechanicalReduction>${motor_wheel_mechanical_reduction}</mechanicalReduction>
-      </actuator>
-    </transmission>
     <link name="${prefix}motor_wheel">
       <visual>
@@ -92,5 +79,4 @@
 			<origin xyz="0 0 0.12" rpy="0 0 0"/>
 		</xacro:unless>
-        <!--inertia ixx="0.01" ixy="0.0" ixz="0.0" iyy="0.01" iyz="0.0" izz="0.01" /-->
         <cylinder_inertia m="${wheel_mass}" r="${wheel_radius}" h="${wheel_width}" />
       </inertial>

Commit message: description: Fix reflect param in fixed_wheel_xl

File: rbvogui_description/urdf/wheels/fixed_wheel_xl.urdf.xacro (robot description, xacro)
@@ -24,11 +24,11 @@
     <!-- TODO: check reflect parameter -->
     <!--MOTOR WHEEL -->
-    <joint name="${prefix}motor_wheel_joint" type="fixed">
+    <joint name="${prefix}fixed_wheel_joint" type="fixed">
       <parent link="${parent}"/>
-      <child link="${prefix}motor_wheel"/>
+      <child link="${prefix}fixed_wheel"/>
       <xacro:insert_block name="origin" />
       <axis xyz="0 0 1" rpy="0 0 0" />
     </joint>
-    <link name="${prefix}motor_wheel">
+    <link name="${prefix}fixed_wheel">
       <visual>
         <!-- HIGH RESOLUTION WHEELS -->
@@ -38,5 +38,5 @@
 		  </xacro:if>
 		  <xacro:unless value="${reflect}">
-			<origin xyz="0 0 0" rpy="0 0 0.0" />
+			<origin xyz="0 0 0.0" rpy="0 0 0" />
 		  </xacro:unless>
           <geometry>
@@ -50,5 +50,5 @@
 		  </xacro:if>
 		  <xacro:unless value="${reflect}">
-			<origin xyz="0 0 0" rpy="0 0 0.0" />
+			<origin xyz="0 0 0" rpy="0 0 0" />
 		  </xacro:unless>
           <geometry>
@@ -65,5 +65,5 @@
 		</xacro:if>
 		<xacro:unless value="${reflect}">
-			<origin xyz="0 0 0" rpy="0 0 0.0" />
+			<origin xyz="0 0 0.0" rpy="0 0 0" />
 		</xacro:unless>
         <geometry>
@@ -79,4 +79,5 @@
 			<origin xyz="0 0 0.12" rpy="0 0 0"/>
 		</xacro:unless>
+     <!--inertia ixx="0.01" ixy="0.0" ixz="0.0" iyy="0.01" iyz="0.0" izz="0.01" /-->
         <cylinder_inertia m="${wheel_mass}" r="${wheel_radius}" h="${wheel_width}" />
       </inertial>
@@ -84,11 +85,12 @@
     <!--WHEEL TIRE -->
     <joint name="${prefix}wheel_joint" type="continuous">
-      <parent link="${prefix}motor_wheel"/>
+      <parent link="${prefix}fixed_wheel"/>
       <child link="${prefix}wheel"/>
+      <xacro:if value="${reflect}">
       <origin xyz="0 0 0" rpy="0 0 0" />
-      <xacro:if value="${reflect}">
-		<axis xyz="0 -1 0" rpy="0 0 0" />
+		<axis xyz="0 1 0" rpy="0 0 0" />
 	  </xacro:if>
       <xacro:unless value="${reflect}">
+       <origin xyz="0 0 0" rpy="0 0 0" />
 		<axis xyz="0 1 0" rpy="0 0 0" />
 	  </xacro:unless>
@@ -137,4 +139,5 @@
       </visual>
       <collision>
+      <!--
         <xacro:if value="${reflect}">
 			<origin xyz="0 0 0" rpy="${M_PI} 0 0" />
@@ -145,4 +148,9 @@
           <geometry>
              <mesh filename="package://rbvogui_description/meshes/wheels/wheel_rbvogui_xl.stl" />
+        </geometry>
+        -->
+        <origin xyz="0 0 0" rpy="${M_PI/2} 0 0" />
+        <geometry>
+          <cylinder radius="${wheel_radius}" length="${wheel_width}"/>
           </geometry>
       </collision>

Commit message: rbvogui_description: added xacro tag to be consistent with Noetic and solved identation errors

File: rbvogui_description/urdf/wheels/fixed_wheel_xl.urdf.xacro (robot description, xacro)
@@ -69,11 +69,11 @@
         <mass value="4" />
         <xacro:if value="${reflect}">
-			<origin xyz="0 0 0.12" rpy="0 0 ${M_PI}"/>
-		</xacro:if>
-		<xacro:unless value="${reflect}">
-			<origin xyz="0 0 0.12" rpy="0 0 0"/>
-		</xacro:unless>
+			    <origin xyz="0 0 0.12" rpy="0 0 ${M_PI}"/>
+		    </xacro:if>
+		    <xacro:unless value="${reflect}">
+			    <origin xyz="0 0 0.12" rpy="0 0 0"/>
+		    </xacro:unless>
         <!-- To do: add real intertia-->
-        <cylinder_inertia m="5" r="0.1425" h="0.14"/>
+        <xacro:cylinder_inertia m="5" r="0.1425" h="0.14"/>
       </inertial>
     </link>

File: rbvogui_description/urdf/wheels/fixed_wheel_xl_offroad.urdf.xacro (robot description, xacro)
@@ -69,11 +69,11 @@
         <mass value="4" />
         <xacro:if value="${reflect}">
-			<origin xyz="0 0 0.12" rpy="0 0 ${M_PI}"/>
-		</xacro:if>
-		<xacro:unless value="${reflect}">
-			<origin xyz="0 0 0.12" rpy="0 0 0"/>
-		</xacro:unless>
+			    <origin xyz="0 0 0.12" rpy="0 0 ${M_PI}"/>
+		    </xacro:if>
+		    <xacro:unless value="${reflect}">
+			    <origin xyz="0 0 0.12" rpy="0 0 0"/>
+		    </xacro:unless>
         <!-- To do: add real intertia-->
-        <cylinder_inertia m="5" r="0.1425" h="0.14"/>
+        <xacro:cylinder_inertia m="5" r="0.1425" h="0.14"/>
       </inertial>
     </link>

File: rbvogui_description/urdf/wheels/motor_wheel_xl.urdf.xacro (robot description, xacro)
@@ -82,11 +82,11 @@
         <mass value="4" />
         <xacro:if value="${reflect}">
-			<origin xyz="0 0 0.12" rpy="0 0 ${M_PI}"/>
-		</xacro:if>
-		<xacro:unless value="${reflect}">
-			<origin xyz="0 0 0.12" rpy="0 0 0"/>
-		</xacro:unless>
+			    <origin xyz="0 0 0.12" rpy="0 0 ${M_PI}"/>
+		    </xacro:if>
+		    <xacro:unless value="${reflect}">
+		    	<origin xyz="0 0 0.12" rpy="0 0 0"/>
+		    </xacro:unless>
         <!-- To do: add real intertia-->
-        <cylinder_inertia m="5" r="0.1425" h="0.14"/>
+        <xacro:cylinder_inertia m="5" r="0.1425" h="0.14"/>
       </inertial>
     </link>

File: rbvogui_description/urdf/wheels/motor_wheel_xl_offroad.urdf.xacro (robot description, xacro)
@@ -82,11 +82,11 @@
         <mass value="4" />
         <xacro:if value="${reflect}">
-			<origin xyz="0 0 0.12" rpy="0 0 ${M_PI}"/>
-		</xacro:if>
-		<xacro:unless value="${reflect}">
-			<origin xyz="0 0 0.12" rpy="0 0 0"/>
-		</xacro:unless>
+			    <origin xyz="0 0 0.12" rpy="0 0 ${M_PI}"/>
+		    </xacro:if>
+		    <xacro:unless value="${reflect}">
+			    <origin xyz="0 0 0.12" rpy="0 0 0"/>
+		    </xacro:unless>
         <!-- To do: add real intertia-->
-        <cylinder_inertia m="5" r="0.1425" h="0.14"/>
+        <xacro:cylinder_inertia m="5" r="0.1425" h="0.14"/>
       </inertial>
     </link>
