Commit message: Added changes to motor_wheel.urdf.xacro file

File: rbvogui_description/urdf/wheels/motor_wheel.urdf.xacro (robot description, xacro)
@@ -2,8 +2,7 @@
 <robot xmlns:xacro="http://www.ros.org/wiki/xacro">
   <xacro:include filename="$(find rbvogui_description)/urdf/wheels/wheel.gazebo.xacro" />
-  <xacro:include filename="$(find rbvogui_description)/urdf/wheels/rubber_wheel.urdf.xacro" />
   <xacro:property name="M_PI" value="3.1415926535897931" />
   <!-- Wheels -->
-  <xacro:property name="wheel_radius" value="0.1175" /> <!-- teorically D: 0.235-->
+  <xacro:property name="wheel_radius" value="0.110" />
   <xacro:property name="wheel_width" value="0.110" />
   <xacro:property name="wheel_mass" value="5.0" />
@@ -46,26 +45,26 @@
     <link name="${prefix}motor_wheel">
       <visual>
-         <!-- HIGH RESOLUTION WHEELS -->
+        <!-- HIGH RESOLUTION WHEELS -->
         <xacro:if value="${hq}">
-          <xacro:if value="${reflect}">
-            <origin xyz="0 0 0.0" rpy="0 0 0" />
-          </xacro:if>
-          <xacro:unless value="${reflect}">
-            <origin xyz="0 0 0.0" rpy="0 0 ${M_PI}" />
-          </xacro:unless>
-            <geometry>
-              <mesh filename="package://rbvogui_description/meshes/wheels/mw_frame.stl" />
-            </geometry>
+		  <xacro:if value="${reflect}">
+			<origin xyz="0 0 0.0" rpy="0 0 0" />
+		  </xacro:if>
+		  <xacro:unless value="${reflect}">
+			<origin xyz="0 0 0.0" rpy="0 0 ${M_PI}" />
+		  </xacro:unless>
+          <geometry>
+            <mesh filename="package://rbvogui_description/meshes/wheels/mw_frame.stl" />
+          </geometry>
         </xacro:if>
-          <!-- LOW RESOLUTION WHEELS -->
+        <!-- LOW RESOLUTION WHEELS -->
         <xacro:unless value="${hq}">
           <xacro:if value="${reflect}">
-            <origin xyz="0 0 0.0" rpy="0 0 0" />
-          </xacro:if>
-          <xacro:unless value="${reflect}">
-            <origin xyz="0 0 0.0" rpy="0 0 ${M_PI}" />
-          </xacro:unless>
+			<origin xyz="0 0 0.0" rpy="0 0 0" />
+		  </xacro:if>
+		  <xacro:unless value="${reflect}">
+			<origin xyz="0 0 0.0" rpy="0 0 ${M_PI}" />
+		  </xacro:unless>
           <geometry>
-            <mesh filename="package://rbvogui_description/meshes/wheels/mw_frame.stl" />
+            <mesh filename="package://rbvogui_description/meshes/wheels/mw_frame.dae" />
           </geometry>
         </xacro:unless>
@@ -75,30 +74,26 @@
       </visual>
       <collision>
-        <xacro:if value="${reflect}">
-          <origin xyz="0 0 0.0" rpy="0 0 0" />
-        </xacro:if>
-        <xacro:unless value="${reflect}">
-          <origin xyz="0 0 0.0" rpy="0 0 ${M_PI}" />
-        </xacro:unless>
-        <geometry>
-          <mesh filename="package://rbvogui_description/meshes/wheels/mw_frame.stl" />
-        </geometry>
+		  <xacro:if value="${reflect}">
+			<origin xyz="0 0 0.0" rpy="0 0 0" />
+		  </xacro:if>
+		  <xacro:unless value="${reflect}">
+			<origin xyz="0 0 0.0" rpy="0 0 ${M_PI}" />
+		  </xacro:unless>
+		  <geometry>
+			<mesh filename="package://rbvogui_description/meshes/wheels/mw_frame.dae" />
+		  </geometry>
       </collision>
       <inertial>
         <mass value="4" />
-          <xacro:if value="${reflect}">
-            <origin xyz="0 0 0.0" rpy="0 0 0"/>
-          </xacro:if>
-        <xacro:unless value="${reflect}">
-          <origin xyz="0 0 0.0" rpy="0 0 ${M_PI}"/>
-        </xacro:unless>
-        <cylinder_inertia m="${wheel_mass}" r="${wheel_radius}" h="${wheel_width}" />
+        <xacro:if value="${reflect}">
+			<origin xyz="0 0 0.0" rpy="0 0 0"/>
+		</xacro:if>
+		<xacro:unless value="${reflect}">
+			<origin xyz="0 0 0.0" rpy="0 0 ${M_PI}"/>
+		</xacro:unless>
+        <xacro:cylinder_inertia m="${wheel_mass}" r="${wheel_radius}" h="${wheel_width}" />
       </inertial>
     </link>
-    <xacro:gazebo_color_wheel_frame prefix="${prefix}"/>
-    <xacro:wheel prefix="${prefix}" parent="${prefix}motor_wheel" reflect="${reflect}" hq="${hq}">
-        <origin xyz="0 0 0" rpy="0 0 0"/>
-    </xacro:wheel>
-    <!--WHEEL TIRE
+    <!--WHEEL TIRE -->
     <joint name="${prefix}wheel_joint" type="continuous">
       <parent link="${prefix}motor_wheel"/>
@@ -126,4 +121,5 @@
     <link name="${prefix}wheel">
       <visual>
+        <!-- HIGH RESOLUTION WHEELS -->
         <xacro:if value="${hq}">
 		  <xacro:if value="${reflect}">
@@ -137,4 +133,5 @@
           </geometry>
         </xacro:if>
+        <!-- LOW RESOLUTION WHEELS -->
         <xacro:unless value="${hq}">
            <xacro:if value="${reflect}">
@@ -171,10 +168,9 @@
 			<origin xyz="0 0 0" rpy="${M_PI/2} 0 0" />
 		</xacro:unless>
-        <cylinder_inertia m="${wheel_mass}" r="${wheel_radius}" h="${wheel_width}" />
+        <xacro:cylinder_inertia m="${wheel_mass}" r="${wheel_radius}" h="${wheel_width}" />
       </inertial>
     </link>
     <xacro:gazebo_color_wheel prefix="${prefix}"/>
     <xacro:gazebo_color_steer_wheel prefix="${prefix}"/>
--->
   </xacro:macro>
 </robot>

Commit message: Revert last commit 6f6ccc1da3faa1cc9425bee59a0e7b81f921d011

File: rbvogui_description/urdf/wheels/motor_wheel.urdf.xacro (robot description, xacro)
@@ -2,7 +2,8 @@
 <robot xmlns:xacro="http://www.ros.org/wiki/xacro">
   <xacro:include filename="$(find rbvogui_description)/urdf/wheels/wheel.gazebo.xacro" />
+  <xacro:include filename="$(find rbvogui_description)/urdf/wheels/rubber_wheel.urdf.xacro" />
   <xacro:property name="M_PI" value="3.1415926535897931" />
   <!-- Wheels -->
-  <xacro:property name="wheel_radius" value="0.110" />
+  <xacro:property name="wheel_radius" value="0.1175" /> <!-- teorically D: 0.235-->
   <xacro:property name="wheel_width" value="0.110" />
   <xacro:property name="wheel_mass" value="5.0" />
@@ -45,26 +46,26 @@
     <link name="${prefix}motor_wheel">
       <visual>
-        <!-- HIGH RESOLUTION WHEELS -->
+         <!-- HIGH RESOLUTION WHEELS -->
         <xacro:if value="${hq}">
-		  <xacro:if value="${reflect}">
-			<origin xyz="0 0 0.0" rpy="0 0 0" />
-		  </xacro:if>
-		  <xacro:unless value="${reflect}">
-			<origin xyz="0 0 0.0" rpy="0 0 ${M_PI}" />
-		  </xacro:unless>
+          <xacro:if value="${reflect}">
+            <origin xyz="0 0 0.0" rpy="0 0 0" />
+          </xacro:if>
+          <xacro:unless value="${reflect}">
+            <origin xyz="0 0 0.0" rpy="0 0 ${M_PI}" />
+          </xacro:unless>
+            <geometry>
+              <mesh filename="package://rbvogui_description/meshes/wheels/mw_frame.stl" />
+            </geometry>
+        </xacro:if>
+          <!-- LOW RESOLUTION WHEELS -->
+        <xacro:unless value="${hq}">
+          <xacro:if value="${reflect}">
+            <origin xyz="0 0 0.0" rpy="0 0 0" />
+          </xacro:if>
+          <xacro:unless value="${reflect}">
+            <origin xyz="0 0 0.0" rpy="0 0 ${M_PI}" />
+          </xacro:unless>
           <geometry>
             <mesh filename="package://rbvogui_description/meshes/wheels/mw_frame.stl" />
-          </geometry>
-        </xacro:if>
-        <!-- LOW RESOLUTION WHEELS -->
-        <xacro:unless value="${hq}">
-          <xacro:if value="${reflect}">
-			<origin xyz="0 0 0.0" rpy="0 0 0" />
-		  </xacro:if>
-		  <xacro:unless value="${reflect}">
-			<origin xyz="0 0 0.0" rpy="0 0 ${M_PI}" />
-		  </xacro:unless>
-          <geometry>
-            <mesh filename="package://rbvogui_description/meshes/wheels/mw_frame.dae" />
           </geometry>
         </xacro:unless>
@@ -74,26 +75,30 @@
       </visual>
       <collision>
-		  <xacro:if value="${reflect}">
-			<origin xyz="0 0 0.0" rpy="0 0 0" />
-		  </xacro:if>
-		  <xacro:unless value="${reflect}">
-			<origin xyz="0 0 0.0" rpy="0 0 ${M_PI}" />
-		  </xacro:unless>
-		  <geometry>
-			<mesh filename="package://rbvogui_description/meshes/wheels/mw_frame.dae" />
-		  </geometry>
+        <xacro:if value="${reflect}">
+          <origin xyz="0 0 0.0" rpy="0 0 0" />
+        </xacro:if>
+        <xacro:unless value="${reflect}">
+          <origin xyz="0 0 0.0" rpy="0 0 ${M_PI}" />
+        </xacro:unless>
+        <geometry>
+          <mesh filename="package://rbvogui_description/meshes/wheels/mw_frame.stl" />
+        </geometry>
       </collision>
       <inertial>
         <mass value="4" />
-        <xacro:if value="${reflect}">
-			<origin xyz="0 0 0.0" rpy="0 0 0"/>
-		</xacro:if>
-		<xacro:unless value="${reflect}">
-			<origin xyz="0 0 0.0" rpy="0 0 ${M_PI}"/>
-		</xacro:unless>
-        <xacro:cylinder_inertia m="${wheel_mass}" r="${wheel_radius}" h="${wheel_width}" />
+          <xacro:if value="${reflect}">
+            <origin xyz="0 0 0.0" rpy="0 0 0"/>
+          </xacro:if>
+        <xacro:unless value="${reflect}">
+          <origin xyz="0 0 0.0" rpy="0 0 ${M_PI}"/>
+        </xacro:unless>
+        <cylinder_inertia m="${wheel_mass}" r="${wheel_radius}" h="${wheel_width}" />
       </inertial>
     </link>
-    <!--WHEEL TIRE -->
+    <xacro:gazebo_color_wheel_frame prefix="${prefix}"/>
+    <xacro:wheel prefix="${prefix}" parent="${prefix}motor_wheel" reflect="${reflect}" hq="${hq}">
+        <origin xyz="0 0 0" rpy="0 0 0"/>
+    </xacro:wheel>
+    <!--WHEEL TIRE
     <joint name="${prefix}wheel_joint" type="continuous">
       <parent link="${prefix}motor_wheel"/>
@@ -121,5 +126,4 @@
     <link name="${prefix}wheel">
       <visual>
-        <!-- HIGH RESOLUTION WHEELS -->
         <xacro:if value="${hq}">
 		  <xacro:if value="${reflect}">
@@ -133,5 +137,4 @@
           </geometry>
         </xacro:if>
-        <!-- LOW RESOLUTION WHEELS -->
         <xacro:unless value="${hq}">
            <xacro:if value="${reflect}">
@@ -168,9 +171,10 @@
 			<origin xyz="0 0 0" rpy="${M_PI/2} 0 0" />
 		</xacro:unless>
-        <xacro:cylinder_inertia m="${wheel_mass}" r="${wheel_radius}" h="${wheel_width}" />
+        <cylinder_inertia m="${wheel_mass}" r="${wheel_radius}" h="${wheel_width}" />
       </inertial>
     </link>
     <xacro:gazebo_color_wheel prefix="${prefix}"/>
     <xacro:gazebo_color_steer_wheel prefix="${prefix}"/>
+-->
   </xacro:macro>
 </robot>
