Commit message: description/rubber_wheel: Set wheel radius to 0.1165

File: rbvogui_description/urdf/wheels/rubber_wheel.urdf.xacro (robot description, xacro)
@@ -4,6 +4,6 @@
   <xacro:property name="M_PI" value="3.1415926535897931" />
   <!-- Wheels -->
-  <xacro:property name="wheel_radius" value="0.1175" />
-  <xacro:property name="wheel_height" value="0.1175" />
+  <xacro:property name="wheel_radius" value="0.1165" /> <!-- rbvogui uses wheels with 0.233 m of diameter-->
+  <xacro:property name="wheel_height" value="0.1165" />
   <xacro:property name="wheel_mass" value="5.0" />
   <!-- in kg-->

Commit message: Added color to rubber wheel

File: rbvogui_description/urdf/wheels/rubber_wheel.urdf.xacro (robot description, xacro)
@@ -27,16 +27,13 @@
     <link name="${prefix}wheel">
       <visual>
-        <material name="dark-gray">
-          <color rgba="0.25 0.25 0.25 1.0"/>
-        </material>
         <!-- HIGH RESOLUTION WHEELS -->
         <xacro:if value="${hq}">
-          <origin xyz="0 0 0" rpy="0 0 0" />
+          <origin xyz="0 0 0" rpy="${M_PI/2} 0 0" />
           <geometry>
             <xacro:if value="${reflect}">
-              <mesh filename="package://rbvogui_description/meshes/wheels/wheel_sxl.stl" />
+              <mesh filename="package://rbvogui_description/meshes/wheels/wheel_sxl_color.dae" />
             </xacro:if>
             <xacro:unless value="${reflect}">
-              <mesh filename="package://rbvogui_description/meshes/wheels/wheel_sxl.stl" />
+              <mesh filename="package://rbvogui_description/meshes/wheels/wheel_sxl_color.dae" />
             </xacro:unless>
           </geometry>
@@ -64,5 +61,5 @@
     <!-- GAZEBO PARAMETERS -->
     <xacro:gazebo_rubber_tire_physics name="${prefix}wheel" />
-    <xacro:gazebo_rubber_tire_material name="${prefix}wheel" />
+    <!--xacro:gazebo_rubber_tire_material name="${prefix}wheel" /-->
   </xacro:macro>
 </robot>

Commit message: Fix wheel spin

File: rbvogui_description/urdf/wheels/rubber_wheel.urdf.xacro (robot description, xacro)
@@ -21,5 +21,10 @@
       <child link="${prefix}wheel"/>
       <xacro:insert_block name="origin" />
-      <axis xyz="0 1 0" rpy="0 0 0" />
+      <xacro:if value="${reflect}">
+        <axis xyz="0 1 0" rpy="0 0 0" />
+      </xacro:if>
+      <xacro:unless value="${reflect}">
+        <axis xyz="0 -1 0" rpy="0 0 0" />
+      </xacro:unless>
       <limit effort="${wheel_joint_effort_limit}" velocity="${wheel_joint_velocity_limit}"/>
       <dynamics damping="${wheel_joint_damping}" friction="${wheel_joint_friction}"/>

File: rbvogui_description/urdf/wheels/steering_wheel.urdf.xacro (robot description, xacro)
@@ -20,5 +20,5 @@
       <child link="${prefix}base_wheel"/>
       <xacro:insert_block name="origin" />
-      <axis xyz="0 0 1" rpy="0 0 0" />
+      <axis xyz="0 0 -1" rpy="0 0 0" />
       <!-- limit effort="${steer_joint_effort_limit}" velocity="${steer_joint_velocity_limit}" lower="-1.5708" upper="1.5708" / -->
       <limit effort="${steer_joint_effort_limit}" velocity="${steer_joint_velocity_limit}" lower="-3.00" upper="3.00"/>
