Commit message: Update urdf links to std robotnik

File: rbvogui_description/robot/rbvogui_std.urdf.xacro (robot description, xacro)
@@ -1,62 +1,75 @@
 <?xml version="1.0"?>
-<!-- RBVogui v3.0 -->
-<robot name="rbvogui" xmlns:xacro="http://www.ros.org/wiki/xacro">
-    <!-- ***************** -->
-    <!-- Imported elements -->
-    <!-- ***************** -->
-    <!-- First we import all posible elements defined in the urdf.xacro files. All these elements are defined as macro:xacros -->
-    <!-- Import rbvogui base elements-->
-    <xacro:include filename="$(find rbvogui_description)/urdf/bases/rbvogui_base_v3.urdf.xacro" />
-    <!-- Import rbvogui wheels -->
-    <xacro:include filename="$(find rbvogui_description)/urdf/wheels/motor_wheel.urdf.xacro" />
-    <xacro:include filename="$(find rbvogui_description)/urdf/wheels/wheel_v3.urdf.xacro" />
-    <!-- Import all available sensors -->
-    <xacro:include filename="$(find robotnik_sensors)/urdf/all_sensors.urdf.xacro" />
-    <xacro:property name="PI" value="3.1415926535897931"/>
-    <xacro:property name="deg2rad" value="0.01745329251"/>
-    <!-- Wheel parameters -->
-    <xacro:property name="wheel_offset_x" value="0.380" />    <!-- x,y,z in translation from base_link to the center of the wheel -->
-    <xacro:property name="wheel_offset_y" value="0.23975" />
-    <xacro:property name="wheel_offset_z" value="0.0" />
-    <!-- Flag to select the high or low quality model -->
-    <xacro:property name="hq" value="true" />
-    <xacro:property name="publish_bf" value="true" />
-    <xacro:arg name="prefix" default="robot_" />
-    <xacro:arg name="gpu" default="true" />
-    <xacro:arg name="load_kinematics_file" default="false"/>
-    <xacro:macro name="rbvogui" params="prefix publish_bf hq load_kinematics_file gpu">
-        <!-- *************** -->
-        <!-- Robots Elements -->
-        <!-- *************** -->
-        <!-- Here we create the robot elements using the xacro:macros imported at the beggining of this file -->
-        <xacro:rbvogui_base prefix="${prefix}" publish_bf="${publish_bf}" hq="${hq}"/>
-        <xacro:motor_wheel prefix="${prefix}front_right_" parent="${prefix}base_link" reflect="false" hq="true">
-            <origin xyz="${wheel_offset_x} -${wheel_offset_y} ${wheel_offset_z}" rpy="0 0 0"/>
-        </xacro:motor_wheel>
-        <xacro:motor_wheel prefix="${prefix}front_left_" parent="${prefix}base_link" reflect="true" hq="true">
-            <origin xyz="${wheel_offset_x} ${wheel_offset_y} ${wheel_offset_z}" rpy="0 0 0"/>
-        </xacro:motor_wheel>
-        <xacro:motor_wheel prefix="${prefix}back_left_" parent="${prefix}base_link" reflect="true" hq="true">
-            <origin xyz="-${wheel_offset_x} ${wheel_offset_y} ${wheel_offset_z}" rpy="0 0 0"/>
-        </xacro:motor_wheel>
-        <xacro:motor_wheel prefix="${prefix}back_right_" parent="${prefix}base_link" reflect="false" hq="true">
-            <origin xyz="-${wheel_offset_x} -${wheel_offset_y} ${wheel_offset_z}" rpy="0 0 0"/>
-        </xacro:motor_wheel>
-        <!-- SENSORS see robotnik_sensors for the specific configuration -->
-        <!-- IMU -->
-        <xacro:sensor_imu_hector prefix="${prefix}imu" parent="${prefix}base_link">
-            <origin xyz="0.3 0.3 0.250" rpy="0 0 0"/>
-        </xacro:sensor_imu_hector>
-        <!-- GPS -->
-        <xacro:sensor_gps prefix="${prefix}gps" parent="${prefix}base_link">
-            <origin xyz="-0.04625 0.0 0.4" rpy="0 0 0"/>
-        </xacro:sensor_gps>
-        <!-- 2d laser -->
-        <xacro:sensor_sick_tim551 prefix="${prefix}front_laser" parent="${prefix}base_link" gpu="${gpu}" min_angle="${-PI/2}" max_angle="${PI/2}" prefix_topic="front_laser">
-            <origin xyz="0.53 0.0 0.153" rpy="${PI} 0 0"/>
-        </xacro:sensor_sick_tim551>
+<robot name="rbvogui" xmlns:xacro="http://wiki.ros.org/xacro">
+  <xacro:include filename="$(find rbvogui_description)/urdf/wheels/steering_wheel.urdf.xacro"/>
+  <xacro:include filename="$(find rbvogui_description)/urdf/bases/rbvogui_base.urdf.xacro"/>
+  <xacro:macro name="rbvogui" params="prefix publish_bf hq">
+    <xacro:property name="M_PI" value="3.1415926535897931" />
+    <xacro:property name="wheel_offset_x" value="0.380"/>
+    <xacro:property name="wheel_offset_y" value="0.23975"/>
+    <xacro:property name="wheel_offset_z" value="-0.012"/>
+    <link name="${prefix}base_footprint" />
+    <joint name="${prefix}base_footprint_joint" type="fixed">
+      <origin xyz="0 0 ${0.1125}" rpy="0 0 0" />
+      <parent link="${prefix}base_footprint"/>
+      <child link="${prefix}base_link" />
+    </joint>
+    <link name="${prefix}base_link"/>
+    <joint name="${prefix}base_joint" type="fixed">
+      <origin xyz="0 0 ${0.132}" rpy="0 0 0" />
+      <parent link="${prefix}base_link"/>
+      <child link="${prefix}case_link" />
+    </joint>
+    <xacro:rbvogui_base prefix="${prefix}" hq="${hq}"/>
+    <xacro:steering_wheel prefix="${prefix}front_left_" parent="${prefix}case_link" reflect="true" hq="true">
+      <origin xyz="${wheel_offset_x} ${wheel_offset_y} ${wheel_offset_z}" rpy="0 0 ${M_PI}"/>
+    </xacro:steering_wheel>
+    <xacro:steering_wheel prefix="${prefix}front_right_" parent="${prefix}case_link" reflect="false" hq="true">
+      <origin xyz="${wheel_offset_x} -${wheel_offset_y} ${wheel_offset_z}" rpy="0 0 0"/>
+    </xacro:steering_wheel>
+    <xacro:steering_wheel prefix="${prefix}rear_left_" parent="${prefix}case_link" reflect="true" hq="true">
+      <origin xyz="-${wheel_offset_x} ${wheel_offset_y} ${wheel_offset_z}" rpy="0 0 ${M_PI}"/>
+    </xacro:steering_wheel>
+    <xacro:steering_wheel prefix="${prefix}rear_right_" parent="${prefix}case_link" reflect="false" hq="true">
+      <origin xyz="-${wheel_offset_x} -${wheel_offset_y} ${wheel_offset_z}" rpy="0 0 0"/>
+    </xacro:steering_wheel>
+    <xacro:macro name="ros2_joint" params="interface jmin jmax prefix name">
+      <joint name="${prefix}${name}_joint">
+        <command_interface name="${interface}">
+          <param name="min">${jmin}</param>
+          <param name="max">${jmax}</param>
+        </command_interface>
+        <state_interface name="position"/>
+        <state_interface name="velocity"/>
+        <state_interface name="effort"/>
+      </joint>
     </xacro:macro>
-    <!-- Gazebo ros control pluggins -->
-    <xacro:ros_control/>
-    <xacro:rbvogui prefix="$(arg prefix)" load_kinematics_file="$(arg load_kinematics_file)" gpu="$(arg gpu)" publish_bf="${publish_bf}" hq="${hq}"/>
+    <ros2_control name="GazeboSystem" type="system">
+      <hardware>
+        <plugin>gazebo_ros2_control/GazeboSystem</plugin>
+      </hardware>
+      <xacro:ros2_joint interface="position" jmin="-2" jmax="2" prefix="${prefix}" name="front_left_base_set"/>
+      <xacro:ros2_joint interface="position" jmin="-2" jmax="2" prefix="${prefix}" name="front_right_base_set"/>
+      <xacro:ros2_joint interface="position" jmin="-2" jmax="2" prefix="${prefix}" name="rear_left_base_set"/>
+      <xacro:ros2_joint interface="position" jmin="-2" jmax="2" prefix="${prefix}" name="rear_right_base_set"/>
+      <xacro:ros2_joint interface="velocity" jmin="-10" jmax="10" prefix="${prefix}" name="front_left_wheel"/>
+      <xacro:ros2_joint interface="velocity" jmin="-10" jmax="10" prefix="${prefix}" name="front_right_wheel"/>
+      <xacro:ros2_joint interface="velocity" jmin="-20" jmax="20" prefix="${prefix}" name="rear_left_wheel"/>
+      <xacro:ros2_joint interface="velocity" jmin="-20" jmax="20" prefix="${prefix}" name="rear_right_wheel"/>
+    </ros2_control>
+  </xacro:macro>
+  <xacro:arg name="robot_id"             default="robot" />
+  <xacro:arg name="prefix"               default="$(arg robot_id)_" />
+  <xacro:arg name="config_controllers"   default="/home/rafaelm/git/robotnikautomation/FRAUNHOFER_RBVOGUI/rbvogui_sim/rbvogui_gazebo/config/controllers2.yaml" />
+  <xacro:property name="hq" value="true" />
+  <xacro:property name="publish_bf" value="true" />
+  <xacro:rbvogui prefix="$(arg prefix)" publish_bf="${publish_bf}" hq="${hq}" />
+  <gazebo>
+    <plugin filename="libgazebo_ros2_control.so" name="robotnik2_gazebo_control">
+      <namespace>$(arg robot_id)</namespace>
+      <parameters>$(arg config_controllers)</parameters>
+      <!--robot_param>robot_description</robot_param-->
+      <!--robot_param_node>robot_state_publisher</robot_param_node-->
+      <!--remaping>$(find rbvogui_description)/config/remapping.yaml</remaping-->
+    </plugin>
+  </gazebo>
 </robot>

File: rbvogui_description/urdf/bases/rbvogui_base.urdf.xacro (robot description, xacro)
@@ -7,5 +7,5 @@
     </xacro:macro>
     <!-- BASE_LINK -->
-    <link name="${prefix}base_link">
+    <link name="${prefix}case_link">
       <inertial>
         <mass value="100.0" />
@@ -36,5 +36,5 @@
       </collision>
     </link>
-    <gazebo reference="${prefix}base_link">
+    <gazebo reference="${prefix}case_link">
       <material>Gazebo/DarkGrey</material>
     </gazebo>
@@ -42,19 +42,19 @@
     <joint name="${prefix}base_logos_joint" type="fixed">
       <origin xyz="0 0 0" rpy="0 0 0 " />
-      <parent link="${prefix}base_link"/>
-      <child link="${prefix}base_logos_link" />
+      <parent link="${prefix}case_link"/>
+      <child link="${prefix}case_logos_link" />
     </joint>
     <!-- Logos -->
-    <link name="${prefix}base_logos_link">
+    <link name="${prefix}case_logos_link">
       <visual>
         <origin xyz="0 0 -0.168" rpy="0 0 0" />
         <xacro:if value="${hq}">
           <geometry>
-            <mesh filename="package://rbvogui_description/meshes/bases/rbvogui_logos_v3.stl" scale="1.001 1.07 1.001"/>
+            <mesh filename="package://rbvogui_description/meshes/bases/rbvogui_logos_v3.stl" scale="1.0001 1.007 1.0001"/>
           </geometry>
         </xacro:if>
         <xacro:unless value="${hq}">
           <geometry>
-            <mesh filename="package://rbvogui_description/meshes/bases/rbvogui_logos_v3.dae" scale="1.001 1.07 1.001"/>
+            <mesh filename="package://rbvogui_description/meshes/bases/rbvogui_logos_v3.dae" scale="1.0001 1.007 1.0001"/>
           </geometry>
         </xacro:unless>
@@ -64,5 +64,5 @@
       </visual>
     </link>
-    <gazebo reference="${prefix}base_logos_link">
+    <gazebo reference="${prefix}case_logos_link">
       <material>Gazebo/Red</material>
     </gazebo>

File: rbvogui_description/urdf/wheels/steering_wheel.urdf.xacro (robot description, xacro)
@@ -1,28 +1,26 @@
 <?xml version="1.0"?>
 <robot xmlns:xacro="http://www.ros.org/wiki/xacro">
-  <xacro:macro name="steer_set" params="prefix parent *origin hq">
+  <!-- Height added: 0.132 m -->
+  <xacro:macro name="steering_wheel" params="prefix parent *origin reflect hq">
+    <xacro:include filename="$(find rbvogui_description)/urdf/wheels/wheel.urdf.xacro"/>
     <xacro:macro name="cylinder_inertia" params="m r h">
       <inertia ixx="${m*(3*r*r+h*h)/12}" ixy = "0" ixz = "0" iyy="${m*(3*r*r+h*h)/12}" iyz = "0" izz="${m*r*r/2}" />
     </xacro:macro>
     <xacro:property name="M_PI" value="3.1415926535897931" />
-    <xacro:property name="wheel_radius" value="0.110" />
-    <xacro:property name="wheel_width" value="0.110" />
-    <xacro:property name="wheel_mass" value="5.0" />
-    <!--MOTOR WHEEL -->
-    <joint name="${prefix}base_set_joint" type="revolute">
+    <joint name="${prefix}steer_joint" type="revolute">
       <xacro:insert_block name="origin" />
       <parent link="${parent}" />
-      <child link="${prefix}base_wheel_link" />
+      <child link="${prefix}steer_link" />
       <axis xyz="0 0 1" />
       <limit effort="100" velocity="100" lower="-${2*M_PI/3}" upper="${2*M_PI/3}" />
     </joint>
-    <link name="${prefix}base_wheel_link" />
-    <joint name="${prefix}set_joint" type="fixed">
-      <parent link="${prefix}base_wheel_link"/>
-      <child link="${prefix}set_wheel_link"/>
-      <origin xyz="0 -0.079 0.132" rpy="${-M_PI/2} 0 0" />
+    <link name="${prefix}steer_link" />
+    <joint name="${prefix}base_wheel_joint" type="fixed">
+      <parent link="${prefix}steer_link"/>
+      <child link="${prefix}base_wheel_link"/>
+      <origin xyz="0 0.079 -0.132" rpy="${M_PI/2} 0 0" />
       <axis xyz="0 0 1" rpy="0 0 0" />
     </joint>
-    <link name="${prefix}set_wheel_link">
+    <link name="${prefix}base_wheel_link">
       <visual>
         <origin xyz="0 0 0.079" rpy="${-M_PI/2} ${M_PI} 0" />
@@ -42,6 +40,6 @@
       <inertial>
         <mass value="4" />
-        <origin xyz="0 0 0.0" rpy="0 0 0"/>
-        <xacro:cylinder_inertia m="${wheel_mass}" r="${wheel_radius}" h="${wheel_width}" />
+        <origin xyz="0 0.05 0.05" rpy="0 0 0"/>
+        <xacro:cylinder_inertia m="5.0" r="0.110" h="0.110" />
       </inertial>
     </link>
@@ -49,4 +47,12 @@
       <material>Gazebo/Red</material>
     </gazebo>
+    <xacro:wheel prefix="${prefix}" parent="${prefix}base_wheel_link" reflect="${reflect}" hq="${hq}">
+      <xacro:if value="${reflect}">
+        <origin xyz="0 0 0.015" rpy="0 0 0" />
+      </xacro:if>
+      <xacro:unless value="${reflect}">
+        <origin xyz="0 0 0.015" rpy="${M_PI} 0 0" />
+      </xacro:unless>
+    </xacro:wheel>
   </xacro:macro>
 </robot>

File: rbvogui_description/urdf/wheels/wheel.urdf.xacro (robot description, xacro)
@@ -1,4 +1,5 @@
 <?xml version="1.0"?>
 <robot xmlns:xacro="http://www.ros.org/wiki/xacro">
+  <!-- Height added: 0.1125 m -->
   <xacro:macro name="wheel" params="prefix parent *origin reflect:=false hq:=true">
     <xacro:macro name="cylinder_inertia" params="m r h">
@@ -18,9 +19,14 @@
       <dynamics damping="0.1" friction="0.1"/>
       <limit effort="1e9" velocity="1000.0"/>
-      <safety_controller k_velocity="0.1" k_position="0.1" soft_lower_limit="-1.0" soft_upper_limit="1.0"/>
+      <safety_controller k_velocity="0.1" k_position="0.1" soft_lower_limit="-${M_PI}" soft_upper_limit="${M_PI}"/>
     </joint>
     <link name="${prefix}wheel_link">
       <inertial>
-        <origin xyz="0 0 ${tire_width/2}" rpy="0 0 0"/>
+        <xacro:if value="${reflect}">
+          <origin xyz="0 0 ${tire_width/2}" rpy="${M_PI/2} 0 0" />
+        </xacro:if>
+        <xacro:unless value="${reflect}">
+          <origin xyz="0 0 -${tire_width/2}" rpy="${M_PI/2} 0 0" />
+        </xacro:unless>
         <mass value="${tire_mass}"/>
         <xacro:cylinder_inertia m="${tire_mass}" r="${tire_radius}" h="${tire_width}"/>
@@ -31,5 +37,5 @@
         </xacro:if>
         <xacro:unless value="${reflect}">
-          <origin xyz="0 0 ${tire_width/2}" rpy="${-M_PI/2} 0 0" />
+          <origin xyz="0 0 -${tire_width/2}" rpy="${M_PI/2} 0 0" />
         </xacro:unless>
         <geometry>
@@ -46,5 +52,10 @@
       </visual>
       <collision>
-        <origin xyz="0 0 ${tire_width/2}" rpy="0 0 0" />
+        <xacro:if value="${reflect}">
+          <origin xyz="0 0 ${tire_width/2}" rpy="0 0 0" />
+        </xacro:if>
+        <xacro:unless value="${reflect}">
+          <origin xyz="0 0 -${tire_width/2}" rpy="0 0 0" />
+        </xacro:unless>
         <geometry>
           <cylinder length="${tire_width}" radius="${tire_radius}" />

Commit message: Added publish bf option

File: rbvogui_description/robot/rbvogui_std.urdf.xacro (robot description, xacro)
@@ -8,10 +8,12 @@
     <xacro:property name="wheel_offset_y" value="0.23975"/>
     <xacro:property name="wheel_offset_z" value="-0.012"/>
-    <link name="${prefix}base_footprint" />
-    <joint name="${prefix}base_footprint_joint" type="fixed">
-      <origin xyz="0 0 ${0.1125}" rpy="0 0 0" />
-      <parent link="${prefix}base_footprint"/>
-      <child link="${prefix}base_link" />
-    </joint>
+    <xacro:if value="${publish_bf}">
+      <link name="${prefix}base_footprint" />
+      <joint name="${prefix}base_footprint_joint" type="fixed">
+        <origin xyz="0 0 ${0.1125}" rpy="0 0 0" />
+        <parent link="${prefix}base_footprint"/>
+        <child link="${prefix}base_link" />
+      </joint>
+    </xacro:if>
     <link name="${prefix}base_link"/>
     <joint name="${prefix}base_joint" type="fixed">
