Commit message: Fixed joints wheel and hitch joints

File: rbvogui_description/urdf/cart/cart.urdf.xacro (robot description, xacro)
@@ -9,5 +9,5 @@
   <xacro:property name="cart_width" value="1.098" />
   <xacro:property name="cart_height" value="0.25" />
-  <xacro:property name="cart_mass" value="30" />
+  <xacro:property name="cart_mass" value="80" />
   <!-- Size wheels -->
   <xacro:property name="wheels_radius" value="0.20" />
@@ -20,8 +20,8 @@
   <xacro:property name="front_wheel_center_dist_y" value="0.245"/>
   <!-- Support front wheel cart -->
-  <xacro:property name="support_length" value="${wheels_radius - front_wheel_radius}" />
+  <xacro:property name="support_length" value="${wheels_radius - front_wheel_radius + 0}" />
   <xacro:property name="support_width" value="0.03" />
   <!-- Hitch -->
-  <xacro:property name="hitch_length" value="0.5" />
+  <xacro:property name="hitch_length" value="0.4" />
   <xacro:property name="hitch_width" value="0.05" />
   <xacro:macro name="cart" params="prefix parent">
@@ -29,22 +29,28 @@
     <link name="${prefix}hitch_z">
       <inertial>
-            <mass value="0.01" />
+            <mass value="1" />
             <origin xyz="0 0 0" rpy="0 0 0" />
-            <xacro:solid_cuboid_inertia w="${0.01}" d="${0.01}" h="${0.01}" m="0.01"/>
+            <xacro:solid_cuboid_inertia w="${0.1}" d="${0.1}" h="${0.1}" m="1"/>
       </inertial>
     </link>
     <link name="${prefix}hitch_y">
       <inertial>
-            <mass value="0.01" />
+            <mass value="1" />
             <origin xyz="0 0 0" rpy="0 0 0" />
-            <xacro:solid_cuboid_inertia w="${0.01}" d="${0.01}" h="${0.01}" m="0.01"/>
+            <xacro:solid_cuboid_inertia w="${0.1}" d="${0.1}" h="${0.1}" m="1"/>
       </inertial>
     </link>
     <link name="${prefix}hitch_x">
       <inertial>
-            <mass value="0.01" />
+            <mass value="1" />
             <origin xyz="0 0 0" rpy="0 0 0" />
-            <xacro:solid_cuboid_inertia w="${0.01}" d="${0.01}" h="${0.01}" m="0.01"/>
-      </inertial>
+            <xacro:solid_cuboid_inertia w="${hitch_length}" d="${hitch_width}" h="${hitch_width}" m="1"/>
+      </inertial>
+      <collision>
+        <origin xyz="-${hitch_length/2} 0.0 0.0" rpy="0.0 0.0 0.0"/>
+        <geometry>
+          <box size="${hitch_length} ${hitch_width} ${hitch_width}"/>
+        </geometry>
+      </collision>
     </link>
     <!-- Hitch to Body -->
@@ -79,7 +85,7 @@
     <link name="${prefix}left_wheel">
       <inertial>
-            <mass value="3" />
-            <origin xyz="0 0 0" rpy="${PI/2} 0 0" />
-            <xacro:solid_cylinder_inertia m="3" r="${wheels_radius}" h="${wheels_width}"/>
+            <mass value="1" />
+            <origin xyz="0 0 0" rpy="${PI/2} 0 0" />
+            <xacro:solid_cylinder_inertia m="1" r="${wheels_radius}" h="${wheels_width}"/>
       </inertial>
       <visual>
@@ -105,7 +111,7 @@
     <link name="${prefix}right_wheel">
       <inertial>
-            <mass value="3" />
-            <origin xyz="0 0 0" rpy="${PI/2} 0 0" />
-            <xacro:solid_cylinder_inertia m="3" r="${wheels_radius}" h="${wheels_width}"/>
+            <mass value="1" />
+            <origin xyz="0 0 0" rpy="${PI/2} 0 0" />
+            <xacro:solid_cylinder_inertia m="1" r="${wheels_radius}" h="${wheels_width}"/>
       </inertial>
       <visual>
@@ -131,7 +137,7 @@
     <link name="${prefix}support_front_right_wheel">
       <inertial>
-            <mass value="0.1" />
+            <mass value="1" />
             <origin xyz="0 0 0" rpy="0 ${PI/2} 0" />
-            <xacro:solid_cuboid_inertia w="${support_length}" d="${support_width}" h="${support_width}" m="0.1"/>
+            <xacro:solid_cuboid_inertia w="${support_length}" d="${support_width}" h="${support_width}" m="1"/>
       </inertial>
       <visual>
@@ -154,7 +160,7 @@
     <link name="${prefix}support_front_left_wheel">
       <inertial>
-            <mass value="0.1" />
+            <mass value="1" />
             <origin xyz="0 0 0" rpy="0 ${PI/2} 0" />
-            <xacro:solid_cuboid_inertia w="${support_length}" d="${support_width}" h="${support_width}" m="0.1"/>
+            <xacro:solid_cuboid_inertia w="${support_length}" d="${support_width}" h="${support_width}" m="1"/>
       </inertial>
       <visual>
@@ -177,7 +183,7 @@
     <link name="${prefix}front_left_wheel">
       <inertial>
-            <mass value="0.1" />
-            <origin xyz="0 0 0" rpy="${PI/2} 0 0" />
-            <xacro:solid_cylinder_inertia m="0.1" r="${front_wheel_radius}" h="${front_wheel_width}"/>
+            <mass value="1" />
+            <origin xyz="0 0 0" rpy="${PI/2} 0 0" />
+            <xacro:solid_cylinder_inertia m="1" r="${front_wheel_radius}" h="${front_wheel_width}"/>
       </inertial>
       <visual>
@@ -203,7 +209,7 @@
     <link name="${prefix}front_right_wheel">
       <inertial>
-            <mass value="0.1" />
-            <origin xyz="0 0 0" rpy="${PI/2} 0 0" />
-            <xacro:solid_cylinder_inertia m="0.1" r="${front_wheel_radius}" h="${front_wheel_width}"/>
+            <mass value="1" />
+            <origin xyz="0 0 0" rpy="${PI/2} 0 0" />
+            <xacro:solid_cylinder_inertia m="1" r="${front_wheel_radius}" h="${front_wheel_width}"/>
       </inertial>
       <visual>

File: rbvogui_description/urdf/cart/cart_joint.urdf.xacro (robot description, xacro)
@@ -4,5 +4,5 @@
     <!-- Robot to Hitch -->
         <joint name="${prefix}hitch_z_joint" type="revolute">
-            <origin xyz="-0.5 0 ${wheels_radius + cart_height/2}" rpy="0.0 0.0 0.0"/>
+            <origin xyz="-0.6 0 ${wheels_radius + cart_height/2}" rpy="0.0 0.0 0.0"/>
             <parent link="${parent}"/>
             <child link="${prefix}hitch_z"/>
@@ -25,8 +25,10 @@
         </joint>
     <!-- Hitch to Body -->
-        <joint name="${prefix}body_joint" type="fixed">
+        <joint name="${prefix}body_joint" type="revolute">
             <origin xyz="${-cart_length/2 -hitch_length} 0 0" rpy="0.0 0.0 0.0"/>
             <parent link="${prefix}hitch_x"/>
             <child link="${prefix}body"/>
+            <axis xyz="0.0 1.0 0.0"/>
+            <limit effort="1000" velocity="2000" lower="-0.2" upper="0.2"/>
         </joint>
     <!-- Left wheel -->

File: rbvogui_description/urdf/ros2_control.urdf.xacro (robot description, xacro)
@@ -11,5 +11,7 @@
           <xacro:if value="${cart}">
             <plugin name="cart_joint_state" filename="libgazebo_ros_joint_state_publisher.so">
-              <namespace>robot</namespace>
+              <ros>
+                <namespace>robot</namespace>
+              </ros>
               <update_rate>30</update_rate>
               <joint_name>robot_cart_hitch_z_joint</joint_name>

Commit message: Fixed inertias

File: rbvogui_description/urdf/cart/cart.urdf.xacro (robot description, xacro)
@@ -31,5 +31,5 @@
             <mass value="1" />
             <origin xyz="0 0 0" rpy="0 0 0" />
-            <xacro:solid_cuboid_inertia w="${0.1}" d="${0.1}" h="${0.1}" m="1"/>
+            <xacro:solid_cuboid_inertia w="${0.01}" d="${0.01}" h="${0.01}" m="10"/>
       </inertial>
     </link>
@@ -38,5 +38,5 @@
             <mass value="1" />
             <origin xyz="0 0 0" rpy="0 0 0" />
-            <xacro:solid_cuboid_inertia w="${0.1}" d="${0.1}" h="${0.1}" m="1"/>
+            <xacro:solid_cuboid_inertia w="${0.01}" d="${0.01}" h="${0.01}" m="10"/>
       </inertial>
     </link>
@@ -44,5 +44,5 @@
       <inertial>
             <mass value="1" />
-            <origin xyz="0 0 0" rpy="0 0 0" />
+            <origin xyz="-${hitch_length/2} 0 0" rpy="0 0 0" />
             <xacro:solid_cuboid_inertia w="${hitch_length}" d="${hitch_width}" h="${hitch_width}" m="1"/>
       </inertial>

Commit message: Changed mesh trolley connection

File: rbvogui_description/urdf/cart/cart.urdf.xacro (robot description, xacro)
@@ -26,5 +26,5 @@
   <xacro:property name="support_width" value="0.03" />
   <!-- Hitch -->
-  <xacro:property name="hitch_length" value="0.215" />
+  <xacro:property name="hitch_length" value="0.3" />
   <xacro:property name="hitch_width" value="0.160" />
   <xacro:property name="hitch_height" value="0.064" />
@@ -34,6 +34,6 @@
   <xacro:property name="bulon_z" value="0.391" />
   <!-- Transform from hitch to chassis UNKOWN -->
-  <xacro:property name="hitch_x" value="-0.620" />
-  <xacro:property name="hitch_z" value="0.161" />
+  <xacro:property name="hitch_x" value="-0.347" />
+  <xacro:property name="hitch_z" value="0.175" />
   <!-- Transform from chassis to wheels -->
   <xacro:property name="front_caster_wheel_x" value="0.620" />
@@ -256,6 +256,6 @@
       <material>Gazebo/Grey</material>
     </gazebo>
-    <!-- Marker0 -->
-    <link name="${prefix}marker0">
+    <!-- Marker00 -->
+    <link name="${prefix}marker00">
       <visual>
         <origin xyz="0.0 0.0 0.0" rpy="0.0 0 0"/>
@@ -265,6 +265,24 @@
       </visual>
     </link>
-    <!-- Marker1 -->
-    <link name="${prefix}marker1">
+    <!-- Marker01 -->
+    <link name="${prefix}marker01">
+      <visual>
+        <origin xyz="0.0 0.0 0.0" rpy="0.0 0 0"/>
+        <geometry>
+          <mesh filename="package://rbvogui_description/meshes/cart/Markers/meshes/Marker0.dae" scale="0.16 0.16 0.16"/>
+        </geometry>
+      </visual>
+    </link>
+    <!-- Marker10 -->
+    <link name="${prefix}marker10">
+      <visual>
+        <origin xyz="0.0 0.0 0.0" rpy="0.0 0 0"/>
+        <geometry>
+          <mesh filename="package://rbvogui_description/meshes/cart/Markers/meshes/Marker1.dae" scale="0.16 0.16 0.16"/>
+        </geometry>
+      </visual>
+    </link>
+    <!-- Marker11 -->
+    <link name="${prefix}marker11">
       <visual>
         <origin xyz="0.0 0.0 0.0" rpy="0.0 0 0"/>

File: rbvogui_description/urdf/cart/cart_joint.urdf.xacro (robot description, xacro)
@@ -7,5 +7,5 @@
         <xacro:if value="${connected}">
             <joint name="${prefix}chassis_joint" type="revolute">
-                <origin xyz="${-cart_length/2 -hitch_length/2} 0 0" rpy="0.0 0.0 0.0"/>
+                <origin xyz="${-cart_length/2 - 0.1} 0 0" rpy="0.0 0.0 0.0"/>
                 <parent link="robot_hitch_x"/>
                 <child link="${prefix}chassis"/>
@@ -87,15 +87,27 @@
             <dynamics damping="0.8" friction="2.0"/>
         </joint>
-    <!-- Marker0 -->
-        <joint name="${prefix}marker0_joint" type="fixed">
-            <origin xyz="0.67 -0.12 0.05" rpy="0.0 0.0 0.0"/>
+    <!-- Marker00 -->
+        <joint name="${prefix}marker00_joint" type="fixed">
+            <origin xyz="0.67 -0.3 0.05" rpy="0.0 0.0 0.0"/>
             <parent link="${prefix}chassis"/>
-            <child link="${prefix}marker0"/>
+            <child link="${prefix}marker00"/>
         </joint>
-    <!-- Marker1 -->
-        <joint name="${prefix}marker1_joint" type="fixed">
-            <origin xyz="0.67 0.12 0.05" rpy="0.0 0.0 0.0"/>
+    <!-- Marker01 -->
+        <joint name="${prefix}marker01_joint" type="fixed">
+            <origin xyz="0.67 0.3 0.05" rpy="0.0 0.0 0.0"/>
             <parent link="${prefix}chassis"/>
-            <child link="${prefix}marker1"/>
+            <child link="${prefix}marker01"/>
+        </joint>
+    <!-- Marker10 -->
+        <joint name="${prefix}marker10_joint" type="fixed">
+            <origin xyz="0.67 -0.08 0.05" rpy="0.0 0.0 0.0"/>
+            <parent link="${prefix}chassis"/>
+            <child link="${prefix}marker10"/>
+        </joint>
+    <!-- Marker11 -->
+        <joint name="${prefix}marker11_joint" type="fixed">
+            <origin xyz="0.67 0.08 0.05" rpy="0.0 0.0 0.0"/>
+            <parent link="${prefix}chassis"/>
+            <child link="${prefix}marker11"/>
         </joint>
     </xacro:macro>

File: rbvogui_description/urdf/cart/cart_robot_connection.urdf.xacro (robot description, xacro)
@@ -7,13 +7,13 @@
   <xacro:property name="bulon_z" value="0.391" />
   <!-- Transform from hitch to chassis UNKOWN -->
-  <xacro:property name="hitch_x" value="-0.620" />
-  <xacro:property name="hitch_z" value="0.161" />
+  <xacro:property name="hitch_x" value="-0.347" />
+  <xacro:property name="hitch_z" value="0.175" />
   <!-- Hitch -->
-  <xacro:property name="hitch_length" value="0.215" />
+  <xacro:property name="hitch_length" value="0.32" />
   <xacro:property name="hitch_width" value="0.160" />
   <xacro:property name="hitch_height" value="0.064" />
   <xacro:macro name="cart_connection" params="prefix connected">
     <!-- Robot to bulon NOMBRE PROVISIONAL SUPONGO??-->
-            <link name="${prefix}bulon">
+            <!-- <link name="${prefix}bulon">
                 <inertial>
                     <mass value="1" />
@@ -38,17 +38,17 @@
                 <parent link="robot_base_link"/>
                 <child link="${prefix}bulon"/>
-            </joint>
+            </joint> -->
             <!-- bulon to Hitch -->
             <link name="${prefix}hitch_z">
             <inertial>
                     <mass value="3" />
-                    <origin xyz="0 0 0" rpy="0 0 0" />
-                    <xacro:solid_cuboid_inertia w="0.215" d="0.064" h="0.160" m="3"/>
+                    <origin xyz="${hitch_length/2} 0 0" rpy="0 0 0" />
+                    <xacro:solid_cuboid_inertia w="${hitch_length}" d="${hitch_height}" h="${hitch_width}" m="3"/>
             </inertial>
             </link>
             <xacro:if value="${connected}">
               <joint name="${prefix}hitch_z_joint" type="revolute">
-                  <origin xyz="${hitch_x - bulon_x} 0 ${hitch_z-bulon_z}" rpy="0.0 0.0 0.0"/>
-                  <parent link="${prefix}bulon"/>
+                  <origin xyz="${hitch_x} 0 ${hitch_z}" rpy="0.0 0.0 0.0"/>
+                  <parent link="robot_base_link"/>
                   <child link="${prefix}hitch_z"/>
                   <axis xyz="0.0 0.0 1.0"/>
@@ -58,6 +58,6 @@
             <xacro:unless value="${connected}">
               <joint name="${prefix}hitch_z_joint" type="fixed">
-                  <origin xyz="${hitch_x - bulon_x} 0 ${hitch_z-bulon_z}" rpy="0.0 0.0 0.0"/>
-                  <parent link="${prefix}bulon"/>
+                  <origin xyz="${hitch_x} 0 ${hitch_z}" rpy="0.0 0.0 0.0"/>
+                  <parent link="robot_base_link"/>
                   <child link="${prefix}hitch_z"/>
               </joint>
@@ -66,6 +66,6 @@
             <inertial>
                     <mass value="3" />
-                    <origin xyz="0 0 0" rpy="0 0 0" />
-                    <xacro:solid_cuboid_inertia w="0.215" d="0.064" h="0.160" m="3"/>
+                    <origin xyz="${hitch_length/2} 0 0" rpy="0 0 0" />
+                    <xacro:solid_cuboid_inertia w="${hitch_length}" d="${hitch_height}" h="${hitch_width}" m="3"/>
             </inertial>
             </link>
@@ -86,26 +86,27 @@
               </joint>
             </xacro:unless>
-            <link name="${prefix}hitch_x">
-            <inertial>
-                    <mass value="3" />
-                    <origin xyz="0 0 0" rpy="0 0 0" />
-                    <xacro:solid_cuboid_inertia w="0.215" d="0.064" h="0.160" m="3"/>
-            </inertial>
-            <visual>
-                <origin xyz="0.0 0.0 0.0" rpy="0.0 0.0 0.0"/>
-                <geometry>
-                <box size="0.215 0.160 0.064"/>
-                </geometry>
-            </visual>
-            <collision>
-                <origin xyz="0.0 0.0 0.0" rpy="0.0 0.0 0.0"/>
-                <geometry>
-                <box size="${hitch_length} ${hitch_width} ${hitch_height}"/>
-                </geometry>
-            </collision>
-            </link>
             <xacro:if value="${connected}">
+              <link name="${prefix}hitch_x">
+                <inertial>
+                        <mass value="3" />
+                        <origin xyz="${hitch_length/2} 0 0" rpy="0 0 0" />
+                        <xacro:solid_cuboid_inertia w="${hitch_length}" d="${hitch_height}" h="${hitch_width}" m="3"/>
+                </inertial>
+                <visual>
+                    <origin xyz="${hitch_length} 0.0 0.0" rpy="-${PI/2} ${PI} ${PI/2}"/>
+                    <geometry>
+                    <!-- <box size="0.215 0.160 0.064"/> -->
+                    <mesh filename="package://rbvogui_description/meshes/cart/trolley_support_closed.stl" scale="1.0 1.0 1.0"/>
+                    </geometry>
+                </visual>
+                <collision>
+                    <origin xyz="${hitch_length/2} 0 0" rpy="0 0 0" />
+                    <geometry>
+                    <box size="${hitch_length} ${hitch_width} ${hitch_height}"/>
+                    </geometry>
+                </collision>
+              </link>
               <joint name="${prefix}hitch_x_joint" type="revolute">
-                  <origin xyz="0.0 0.0 0.0" rpy="0.0 0.0 0.0"/>
+                  <origin xyz="${-hitch_length} 0.0 0.0" rpy="0.0 0.0 0.0"/>
                   <parent link="${prefix}hitch_y"/>
                   <child link="${prefix}hitch_x"/>
@@ -115,6 +116,26 @@
             </xacro:if>
             <xacro:unless value="${connected}">
+              <link name="${prefix}hitch_x">
+                <inertial>
+                        <mass value="3" />
+                        <origin xyz="${hitch_length/2} 0 0" rpy="0 0 0" />
+                        <xacro:solid_cuboid_inertia w="${hitch_length}" d="${hitch_height}" h="${hitch_width}" m="3"/>
+                </inertial>
+                <visual>
+                    <origin xyz="${hitch_length} 0.0 0.0" rpy="-${PI/2} ${PI} ${PI/2}"/>
+                    <geometry>
+                    <!-- <box size="0.215 0.160 0.064"/> -->
+                    <mesh filename="package://rbvogui_description/meshes/cart/trolley_support.stl" scale="1.0 1.0 1.0"/>
+                    </geometry>
+                </visual>
+                <collision>
+                    <origin xyz="${hitch_length/2} 0 0" rpy="0 0 0" />
+                    <geometry>
+                    <box size="${hitch_length} ${hitch_width} ${hitch_height}"/>
+                    </geometry>
+                </collision>
+              </link>
               <joint name="${prefix}hitch_x_joint" type="fixed">
-                  <origin xyz="0.0 0.0 0.0" rpy="0.0 0.0 0.0"/>
+                  <origin xyz="${-hitch_length} 0.0 0.0" rpy="0.0 0.0 0.0"/>
                   <parent link="${prefix}hitch_y"/>
                   <child link="${prefix}hitch_x"/>

Commit message: Fix position

File: rbvogui_description/urdf/cart/cart.urdf.xacro (robot description, xacro)
@@ -5,4 +5,5 @@
   <xacro:include filename="$(find rbvogui_description)/urdf/cart/robot_cart_connection.urdf.xacro" />
   <xacro:include filename="$(find rbvogui_description)/urdf/cart/markers.urdf.xacro" />
+  <xacro:include filename="$(find robotnik_sensors)/urdf/all_sensors.urdf.xacro" />
   <xacro:arg name="prefix" default="robot_" />
   <xacro:arg name="connected" default="false" />
@@ -272,4 +273,8 @@
       <material>Gazebo/Grey</material>
     </gazebo>
+    <!-- hokuyo ust10 -->
+    <xacro:sensor_hokuyo_ust10lx prefix="${prefix}rear_laser" parent="${prefix}chassis" gpu="false" prefix_topic="/${prefix}/rear_laser">
+        <origin xyz="-0.63 0.0 -0.023" rpy="${PI} 0 ${-PI*3/4}"/>
+    </xacro:sensor_hokuyo_ust10lx>
     <xacro:cart_joints prefix="${prefix}" connected="${connected}"/>
     <xacro:markers prefix="${prefix}"/>

File: rbvogui_description/urdf/cart/robot_cart_connection.urdf.xacro (robot description, xacro)
@@ -19,5 +19,5 @@
         <inertial>
           <mass value="3" />
-          <origin xyz="0.0 0 0" rpy="0 0 0" />
+          <origin xyz="0.0 0.0 0.0" rpy="-${PI/2} ${PI} ${PI/2}"/>
           <xacro:solid_cuboid_inertia w="${hitch_length}" d="${hitch_height}" h="${hitch_width}" m="3"/>
         </inertial>
@@ -40,5 +40,5 @@
         <inertial>
           <mass value="3" />
-          <origin xyz="0.0 0 0" rpy="0 0 0" />
+          <origin xyz="0.0 0.0 0.0" rpy="-${PI/2} ${PI} ${PI/2}"/>
           <xacro:solid_cuboid_inertia w="${hitch_length}" d="${hitch_height}" h="${hitch_width}" m="3"/>
         </inertial>
@@ -67,11 +67,11 @@
         <link name="${prefix}hitch_z">
           <inertial>
-            <mass value="3" />
+            <mass value="1" />
             <origin xyz="0.0 0 0" rpy="0 0 0" />
-            <xacro:solid_cuboid_inertia w="${hitch_length}" d="${hitch_height}" h="${hitch_width}" m="3"/>
+            <xacro:solid_cuboid_inertia w="${0.1}" d="${0.1}" h="${0.1}" m="1"/>
           </inertial>
         </link>
         <joint name="${prefix}hitch_z_joint" type="revolute">
-          <origin xyz="${hitch_x} 0 ${hitch_z}" rpy="0.0 0.0 0.0"/>
+          <origin xyz="-0.34 0 0" rpy="0.0 0.0 0.0"/>
           <parent link="${prefix}bulon"/>
           <child link="${prefix}hitch_z"/>
@@ -81,7 +81,7 @@
         <link name="${prefix}hitch_y">
           <inertial>
-            <mass value="3" />
+            <mass value="1" />
             <origin xyz="0.0 0 0" rpy="0 0 0" />
-            <xacro:solid_cuboid_inertia w="${hitch_length}" d="${hitch_height}" h="${hitch_width}" m="3"/>
+            <xacro:solid_cuboid_inertia w="${0.1}" d="${0.1}" h="${0.1}" m="1"/>
           </inertial>
         </link>
@@ -95,7 +95,7 @@
         <link name="${prefix}hitch_x">
           <inertial>
-            <mass value="3" />
+            <mass value="1" />
             <origin xyz="0.0 0 0" rpy="0 0 0" />
-            <xacro:solid_cuboid_inertia w="${hitch_length}" d="${hitch_height}" h="${hitch_width}" m="3"/>
+            <xacro:solid_cuboid_inertia w="${0.1}" d="${0.1}" h="${0.1}" m="1"/>
           </inertial>
         </link>
@@ -104,5 +104,5 @@
           <parent link="${prefix}hitch_y"/>
           <child link="${prefix}hitch_x"/>
-          <axis xyz="1.0 9.0 0.0"/>
+          <axis xyz="1.0 0.0 0.0"/>
           <limit effort="1000" velocity="2000" lower="${-PI/9}" upper="${PI/9}"/>
         </joint>

Commit message: Add hokuyo in cart

File: rbvogui_description/urdf/cart/cart.urdf.xacro (robot description, xacro)
@@ -274,6 +274,6 @@
     </gazebo>
     <!-- hokuyo ust10 -->
-    <xacro:sensor_hokuyo_ust10lx prefix="${prefix}rear_laser" parent="${prefix}chassis" gpu="false" prefix_topic="/${prefix}/rear_laser">
-        <origin xyz="-0.63 0.0 -0.023" rpy="${PI} 0 ${-PI*3/4}"/>
+    <xacro:sensor_hokuyo_ust10lx prefix="${prefix}rear_laser" parent="${prefix}chassis" gpu="false" prefix_topic="/${prefix}rear_laser">
+        <origin xyz="-0.63 0.0 -0.023" rpy="${PI} 0 ${-PI/2}"/>
     </xacro:sensor_hokuyo_ust10lx>
     <xacro:cart_joints prefix="${prefix}" connected="${connected}"/>
