Commit message: (feat): prepare packages and config files

File: rbvogui_description/urdf/cart/cart.urdf.xacro (robot description, xacro)
@@ -1,310 +1,11 @@
 <?xml version="1.0"?>
 <robot xmlns:xacro="http://www.ros.org/wiki/xacro" name="cart">
-  <xacro:include filename="$(find rbvogui_description)/urdf/inertia.urdf.xacro" />
-  <xacro:include filename="$(find rbvogui_description)/urdf/cart/cart_joint.urdf.xacro" />
-  <xacro:include filename="$(find rbvogui_description)/urdf/cart/robot_cart_connection.urdf.xacro" />
-  <xacro:include filename="$(find rbvogui_description)/urdf/cart/markers.urdf.xacro" />
-  <xacro:include filename="$(find robotnik_sensors)/urdf/all_sensors.urdf.xacro" />
+  <xacro:include filename="$(find rbvogui_description)/urdf/cart/cart_base.urdf.xacro" />
+  <!-- <xacro:include filename="$(find rbvogui_description)/urdf/cart/markers.urdf.xacro" /> -->
   <xacro:arg name="prefix" default="robot_" />
   <xacro:arg name="connected" default="false" />
-  <!-- Math -->
-  <xacro:property name="PI" value="3.141592" />
-  <!-- Size cart -->
-  <xacro:property name="cart_length" value="1.3" />
-  <xacro:property name="cart_width" value="1.3" />
-  <xacro:property name="cart_height" value="0.23" />
-  <xacro:property name="cart_mass" value="80" />
-  <!-- Size wheels -->
-  <xacro:property name="wheels_radius" value="0.225" />
-  <xacro:property name="wheels_width" value="0.08" />
-  <xacro:property name="wheels_center_dist_x" value="0.41" />
-  <!-- Size front wheel-->
-  <xacro:property name="front_wheel_radius" value="0.08" />
-  <xacro:property name="front_wheel_width" value="0.05" />
-  <xacro:property name="front_wheel_center_dist_x" value="0.331" />
-  <xacro:property name="front_wheel_center_dist_y" value="0.245"/>
-  <!-- Support front wheel cart -->
-  <xacro:property name="support_length" value="${wheels_radius - front_wheel_radius + 0}" />
-  <xacro:property name="support_width" value="0.03" />
-  <!-- Hitch -->
-  <xacro:property name="hitch_length" value="0.3" />
-  <xacro:property name="hitch_width" value="0.160" />
-  <xacro:property name="hitch_height" value="0.064" />
-  <!-- NEW CART VALUES -->
-  <!-- Transform from robot_base_link to bulon -->
-  <xacro:property name="bulon_x" value="-0.669" />
-  <xacro:property name="bulon_z" value="0.391" />
-  <!-- Transform from hitch to chassis UNKOWN -->
-  <xacro:property name="hitch_x" value="-0.347" />
-  <xacro:property name="hitch_z" value="0.175" />
-  <!-- Transform from chassis to wheels -->
-  <xacro:property name="front_caster_wheel_x" value="0.620" />
-  <xacro:property name="front_caster_wheel_y" value="0.6045" />
-  <xacro:property name="front_caster_wheel_z" value="-0.11201" />
-  <xacro:property name="rear_wheel_x" value="-0.40883" />
-  <xacro:property name="rear_wheel_y" value="0.5895" />
-  <xacro:property name="rear_wheel_z" value="-0.075" />
-  <!-- Transform from front_caster_wheel to front_wheel -->
-  <xacro:property name="front_wheel_x" value="-0.04545" />
-  <xacro:property name="front_wheel_z" value="-0.115" />
-  <xacro:macro name="cart" params="prefix connected">
-    <xacro:unless value="${connected}">
-      <link name="${prefix}base_footprint"/>
-    </xacro:unless>
-    <!-- Lanza -->
-    <link name="${prefix}lanza">
-      <visual>
-        <origin xyz="0.0 0.0 0.0" rpy="0.0 0 0"/>
-        <geometry>
-          <mesh filename="package://rbvogui_description/meshes/cart/lanza.stl" scale="1.0 1.0 1.0"/>
-        </geometry>
-      </visual>
-      <collision>
-        <origin xyz="0.0 0.0 0.0" rpy="0.0 0.0 0.0"/>
-        <geometry>
-          <mesh filename="package://rbvogui_description/meshes/cart/lanza.stl" scale="1.0 1.0 1.0"/>
-        </geometry>
-      </collision>
-    </link>
-    <!-- Chassis -->
-    <link name="${prefix}chassis">
-      <inertial>
-        <mass value="${cart_mass}" />
-        <origin xyz="-0.1 0 -0.1" rpy="0 0 0" />
-        <inertia ixx="${(cart_mass*(cart_width*cart_width+cart_height*cart_height))/12}" ixy="0" ixz="0"
-                  iyy="${(cart_mass*(cart_length*cart_length+cart_height*cart_height))/12}" iyz="0"
-                  izz="${(cart_mass*(cart_length*cart_length+cart_width*cart_width))/12}" />
-      </inertial>
-      <visual>
-        <origin xyz="0.0 0.0 0" rpy="0 0.0 0"/>
-        <geometry>
-          <mesh filename="package://rbvogui_description/meshes/cart/cart.stl" scale="1.0 1.0 1.0"/>
-        </geometry>
-        <material name="red">
-          <color rgba="0.9 0.9 0.9 1"/>
-        </material>
-      </visual>
-      <collision>
-        <origin xyz="0.0 0.0 0.0" rpy="0.0 0.0 0.0"/>
-        <geometry>
-          <box size="${cart_length} ${cart_width} ${cart_height}"/>
-        </geometry>
-      </collision>
-    </link>
-    <gazebo reference="${prefix}chassis">
-      <material>Gazebo/Red</material>
-    </gazebo>
-    <!-- Rear Left wheel -->
-    <link name="${prefix}rear_left_wheel">
-      <inertial>
-            <mass value="3" />
-            <origin xyz="0 0 0" rpy="${PI/2} 0 0" />
-            <xacro:solid_cylinder_inertia m="3" r="${wheels_radius}" h="${wheels_width}"/>
-      </inertial>
-      <visual>
-        <origin xyz="0.0 0.0 0.0" rpy="0 0.0 0"/>
-        <geometry>
-          <mesh filename="package://rbvogui_description/meshes/cart/back_wheel.stl" scale="1.0 1.0 1.0"/>
-        </geometry>
-        <material name="black">
-          <color rgba="0.2 0.2 0.2 0.8"/>
-        </material>
-      </visual>
-      <collision>
-        <origin xyz="0.0 0.0 0.0" rpy="${PI/2} 0.0 0.0"/>
-        <geometry>
-          <cylinder radius="${wheels_radius}" length="${wheels_width}"/>
-        </geometry>
-        <contact_coefficients mu="1.0" kp="1.0" kd="1.0" />
-      </collision>
-    </link>
-    <gazebo reference="${prefix}rear_left_wheel">
-      <material>Gazebo/Grey</material>
-    </gazebo>
-    <!-- Rear Right wheel -->
-    <link name="${prefix}rear_right_wheel">
-      <inertial>
-            <mass value="3" />
-            <origin xyz="0 0 0" rpy="${PI/2} 0 0" />
-            <xacro:solid_cylinder_inertia m="3" r="${wheels_radius}" h="${wheels_width}"/>
-      </inertial>
-      <visual>
-        <origin xyz="0.0 0.0 0.0" rpy="0 0.0 0"/>
-        <geometry>
-          <mesh filename="package://rbvogui_description/meshes/cart/back_wheel.stl" scale="1.0 1.0 1.0"/>
-        </geometry>
-        <material name="black">
-          <color rgba="0.1 0.1 0.1 1"/>
-        </material>
-      </visual>
-      <collision>
-        <origin xyz="0.0 0.0 0.0" rpy="${PI/2} 0.0 0.0"/>
-        <geometry>
-          <cylinder radius="${wheels_radius}" length="${wheels_width}"/>
-        </geometry>
-        <contact_coefficients mu="1.0" kp="1.0" kd="1.0" />
-      </collision>
-    </link>
-    <gazebo reference="${prefix}rear_right_wheel">
-      <material>Gazebo/Grey</material>
-    </gazebo>
-    <!-- Front Right Wheel base support -->
-    <link name="${prefix}front_right_wheel_base_support">
-      <visual>
-        <origin xyz="0.0 0.0 0.0" rpy="0 0 0"/>
-        <geometry>
-          <mesh filename="package://rbvogui_description/meshes/cart/base_support_wheel.stl" scale="1.0 1.0 1.0"/>
-        </geometry>
-      </visual>
-    </link>
-    <gazebo reference="${prefix}front_right_wheel_base_support">
-      <material>Gazebo/Red</material>
-    </gazebo>
-    <!-- Front Left Wheel base support -->
-    <link name="${prefix}front_left_wheel_base_support">
-      <visual>
-        <origin xyz="0.0 0.0 0.0" rpy="0 0 0"/>
-        <geometry>
-          <mesh filename="package://rbvogui_description/meshes/cart/base_support_wheel.stl" scale="1.0 1.0 1.0"/>
-        </geometry>
-      </visual>
-    </link>
-    <gazebo reference="${prefix}front_left_wheel_base_support">
-      <material>Gazebo/Red</material>
-    </gazebo>
-    <!-- Front Right Wheel support -->
-    <link name="${prefix}front_right_wheel_support">
-      <inertial>
-            <mass value="1" />
-            <origin xyz="0 0 0" rpy="0 ${PI/2} 0" />
-            <xacro:solid_cuboid_inertia w="${support_length}" d="${support_width}" h="${support_width}" m="1"/>
-      </inertial>
-      <visual>
-        <origin xyz="0.0 0.0 0.0" rpy="0 0 -${40*PI/180}"/>
-        <geometry>
-          <mesh filename="package://rbvogui_description/meshes/cart/support_wheel.stl" scale="1.0 1.0 1.0"/>
-        </geometry>
-      </visual>
-      <collision>
-        <origin xyz="0.0 0.0 0.0" rpy="0.0 ${PI/2} 0.0"/>
-        <geometry>
-          <box size="${support_length} ${support_width} ${support_width}"/>
-        </geometry>
-      </collision>
-    </link>
-    <gazebo reference="${prefix}front_right_wheel_support">
-      <material>Gazebo/Red</material>
-    </gazebo>
-    <!-- Front Left Wheel support -->
-    <link name="${prefix}front_left_wheel_support">
-      <inertial>
-            <mass value="1" />
-            <origin xyz="0 0 0" rpy="0 ${PI/2} 0" />
-            <xacro:solid_cuboid_inertia w="${support_length}" d="${support_width}" h="${support_width}" m="1"/>
-      </inertial>
-      <visual>
-        <origin xyz="0.0 0.0 0.0" rpy="0 0 -${40*PI/180}"/>
-        <geometry>
-          <mesh filename="package://rbvogui_description/meshes/cart/support_wheel.stl" scale="1.0 1.0 1.0"/>
-        </geometry>
-      </visual>
-      <collision>
-        <origin xyz="0.0 0.0 0.0" rpy="0.0 ${PI/2} 0.0"/>
-        <geometry>
-          <box size="${support_length} ${support_width} ${support_width}"/>
-        </geometry>
-      </collision>
-    </link>
-    <gazebo reference="${prefix}front_left_wheel_support">
-      <material>Gazebo/Red</material>
-    </gazebo>
-    <!-- Front Left wheel -->
-    <link name="${prefix}front_left_wheel">
-      <inertial>
-            <mass value="1" />
-            <origin xyz="0 0 0" rpy="${PI/2} 0 0" />
-            <xacro:solid_cylinder_inertia m="1" r="${front_wheel_radius}" h="${front_wheel_width}"/>
-      </inertial>
-      <visual>
-        <origin xyz="0.0 0.0 0.0" rpy="0.0 0 ${PI/2}"/>
-        <geometry>
-          <mesh filename="package://rbvogui_description/meshes/cart/front_wheel.stl" scale="1.0 1.0 1.0"/>
-        </geometry>
-        <material name="black">
-          <color rgba="0.1 0.1 0.1 1"/>
-        </material>
-      </visual>
-      <collision>
-        <origin xyz="0.0 0.0 0.0" rpy="${PI/2} 0.0 0.0"/>
-        <geometry>
-          <cylinder radius="${front_wheel_radius}" length="${front_wheel_width}"/>
-        </geometry>
-        <contact_coefficients mu="1.0" kp="1.0" kd="1.0" />
-      </collision>
-    </link>
-    <gazebo reference="${prefix}front_left_wheel">
-      <material>Gazebo/Grey</material>
-    </gazebo>
-    <!-- Front Right wheel -->
-    <link name="${prefix}front_right_wheel">
-      <inertial>
-            <mass value="1" />
-            <origin xyz="0 0 0" rpy="${PI/2} 0 0" />
-            <xacro:solid_cylinder_inertia m="1" r="${front_wheel_radius}" h="${front_wheel_width}"/>
-      </inertial>
-      <visual>
-        <origin xyz="0.0 0.0 0.0" rpy="0.0 0 ${PI/2}"/>
-        <geometry>
-          <mesh filename="package://rbvogui_description/meshes/cart/front_wheel.stl" scale="1.0 1.0 1.0"/>
-        </geometry>
-        <material name="black">
-          <color rgba="0.1 0.1 0.1 1"/>
-        </material>
-      </visual>
-      <collision>
-        <origin xyz="0.0 0.0 0.0" rpy="${PI/2} 0.0 0.0"/>
-        <geometry>
-          <cylinder radius="${front_wheel_radius}" length="${front_wheel_width}"/>
-        </geometry>
-        <contact_coefficients mu="1.0" kp="1.0" kd="1.0" />
-      </collision>
-    </link>
-    <gazebo reference="${prefix}front_right_wheel">
-      <material>Gazebo/Grey</material>
-    </gazebo>
-    <!-- hokuyo ust10 -->
-    <xacro:sensor_hokuyo_ust10lx prefix="${prefix}rear_laser" parent="${prefix}chassis" gpu="false" prefix_topic="/${prefix}rear_laser">
-        <origin xyz="-0.63 0.0 -0.023" rpy="${PI} 0 ${-PI/2}"/>
-    </xacro:sensor_hokuyo_ust10lx>
-    <xacro:cart_joints prefix="${prefix}" connected="${connected}"/>
-    <xacro:markers prefix="${prefix}"/>
-    <gazebo>
-      <plugin name="cart_joint_state" filename="libgazebo_ros_joint_state_publisher.so">
-        <ros>
-          <xacro:if value="${connected}">
-            <namespace>robot</namespace>
-          </xacro:if>
-          <xacro:unless value="${connected}">
-            <namespace>robot/cart</namespace>
-          </xacro:unless>
-        </ros>
-        <update_rate>30</update_rate>
-        <xacro:if value="${connected}">
-          <joint_name>robot_hitch_x_joint</joint_name>
-          <joint_name>robot_hitch_y_joint</joint_name>
-          <joint_name>robot_hitch_z_joint</joint_name>
-          <joint_name>${prefix}chassis_joint</joint_name>
-        </xacro:if>
-        <joint_name>${prefix}rear_left_wheel_joint</joint_name>
-        <joint_name>${prefix}rear_right_wheel_joint</joint_name>
-        <joint_name>${prefix}front_right_wheel_support_joint</joint_name>
-        <joint_name>${prefix}front_left_wheel_support_joint</joint_name>
-        <joint_name>${prefix}front_right_wheel_joint</joint_name>
-        <joint_name>${prefix}front_left_wheel_joint</joint_name>
-      </plugin>
-    </gazebo>
-  </xacro:macro>
-  <xacro:unless value="$(arg connected)">
-    <xacro:cart prefix="$(arg prefix)cart_" connected="$(arg connected)"/>
-  </xacro:unless>
+  <xacro:arg name="namespace" default="robot" />
+  <xacro:cart_base prefix="$(arg prefix)" connected="$(arg connected)" namespace="$(arg namespace)">
+  </xacro:cart_base>
+  <!-- <xacro:markers prefix="${prefix}"/> -->
 </robot>

File: rbvogui_description/urdf/cart/robot_cart_connection.urdf.xacro (robot description, xacro)
@@ -3,15 +3,12 @@
   <xacro:arg name="prefix" default="robot_" />
   <xacro:arg name="connected" default="true" />
-  <!-- Transform from robot_base_link to bulon -->
-  <xacro:property name="bulon_x" value="-0.669" />
-  <xacro:property name="bulon_z" value="0.391" />
   <!-- Transform from hitch to chassis UNKOWN -->
   <xacro:property name="hitch_x" value="-0.347" />
-  <xacro:property name="hitch_z" value="0.22" />
+  <xacro:property name="hitch_z" value="0.3" />
   <!-- Hitch -->
   <xacro:property name="hitch_length" value="0.32" />
   <xacro:property name="hitch_width" value="0.160" />
   <xacro:property name="hitch_height" value="0.064" />
-  <xacro:macro name="cart_connection" params="prefix connected">
+  <xacro:macro name="cart_connection" params="prefix connected parent">
     <xacro:if value="${connected}">
       <!-- Bulon -->
@@ -60,5 +57,5 @@
     <joint name="${prefix}bulon_joint" type="fixed">
         <origin xyz="${hitch_x} 0.0 ${hitch_z}" rpy="0.0 0.0 0.0"/>
-        <parent link="${prefix}base_link"/>
+        <parent link="${parent}"/>
         <child link="${prefix}bulon"/>
     </joint>

File: rbvogui_description/urdf/ros2_control.urdf.xacro (robot description, xacro)
@@ -1,11 +1,11 @@
 <?xml version="1.0"?>
 <robot xmlns:xacro="http://wiki.ros.org/xacro">
-    <xacro:macro name="ros2_control" params="prefix">
+    <xacro:macro name="ros2_control" params="prefix robot_id controllers">
         <gazebo>
           <plugin name="ros_control" filename="libgazebo_ros2_control.so">
-            <namespace>robot</namespace>
+            <namespace>${robot_id}</namespace>
             <robot_param>robot_description</robot_param>
             <robot_param_node>robot_state_publisher</robot_param_node>
-            <parameters>$(find rbvogui_gazebo)/config/base_controller.yaml</parameters>
+            <parameters>${controllers}</parameters>
           </plugin>
         </gazebo>
